File: LauriFilter.sch (EAGLE design)
At the start: 37 parts, among them IC2 IC_74HC595-SOIC-16

Commit message: pre order fixes
Parts:
- added D1: BAS70-04, diode:BAS70-04
- added JP1: M02PTH, SparkFun-Connectors:M02PTH
- added R14, R15: 300, OPL:R
- added R16: 300, OPL:R-0603
Connections:
- new net N$11: R14.1, U$1.OUT_L
- new net N$12: R15.1, U$1.OUT_R
- new net N$13: D1.C1A2, R16.2, U$1.OUT_DAC
- new net N$20: JP1.2, R16.1
- net 3.3V: now also D1.C2
- net GND: now also D1.A1, JP1.1
- net N$5: now also R14.2; no longer U$1.OUT_L
- net N$6: now also R15.2; no longer U$1.OUT_R
Changed lines of the file:
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@@
 </variantdefs>
 <classes>
-<class number="0" name="default" width="0" drill="0">
+<class number="0" name="default" width="0.2032" drill="0">
 </class>
 </classes>
@@
 <part name="SUPPLY5" library="SparkFun-Aesthetics" deviceset="3.3V" device=""/>
 <part name="R13" library="OPL" deviceset="R*" device="-0603" value="100k"/>
+<part name="R14" library="OPL" deviceset="R*" device="" value="300"/>
+<part name="R15" library="OPL" deviceset="R*" device="" value="300"/>
+<part name="JP1" library="SparkFun-Connectors" deviceset="M02" device="PTH"/>
+<part name="GND22" library="SparkFun-Aesthetics" deviceset="GND" device=""/>
+<part name="D1" library="diode" deviceset="BAS70-04" device=""/>
+<part name="GND32" library="SparkFun-Aesthetics" deviceset="GND" device=""/>
+<part name="SUPPLY6" library="SparkFun-Aesthetics" deviceset="3.3V" device=""/>
+<part name="R16" library="OPL" deviceset="R*" device="-0603" value="300"/>
 </parts>
 <sheets>
@@
 <instance part="SUPPLY5" gate="G$1" x="-35.56" y="133.35"/>
 <instance part="R13" gate="R" x="-39.37" y="35.56"/>
+<instance part="R14" gate="R" x="86.36" y="22.86"/>
+<instance part="R15" gate="R" x="86.36" y="20.32"/>
+<instance part="JP1" gate="G$1" x="142.24" y="-10.16" rot="R180"/>
+<instance part="GND22" gate="1" x="129.54" y="-7.62" rot="R180"/>
+<instance part="D1" gate="G$1" x="106.68" y="-5.08" rot="MR0"/>
+<instance part="GND32" gate="1" x="111.76" y="-12.7"/>
+<instance part="SUPPLY6" gate="G$1" x="101.6" y="-10.16" rot="R180"/>
+<instance part="R16" gate="R" x="115.57" y="-2.54" rot="R180"/>
 </instances>
 <busses>
@@
 <pinref part="GND21" gate="1" pin="GND"/>
 </segment>
+<segment>
+<pinref part="JP1" gate="G$1" pin="1"/>
+<pinref part="GND22" gate="1" pin="GND"/>
+<wire x1="129.54" y1="-10.16" x2="134.62" y2="-10.16" width="0.1524" layer="91"/>
+</segment>
+<segment>
+<pinref part="D1" gate="G$1" pin="A1"/>
+<pinref part="GND32" gate="1" pin="GND"/>
+<wire x1="111.76" y1="-5.08" x2="111.76" y2="-10.16" width="0.1524" layer="91"/>
+</segment>
 </net>
 <net name="N$1" class="0">
@@
 <net name="N$5" class="0">
 <segment>
-<pinref part="U$1" gate="G$1" pin="OUT_L"/>
-<wire x1="63.5" y1="22.86" x2="114.3" y2="22.86" width="0.1524" layer="91"/>
+<wire x1="90.17" y1="22.86" x2="114.3" y2="22.86" width="0.1524" layer="91"/>
 <wire x1="114.3" y1="22.86" x2="114.3" y2="40.64" width="0.1524" layer="91"/>
 <pinref part="U$7" gate="G$1" pin="TIP"/>
 <wire x1="114.3" y1="40.64" x2="144.78" y2="40.64" width="0.1524" layer="91"/>
+<pinref part="R14" gate="R" pin="2"/>
 </segment>
 </net>
 <net name="N$6" class="0">
 <segment>
-<pinref part="U$1" gate="G$1" pin="OUT_R"/>
-<wire x1="63.5" y1="20.32" x2="121.92" y2="20.32" width="0.1524" layer="91"/>
 <pinref part="U$8" gate="G$1" pin="TIP"/>
+<pinref part="R15" gate="R" pin="2"/>
+<wire x1="90.17" y1="20.32" x2="121.92" y2="20.32" width="0.1524" layer="91"/>
 </segment>
 </net>
@@
 <pinref part="SUPPLY5" gate="G$1" pin="3.3V"/>
 </segment>
+<segment>
+<pinref part="D1" gate="G$1" pin="C2"/>
+<pinref part="SUPPLY6" gate="G$1" pin="3.3V"/>
+<wire x1="101.6" y1="-5.08" x2="101.6" y2="-10.16" width="0.1524" layer="91"/>
+</segment>
 </net>
 <net name="MODE1_A" class="0">
@@
 </segment>
 </net>
+<net name="N$11" class="0">
+<segment>
+<pinref part="R14" gate="R" pin="1"/>
+<pinref part="U$1" gate="G$1" pin="OUT_L"/>
+<wire x1="63.5" y1="22.86" x2="82.55" y2="22.86" width="0.1524" layer="91"/>
+</segment>
+</net>
+<net name="N$12" class="0">
+<segment>
+<pinref part="R15" gate="R" pin="1"/>
+<pinref part="U$1" gate="G$1" pin="OUT_R"/>
+<wire x1="63.5" y1="20.32" x2="82.55" y2="20.32" width="0.1524" layer="91"/>
+</segment>
+</net>
+<net name="N$13" class="0">
+<segment>
+<pinref part="U$1" gate="G$1" pin="OUT_DAC"/>
+<wire x1="63.5" y1="15.24" x2="88.9" y2="15.24" width="0.1524" layer="91"/>
+<wire x1="88.9" y1="15.24" x2="88.9" y2="-2.54" width="0.1524" layer="91"/>
+<wire x1="88.9" y1="-2.54" x2="106.68" y2="-2.54" width="0.1524" layer="91"/>
+<pinref part="D1" gate="G$1" pin="C1A2"/>
+<wire x1="106.68" y1="-2.54" x2="111.76" y2="-2.54" width="0.1524" layer="91"/>
+<junction x="106.68" y="-2.54"/>
+<pinref part="R16" gate="R" pin="2"/>
+</segment>
+</net>
+<net name="N$20" class="0">
+<segment>
+<pinref part="JP1" gate="G$1" pin="2"/>
+<pinref part="R16" gate="R" pin="1"/>
+<wire x1="119.38" y1="-2.54" x2="121.92" y2="-2.54" width="0.1524" layer="91"/>
+<wire x1="121.92" y1="-2.54" x2="121.92" y2="-12.7" width="0.1524" layer="91"/>
+<wire x1="121.92" y1="-12.7" x2="134.62" y2="-12.7" width="0.1524" layer="91"/>
+</segment>
+</net>
