File: Eurorack Set 2/TestBench.brd (EAGLE design)
At the start: 140 x 138.5 mm, 12 parts

Commit message: small cosmetic changes-  reversed the led polarity
Parts:
- moved U$3 183.8 mm to (31.0, 41.0)
Changed lines of the file:
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@@
 <element name="U$2" library="EurorackModularParts" package="POWER_16" value="POWER" x="125.73" y="115.57" rot="R270"/>
 <element name="J1" library="dp_devices" package="DC_BARREL_JACK_PTH_2MM" value="" x="129" y="135" rot="R180"/>
-<element name="U$3" library="zephod-components" package="PROTO_10_24" value="PROTOAREA" x="161" y="171"/>
+<element name="U$3" library="zephod-components" package="PROTO_10_24" value="PROTOAREA" x="31" y="41"/>
 <element name="U$4" library="EurorackModularParts" package="OG-POTS_ALPS_POT_VERTICAL" value="" x="130" y="15"/>
 <element name="U$5" library="EurorackModularParts" package="OG-POTS_ALPS_POT_VERTICAL" value="" x="130" y="35"/>
