File: Eurorack Set 2/ScaleOffset-R2.brd (EAGLE design)
At the start: 29.1 x 106.5 mm, 26 parts, among them IC3 TL074D

Commit message: More bodges... different led setup for scaleoffset, gaterhythm still has buttons reversed
Parts:
- added C2, C3: (no value), OPL:AVX-A
Connections:
- removed net N$9: IC3.14, LED1.K
- new net N$2: LED1.A, R7.2
- net -12V: now also C3.-
- net 12V: now also C2.+
- net GND: now also C2.-, C3.+, LED1.K; no longer R7.1
- net N$11: now also IC3.14, R7.1; no longer LED1.A, R7.2
Routing:
- net N$11: track 21.6 -> 5.30 mm, vias 2 -> 0
- net N$9: track 14.9 -> 0.00 mm, vias 2 -> 0
- net N$2: track 0.00 -> 13.9 mm
- net GND: track 72.2 -> 67.9 mm
- net -12V: vias 2 -> 0
Changed lines of the file:
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@@
 <element name="R10" library="OPL" package="C0805" value="51" x="22.86" y="45.72" rot="R270"/>
 <element name="R11" library="OPL" package="C0805" value="51" x="7.62" y="45.72" rot="R270"/>
+<element name="C2" library="OPL" package="AVX-A" value="" x="1.905" y="-22.86"/>
+<element name="C3" library="OPL" package="AVX-A" value="" x="1.905" y="-26.67"/>
 </elements>
 <signals>
@@
 <contactref element="U$5" pad="5"/>
 <contactref element="C1" pad="1"/>
-<contactref element="R7" pad="1"/>
 <contactref element="OUT2" pad="RING@1"/>
 <contactref element="C4" pad="2"/>
@@
 <contactref element="GATE" pad="RING@2"/>
 <contactref element="GATE" pad="RING@1"/>
-<wire x1="7.493" y1="57.912" x2="7.493" y2="53.975" width="0.254" layer="1"/>
-<wire x1="9.271" y1="59.69" x2="7.493" y2="57.912" width="0.254" layer="1"/>
-<wire x1="10.855" y1="59.69" x2="9.271" y2="59.69" width="0.254" layer="1"/>
 <wire x1="5.461" y1="62.357" x2="3.937" y2="62.357" width="0.254" layer="1"/>
 <wire x1="3.937" y1="62.357" x2="3.175" y2="62.357" width="0.254" layer="1"/>
@@
 <wire x1="10.922" y1="62.23" x2="11.43" y2="61.722" width="0.254" layer="1"/>
 <wire x1="10.922" y1="62.23" x2="10.855" y2="62.23" width="0.254" layer="1"/>
-<wire x1="10.855" y1="62.23" x2="9.271" y2="62.23" width="0.254" layer="1"/>
-<wire x1="9.271" y1="62.23" x2="5.655" y2="62.23" width="0.254" layer="1"/>
-<wire x1="9.271" y1="62.23" x2="9.271" y2="59.69" width="0.254" layer="1"/>
 <wire x1="11.82" y1="76.2" x2="10.033" y2="76.2" width="0.254" layer="1"/>
 <wire x1="10.033" y1="76.2" x2="3.42" y2="76.2" width="0.254" layer="1"/>
@@
 <via x="3.937" y="63.246" extent="1-16" drill="0.3048"/>
 <via x="2.413" y="64.77" extent="1-16" drill="0.3048"/>
+<contactref element="LED1" pad="K"/>
+<wire x1="8.763" y1="59.69" x2="10.855" y2="59.69" width="0.254" layer="1"/>
+<wire x1="6.223" y1="62.23" x2="8.763" y2="59.69" width="0.254" layer="1"/>
+<wire x1="5.655" y1="62.23" x2="6.223" y2="62.23" width="0.254" layer="1"/>
+<wire x1="5.655" y1="62.23" x2="10.855" y2="62.23" width="0.254" layer="1"/>
+<contactref element="C2" pad="-"/>
+<contactref element="C3" pad="+"/>
+<wire x1="3.175" y1="-22.86" x2="0.635" y2="-26.67" width="0" layer="19" extent="1-1"/>
+<wire x1="3.42" y1="10.16" x2="3.175" y2="-22.86" width="0" layer="19" extent="1-16"/>
 </signal>
 <signal name="N$1">
@@
 <via x="19.558" y="44.958" extent="1-16" drill="0.3048"/>
 <via x="20.701" y="46.101" extent="1-16" drill="0.3048"/>
+<contactref element="C2" pad="+"/>
+<wire x1="0.635" y1="-22.86" x2="13.97" y2="24.13" width="0" layer="19" extent="1-1"/>
 </signal>
 <signal name="-12V">
@@
 <wire x1="5.588" y1="60.96" x2="5.655" y2="60.96" width="0.254" layer="1"/>
 <wire x1="6.223" y1="60.96" x2="5.655" y2="60.96" width="0.254" layer="1"/>
-<wire x1="7.874" y1="59.309" x2="6.223" y2="60.96" width="0.254" layer="1"/>
-<wire x1="9.017" y1="58.166" x2="7.874" y2="59.309" width="0.254" layer="16"/>
-<wire x1="9.017" y1="56.515" x2="9.017" y2="58.166" width="0.254" layer="1"/>
-<wire x1="16.256" y1="49.276" x2="9.017" y2="56.515" width="0.254" layer="1"/>
+<wire x1="9.398" y1="57.785" x2="6.223" y2="60.96" width="0.254" layer="1"/>
+<wire x1="9.398" y1="56.134" x2="9.398" y2="57.785" width="0.254" layer="1"/>
+<wire x1="16.256" y1="49.276" x2="9.398" y2="56.134" width="0.254" layer="1"/>
 <wire x1="20.193" y1="49.276" x2="20.066" y2="49.276" width="0.254" layer="1"/>
 <wire x1="20.066" y1="49.276" x2="16.256" y2="49.276" width="0.254" layer="1"/>
@@
 <wire x1="20.066" y1="49.276" x2="20.066" y2="45.847" width="0.254" layer="1"/>
 <wire x1="20.066" y1="49.276" x2="20.28" y2="49.18" width="0.254" layer="1"/>
-<via x="7.874" y="59.309" extent="1-16" drill="0.3048"/>
-<via x="9.017" y="58.166" extent="1-16" drill="0.3048"/>
+<contactref element="C3" pad="-"/>
+<wire x1="3.175" y1="-26.67" x2="24.13" y2="24.13" width="0" layer="19" extent="1-1"/>
 </signal>
 <signal name="OFFSET">
@@
 <via x="14.478" y="51.943" extent="1-16" drill="0.3048"/>
 </signal>
-<signal name="N$9">
-<contactref element="LED1" pad="K"/>
+<signal name="N$11">
+<contactref element="IC3" pad="13"/>
 <contactref element="IC3" pad="14"/>
-<wire x1="5.715" y1="55.753" x2="5.715" y2="57.15" width="0.254" layer="1"/>
-<wire x1="6.731" y1="54.737" x2="5.715" y2="55.753" width="0.254" layer="1"/>
-<wire x1="11.684" y1="49.784" x2="6.731" y2="54.737" width="0.254" layer="16"/>
-<wire x1="15.113" y1="46.355" x2="11.684" y2="49.784" width="0.254" layer="1"/>
-<wire x1="15.24" y1="46.355" x2="15.113" y2="46.355" width="0.254" layer="1"/>
+<contactref element="R7" pad="1"/>
+<wire x1="7.493" y1="55.372" x2="7.493" y2="53.975" width="0.254" layer="1"/>
+<wire x1="5.715" y1="57.15" x2="7.493" y2="55.372" width="0.254" layer="1"/>
+<wire x1="5.715" y1="57.15" x2="5.715" y2="58.42" width="0.254" layer="1"/>
+<wire x1="5.715" y1="58.42" x2="5.655" y2="58.42" width="0.254" layer="1"/>
 <wire x1="5.715" y1="57.15" x2="5.655" y2="57.15" width="0.254" layer="1"/>
-<via x="6.731" y="54.737" extent="1-16" drill="0.3048"/>
-<via x="11.684" y="49.784" extent="1-16" drill="0.3048"/>
-</signal>
-<signal name="N$11">
-<contactref element="R7" pad="2"/>
-<contactref element="LED1" pad="A"/>
-<contactref element="IC3" pad="13"/>
-<wire x1="9.017" y1="55.88" x2="9.017" y2="55.753" width="0.254" layer="1"/>
-<wire x1="9.017" y1="55.753" x2="9.017" y2="53.975" width="0.254" layer="1"/>
-<wire x1="8.128" y1="56.769" x2="9.017" y2="55.88" width="0.254" layer="1"/>
-<wire x1="8.128" y1="57.658" x2="8.128" y2="56.769" width="0.254" layer="1"/>
-<wire x1="7.239" y1="58.547" x2="8.128" y2="57.658" width="0.254" layer="16"/>
-<wire x1="5.842" y1="58.547" x2="7.239" y2="58.547" width="0.254" layer="1"/>
-<wire x1="5.715" y1="58.42" x2="5.842" y2="58.547" width="0.254" layer="1"/>
-<wire x1="5.715" y1="58.42" x2="5.655" y2="58.42" width="0.254" layer="1"/>
-<wire x1="15.24" y1="44.577" x2="15.24" y2="43.815" width="0.254" layer="1"/>
-<wire x1="11.049" y1="48.768" x2="15.24" y2="44.577" width="0.254" layer="1"/>
-<wire x1="11.049" y1="52.959" x2="11.049" y2="48.768" width="0.254" layer="1"/>
-<wire x1="11.176" y1="53.086" x2="11.049" y2="52.959" width="0.254" layer="1"/>
-<wire x1="11.176" y1="53.594" x2="11.176" y2="53.086" width="0.254" layer="1"/>
-<wire x1="9.017" y1="55.753" x2="11.176" y2="53.594" width="0.254" layer="1"/>
-<via x="8.128" y="57.658" extent="1-16" drill="0.3048"/>
-<via x="7.239" y="58.547" extent="1-16" drill="0.3048"/>
 </signal>
 <signal name="FBOUT2">
@@
 <via x="7.62" y="42.291" extent="1-16" drill="0.3048"/>
 </signal>
+<signal name="N$2">
+<contactref element="LED1" pad="A"/>
+<contactref element="R7" pad="2"/>
+<wire x1="10.795" y1="53.975" x2="9.017" y2="53.975" width="0.254" layer="1"/>
+<wire x1="11.176" y1="53.594" x2="10.795" y2="53.975" width="0.254" layer="1"/>
+<wire x1="11.176" y1="51.435" x2="11.176" y2="53.594" width="0.254" layer="1"/>
+<wire x1="11.049" y1="51.308" x2="11.176" y2="51.435" width="0.254" layer="1"/>
+<wire x1="11.049" y1="48.006" x2="11.049" y2="51.308" width="0.254" layer="1"/>
+<wire x1="15.24" y1="43.815" x2="11.049" y2="48.006" width="0.254" layer="1"/>
+</signal>
 </signals>

Commit message: Fiducials!
Parts:
- added U$1, U$2, U$3, U$4: FIDUCIAL, adafruit:FIDUCIAL_1MM
- moved C2 77.1 mm to (14.0, 53.3), turned to 270 degrees
- moved C3 76.6 mm to (14.6, 48.9)
Routing:
- net GND: track 67.9 -> 74.7 mm
- net 12V: track 52.6 -> 58.7 mm, vias 2 -> 3
- net -12V: track 50.1 -> 54.0 mm
- net OFFSET: track 20.4 -> 22.6 mm
Changed lines of the file:
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@@
 <setting verticaltext="up"/>
 </settings>
-<grid distance="25" unitdist="mil" unit="mil" style="lines" multiple="1" display="yes" altdistance="0.025" altunitdist="inch" altunit="inch"/>
+<grid distance="50" unitdist="mil" unit="mil" style="lines" multiple="1" display="yes" altdistance="0.025" altunitdist="inch" altunit="inch"/>
 <layers>
 <layer number="1" name="Top" color="4" fill="1" visible="yes" active="yes"/>
@@
 <element name="R10" library="OPL" package="C0805" value="51" x="22.86" y="45.72" rot="R270"/>
 <element name="R11" library="OPL" package="C0805" value="51" x="7.62" y="45.72" rot="R270"/>
-<element name="C2" library="OPL" package="AVX-A" value="" x="1.905" y="-22.86"/>
-<element name="C3" library="OPL" package="AVX-A" value="" x="1.905" y="-26.67"/>
+<element name="C2" library="OPL" package="AVX-A" value="" x="13.97" y="53.34" rot="R270"/>
+<element name="C3" library="OPL" package="AVX-A" value="" x="14.605" y="48.895"/>
+<element name="U$1" library="adafruit" package="FIDUCIAL_1MM" value="FIDUCIAL" x="2.54" y="21.59"/>
+<element name="U$2" library="adafruit" package="FIDUCIAL_1MM" value="FIDUCIAL" x="26.67" y="21.59"/>
+<element name="U$3" library="adafruit" package="FIDUCIAL_1MM" value="FIDUCIAL" x="2.54" y="86.36"/>
+<element name="U$4" library="adafruit" package="FIDUCIAL_1MM" value="FIDUCIAL" x="26.035" y="86.36"/>
 </elements>
 <signals>
@@
 <contactref element="C2" pad="-"/>
 <contactref element="C3" pad="+"/>
-<wire x1="3.175" y1="-22.86" x2="0.635" y2="-26.67" width="0" layer="19" extent="1-1"/>
-<wire x1="3.42" y1="10.16" x2="3.175" y2="-22.86" width="0" layer="19" extent="1-16"/>
+<wire x1="13.335" y1="51.435" x2="13.335" y2="48.895" width="0.254" layer="1"/>
+<wire x1="13.97" y1="52.07" x2="13.335" y2="51.435" width="0.254" layer="1"/>
+<wire x1="13.335" y1="48.26" x2="13.335" y2="48.895" width="0.254" layer="1"/>
+<wire x1="15.24" y1="46.355" x2="13.335" y2="48.26" width="0.254" layer="1"/>
 </signal>
 <signal name="N$1">
@@
 <wire x1="14.732" y1="61.214" x2="13.716" y2="60.198" width="0.254" layer="1"/>
 <wire x1="15.875" y1="61.214" x2="14.732" y2="61.214" width="0.254" layer="1"/>
-<wire x1="25.4" y1="51.689" x2="15.875" y2="61.214" width="0.254" layer="1"/>
+<wire x1="25.4" y1="51.689" x2="18.2245" y2="58.8645" width="0.254" layer="1"/>
+<wire x1="18.2245" y1="58.8645" x2="15.875" y2="61.214" width="0.254" layer="1"/>
 <wire x1="25.4" y1="49.276" x2="25.4" y2="51.689" width="0.254" layer="1"/>
 <wire x1="25.4" y1="49.276" x2="25.44" y2="49.18" width="0.254" layer="1"/>
-<wire x1="13.97" y1="39.37" x2="13.97" y2="26.67" width="0.254" layer="1"/>
-<wire x1="19.558" y1="44.958" x2="13.97" y2="39.37" width="0.254" layer="1"/>
-<wire x1="20.701" y1="46.101" x2="19.558" y2="44.958" width="0.254" layer="16"/>
-<wire x1="22.479" y1="47.879" x2="20.701" y2="46.101" width="0.254" layer="1"/>
-<wire x1="23.876" y1="47.879" x2="22.479" y2="47.879" width="0.254" layer="1"/>
-<wire x1="25.273" y1="49.276" x2="23.876" y2="47.879" width="0.254" layer="1"/>
-<wire x1="25.273" y1="49.276" x2="25.44" y2="49.18" width="0.254" layer="1"/>
-<via x="19.558" y="44.958" extent="1-16" drill="0.3048"/>
-<via x="20.701" y="46.101" extent="1-16" drill="0.3048"/>
 <contactref element="C2" pad="+"/>
-<wire x1="0.635" y1="-22.86" x2="13.97" y2="24.13" width="0" layer="19" extent="1-1"/>
+<wire x1="18.2245" y1="58.8645" x2="13.97" y2="54.61" width="0.254" layer="1"/>
+<wire x1="26.797" y1="47.879" x2="25.527" y2="49.149" width="0.254" layer="16"/>
+<wire x1="26.797" y1="39.878" x2="26.797" y2="47.879" width="0.254" layer="1"/>
+<wire x1="20.828" y1="33.909" x2="26.797" y2="39.878" width="0.254" layer="1"/>
+<wire x1="19.558" y1="32.639" x2="20.828" y2="33.909" width="0.254" layer="16"/>
+<wire x1="19.558" y1="32.258" x2="19.558" y2="32.639" width="0.254" layer="1"/>
+<wire x1="13.97" y1="26.67" x2="19.558" y2="32.258" width="0.254" layer="1"/>
+<wire x1="25.527" y1="49.149" x2="25.44" y2="49.18" width="0.254" layer="16"/>
+<via x="26.797" y="47.879" extent="1-16" drill="0.3048"/>
+<via x="20.828" y="33.909" extent="1-16" drill="0.3048"/>
+<via x="19.558" y="32.639" extent="1-16" drill="0.3048"/>
 </signal>
 <signal name="-12V">
@@
 <wire x1="5.588" y1="60.96" x2="5.461" y2="60.833" width="0.254" layer="1"/>
 <wire x1="5.588" y1="60.96" x2="5.655" y2="60.96" width="0.254" layer="1"/>
+<contactref element="C3" pad="-"/>
+<wire x1="19.939" y1="48.895" x2="18.923" y2="48.895" width="0.254" layer="1"/>
+<wire x1="18.923" y1="48.895" x2="17.018" y2="48.895" width="0.254" layer="1"/>
+<wire x1="17.018" y1="48.895" x2="15.875" y2="48.895" width="0.254" layer="1"/>
+<wire x1="20.193" y1="49.149" x2="19.939" y2="48.895" width="0.254" layer="1"/>
+<wire x1="20.193" y1="49.149" x2="20.28" y2="49.18" width="0.254" layer="1"/>
 <wire x1="6.223" y1="60.96" x2="5.655" y2="60.96" width="0.254" layer="1"/>
 <wire x1="9.398" y1="57.785" x2="6.223" y2="60.96" width="0.254" layer="1"/>
 <wire x1="9.398" y1="56.134" x2="9.398" y2="57.785" width="0.254" layer="1"/>
-<wire x1="16.256" y1="49.276" x2="9.398" y2="56.134" width="0.254" layer="1"/>
-<wire x1="20.193" y1="49.276" x2="20.066" y2="49.276" width="0.254" layer="1"/>
-<wire x1="20.066" y1="49.276" x2="16.256" y2="49.276" width="0.254" layer="1"/>
-<wire x1="20.193" y1="49.276" x2="20.28" y2="49.18" width="0.254" layer="1"/>
+<wire x1="12.446" y1="53.086" x2="9.398" y2="56.134" width="0.254" layer="1"/>
+<wire x1="14.732" y1="53.086" x2="12.446" y2="53.086" width="0.254" layer="1"/>
+<wire x1="18.923" y1="48.895" x2="14.732" y2="53.086" width="0.254" layer="1"/>
 <wire x1="24.13" y1="27.432" x2="24.13" y2="26.67" width="0.254" layer="1"/>
 <wire x1="20.193" y1="31.369" x2="24.13" y2="27.432" width="0.254" layer="1"/>
 <wire x1="20.193" y1="45.72" x2="20.193" y2="31.369" width="0.254" layer="1"/>
-<wire x1="20.066" y1="45.847" x2="20.193" y2="45.72" width="0.254" layer="1"/>
-<wire x1="20.066" y1="49.276" x2="20.066" y2="45.847" width="0.254" layer="1"/>
-<wire x1="20.066" y1="49.276" x2="20.28" y2="49.18" width="0.254" layer="1"/>
-<contactref element="C3" pad="-"/>
-<wire x1="3.175" y1="-26.67" x2="24.13" y2="24.13" width="0" layer="19" extent="1-1"/>
+<wire x1="17.018" y1="48.895" x2="20.193" y2="45.72" width="0.254" layer="1"/>
 </signal>
 <signal name="OFFSET">
 <contactref element="OFFSET" pad="P$2"/>
 <contactref element="R4" pad="1"/>
-<wire x1="6.223" y1="53.975" x2="5.207" y2="53.975" width="0.254" layer="1"/>
-<wire x1="7.366" y1="52.832" x2="6.223" y2="53.975" width="0.254" layer="1"/>
-<wire x1="9.906" y1="52.832" x2="7.366" y2="52.832" width="0.254" layer="1"/>
-<wire x1="11.684" y1="51.054" x2="9.906" y2="52.832" width="0.254" layer="16"/>
-<wire x1="13.589" y1="51.054" x2="11.684" y2="51.054" width="0.254" layer="1"/>
-<wire x1="14.478" y1="51.943" x2="13.589" y2="51.054" width="0.254" layer="16"/>
-<wire x1="20.193" y1="51.943" x2="14.478" y2="51.943" width="0.254" layer="1"/>
-<wire x1="22.86" y1="49.276" x2="20.193" y2="51.943" width="0.254" layer="1"/>
+<wire x1="8.255" y1="50.927" x2="5.207" y2="53.975" width="0.254" layer="1"/>
+<wire x1="9.271" y1="49.911" x2="8.255" y2="50.927" width="0.254" layer="16"/>
+<wire x1="11.684" y1="49.911" x2="9.271" y2="49.911" width="0.254" layer="1"/>
+<wire x1="15.24" y1="53.467" x2="11.684" y2="49.911" width="0.254" layer="16"/>
+<wire x1="18.669" y1="53.467" x2="15.24" y2="53.467" width="0.254" layer="1"/>
+<wire x1="22.86" y1="49.276" x2="18.669" y2="53.467" width="0.254" layer="1"/>
 <wire x1="22.86" y1="49.276" x2="22.86" y2="49.18" width="0.254" layer="1"/>
-<via x="9.906" y="52.832" extent="1-16" drill="0.3048"/>
-<via x="11.684" y="51.054" extent="1-16" drill="0.3048"/>
-<via x="13.589" y="51.054" extent="1-16" drill="0.3048"/>
-<via x="14.478" y="51.943" extent="1-16" drill="0.3048"/>
+<via x="8.255" y="50.927" extent="1-16" drill="0.3048"/>
+<via x="9.271" y="49.911" extent="1-16" drill="0.3048"/>
+<via x="11.684" y="49.911" extent="1-16" drill="0.3048"/>
+<via x="15.24" y="53.467" extent="1-16" drill="0.3048"/>
 </signal>
 <signal name="N$11">
@@
 <contactref element="R7" pad="2"/>
 <wire x1="10.795" y1="53.975" x2="9.017" y2="53.975" width="0.254" layer="1"/>
-<wire x1="11.176" y1="53.594" x2="10.795" y2="53.975" width="0.254" layer="1"/>
-<wire x1="11.176" y1="51.435" x2="11.176" y2="53.594" width="0.254" layer="1"/>
-<wire x1="11.049" y1="51.308" x2="11.176" y2="51.435" width="0.254" layer="1"/>
-<wire x1="11.049" y1="48.006" x2="11.049" y2="51.308" width="0.254" layer="1"/>
-<wire x1="15.24" y1="43.815" x2="11.049" y2="48.006" width="0.254" layer="1"/>
+<wire x1="12.319" y1="52.451" x2="10.795" y2="53.975" width="0.254" layer="1"/>
+<wire x1="12.319" y1="46.736" x2="12.319" y2="52.451" width="0.254" layer="1"/>
+<wire x1="15.24" y1="43.815" x2="12.319" y2="46.736" width="0.254" layer="1"/>
 </signal>
 </signals>
