File: Eurorack Set 2/MiniBus.sch (EAGLE design)
At the start: 32 parts

Commit message: Finally some updates...
Parts:
- added H1, H2, H3, H4, H5, H6: MOUNT-HOLE, zephod-components:MOUNT-HOLE
Changed lines of the file:
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@@
 </variantdefs>
 <classes>
-<class number="0" name="default" width="0" drill="0">
+<class number="0" name="default" width="0.508" drill="0">
 </class>
 </classes>
@@
 <part name="GND9" library="SparkFun-Aesthetics" deviceset="GND" device=""/>
 <part name="GND10" library="SparkFun-Aesthetics" deviceset="GND" device=""/>
+<part name="H1" library="zephod-components" deviceset="MOUNT-HOLE" device=""/>
+<part name="H2" library="zephod-components" deviceset="MOUNT-HOLE" device=""/>
+<part name="H3" library="zephod-components" deviceset="MOUNT-HOLE" device=""/>
+<part name="H4" library="zephod-components" deviceset="MOUNT-HOLE" device=""/>
+<part name="H5" library="zephod-components" deviceset="MOUNT-HOLE" device=""/>
+<part name="H6" library="zephod-components" deviceset="MOUNT-HOLE" device=""/>
 </parts>
 <sheets>
@@
 <instance part="GND9" gate="1" x="12.7" y="139.7" rot="R180"/>
 <instance part="GND10" gate="1" x="66.04" y="119.38"/>
+<instance part="H1" gate="G$1" x="27.94" y="193.04"/>
+<instance part="H2" gate="G$1" x="7.62" y="193.04"/>
+<instance part="H3" gate="G$1" x="27.94" y="187.96"/>
+<instance part="H4" gate="G$1" x="63.5" y="187.96"/>
+<instance part="H5" gate="G$1" x="2.54" y="208.28"/>
+<instance part="H6" gate="G$1" x="-20.32" y="187.96"/>
 </instances>
 <busses>
