File: Eurorack Set 3/Melody.brd (EAGLE design)
At the start: 39.3 x 106.5 mm, 72 parts, among them IC1 LD1117AS33TR, IC2 MCP6004, IC4 7905, Q2 MMBT3904, U1 MKL02Z32VFK4

Commit message: Melody And Screwdriver Updates
Parts:
- removed GATE: Gate, EurorackModularParts:3.5MM-JACK-SWITCH-13MM-INPUT
- removed LED1, LED2, LED3: (no value), SparkFun-LED:LED3MM
- removed R23: 10k, OPL:R0603
- removed U$11, U$9: FIDUCIAL, adafruit:FIDUCIAL_1MM
- removed U$3, U$6: SWITCH_W_LED_PB6149L-X-102WHITE, zephod-components:PB6149L
- added CLOCK: Clock, EurorackModularParts:3.5MM-JACK-SWITCH-13MM-INPUT
- added JP2: (no value), SparkFun-Connectors:1X04
- added Q1: MMBT3904, transistor:SOT23-BEC
- added RESET: Reset, EurorackModularParts:3.5MM-JACK-SWITCH-13MM-INPUT
- added SW1: EC12E_SW, switch-alps:ALPS_EC12E_SW
- added U$12: 0.49"OLEDFOLDED, zephod-tft:0.49"-FPC-0.7-14-FOLDED
- R18: value 2k -> 100k
- R19, R22: value 56 -> 33k
- R20: value 2k -> 10k
- R21: value 2k -> 33k
- U$2: value EURORACK_PCB8HP -> EURORACK_PCB12HP; device EurorackModularParts:EURORACK8HPPCB -> EurorackModularParts:EURORACK12HPPCB
- U$4: value FIDUCIAL -> GATE2; device adafruit:FIDUCIAL_1MM -> EurorackModularParts:3.5MM-JACK-SWITCH-13MM-OUTPUT
- U$5: value FIDUCIAL -> GATE1; device adafruit:FIDUCIAL_1MM -> EurorackModularParts:3.5MM-JACK-SWITCH-13MM-OUTPUT
- U$7: value Out 2 -> CV2
- U$8: value Out 1 -> CV1
- moved U$4 92.4 mm to (38.1, 10.2)
- moved R18 91.8 mm to (20.3, 87.0)
- moved R21 83.7 mm to (45.7, 84.5), turned to 0 degrees
- moved R20 79.6 mm to (26.7, 80.6), turned to 0 degrees
- moved C8 77.5 mm to (58.2, 43.8), turned to 180 degrees
- moved C12 77.1 mm to (57.4, 41.3), turned to 0 degrees
- moved IC1 77.1 mm to (56.5, 49.5)
- moved C11 76.7 mm to (56.1, 55.8)
- moved C13 76.7 mm to (56.1, 58.3)
- moved R19 76.5 mm to (45.7, 89.5), turned to 0 degrees
- moved D1 73.0 mm to (49.5, 50.2)
- moved D2 72.5 mm to (49.5, 60.3), turned to 0 degrees
- moved Q2 72.2 mm to (25.4, 103.5), turned to 270 degrees
- moved U$1 71.6 mm to (42.5, 54.0)
- moved R17 70.3 mm to (10.2, 10.2)
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Connections:
- removed net LED1: U$6.LEDPOS, U1.1
- removed net LED2: LED1.A, U1.20
- removed net LED3: LED2.A, U1.14
- removed net LED4: LED3.A, U1.13
- removed net N$1: JP1.3, U1.5
- removed net N$19: R22.1, U$3.LEDNEG
- removed net SW1: U$6.1, U$6.2, U1.2
- removed net SW2: R23.1, U$3.1, U$3.2, U1.17
- removed net SW2LED: R22.2, U1.18
- new net ENC_A: R19.2, SW1.A, U1.5
- new net ENC_B: R21.2, SW1.B, U1.6
- new net ENC_S: R22.2, SW1.E, U1.20
- new net RESET: Q1.C, R20.1, U1.13
- new net SCL: JP1.3, U1.17
- new net SDA: JP1.2, U1.18
- net 3.3V: now also R13.P$3, R14.P$3, R17.P$3, R19.1, R20.2, R21.1, R22.1, R90.P$3; no longer R13.P$1, R14.P$1, R17.P$1, R23.2, R90.P$1, U$3.LEDPOS
- net GND: now also CLOCK.RING@1, CLOCK.RING@2, Q1.E, R13.P$1, R14.P$1, R17.P$1, R90.P$1, RESET.RING@1, RESET.RING@2, SW1.C, SW1.D; no longer GATE.RING@1, GATE.RING@2, R13.P$3, R14.P$3, R17.P$3, R18.2, R19.2, R20.2, R21.2, R90.P$3, U$3.3, U$3.4, U$6.3, U$6.4
- net N$14: now also U1.1; no longer R19.1, U$6.LEDNEG
- net N$15: now also Q1.B, R18.2; no longer LED3.K, R18.1
- net N$16: now also R18.1, RESET.TIP@1, RESET.TIP@2; no longer LED2.K, R20.1
- net N$17: now also U1.2; no longer LED1.K, R21.1
- net N$2: now also U1.14; no longer JP1.2, U1.6
- net N$43: now also CLOCK.TIP@1, CLOCK.TIP@2; no longer GATE.TIP@1, GATE.TIP@2
- net RACK_GATE: now also CLOCK.SWITCH@1, CLOCK.SWITCH@2, RESET.SWITCH@1, RESET.SWITCH@2; no longer GATE.SWITCH@1, GATE.SWITCH@2
Other:
- board size 39.3 x 106.5 mm -> 59.6 x 106.5 mm

Commit message: Melody progress
Parts:
- removed U$5: GATE1, EurorackModularParts:3.5MM-JACK-SWITCH-13MM-OUTPUT
- U$4: value GATE2 -> ACCENT
- U$7: value CV2 -> NOTE
- U$8: value CV1 -> VELOCITY
Changed lines of the file:
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@@
 <element name="IN1" library="EurorackModularParts" package="3.5MM-JACK-SWITCH-13MM-INPUT" value="In 2" x="12.7" y="45.72"/>
 <element name="IN2" library="EurorackModularParts" package="3.5MM-JACK-SWITCH-13MM-INPUT" value="In 1" x="12.7" y="63.5"/>
-<element name="U$7" library="EurorackModularParts" package="3.5MM-JACK-SWITCH-13MM-OUTPUT" value="CV2" x="53.34" y="10.16"/>
-<element name="U$8" library="EurorackModularParts" package="3.5MM-JACK-SWITCH-13MM-OUTPUT" value="CV1" x="53.34" y="27.94"/>
+<element name="U$7" library="EurorackModularParts" package="3.5MM-JACK-SWITCH-13MM-OUTPUT" value="NOTE" x="53.34" y="10.16"/>
+<element name="U$8" library="EurorackModularParts" package="3.5MM-JACK-SWITCH-13MM-OUTPUT" value="VELOCITY" x="53.34" y="27.94"/>
 <element name="U$2" library="EurorackModularParts" package="EURORACK12HPPCB" value="EURORACK_PCB12HP" x="0.67" y="0"/>
 <element name="D3" library="diode" package="SOT23" value="BAS70-04" x="16.74" y="36.735" rot="R270"/>
@@
 <element name="R20" library="OPL" package="R0603" value="10k" x="26.67" y="80.645"/>
 <element name="RESET" library="EurorackModularParts" package="3.5MM-JACK-SWITCH-13MM-INPUT" value="Reset" x="12.7" y="81.28"/>
-<element name="U$4" library="EurorackModularParts" package="3.5MM-JACK-SWITCH-13MM-OUTPUT" value="GATE2" x="38.1" y="10.16"/>
-<element name="U$5" library="EurorackModularParts" package="3.5MM-JACK-SWITCH-13MM-OUTPUT" value="GATE1" x="38.1" y="27.94"/>
+<element name="U$4" library="EurorackModularParts" package="3.5MM-JACK-SWITCH-13MM-OUTPUT" value="ACCENT" x="38.1" y="10.16"/>
 <element name="JP2" library="SparkFun-Connectors" package="1X04" value="" x="31.75" y="104.14"/>
 <element name="SW1" library="switch-alps" package="ALPS_EC12E_SW" value="EC12E_SW" x="52.07" y="97.79">

Commit message: Melody Updates
Parts:
- removed JP1, JP2: (no value), SparkFun-Connectors:1X04
- removed R13: A, EurorackModularParts:OG-POTS_ALPS_POT_VERTICAL
- removed R90: C, EurorackModularParts:OG-POTS_ALPS_POT_VERTICAL
- removed SW1: EC12E_SW, switch-alps:ALPS_EC12E_SW
- removed U$12: 0.49"OLEDFOLDED, zephod-tft:0.49"-FPC-0.7-14-FOLDED
- removed U$4: ACCENT, EurorackModularParts:3.5MM-JACK-SWITCH-13MM-OUTPUT
- added ACCENT: ACCENT, EurorackModularParts:3.5MM-JACK-SWITCH-13MM-OUTPUT
- added BEAT: Beat, EurorackModularParts:3.5MM-JACK-SWITCH-13MM-OUTPUT
- added BUTTON_ALGO, BUTTON_BEATS, BUTTON_SCALE, BUTTON_TPB: BUTTON-4P-3100010P1, zephod-components:4P-SMD-6.0X6.0X5.0H
- added C20, C7: 100nF, OPL:C0603
- added C5: 10uF, OPL:AVX-A
- added C6: 1uF, OPL:C0603
- added CLOCKOUT_JACK: Clock Out, EurorackModularParts:3.5MM-JACK-SWITCH-13MM-OUTPUT
- added D5: BAS70-04, diode:SOT23
- added GATE: GATE, EurorackModularParts:3.5MM-JACK-SWITCH-13MM-OUTPUT
- added IC3, IC5: IC_74HC595-SOIC-16, dp_devices:SOIC-16
- added IC6: MCP6004, gm-ics:SO14
- added INTENSITY: INTENSITY, EurorackModularParts:3.5MM-JACK-SWITCH-13MM-INPUT
- added LED10_BEAT, LED11_LOOP, LED12_GATE, LED9_CLOCK, LED_ALGO_FOURCHORD, LED_ALGO_GOA, LED_ALGO_PSYCH, LED_BEAT_16, LED_BEAT_2, LED_BEAT_4, LED_BEAT_8, LED_SCALE_DORIAN, LED_SCALE_MAJOR, LED_SCALE_MINOR, LED_SCALE_PENTA, LED_TPB_2, LED_TPB_3, LED_TPB_4, LED_TPB_6: (no value), SparkFun-LED:LED3MM
- added LED_ALGO_FLAT: WHITE_WITH_11MM_SPACER, SparkFun-LED:LED3MM
- added LOOP: Loop, EurorackModularParts:3.5MM-JACK-SWITCH-13MM-OUTPUT
- added POT_IN1: A, EurorackModularParts:OG-POTS_ALPS_POT_VERTICAL
- added POT_IN2: B, EurorackModularParts:OG-POTS_ALPS_POT_VERTICAL
- added POT_TEMPO: TEMPO, EurorackModularParts:OG-POTS_ALPS_POT_VERTICAL
- added Q3, Q4, Q5, Q6, Q7, Q8: MMBT3904, transistor:SOT23-BEC
- added R23, R26, R27, R28, R30, R38, R40, R42, R44, R46: 100k, OPL:R0603
- added R29: 100, OPL:R0603
- added R31, R32, R33, R34, R35: 2k, OPL:R1206-8
- added R36: 10k, OPL:R1206-8
- added R37, R39, R41, R43, R45: 10k, OPL:R0603
- added TICK: Tick, EurorackModularParts:3.5MM-JACK-SWITCH-13MM-OUTPUT
- added U2: LM4040DIM3-5.0, FarnellThings:SOT95P237X112-3N
- C14, C4: value 10uF -> 100nF; device OPL:AVX-A -> OPL:C0603
- C16: value 100nF -> 3.3n
- CLOCK: value Clock -> Clock In
- IC4: value 7905 -> IC_74HC595-SOIC-16; device linear:TO220H -> dp_devices:SOIC-16
- IN1: value In 2 -> In 1
- IN2: value In 1 -> In 2
- R14: value D -> 100k; device EurorackModularParts:OG-POTS_ALPS_POT_VERTICAL -> OPL:R0603
- R17: value B -> D
- R19: value 33k -> 10k
- R21: value 33k -> 100k
- moved IC4 167.2 mm to (207.0, 12.7)
- moved C14 164.2 mm to (213.4, 10.2), turned to 90 degrees
- moved C4 152.4 mm to (196.8, 12.7)
- moved R10 116.3 mm to (134.5, 46.6)
- moved IC2 113.7 mm to (135.2, 29.2)
- moved R11 113.7 mm to (137.6, 45.3)
- moved R3 113.7 mm to (142.2, 23.9)
- moved C1 113.7 mm to (138.3, 36.8)
- moved C10 113.7 mm to (144.8, 33.3)
- moved C15 113.7 mm to (131.8, 21.8)
- moved C18 113.7 mm to (135.3, 23.8)
- moved C19 113.7 mm to (134.8, 34.8)
- moved C2 113.7 mm to (138.8, 23.8)
- moved C3 113.7 mm to (131.3, 34.8)
- moved C9 113.7 mm to (144.8, 28.3)
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Connections:
- net GATE renamed CLOCK_IN
- removed net ENC_A: R19.2, SW1.A, U1.5
- removed net ENC_B: R21.2, SW1.B, U1.6
- removed net ENC_S: R22.2, SW1.E, U1.20
- removed net KNOB_A: R90.P$2, U1.19
- removed net KNOB_B: R13.P$2, U1.9
- removed net KNOB_C: R14.P$2, U1.10
- removed net KNOB_D: R17.P$2, U1.21
- removed net VEE: C17.1, C19.2, C4.-, D2.A, IC2.11, IC4.2
- removed net VIN: C11.2, C13.+, C18.2, D1.C, IC1.3, IC2.4
- new net -12V: C19.2, C20.1, C5.-, D2.A, IC2.11, IC6.11, R26.1
- new net 12V: C11.2, C13.+, C17.1, C18.2, D1.C, IC1.3, IC2.4, IC6.4, R19.2, R37.2, R39.2, R41.2, R43.2, R45.2
- new net ADC_3: U1.21
- new net BUTTON_ALGO: BUTTON_ALGO.1, BUTTON_ALGO.4, R36.1
- new net BUTTON_BEATS: BUTTON_BEATS.1, BUTTON_BEATS.4, R36.4
- new net BUTTON_SCALE: BUTTON_SCALE.1, BUTTON_SCALE.4, R36.3
- new net BUTTON_TPB: BUTTON_TPB.1, BUTTON_TPB.4, R36.2
- new net KNOB_IN1: POT_IN1.P$2, R23.2
- new net KNOB_IN2: POT_IN2.P$2, R27.2
- new net KNOB_INTENSITY: R17.P$2, R30.2
- new net KNOB_TEMPO: POT_TEMPO.P$2, U1.10
- new net N$1: IC3.12
- new net N$19: IC3.11
- new net N$22: IC3.14
- new net N$23: R21.1
- new net N$25: Q3.B, R21.2
- new net N$26: IC4.11
- new net N$27: IC4.12
- new net N$28: IC3.9, IC4.14
- new net N$29: ACCENT.TIP@1, ACCENT.TIP@2, Q3.C, R19.1
- new net N$30: IC5.11
- new net N$31: IC5.12
- new net N$32: IC4.9, IC5.14
- new net N$33: INTENSITY.TIP@1, INTENSITY.TIP@2, R14.2
- new net N$34: C16.1, IC6.2, R14.1, R22.2, R28.1, R30.1
- new net N$35: IC3.15, R31.8
- new net N$36: IC3.1, R31.7
- new net N$37: IC3.2, R31.6
- new net N$38: IC3.3, R31.5
- new net N$39: IC3.4, R32.8
- new net N$40: IC3.5, R32.2
- new net N$41: IC3.6, R32.3
- new net N$42: IC3.7, R32.4
- new net N$44: IC5.15, R35.4
- new net N$45: IC5.1, R35.3
- new net N$46: IC5.2, R35.2
- new net N$47: IC5.3, R35.1
- new net N$48: IC4.15, R33.4
- new net N$49: IC4.1, R33.3
- new net N$50: IC4.2, R33.2
- new net N$51: IC4.3, R33.1
- new net N$52: IC4.4, R34.4
- new net N$53: IC4.5, R34.3
- new net N$54: IC4.6, R34.2
- new net N$55: IC4.7, R34.1
- new net N$56: R38.1
- new net N$57: Q4.B, R38.2
- new net N$58: GATE.TIP@1, GATE.TIP@2, Q4.C, R37.1
- new net N$59: R40.1
- new net N$60: Q5.B, R40.2
- new net N$61: CLOCKOUT_JACK.TIP@1, CLOCKOUT_JACK.TIP@2, Q5.C, R39.1
- new net N$62: R42.1
- new net N$63: Q6.B, R42.2
- new net N$65: Q6.C, R41.1, TICK.TIP@1, TICK.TIP@2
- new net N$67: R44.1
- new net N$68: Q7.B, R44.2
- new net N$69: BEAT.TIP@1, BEAT.TIP@2, Q7.C, R43.1
- new net N$70: R46.1
- new net N$71: Q8.B, R46.2
- new net N$72: LOOP.TIP@1, LOOP.TIP@2, Q8.C, R45.1
- net 3.3V: now also C14.2, C4.2, C7.2, CLOCK.SWITCH@1, CLOCK.SWITCH@2, D5.2, IC3.10, IC3.16, IC4.10, IC4.16, IC5.10, IC5.16, POT_IN1.P$3, POT_IN2.P$3, POT_TEMPO.P$3, R36.5, R36.6, R36.7, R36.8; no longer JP1.4, R13.P$3, R14.P$3, R19.1, R21.1, R22.1, R90.P$3
- net ADC_1: now also D5.3, R29.1
- net ADC_1_PRE: now also C16.2, IC6.1, R22.1, R29.2
- net GND: now also ACCENT.RING@1, ACCENT.RING@2, BEAT.RING@1, BEAT.RING@2, BUTTON_ALGO.2, BUTTON_ALGO.3, BUTTON_BEATS.2, BUTTON_BEATS.3, BUTTON_SCALE.2, BUTTON_SCALE.3, BUTTON_TPB.2, BUTTON_TPB.3, C14.1, C20.2, C4.1, C5.+, C6.1, C7.1, CLOCKOUT_JACK.RING@1, CLOCKOUT_JACK.RING@2, D5.1, GATE.RING@1, GATE.RING@2, IC3.13, IC3.8, IC4.13, IC4.8, IC5.13, IC5.8, IC6.3, INTENSITY.RING@1, INTENSITY.RING@2, INTENSITY.SWITCH@1, INTENSITY.SWITCH@2, LED10_BEAT.K, LED11_LOOP.K, LED12_GATE.K, LED9_CLOCK.K, LED_ALGO_FLAT.K, LED_ALGO_FOURCHORD.K, LED_ALGO_GOA.K, LED_ALGO_PSYCH.K, LED_BEAT_16.K, LED_BEAT_2.K, LED_BEAT_4.K, LED_BEAT_8.K, LED_SCALE_DORIAN.K, LED_SCALE_MAJOR.K, LED_SCALE_MINOR.K, LED_SCALE_PENTA.K, LED_TPB_2.K, LED_TPB_3.K, LED_TPB_4.K, LED_TPB_6.K, LOOP.RING@1, LOOP.RING@2, POT_IN1.P$1, POT_IN2.P$1, POT_TEMPO.P$1, Q3.E, Q4.E, Q5.E, Q6.E, Q7.E, Q8.E, RESET.SWITCH@1, RESET.SWITCH@2, TICK.RING@1, TICK.RING@2, U2.1; no longer C14.+, C16.2, C4.+, IC4.1, JP1.1, R13.P$1, R14.P$1, R90.P$1, SW1.C, SW1.D
- net N$4: now also R23.1
- net N$8: now also R27.1
- net RACK_GATE: no longer CLOCK.SWITCH@1, CLOCK.SWITCH@2, RESET.SWITCH@1, RESET.SWITCH@2
- net REF_-5V: now also C6.2, R26.2, R28.2, U2.2; no longer C14.-, C16.1, IC4.3
- net SCL: no longer JP1.3
- net SDA: no longer JP1.2

Commit message: Melody Updates
Parts:
- removed IC3, IC4, IC5: IC_74HC595-SOIC-16, dp_devices:SOIC-16
- added U3, U4, U5: 74HC595BQ, FarnellThings:QFN50P250X350X100-17N
- POT_IN1: value A -> SEED A
- POT_IN2: value B -> SEED B
- R17: value D -> INTENSITY
- moved R34 215.7 mm to (3.81, 74.9), turned to 0 degrees
- moved R33 205.2 mm to (5.08, 59.7), turned to 0 degrees
- moved C4 192.9 mm to (8.89, 55.9), turned to 270 degrees
- moved R32 153.9 mm to (40.6, 74.9)
- moved R31 143.2 mm to (40.6, 59.7), turned to 180 degrees
- moved R35 135.4 mm to (92.7, 57.1), turned to 0 degrees
- moved C7 133.3 mm to (41.9, 53.3)
- moved C14 126.1 mm to (94.0, 50.8), turned to 270 degrees
- moved R36 32.9 mm to (24.1, 72.4)
- moved U1 14.4 mm to (94.0, 65.4)
- moved RESET 3.81 mm to (38.1, 99.1)
- moved POT_TEMPO 2.54 mm to (22.9, 99.1)
- renumbered BUTTON_ALGO to B_ALGO, BUTTON_BEATS to B_BEATS, BUTTON_SCALE to B_SCALE, BUTTON_TPB to B_TPB, U$7 to NOTE, U$8 to VELOCITY
Connections:
- net ADC_2 renamed ADC_IN2
- removed net ADC_1: D3.3, D5.3, R10.1, R29.1, U1.15
- removed net ADC_3: U1.21
- new net ADC_IN1: D3.3, R10.1, U1.15
- new net ADC_INTENSITY: D5.3, R29.1, U1.21
- new net ADC_INTENSITY_PRE: C16.2, IC6.1, R22.1, R29.2
- new net N$73: LED_ALGO_GOA.A, R34.5
- new net N$74: LED_ALGO_FLAT.A, R34.6
- new net N$75: LED_ALGO_PSYCH.A, R34.7
- new net N$76: LED_ALGO_FOURCHORD.A, R34.8
- new net N$77: LED_SCALE_MINOR.A, R33.7
- new net N$78: LED_SCALE_PENTA.A, R33.8
- new net N$79: LED_BEAT_16.A, R31.1
- new net N$80: LED_BEAT_8.A, R31.2
- new net N$81: LED_BEAT_4.A, R31.3
- new net N$82: LED_BEAT_2.A, R31.4
- new net N$83: LED_TPB_2.A, R32.8
- new net N$84: LED_TPB_3.A, R32.7
- new net N$85: LED_TPB_4.A, R32.6
- new net N$86: LED_TPB_6.A, R32.5
- new net N$87: U3.14
- new net N$88: U5.9
- new net N$89: U4.9
- net 3.3V: now also U3.10, U3.16, U4.10, U4.16, U5.10, U5.16; no longer IC3.10, IC3.16, IC4.10, IC4.16, IC5.10, IC5.16
- net ADC_1_PRE: no longer C16.2, IC6.1, R22.1, R29.2
- net GND: now also U3.13, U3.17, U3.8, U4.13, U4.17, U4.8, U5.13, U5.17, U5.8; no longer IC3.13, IC3.8, IC4.13, IC4.8, IC5.13, IC5.8
- net N$1: now also U4.12; no longer IC3.12
- net N$19: now also U4.11; no longer IC3.11
- net N$22: now also U4.14; no longer IC3.14
- net N$26: now also U5.11; no longer IC4.11
- net N$27: now also U5.12; no longer IC4.12
- net N$28: now also LED_SCALE_DORIAN.A, R33.5; no longer IC3.9, IC4.14
- net N$30: now also U3.11; no longer IC5.11
- net N$31: now also U3.12; no longer IC5.12
- net N$32: now also LED_SCALE_MAJOR.A, R33.6; no longer IC4.9, IC5.14
- net N$35: now also U4.15; no longer IC3.15
- net N$36: now also U4.1; no longer IC3.1
- net N$37: now also U4.2; no longer IC3.2
- net N$38: now also U4.3; no longer IC3.3
- net N$39: now also R32.4, U4.4; no longer IC3.4, R32.8
- net N$40: now also R32.3, U4.5; no longer IC3.5, R32.2
- net N$41: now also R32.2, U4.6; no longer IC3.6, R32.3
- net N$42: now also R32.1, U4.7; no longer IC3.7, R32.4
- net N$44: now also U3.15; no longer IC5.15
- net N$45: now also U3.1; no longer IC5.1
- net N$46: now also U3.2; no longer IC5.2
- net N$47: now also U3.3; no longer IC5.3
- net N$48: now also U5.15; no longer IC4.15
- net N$49: now also U5.1; no longer IC4.1
- net N$50: now also U5.2; no longer IC4.2
- net N$51: now also U5.3; no longer IC4.3
- net N$52: now also U5.4; no longer IC4.4
- net N$53: now also U5.5; no longer IC4.5
- net N$54: now also U5.6; no longer IC4.6
- net N$55: now also U5.7; no longer IC4.7

Commit message: Melody Updates
Parts:
- removed C20: 100nF, OPL:C0603
- removed C9: 1uF, OPL:C0603
- removed D1, D2: 1N5819HW, diode:SOD123
- removed D5: BAS70-04, diode:SOT23
- removed IC2, IC6: MCP6004, gm-ics:SO14
- removed R35: 2k, OPL:R1206-8
- added C21: 100nF, OPL:C0603
- added IC3: TL074D, EurorackModularParts:SO14
- added IC4: MCP6004, EurorackModularParts:SO14
- added LED_ACCENT: WHITE 3MM WITH 11MM HOLDER, SparkFun-LED:LED3MM
- added R13, R47, R48, R49, R50, R51: 2k, OPL:R0603
- added R52, R53: 100k, OPL:R0603
- added U6: 24LC00T-I/OT, EurorackModularParts:SOT95P290X145-5N
- C11: value 100Nf -> 100nF
- C13: value 10Uf -> 10uF
- D3, D4: value BAS70-04 -> MRA4004T3G; device diode:SOT23 -> OPL:DO-214AC
- LED_ALGO_FOURCHORD, LED_ALGO_GOA, LED_ALGO_PSYCH, LED_BEAT, LED_BEAT_16, LED_BEAT_2, LED_BEAT_4, LED_BEAT_8, LED_GATE, LED_LOOP, LED_SCALE_DORIAN, LED_SCALE_MAJOR, LED_SCALE_MINOR, LED_SCALE_PENTA, LED_TICK, LED_TPB_2, LED_TPB_3, LED_TPB_4, LED_TPB_6: value (none) -> WHITE 3MM WITH 11MM HOLDER
- R1, R14, R16: value 100k -> 100k 1%
- R10: value 100 -> 2k
- R11, R29: value 100 -> 10k
- R12, R2, R22: value 33k -> 33k 1%
- R15, R3: value 100k -> 49.9k 1%
- R23, R27, R30: value 100k -> 33k 1%
- R24, R25: value 51 -> 100
- R26: value 100k -> 10k
- R28: value 100k -> 49.9k
- R5, R8: value 100k -> 25.5k 1%
- R7, R9: value 33k -> 10.2k 1%
- moved R11 133.2 mm to (13.3, 93.3), turned to 0 degrees
- moved R3 118.4 mm to (24.8, 38.7), turned to 90 degrees
- moved C10 114.6 mm to (31.8, 51.8), turned to 0 degrees
- moved C13 110.7 mm to (3.31, 42.1), turned to 90 degrees
- moved C11 107.5 mm to (5.82, 41.5), turned to 270 degrees
- moved U$1 106.3 mm to (10.8, 19.7), turned to 180 degrees
- moved U$10 105.1 mm to (31.6, 42.3)
- moved R7 104.7 mm to (33.0, 36.8)
- moved R9 104.6 mm to (31.1, 36.8)
- moved R5 104.1 mm to (34.9, 28.2)
- moved C19 104.0 mm to (33.0, 13.3), turned to 90 degrees
- moved R8 103.8 mm to (30.5, 12.1)
- moved C6 103.8 mm to (11.4, 57.8), turned to 90 degrees
- moved C2 103.6 mm to (35.3, 26.4)
- moved R4 103.3 mm to (33.7, 9.94), turned to 0 degrees
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- renumbered LED10_BEAT to LED_BEAT, LED11_LOOP to LED_LOOP, LED12_GATE to LED_GATE, LED9_CLOCK to LED_TICK
Connections:
- net N$5 renamed SWD_CLK
- net N$7 renamed SWD_DIO
- net RESET renamed RESET_PATTERN
- removed net ADC_1_PRE: C15.2, IC2.1, R10.2, R12.1
- removed net ADC_2_PRE: C1.2, IC2.8, R11.2, R2.1
- removed net ADC_INTENSITY_PRE: C16.2, IC6.1, R22.1, R29.2
- removed net N$1 (its old number): U4.12
- removed net N$19 (its old number): U4.11
- removed net N$22: U4.14
- removed net N$23: R21.1
- removed net N$26 (its old number): U5.11
- removed net N$27 (its old number): U5.12
- removed net N$30 (its old number): U3.11
- removed net N$31 (its old number): U3.12
- removed net N$44: R35.4, U3.15
- removed net N$45: R35.3, U3.1
- removed net N$46: R35.2, U3.2
- removed net N$47: R35.1, U3.3
- removed net N$50: R33.2, U5.2
- removed net N$51: R33.1, U5.3
- removed net N$52: R34.4, U5.4
- removed net N$53: R34.3, U5.5
- removed net N$54: R34.2, U5.6
- removed net N$55: R34.1, U5.7
- removed net N$56: R38.1
- removed net N$59: R40.1
- removed net N$62: R42.1
- removed net N$67: R44.1
- removed net N$70: R46.1
- removed net N$87: U3.14
- removed net PTA1: SWD1.10, U1.23
- removed net RACK_GATE: U$1.15, U$1.16
- new net CLOCK: U1.1, U3.11, U4.11, U5.11
- new net CPU_RESET: R29.2, SWD1.10, U1.23
- new net LATCH: U1.19, U3.12, U4.12, U5.12
- new net N$37: R34.4, U5.15
- new net N$38: R34.3, U5.1
- new net N$39: R34.2, U5.2
- new net N$40: R34.1, U5.3
- new net N$41: R33.4, U5.4
- new net N$42: R33.3, U5.5
- new net N$90: LED_TICK.A, R13.1
- new net N$91: LED_LOOP.A, R48.1
- new net N$92: LED_GATE.A, R49.1
- new net N$93: LED_BEAT.A, R47.1
- new net N$94: IC3.7, R25.2, R52.2
- new net N$95: LED_ACCENT.A, R10.1
- new net N$96: CLOCK.SWITCH@1, CLOCK.SWITCH@2, R11.1
- new net N$97: IC4.5, IC4.7
- new net OUT_ACCENT: R10.2, R21.1, U3.4
- new net OUT_BEAT: R44.1, R47.2, U3.2
- new net OUT_CLOCK: R40.1, U3.15
- new net OUT_GATE: R38.1, R49.2, U3.5
- new net OUT_LOOP: R46.1, R48.2, U3.3
- new net OUT_TICK: R13.2, R42.1, U3.1
- new net SHIFTERS: U1.2, U5.14
- net -12V: now also D4.1, IC3.11; no longer C20.1, D2.A, IC2.11, IC6.11
- net 12V: now also D3.2, IC3.4, R11.2; no longer C17.1, D1.C, IC2.4, IC6.4
- net 3.3V: now also C17.1, C21.2, IC4.4, POT_IN1.P$1, POT_IN2.P$1, R17.P$1, R29.1, R50.1, R51.1, U6.5; no longer C9.2, CLOCK.SWITCH@1, CLOCK.SWITCH@2, D3.2, D4.2, D5.2, POT_IN1.P$3, POT_IN2.P$3, R17.P$3
- net ADC_IN1: now also C15.2, IC4.8, R12.1; no longer D3.3, R10.1
- net ADC_IN2: now also C1.2, IC4.1, R2.1; no longer D4.3, R11.1
- net ADC_INTENSITY: now also C16.2, IC4.14, R22.1; no longer D5.3, R29.1
- net BUTTON_ALGO: now also U1.9
- net BUTTON_BEATS: now also U1.6
- net BUTTON_SCALE: now also U1.5
- net BUTTON_TPB: now also U1.20
- net CLOCK_IN: now also U1.14
- net GND: now also C21.1, IC3.10, IC3.12, IC3.3, IC3.5, IC4.10, IC4.11, IC4.12, IC4.3, IC4.6, LED_ACCENT.K, POT_IN1.P$3, POT_IN2.P$3, R17.P$3, U6.2; no longer C20.2, C9.1, D3.1, D4.1, D5.1, IC2.10, IC2.12, IC2.3, IC2.5, IC6.3, POT_IN1.P$1, POT_IN2.P$1, R17.P$1
- net N$10: now also IC3.9; no longer IC2.13, R4.2
- net N$13: now also D3.1; no longer D1.A
- net N$14: now also IC3.14, R24.2, R6.2; no longer U1.1
- net N$17: now also IC3.6, R52.1, R53.2; no longer U1.2
- net N$18: now also IC3.8, R4.1; no longer IC2.14, R24.2
- net N$2: now also IC3.13, R4.2, R6.1; no longer U1.14
- net N$24: now also IC3.1, R53.1; no longer IC2.7, R25.2
- net N$28: now also R33.6; no longer R33.5
- net N$32: now also R33.5; no longer R33.6
- net N$34: now also IC4.13; no longer IC6.2
- net N$4: now also IC4.9; no longer IC2.2
- net N$48: now also R33.2, U5.6; no longer R33.4, U5.15
- net N$49: now also R33.1, U5.7; no longer R33.3, U5.1
- net N$64: now also D4.2; no longer D2.C
- net N$73: now also R34.6; no longer R34.5
- net N$74: now also R34.5; no longer R34.6
- net N$79: now also R31.3; no longer R31.1
- net N$8: now also IC4.2; no longer IC2.9
- net N$81: now also R31.1; no longer R31.3
- net N$85: now also R32.5; no longer R32.6
- net N$86: now also R32.6; no longer R32.5
- net N$88: now also U4.14
- net N$89: now also U3.14
- net N$9: now also IC3.2; no longer IC2.6, R6.1
- net REF_-5V: no longer R4.1, R6.2
- net SCL: now also R50.2, U6.1
- net SDA: now also R51.2, U6.3
Routing:
- net GND: track 0.00 -> 361.2 mm, vias 0 -> 27
- net 3.3V: track 0.00 -> 246.8 mm, vias 0 -> 16
- net 12V: track 0.00 -> 197.4 mm, vias 0 -> 20
- net OUT_GATE: track 0.00 -> 96.6 mm, vias 0 -> 6
- net CLOCK: track 0.00 -> 84.7 mm, vias 0 -> 12
- net -12V: track 0.00 -> 83.9 mm, vias 0 -> 6
- net LATCH: track 0.00 -> 78.6 mm, vias 0 -> 17
- net CLOCK_IN: track 0.00 -> 78.2 mm, vias 0 -> 13
- net BUTTON_SCALE: track 0.00 -> 70.3 mm, vias 0 -> 8
- net RESET_PATTERN: track 0.00 -> 63.7 mm, vias 0 -> 10
- net KNOB_TEMPO: track 0.00 -> 63.1 mm, vias 0 -> 11
- net BUTTON_ALGO: track 0.00 -> 60.0 mm, vias 0 -> 10
- net OUT_ACCENT: track 0.00 -> 59.8 mm, vias 0 -> 2
- net OUT_LOOP: track 0.00 -> 54.6 mm, vias 0 -> 8
- net N$34: track 0.00 -> 54.0 mm, vias 0 -> 2
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