File: Eurorack Set 3/LEDDistortionV2.brd (EAGLE design)
At the start: 19 x 106.5 mm, 52 parts, among them IC1 TL072, IC2 TL072

Commit message: Final tweaks for the order - initial bom update for tuesday
Connections:
- net GND: now also U$2.RING@3, U$2.SWITCH@3, U$3.RING@3, U$6.RING@3; no longer U$2.RING@1, U$2.RING@2, U$2.SWITCH@1, U$2.SWITCH@2, U$3.RING@1, U$3.RING@2, U$6.RING@1, U$6.RING@2
- net N$12: now also U$6.TIP@3; no longer U$6.TIP@1, U$6.TIP@2
- net N$5: now also U$3.TIP@3; no longer U$3.TIP@1, U$3.TIP@2
- net N$6: now also U$2.TIP@3; no longer U$2.TIP@1, U$2.TIP@2
Routing:
- net GND: track 220.4 -> 194.8 mm
Changed lines of the file:
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@@
 <element name="C8" library="OPL" package="AVX-A" value="10u" x="16.51" y="86.995" rot="MR180"/>
 <element name="U$1" library="EurorackModularParts" package="POWER_10" value="POWER_SIMPLE10" x="10.16" y="90.805" rot="MR0"/>
-<element name="U$2" library="EurorackModularParts" package="3.5MM-JACK-SWITCH-13MM-INPUT" value="IN" x="7.62" y="99.06"/>
-<element name="U$3" library="EurorackModularParts" package="3.5MM-JACK-SWITCH-13MM-OUTPUT" value="OUT2" x="12.7" y="44.45"/>
+<element name="U$2" library="EurorackModularParts" package="3.5MM-JACK-SWITCH-13MM-INPUT" value="IN" x="7.62" y="99.06">
+<attribute name="DESC" value="Input" x="7.62" y="99.06" size="1.778" layer="27" display="off"/>
+<attribute name="MPN" value="PJ-341" x="7.62" y="99.06" size="1.778" layer="27" display="off"/>
+<attribute name="VALUE" value="PJ-341" x="7.62" y="99.06" size="1.778" layer="27" display="off"/>
+</element>
+<element name="U$3" library="EurorackModularParts" package="3.5MM-JACK-SWITCH-13MM-OUTPUT" value="OUT2" x="12.7" y="44.45">
+<attribute name="DESC" value="Output" x="12.7" y="44.45" size="1.778" layer="27" display="off"/>
+<attribute name="MPN" value="PJ-341" x="12.7" y="44.45" size="1.778" layer="27" display="off"/>
+<attribute name="VALUE" value="PJ-341" x="12.7" y="44.45" size="1.778" layer="27" display="off"/>
+</element>
 <element name="R1" library="OPL" package="C0805" value="TBD" x="15.875" y="76.835" rot="MR0"/>
 <element name="R2" library="OPL" package="C0805" value="100k" x="15.875" y="73.66" rot="MR270"/>
 <element name="LED1" library="SparkFun-LED" package="LED3MM" value="REDBLUE" x="3.81" y="6.35" rot="R90"/>
-<element name="GAIN1" library="EurorackModularParts" package="OG-POTS_ALPS_POT_VERTICAL" value="100k" x="10.16" y="83.82"/>
-<element name="POST1" library="EurorackModularParts" package="OG-POTS_ALPS_POT_VERTICAL" value="100k" x="10.16" y="60.96"/>
+<element name="GAIN1" library="EurorackModularParts" package="OG-POTS_ALPS_POT_VERTICAL" value="100k" x="10.16" y="83.82">
+<attribute name="DESC" value="Parameter" x="10.16" y="83.82" size="1.778" layer="27" display="off"/>
+</element>
+<element name="POST1" library="EurorackModularParts" package="OG-POTS_ALPS_POT_VERTICAL" value="100k" x="10.16" y="60.96">
+<attribute name="DESC" value="Parameter" x="10.16" y="60.96" size="1.778" layer="27" display="off"/>
+</element>
 <element name="R4" library="OPL" package="C0805" value="100k" x="4.445" y="72.39" rot="MR270"/>
 <element name="R3" library="OPL" package="C0805" value="100" x="1.905" y="72.39" rot="MR90"/>
@@
 <element name="IC2" library="EurorackModularParts" package="SO08" value="TL072" x="10.16" y="29.21" rot="MR270"/>
 <element name="R7" library="OPL" package="C0805" value="330" x="18.415" y="30.48" rot="MR90"/>
-<element name="U$6" library="EurorackModularParts" package="3.5MM-JACK-SWITCH-13MM-OUTPUT" value="OUT1" x="12.7" y="6.35"/>
+<element name="U$6" library="EurorackModularParts" package="3.5MM-JACK-SWITCH-13MM-OUTPUT" value="OUT1" x="12.7" y="6.35">
+<attribute name="DESC" value="Output" x="12.7" y="6.35" size="1.778" layer="27" display="off"/>
+<attribute name="MPN" value="PJ-341" x="12.7" y="6.35" size="1.778" layer="27" display="off"/>
+<attribute name="VALUE" value="PJ-341" x="12.7" y="6.35" size="1.778" layer="27" display="off"/>
+</element>
 <element name="R8" library="OPL" package="C0805" value="TBD" x="18.415" y="34.925" rot="MR90"/>
 <element name="R9" library="OPL" package="C0805" value="100k" x="16.51" y="30.48" rot="MR270"/>
 <element name="LED2" library="SparkFun-LED" package="LED3MM" value="BLUERED" x="3.81" y="44.45" rot="R90"/>
-<element name="POST2" library="EurorackModularParts" package="OG-POTS_ALPS_POT_VERTICAL" value="100k" x="10.16" y="22.86"/>
+<element name="POST2" library="EurorackModularParts" package="OG-POTS_ALPS_POT_VERTICAL" value="100k" x="10.16" y="22.86">
+<attribute name="DESC" value="Parameter" x="10.16" y="22.86" size="1.778" layer="27" display="off"/>
+</element>
 <element name="R10" library="OPL" package="C0805" value="100k" x="3.81" y="29.21" rot="MR270"/>
 <element name="R12" library="OPL" package="C0805" value="100" x="1.905" y="29.21" rot="MR90"/>
@@
 <contactref element="U$1" pad="5"/>
 <contactref element="U$1" pad="7"/>
-<contactref element="U$2" pad="RING@2"/>
-<contactref element="U$2" pad="RING@1"/>
-<contactref element="U$2" pad="SWITCH@2"/>
-<contactref element="U$2" pad="SWITCH@1"/>
-<contactref element="U$3" pad="RING@2"/>
-<contactref element="U$3" pad="RING@1"/>
+<contactref element="U$2" pad="RING@3"/>
+<contactref element="U$2" pad="SWITCH@3"/>
+<contactref element="U$3" pad="RING@3"/>
 <contactref element="IC1" pad="3"/>
 <contactref element="LED1" pad="K"/>
@@
 <contactref element="POST1" pad="P$1"/>
 <contactref element="IC1" pad="5"/>
-<contactref element="U$6" pad="RING@2"/>
-<contactref element="U$6" pad="RING@1"/>
+<contactref element="U$6" pad="RING@3"/>
 <contactref element="IC2" pad="3"/>
 <contactref element="LED2" pad="K"/>
@@
 <wire x1="7.62" y1="7.62" x2="7.62" y2="16.129" width="0.3048" layer="1"/>
 <wire x1="7.62" y1="16.129" x2="7.58" y2="16.16" width="0.3048" layer="1"/>
-<wire x1="5.08" y1="6.35" x2="9" y2="6.35" width="0.3048" layer="16"/>
-<wire x1="3.81" y1="7.62" x2="5.08" y2="6.35" width="0.3048" layer="16"/>
 <wire x1="7.747" y1="16.383" x2="7.747" y2="27.178" width="0.3048" layer="16"/>
 <wire x1="7.62" y1="16.256" x2="7.747" y2="16.383" width="0.3048" layer="16"/>
@@
 <wire x1="8.89" y1="44.45" x2="9" y2="44.45" width="0.3048" layer="1"/>
 <wire x1="7.493" y1="49.403" x2="7.493" y2="54.229" width="0.3048" layer="16"/>
-<wire x1="3.81" y1="45.72" x2="5.715" y2="47.625" width="0.3048" layer="16"/>
-<wire x1="5.715" y1="47.625" x2="7.493" y2="49.403" width="0.3048" layer="16"/>
+<wire x1="3.81" y1="45.72" x2="7.493" y2="49.403" width="0.3048" layer="16"/>
 <wire x1="7.493" y1="54.229" x2="7.58" y2="54.26" width="0.3048" layer="16"/>
-<wire x1="5.715" y1="47.625" x2="8.89" y2="44.45" width="0.3048" layer="16"/>
+<wire x1="8.255" y1="43.815" x2="8.255" y2="37.084" width="0.3048" layer="16"/>
+<wire x1="8.89" y1="44.45" x2="8.255" y2="43.815" width="0.3048" layer="16"/>
 <wire x1="8.89" y1="44.45" x2="9" y2="44.45" width="0.3048" layer="16"/>
-<wire x1="8.255" y1="44.958" x2="8.255" y2="37.084" width="0.3048" layer="16"/>
-<wire x1="8.255" y1="44.958" x2="9" y2="44.45" width="0.3048" layer="16"/>
 <wire x1="5.08" y1="56.769" x2="5.08" y2="57.912" width="0.3048" layer="16"/>
 <wire x1="7.493" y1="54.356" x2="5.08" y2="56.769" width="0.3048" layer="1"/>
 <wire x1="5.08" y1="57.912" x2="3.175" y2="58.115" width="0.3048" layer="16"/>
 <wire x1="7.493" y1="54.356" x2="7.58" y2="54.26" width="0.3048" layer="1"/>
-<wire x1="11.32" y1="99.06" x2="10.16" y2="99.06" width="0.3048" layer="16"/>
-<wire x1="10.16" y1="99.06" x2="3.92" y2="99.06" width="0.3048" layer="16"/>
-<wire x1="11.32" y1="99.06" x2="10.033" y2="99.06" width="0.3048" layer="1"/>
-<wire x1="10.033" y1="99.06" x2="3.92" y2="99.06" width="0.3048" layer="1"/>
+<wire x1="11.32" y1="99.06" x2="9.906" y2="99.06" width="0.3048" layer="1"/>
+<wire x1="9.906" y1="99.06" x2="3.92" y2="99.06" width="0.3048" layer="1"/>
 <wire x1="12.7" y1="89.535" x2="15.24" y2="86.995" width="0.3048" layer="16"/>
 <wire x1="7.62" y1="89.535" x2="5.08" y2="86.995" width="0.3048" layer="16"/>
@@
 <wire x1="10.16" y1="92.075" x2="12.7" y2="92.075" width="0.3048" layer="1"/>
 <wire x1="10.16" y1="89.535" x2="12.7" y2="89.535" width="0.3048" layer="1"/>
-<wire x1="10.033" y1="92.202" x2="10.033" y2="99.06" width="0.3048" layer="1"/>
-<wire x1="10.033" y1="92.202" x2="10.16" y2="92.075" width="0.3048" layer="1"/>
-<wire x1="10.16" y1="92.075" x2="10.16" y2="99.06" width="0.3048" layer="16"/>
+<wire x1="9.906" y1="92.202" x2="9.906" y2="99.06" width="0.3048" layer="1"/>
+<wire x1="9.906" y1="92.202" x2="10.16" y2="92.075" width="0.3048" layer="1"/>
 <wire x1="4.699" y1="80.01" x2="4.064" y2="80.01" width="0.3048" layer="16"/>
 <wire x1="7.493" y1="77.216" x2="4.699" y2="80.01" width="0.3048" layer="16"/>
@@
 </signal>
 <signal name="N$6">
-<contactref element="U$2" pad="TIP@1"/>
-<contactref element="U$2" pad="TIP@2"/>
+<contactref element="U$2" pad="TIP@3"/>
 <contactref element="GAIN1" pad="P$2"/>
 <wire x1="10.16" y1="85.471" x2="10.16" y2="77.12" width="0.3048" layer="1"/>
@@
 </signal>
 <signal name="N$5">
-<contactref element="U$3" pad="TIP@1"/>
-<contactref element="U$3" pad="TIP@2"/>
+<contactref element="U$3" pad="TIP@3"/>
 <contactref element="R3" pad="1"/>
 <wire x1="3.81" y1="69.596" x2="1.905" y2="71.501" width="0.3048" layer="16"/>
@@
 </signal>
 <signal name="N$12">
-<contactref element="U$6" pad="TIP@1"/>
-<contactref element="U$6" pad="TIP@2"/>
+<contactref element="U$6" pad="TIP@3"/>
 <contactref element="R12" pad="1"/>
 <wire x1="1.905" y1="19.304" x2="1.905" y2="28.321" width="0.3048" layer="16"/>
