File: Eurorack Set 3/SimpleTrigger.sch (EAGLE design)
At the start: 16 parts

Commit message: 4io frontpanel, trigger thinner
Parts:
- U$9: value EURORACK_PCB4HP -> EURORACK_PCB2HP; device EurorackModularParts:EURORACK_PCB4HP -> EurorackModularParts:EURORACK_PCB2HP
Changed lines of the file:
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@@
 <setting verticaltext="up"/>
 </settings>
-<grid distance="0.05" unitdist="inch" unit="inch" style="lines" multiple="1" display="no" altdistance="0.01" altunitdist="inch" altunit="inch"/>
+<grid distance="0.1" unitdist="inch" unit="inch" style="lines" multiple="1" display="no" altdistance="0.01" altunitdist="inch" altunit="inch"/>
 <layers>
 <layer number="1" name="Top" color="4" fill="1" visible="yes" active="no"/>
@@
 <part name="GND5" library="SparkFun-Aesthetics" deviceset="GND" device=""/>
 <part name="GND6" library="SparkFun-Aesthetics" deviceset="GND" device=""/>
-<part name="U$9" library="EurorackModularParts" deviceset="EURORACK_PCB" device="4HP" value="EURORACK_PCB4HP"/>
+<part name="U$9" library="EurorackModularParts" deviceset="EURORACK_PCB" device="2HP" value="EURORACK_PCB2HP"/>
 <part name="U$10" library="zephod-components" deviceset="SWITCH_W_LED_PB6149L-X-102" device="WHITE"/>
 <part name="U$11" library="EurorackModularParts" deviceset="AUDIO-JACK" device="OUTPUT" value="PJ-341"/>
