File: Eurorack Set 4/Tuesday(MelodyR2).brd (EAGLE design)
At the start: 59.6 x 106.5 mm, 141 parts, among them IC1 LD1117AS33TR, IC3 TL074D, IC4 MCP6004, Q1 MMBT3904, Q2 MMBT3904, Q3 MMBT3904, Q4 MMBT3904, Q5 MMBT3904, Q6 MMBT3904, Q7 MMBT3904, Q8 MMBT3904, U1 MKL02Z32VFK4, U2 LM4040DIM3-5.0, U3 74HC595BQ, U4 74HC595BQ, U5 74HC595BQ, U6 24LC00T-I/OT

Commit message: eeprom pinout update
Parts:
- moved U$1 0.50 mm to (10.8, 19.2)
Routing:
- net GND: track 243.9 -> 276.6 mm, vias 30 -> 36
- net N$34: track 57.2 -> 64.4 mm, vias 6 -> 8
- net N$24: track 15.2 -> 10.3 mm, vias 2 -> 0
- net N$17: track 11.3 -> 8.18 mm, vias 2 -> 0
- net -12V: track 77.6 -> 74.5 mm
- net N$10: track 26.3 -> 27.8 mm
- net N$13: track 6.27 -> 7.60 mm
- net 12V: track 190.3 -> 191.3 mm, vias 10 -> 8
- net N$94: track 8.38 -> 7.72 mm, vias 2 -> 0
- net N$64: track 14.3 -> 14.9 mm
- net REF_-5V: vias 8 -> 6

Commit message: Tuesday r2 handrouted & panel details
Parts:
- removed LED_ALGO_FOURCHORD, LED_ALGO_PSYCH: WHITE 3MM WITH 11MM HOLDER, SparkFun-LED:LED3MM
- added D1, D2: MRA4004T3G, OPL:DO-214AC
- C18, C19: value 100nF 16V+ -> 100nF
- C6: value 1uF -> 100nF
- D3, D4: value MRA4004T3G -> WHITE 3MM WITH 11MM HOLDER; device OPL:DO-214AC -> SparkFun-LED:LED3MM
- D5: value WHITE_WITH_11MM_SPACER -> WHITE 3MM WITH 11MM HOLDER
- R1, R14, R16: value 100k 1% -> 100k
- R10, R13, R31, R32, R33, R34, R47, R48, R49: value 2k -> 1k
- R12, R2, R22, R23, R27, R30: value 33k 1% -> 33k
- R15, R3: value 49.9k 1% -> 51k
- R17: value INTENSITY -> 10kB
- R28: value 49.9k -> 51k
- R5, R8: value 25.5k 1% -> 30k
- R68: value SEED A -> 10kB
- R69: value SEED B -> 10kB
- R7, R9: value 10.2k 1% -> 12k
- R70: value TEMPO -> 10kB
- U6: value 24LC00T-I/OT -> 24LC16T-I/OT
- moved D4 66.1 mm to (17.8, 78.7), turned to 270 degrees
- moved D3 57.2 mm to (17.8, 83.8), turned to 270 degrees
- moved R3 18.7 mm to (42.5, 32.8), turned to 180 degrees
- moved R10 15.4 mm to (53.5, 17.0), turned to 180 degrees
- moved R29 11.5 mm to (15.3, 55.7)
- moved R42 7.00 mm to (52.0, 88.2), turned to 0 degrees
- moved R24 6.80 mm to (39.2, 16.8), turned to 180 degrees
- moved R27 4.00 mm to (15.0, 34.1), turned to 270 degrees
- moved R19 3.66 mm to (51.9, 31.8), turned to 180 degrees
- moved TP1 3.64 mm to (37.9, 45.0)
- moved R21 1.82 mm to (57.8, 37.0), turned to 270 degrees
- moved SWD1 1.75 mm to (18.5, 58.1)
- moved Q6 1.12 mm to (55.8, 89.5), turned to 0 degrees
- moved C10 0.25 mm to (32.0, 50.8)
- moved Q3 0.25 mm to (56.8, 31.8)
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- renumbered ACCENT to J7, BEAT to J10, B_ALGO to B1, B_BEATS to B4, B_SCALE to B3, B_TPB to B2, CLOCK to J4, CLOCKOUT_JACK to J6, GATE to J8, IN1 to J2, IN2 to J3, INTENSITY to J1, LED_ACCENT to D20, LED_ALGO_FLAT to D5, LED_ALGO_GOA to D6, LED_BEAT to D21, LED_BEAT_16 to D11, LED_BEAT_2 to D14, LED_BEAT_4 to D13, LED_BEAT_8 to D12, LED_GATE to D23, LED_LOOP to D22, LED_SCALE_DORIAN to D7, LED_SCALE_MAJOR to D8, LED_SCALE_MINOR to D9, LED_SCALE_PENTA to D10, LED_TICK to D19, LED_TPB_2 to D15, LED_TPB_3 to D16, LED_TPB_4 to D17, LED_TPB_6 to D18, LOOP to J11, NOTE to J12, POT_IN1 to R68, POT_IN2 to R69, POT_TEMPO to R70, RESET to J5, TICK to J9, U$1 to J14, U$10 to U7, U$19 to PRETTY1, U$2 to OUTLINE, U$4 to FID3, U$7 to FID2, U$8 to FID1, VELOCITY to J13
Connections:
- net N$22 renamed D21
- net -12V: now also D2.1; no longer D4.1
- net 12V: now also D1.2; no longer D3.2
- net 3.3V: now also U6.4; no longer U6.5
- net GND: now also D3.K, D4.K, U6.5; no longer LED_ALGO_FOURCHORD.K, LED_ALGO_PSYCH.K
- net N$13: now also D1.1; no longer D3.1
- net N$64: now also D2.2; no longer D4.2
- net N$75: now also D4.A; no longer LED_ALGO_PSYCH.A
- net N$76: now also D3.A; no longer LED_ALGO_FOURCHORD.A
Routing:
- net GND: track 276.6 -> 82.4 mm, vias 36 -> 37
- net 3.3V: track 308.4 -> 341.6 mm, vias 21 -> 23
- net -12V: track 74.5 -> 100.4 mm, vias 10 -> 6
- net OUT_ACCENT: track 63.3 -> 88.9 mm, vias 10 -> 2
- net OUT_GATE: track 100.8 -> 118.4 mm, vias 10 -> 0
- net 12V: track 191.3 -> 205.5 mm, vias 8 -> 20
- net N$23: track 14.2 -> 2.95 mm, vias 2 -> 0
- net BUTTON_TPB: track 37.7 -> 47.4 mm, vias 7 -> 1
- net N$65: track 7.14 -> 16.3 mm
- net CLOCK: track 67.6 -> 76.6 mm, vias 12 -> 10
- net LATCH: track 79.1 -> 70.7 mm, vias 14 -> 8
- net KNOB_TEMPO: track 59.3 -> 67.2 mm, vias 10 -> 2
- net N$34: track 64.4 -> 57.1 mm, vias 8 -> 6
- net CLOCK_IN: track 69.7 -> 76.5 mm, vias 4 -> 8
- net SHIFTERS: track 41.4 -> 47.9 mm, vias 4 -> 6
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