File: Eurorack Set 5/CodecDelay.brd (EAGLE design)
At the start: 39.3 x 106.5 mm, 48 parts, among them IC2 IC_74HC595-SOIC-16

Commit message: VCA updates
Parts:
- moved U$20 170.4 mm to (58.4, 91.4)
- moved U$21 161.5 mm to (33.0, 91.4)
- moved U$19 145.1 mm to (58.4, 67.3)
- moved U$11 116.7 mm to (33.0, 71.1)
- moved U$14 114.1 mm to (82.5, 58.4)
- moved U$9 97.3 mm to (57.1, 45.7)
- moved U$10 93.5 mm to (33.0, 52.1)
- moved U$5 4.58 mm to (63.5, 29.2)
Changed lines of the file:
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@@
 <attribute name="VALUE" value="PJ-341" x="10.16" y="76.2" size="1.778" layer="27" display="off"/>
 </element>
-<element name="U$5" library="EurorackModularParts" package="3.5MM-JACK-SWITCH-13MM-INPUT" value="IN 1" x="67.31" y="26.67">
-<attribute name="DESC" value="Input" x="67.31" y="26.67" size="1.778" layer="27" display="off"/>
-<attribute name="MPN" value="PJ-341" x="67.31" y="26.67" size="1.778" layer="27" display="off"/>
-<attribute name="VALUE" value="PJ-341" x="67.31" y="26.67" size="1.778" layer="27" display="off"/>
+<element name="U$5" library="EurorackModularParts" package="3.5MM-JACK-SWITCH-13MM-INPUT" value="IN 1" x="63.5" y="29.21">
+<attribute name="DESC" value="Input" x="63.5" y="29.21" size="1.778" layer="27" display="off"/>
+<attribute name="MPN" value="PJ-341" x="63.5" y="29.21" size="1.778" layer="27" display="off"/>
+<attribute name="VALUE" value="PJ-341" x="63.5" y="29.21" size="1.778" layer="27" display="off"/>
 </element>
 <element name="U$6" library="EurorackModularParts" package="3.5MM-JACK-SWITCH-13MM-INPUT" value="IN 2" x="95.25" y="35.56">
@@
 <element name="U$17" library="adafruit" package="FIDUCIAL_1MM" value="FIDUCIAL" x="2.54" y="3.81"/>
 <element name="U$18" library="adafruit" package="FIDUCIAL_1MM" value="FIDUCIAL" x="37.465" y="3.81"/>
-<element name="U$14" library="EurorackModularParts" package="OG-POTS_ALPS_POT_VERTICAL" value="DRIVE" x="-7.62" y="-11.43">
-<attribute name="DESC" value="Temperature" x="-7.62" y="-11.43" size="1.778" layer="27" display="off"/>
-</element>
-<element name="U$9" library="EurorackModularParts" package="OG-POTS_ALPS_POT_VERTICAL" value="DRIVE" x="-21.59" y="-11.43">
-<attribute name="DESC" value="Feedback" x="-21.59" y="-11.43" size="1.778" layer="27" display="off"/>
-</element>
-<element name="U$10" library="EurorackModularParts" package="OG-POTS_ALPS_POT_VERTICAL" value="DRIVE" x="-35.56" y="-11.43">
-<attribute name="DESC" value="Mix" x="-35.56" y="-11.43" size="1.778" layer="27" display="off"/>
-</element>
-<element name="U$11" library="EurorackModularParts" package="OG-POTS_ALPS_POT_VERTICAL" value="DRIVE" x="-49.53" y="-11.43">
-<attribute name="DESC" value="CV Amt" x="-49.53" y="-11.43" size="1.778" layer="27" display="off"/>
-</element>
-<element name="U$19" library="EurorackModularParts" package="OG-POTS_ALPS_POT_VERTICAL" value="DRIVE" x="-63.5" y="-11.43">
-<attribute name="DESC" value="Time" x="-63.5" y="-11.43" size="1.778" layer="27" display="off"/>
-</element>
-<element name="U$20" library="EurorackModularParts" package="OG-POTS_ALPS_POT_VERTICAL" value="DRIVE" x="-77.47" y="-11.43">
-<attribute name="DESC" value="Ducking" x="-77.47" y="-11.43" size="1.778" layer="27" display="off"/>
-</element>
-<element name="U$21" library="EurorackModularParts" package="OG-POTS_ALPS_POT_VERTICAL" value="DRIVE" x="-91.44" y="-11.43">
-<attribute name="DESC" value="Multitap Amt" x="-91.44" y="-11.43" size="1.778" layer="27" display="off"/>
+<element name="U$14" library="EurorackModularParts" package="OG-POTS_ALPS_POT_VERTICAL" value="DRIVE" x="82.55" y="58.42">
+<attribute name="DESC" value="Temperature" x="82.55" y="58.42" size="1.778" layer="27" display="off"/>
+</element>
+<element name="U$9" library="EurorackModularParts" package="OG-POTS_ALPS_POT_VERTICAL" value="DRIVE" x="57.15" y="45.72">
+<attribute name="DESC" value="Feedback" x="57.15" y="45.72" size="1.778" layer="27" display="off"/>
+</element>
+<element name="U$10" library="EurorackModularParts" package="OG-POTS_ALPS_POT_VERTICAL" value="DRIVE" x="33.02" y="52.07">
+<attribute name="DESC" value="Mix" x="33.02" y="52.07" size="1.778" layer="27" display="off"/>
+</element>
+<element name="U$11" library="EurorackModularParts" package="OG-POTS_ALPS_POT_VERTICAL" value="DRIVE" x="33.02" y="71.12">
+<attribute name="DESC" value="CV Amt" x="33.02" y="71.12" size="1.778" layer="27" display="off"/>
+</element>
+<element name="U$19" library="EurorackModularParts" package="OG-POTS_ALPS_POT_VERTICAL" value="DRIVE" x="58.42" y="67.31">
+<attribute name="DESC" value="Time" x="58.42" y="67.31" size="1.778" layer="27" display="off"/>
+</element>
+<element name="U$20" library="EurorackModularParts" package="OG-POTS_ALPS_POT_VERTICAL" value="DRIVE" x="58.42" y="91.44">
+<attribute name="DESC" value="Ducking" x="58.42" y="91.44" size="1.778" layer="27" display="off"/>
+</element>
+<element name="U$21" library="EurorackModularParts" package="OG-POTS_ALPS_POT_VERTICAL" value="DRIVE" x="33.02" y="91.44">
+<attribute name="DESC" value="Multitap Amt" x="33.02" y="91.44" size="1.778" layer="27" display="off"/>
 </element>
 </elements>
@@
 <contactref element="U$11" pad="P$1"/>
 <wire x1="102.98" y1="26.67" x2="91.55" y2="35.56" width="0" layer="19" extent="1-1"/>
-<wire x1="71.01" y1="26.67" x2="91.55" y2="35.56" width="0" layer="19" extent="1-1"/>
-<wire x1="63.61" y1="26.67" x2="71.01" y2="26.67" width="0" layer="19" extent="1-1"/>
-<wire x1="66.15" y1="12.7" x2="63.61" y2="26.67" width="0" layer="19" extent="1-1"/>
-<wire x1="37.465" y1="36.195" x2="63.61" y2="26.67" width="0" layer="19" extent="1-1"/>
+<wire x1="67.2" y1="29.21" x2="91.55" y2="35.56" width="0" layer="19" extent="1-1"/>
+<wire x1="59.8" y1="29.21" x2="67.2" y2="29.21" width="0" layer="19" extent="1-1"/>
+<wire x1="66.15" y1="12.7" x2="59.8" y2="29.21" width="0" layer="19" extent="1-1"/>
+<wire x1="37.465" y1="36.195" x2="59.8" y2="29.21" width="0" layer="19" extent="1-1"/>
 <wire x1="30.48" y1="38.1" x2="37.465" y2="36.195" width="0" layer="19" extent="1-1"/>
 <wire x1="21.59" y1="38.1" x2="30.48" y2="38.1" width="0" layer="19" extent="1-1"/>
@@
 <wire x1="13.86" y1="96.52" x2="13.86" y2="76.2" width="0" layer="19" extent="1-1"/>
 <wire x1="6.46" y1="96.52" x2="13.86" y2="96.52" width="0" layer="19" extent="1-1"/>
-<wire x1="-10.2" y1="-18.13" x2="4.445" y2="1.27" width="0" layer="19" extent="1-1"/>
-<wire x1="-24.17" y1="-18.13" x2="-10.2" y2="-18.13" width="0" layer="19" extent="1-1"/>
-<wire x1="-38.14" y1="-18.13" x2="-24.17" y2="-18.13" width="0" layer="19" extent="1-1"/>
-<wire x1="-52.11" y1="-18.13" x2="-38.14" y2="-18.13" width="0" layer="19" extent="1-1"/>
-<wire x1="-66.08" y1="-18.13" x2="-52.11" y2="-18.13" width="0" layer="19" extent="1-1"/>
-<wire x1="-80.05" y1="-18.13" x2="-66.08" y2="-18.13" width="0" layer="19" extent="1-1"/>
-<wire x1="-94.02" y1="-18.13" x2="-80.05" y2="-18.13" width="0" layer="19" extent="1-1"/>
+<wire x1="79.97" y1="51.72" x2="4.445" y2="1.27" width="0" layer="19" extent="1-1"/>
+<wire x1="54.57" y1="39.02" x2="79.97" y2="51.72" width="0" layer="19" extent="1-1"/>
+<wire x1="30.44" y1="45.37" x2="54.57" y2="39.02" width="0" layer="19" extent="1-1"/>
+<wire x1="30.44" y1="64.42" x2="30.44" y2="45.37" width="0" layer="19" extent="1-1"/>
+<wire x1="55.84" y1="60.61" x2="30.44" y2="64.42" width="0" layer="19" extent="1-1"/>
+<wire x1="55.84" y1="84.74" x2="55.84" y2="60.61" width="0" layer="19" extent="1-1"/>
+<wire x1="30.44" y1="84.74" x2="55.84" y2="84.74" width="0" layer="19" extent="1-1"/>
 </signal>
 <signal name="N$1">
 <contactref element="U$5" pad="TIP@3"/>
 <contactref element="U$1" pad="IN_L"/>
-<wire x1="67.31" y1="31.17" x2="67.31" y2="31.17" width="0" layer="19" extent="1-16"/>
-<wire x1="6.985" y1="1.27" x2="67.31" y2="31.17" width="0" layer="19" extent="1-1"/>
+<wire x1="63.5" y1="33.71" x2="63.5" y2="33.71" width="0" layer="19" extent="1-16"/>
+<wire x1="6.985" y1="1.27" x2="63.5" y2="33.71" width="0" layer="19" extent="1-1"/>
 </signal>
 <signal name="N$2">
@@
 <contactref element="U$21" pad="P$3"/>
 <contactref element="U$20" pad="P$3"/>
-<wire x1="-74.89" y1="-18.13" x2="-88.86" y2="-18.13" width="0" layer="19" extent="1-1"/>
-<wire x1="-60.92" y1="-18.13" x2="-74.89" y2="-18.13" width="0" layer="19" extent="1-1"/>
-<wire x1="-46.95" y1="-18.13" x2="-60.92" y2="-18.13" width="0" layer="19" extent="1-1"/>
-<wire x1="-32.98" y1="-18.13" x2="-46.95" y2="-18.13" width="0" layer="19" extent="1-1"/>
-<wire x1="-19.01" y1="-18.13" x2="-32.98" y2="-18.13" width="0" layer="19" extent="1-1"/>
-<wire x1="-5.04" y1="-18.13" x2="-19.01" y2="-18.13" width="0" layer="19" extent="1-1"/>
-<wire x1="17.72" y1="20.955" x2="-5.04" y2="-18.13" width="0" layer="19" extent="16-16"/>
+<wire x1="61" y1="84.74" x2="35.6" y2="84.74" width="0" layer="19" extent="1-1"/>
+<wire x1="61" y1="60.61" x2="61" y2="84.74" width="0" layer="19" extent="1-1"/>
+<wire x1="35.6" y1="64.42" x2="61" y2="60.61" width="0" layer="19" extent="1-1"/>
+<wire x1="35.6" y1="45.37" x2="35.6" y2="64.42" width="0" layer="19" extent="1-1"/>
+<wire x1="59.73" y1="39.02" x2="35.6" y2="45.37" width="0" layer="19" extent="1-1"/>
+<wire x1="85.13" y1="51.72" x2="59.73" y2="39.02" width="0" layer="19" extent="1-1"/>
+<wire x1="17.72" y1="20.955" x2="85.13" y2="51.72" width="0" layer="19" extent="16-16"/>
 <wire x1="17.72" y1="28.575" x2="17.72" y2="20.955" width="0" layer="19" extent="16-16"/>
 <wire x1="19.558" y1="30.48" x2="17.72" y2="28.575" width="0" layer="19" extent="16-16"/>
