File: Eurorack Set 5/LFO.brd (EAGLE design)
At the start: 39.3 x 106.5 mm, 117 parts, among them IC1 LD1117AS33TR, IC3 TL074D, IC4 MCP6004, J1 PJ-341, J12 PJ-341, J13 PJ-341, J14 POWER, J2 PJ-341, J3 PJ-341, J4 PJ-341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

Commit message: Many tweaks for frontpanel setup
Parts:
- added C14: 100nF, OPL:C0603
- moved C11 31.7 mm to (6.35, 3.17)
- moved C13 30.7 mm to (6.35, 1.27)
- moved IC1 27.3 mm to (8.89, 7.62), turned to 270 degrees
- moved C8 24.1 mm to (8.25, 12.3)
- moved C10 20.8 mm to (12.6, 47.2), turned to 180 degrees
- moved D2 20.6 mm to (14.9, 26.1), turned to 0 degrees
- moved R25 17.4 mm to (25.3, 12.4), turned to 0 degrees
- moved R24 17.0 mm to (37.6, 12.4), turned to 0 degrees
- moved D3 12.7 mm to (33.0, 26.7), turned to 90 degrees
- moved D40 12.7 mm to (20.3, 26.7), turned to 0 degrees
- moved Q3 12.7 mm to (25.8, 30.5), turned to 90 degrees
- moved R19 11.7 mm to (25.4, 34.3)
- moved Q1 9.00 mm to (6.35, 34.8), turned to 270 degrees
- moved R10 8.82 mm to (25.4, 26.0), turned to 0 degrees
- moved FID2 7.62 mm to (38.6, 1.82)
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Connections:
- net 3.3V: now also C14.2
- net GND: now also C14.1
Routing:
- net LATCH: track 0.00 -> 97.8 mm, vias 0 -> 9
- net CLOCK: track 0.00 -> 87.1 mm, vias 0 -> 13
- net 3.3V: track 156.2 -> 233.1 mm, vias 1 -> 8
- net N$94: track 0.00 -> 71.5 mm, vias 0 -> 8
- net RESET_PATTERN: track 4.13 -> 72.4 mm, vias 0 -> 8
- net SHIFTERS: track 0.00 -> 67.8 mm, vias 0 -> 6
- net 12V: track 43.5 -> 97.5 mm, vias 0 -> 8
- net N$14: track 2.89 -> 55.2 mm, vias 0 -> 2
- net -12V: track 92.4 -> 135.7 mm, vias 0 -> 4
- net N$10: track 4.47 -> 45.3 mm, vias 0 -> 2
- net KNOB_PHASE: track 0.00 -> 40.7 mm, vias 0 -> 6
- net N$4: track 6.30 -> 45.8 mm, vias 0 -> 8
- net ADC_FREQ: track 0.00 -> 37.2 mm, vias 0 -> 6
- net ADC_SHAPE: track 4.52 -> 38.7 mm, vias 0 -> 6
- net KNOB_FREQ: track 0.00 -> 27.8 mm, vias 0 -> 4
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
Commit message: Doublechecks & artwork prep
Changed lines of the file:
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@@
 <?xml version="1.0" encoding="utf-8"?>
 <!DOCTYPE eagle SYSTEM "eagle.dtd">
-<eagle version="6.5.0">
+<eagle version="7.7.0">
 <drawing>
 <settings>
@@
 <pass name="Default">
 <param name="RoutingGrid" value="4.92125984mil"/>
+<param name="AutoGrid" value="1"/>
+<param name="Efforts" value="0"/>
+<param name="TopRouterVariant" value="1"/>
 <param name="tpViaShape" value="round"/>
 <param name="PrefDir.1" value="*"/>
@@
 <contactref element="IC4" pad="4"/>
 <contactref element="C17" pad="1"/>
-<contactref element="C17" pad="1"/>
 <contactref element="R29" pad="1"/>
 <contactref element="R17" pad="P$3"/>
@@
 <wire x1="5.588" y1="3.175" x2="5.08" y2="2.667" width="0.381" layer="1"/>
 <wire x1="5.08" y1="2.667" x2="5.08" y2="1.27" width="0.381" layer="1"/>
-<wire x1="23.494003125" y1="8.621003125" x2="15.098003125" y2="8.621003125" width="0.381" layer="1"/>
-<wire x1="38.375003125" y1="23.375003125" x2="23.494003125" y2="8.621003125" width="0.381" layer="1"/>
+<wire x1="23.988003125" y1="8.621003125" x2="15.098003125" y2="8.621003125" width="0.381" layer="1"/>
 <wire x1="39.625003125" y1="24.625003125" x2="38.375003125" y2="23.375003125" width="0.381" layer="16"/>
 <wire x1="39.625003125" y1="33.375003125" x2="39.625003125" y2="24.625003125" width="0.381" layer="1"/>
@@
 <wire x1="13.208" y1="4.572" x2="6.488" y2="4.572" width="0.381" layer="1"/>
 <wire x1="6.488" y1="4.572" x2="5.74" y2="5.32" width="0.381" layer="1"/>
+<wire x1="23.988003125" y1="8.621003125" x2="30.353" y2="14.986" width="0.381" layer="1"/>
+<wire x1="30.353" y1="14.986" x2="30.353" y2="15.353" width="0.381" layer="1"/>
+<wire x1="30.353" y1="15.353" x2="38.375003125" y2="23.375003125" width="0.381" layer="1"/>
 </signal>
 <signal name="N$25">
