File: Eurorack Set 5/TuesdayR3.brd (EAGLE design)
At the start: 59.6 x 106.5 mm, 152 parts, among them IC1 LD1117AS33TR, IC3 TL074D, IC4 MCP6004, J1 PJ-341, J10 PJ-341, J11 PJ-341, J12 PJ-341, J13 PJ-341, J14 POWER, J2 PJ-341, J3 PJ-341, J4 PJ-341, J5 PJ-341, J6 PJ-341, J7 PJ-341, J8 PJ-341, J9 PJ-341, Q1 MMBT3904, Q2 MMBT3904, Q3 MMBT3904, Q4 MMBT3904, Q5 MMBT3904, Q6 MMBT3904, Q7 MMBT3904, Q8 MMBT3904, U1 MKL02Z32VFK4, U2 LM4040DIM3-5.0, U3 74HC595BQ, U4 74HC595BQ, U5 74HC595BQ, U6 24LC16T-I/OT, U7 MCP4822-E/SN

Commit message: Tuesday bom fix (LD1117 wrong version)
Parts:
- IC1: value LD1117AS33TR -> LD1117S33CTR
Changed lines of the file:
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@@
 <attribute name="MPN" value="TAJB106K020RNJ" x="3.19" y="41.5" size="1.778" layer="27" rot="R90" display="off"/>
 </element>
-<element name="IC1" library="ld-components" package="SOT223" value="LD1117AS33TR" x="11.43" y="41.275" rot="R270">
+<element name="IC1" library="ld-components" package="SOT223" value="LD1117S33CTR" x="11.43" y="41.275" rot="R270">
 <attribute name="OC_FARNELL" value="1467776" x="11.43" y="41.275" size="1.778" layer="27" rot="R270" display="off"/>
 <attribute name="MF" value="STMICROELECTRONICS" x="11.43" y="41.275" size="1.778" layer="27" rot="R270" display="off"/>

Commit message: Assembly data fixes, VCA revision (lm13700 pinout reversal!), Wobbler revision (better opamp scaling)
Parts:
- removed FID1, FID2, FID3: FIDUCIAL, adafruit:FIDUCIAL_1MM
Other:
- board text added: "J1"
- board text added: "J10"
- board text added: "J11"
- board text added: "J12"
- board text added: "J13"
- board text added: "J14"
- board text added: "J2"
- board text added: "J3"
- board text added: "J4"
- board text added: "J5"
- board text added: "J6"
- board text added: "J7"
- board text added: "J8"
- board text added: "J9"
- board text added: "R17"
- board text added: "R68"
- board text added: "R69"
- board text added: "R70"
- board text added: "U1"
