File: Eurorack Set 8 - Second Production Run/AddMixShift.brd (EAGLE design)
At the start: 19 x 106.5 mm, 49 parts

Commit message: Many production tweaks for wobbler/edgecutter.
Parts:
- D3, D4: value (none) -> 3mm YELLOW
- U$8: value (none) -> 100K LINEAR
- U$9: value (none) -> 100k AUDIO
- renumbered U$11 to IC2, U$12 to IC3, U$7 to IC1
Changed lines of the file:
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@@
 <setting verticaltext="up"/>
 </settings>
-<grid distance="25" unitdist="mil" unit="mil" style="dots" multiple="1" display="yes" altdistance="0.025" altunitdist="inch" altunit="inch"/>
+<grid distance="50" unitdist="mil" unit="mil" style="lines" multiple="1" display="yes" altdistance="0.025" altunitdist="inch" altunit="inch"/>
 <layers>
 <layer number="1" name="Top" color="4" fill="1" visible="yes" active="yes"/>
@@
 <attribute name="DESC" value="Input B" x="10.16" y="86.36" size="1.778" layer="27" display="off"/>
 </element>
-<element name="U$8" library="EurorackModularParts" package="OG-POTS_ALPS_POT_VERTICAL" value="" x="10.16" y="57.15" rot="R90">
+<element name="U$8" library="EurorackModularParts" package="OG-POTS_ALPS_POT_VERTICAL" value="100K LINEAR" x="10.16" y="57.15" rot="R90">
 <attribute name="DESC" value="Parameter" x="10.16" y="57.15" size="1.778" layer="27" rot="R90" display="off"/>
 </element>
-<element name="U$9" library="EurorackModularParts" package="OG-POTS_ALPS_POT_VERTICAL" value="" x="10.16" y="72.39" rot="R90">
+<element name="U$9" library="EurorackModularParts" package="OG-POTS_ALPS_POT_VERTICAL" value="100k AUDIO" x="10.16" y="72.39" rot="R90">
 <attribute name="DESC" value="Parameter" x="10.16" y="72.39" size="1.778" layer="27" rot="R90" display="off"/>
 </element>
@@
 <element name="R13" library="OPL" package="R0603" value="100" x="5.715" y="22.86" rot="R180"/>
 <element name="R14" library="OPL" package="R0603" value="100" x="12.065" y="22.86"/>
-<element name="U$7" library="EurorackModularParts" package="SO08" value="TL072" x="11.43" y="41.91" rot="R270"/>
-<element name="U$11" library="EurorackModularParts" package="SO08" value="TL072" x="10.16" y="31.115"/>
+<element name="IC1" library="EurorackModularParts" package="SO08" value="TL072" x="11.43" y="41.91" rot="R270"/>
+<element name="IC2" library="EurorackModularParts" package="SO08" value="TL072" x="10.16" y="31.115"/>
 <element name="C3" library="OPL" package="C0603" value="100nF" x="8.255" y="36.83" rot="R270"/>
 <element name="C4" library="OPL" package="C0603" value="100nF" x="12.065" y="25.4" rot="R270"/>
-<element name="U$12" library="EurorackModularParts" package="SO08" value="TL072" x="3.81" y="31.115"/>
+<element name="IC3" library="EurorackModularParts" package="SO08" value="TL072" x="3.81" y="31.115"/>
 <element name="R15" library="OPL" package="R0603" value="100K" x="5.715" y="36.83" rot="R90"/>
 <element name="R16" library="OPL" package="R0603" value="100K" x="4.445" y="36.83" rot="R90"/>
@@
 <element name="C5" library="OPL" package="C0603" value="100nF" x="1.905" y="36.83" rot="R270"/>
 <element name="C6" library="OPL" package="C0603" value="100nF" x="5.715" y="25.4" rot="R270"/>
-<element name="D3" library="EurorackModularParts" package="3MMLED" value="" x="6.35" y="48.26"/>
-<element name="D4" library="EurorackModularParts" package="3MMLED" value="" x="13.97" y="48.26" rot="R180"/>
+<element name="D3" library="EurorackModularParts" package="3MMLED" value="3mm YELLOW" x="6.35" y="48.26"/>
+<element name="D4" library="EurorackModularParts" package="3MMLED" value="3mm YELLOW" x="13.97" y="48.26" rot="R180"/>
 <element name="R18" library="OPL" package="R0603" value="1k" x="9.525" y="48.26" rot="R270"/>
 <element name="R19" library="OPL" package="R0603" value="100K" x="3.175" y="25.4" rot="R90"/>
@@
 <contactref element="U$3" pad="RING@3"/>
 <contactref element="U$5" pad="RING@3"/>
-<contactref element="U$7" pad="3"/>
-<contactref element="U$7" pad="5"/>
-<contactref element="U$11" pad="3"/>
-<contactref element="U$11" pad="5"/>
+<contactref element="IC1" pad="3"/>
+<contactref element="IC1" pad="5"/>
+<contactref element="IC2" pad="3"/>
+<contactref element="IC2" pad="5"/>
 <contactref element="C3" pad="1"/>
 <contactref element="C4" pad="2"/>
-<contactref element="U$12" pad="5"/>
+<contactref element="IC3" pad="5"/>
 <contactref element="U$17" pad="RING@3"/>
 <contactref element="C6" pad="2"/>
@@
 <contactref element="D3" pad="+"/>
 <contactref element="D4" pad="-"/>
-<contactref element="U$12" pad="3"/>
+<contactref element="IC3" pad="3"/>
 <wire x1="15.24" y1="43.815" x2="17.907" y2="43.815" width="0" layer="19" extent="1-16"/>
 <wire x1="14.03" y1="40.005" x2="15.24" y2="38.735" width="0" layer="19" extent="1-16"/>
@@
 <contactref element="C11" pad="+"/>
 <contactref element="U$8" pad="P$3"/>
-<contactref element="U$11" pad="8"/>
-<contactref element="U$7" pad="8"/>
+<contactref element="IC2" pad="8"/>
+<contactref element="IC1" pad="8"/>
 <contactref element="C3" pad="2"/>
-<contactref element="U$12" pad="8"/>
+<contactref element="IC3" pad="8"/>
 <contactref element="C5" pad="2"/>
 <wire x1="16.383" y1="43.815" x2="16.86" y2="59.73" width="0" layer="19" extent="1-1"/>
@@
 <contactref element="D2" pad="1"/>
 <contactref element="C12" pad="-"/>
-<contactref element="U$11" pad="4"/>
-<contactref element="U$7" pad="4"/>
+<contactref element="IC2" pad="4"/>
+<contactref element="IC1" pad="4"/>
 <contactref element="C4" pad="1"/>
-<contactref element="U$12" pad="4"/>
+<contactref element="IC3" pad="4"/>
 <contactref element="C6" pad="1"/>
 <wire x1="8.83" y1="40.005" x2="16.86" y2="54.57" width="0" layer="19" extent="1-1"/>
@@
 <contactref element="R10" pad="1"/>
 <contactref element="R12" pad="2"/>
-<contactref element="U$7" pad="7"/>
+<contactref element="IC1" pad="7"/>
 <wire x1="14.03" y1="42.545" x2="16.383" y2="42.545" width="0" layer="19" extent="1-1"/>
 <wire x1="9.652" y1="22.86" x2="14.03" y2="42.545" width="0" layer="19" extent="1-1"/>
@@
 <contactref element="R3" pad="2"/>
 <contactref element="R2" pad="2"/>
-<contactref element="U$7" pad="2"/>
+<contactref element="IC1" pad="2"/>
 <wire x1="2.54" y1="85.598" x2="17.78" y2="85.598" width="0" layer="19" extent="1-1"/>
 <wire x1="15.113" y1="65.405" x2="17.78" y2="85.598" width="0" layer="19" extent="1-1"/>
@@
 <contactref element="R6" pad="1"/>
 <contactref element="R7" pad="1"/>
-<contactref element="U$7" pad="1"/>
+<contactref element="IC1" pad="1"/>
 <contactref element="R20" pad="1"/>
 <wire x1="4.953" y1="43.815" x2="8.83" y2="43.815" width="0" layer="19" extent="1-1"/>
@@
 <contactref element="R11" pad="2"/>
 <contactref element="R12" pad="1"/>
-<contactref element="U$7" pad="6"/>
+<contactref element="IC1" pad="6"/>
 <wire x1="14.03" y1="41.275" x2="17.907" y2="42.545" width="0" layer="19" extent="1-1"/>
 <wire x1="6.477" y1="41.275" x2="14.03" y2="41.275" width="0" layer="19" extent="1-1"/>
@@
 <contactref element="R6" pad="2"/>
 <contactref element="R8" pad="1"/>
-<contactref element="U$11" pad="2"/>
+<contactref element="IC2" pad="2"/>
 <wire x1="8.255" y1="26.162" x2="9.525" y2="28.515" width="0" layer="19" extent="1-1"/>
 <wire x1="9.525" y1="24.638" x2="8.255" y2="26.162" width="0" layer="19" extent="1-1"/>
@@
 <contactref element="R7" pad="2"/>
 <contactref element="R9" pad="1"/>
-<contactref element="U$11" pad="6"/>
+<contactref element="IC2" pad="6"/>
 <wire x1="9.525" y1="37.592" x2="2.54" y2="42.418" width="0" layer="19" extent="1-1"/>
 <wire x1="10.795" y1="33.715" x2="9.525" y2="37.592" width="0" layer="19" extent="1-1"/>
@@
 <contactref element="R8" pad="2"/>
 <contactref element="R13" pad="1"/>
-<contactref element="U$11" pad="1"/>
+<contactref element="IC2" pad="1"/>
 <wire x1="9.525" y1="26.162" x2="8.255" y2="28.515" width="0" layer="19" extent="1-1"/>
 <wire x1="6.477" y1="22.86" x2="9.525" y2="26.162" width="0" layer="19" extent="1-1"/>
@@
 <contactref element="R9" pad="2"/>
 <contactref element="R14" pad="1"/>
-<contactref element="U$11" pad="7"/>
+<contactref element="IC2" pad="7"/>
 <contactref element="R15" pad="2"/>
 <wire x1="9.525" y1="33.715" x2="9.525" y2="36.068" width="0" layer="19" extent="1-1"/>
@@
 </signal>
 <signal name="N$17">
-<contactref element="U$12" pad="6"/>
+<contactref element="IC3" pad="6"/>
 <contactref element="R15" pad="1"/>
 <contactref element="R16" pad="2"/>
@@
 <signal name="N$18">
 <contactref element="R16" pad="1"/>
-<contactref element="U$12" pad="7"/>
+<contactref element="IC3" pad="7"/>
 <contactref element="R17" pad="1"/>
 <wire x1="3.175" y1="36.068" x2="4.445" y2="36.068" width="0" layer="19" extent="1-1"/>
@@
 </signal>
 <signal name="N$24">
-<contactref element="U$12" pad="1"/>
+<contactref element="IC3" pad="1"/>
 <contactref element="R18" pad="2"/>
 <contactref element="R19" pad="1"/>
@@
 </signal>
 <signal name="N$25">
-<contactref element="U$12" pad="2"/>
+<contactref element="IC3" pad="2"/>
 <contactref element="R20" pad="2"/>
 <contactref element="R19" pad="2"/>

Commit message: Moved TuesdayR4 to new folder, updated library components to match latest insights.
Parts:
- removed U$14, U$16: 100K, adafruit:TC33X
- added C10, C13, C14, C7, C8, C9: 22pf, OPL:C0603
- R1, R11, R12, R15, R16, R6, R7, R8, R9: value 100K -> 100K 0.1%
- R4, R5: value 90K -> 100k 0.1%
- U$8: value 100K LINEAR -> 10K LINEAR
- moved R20 23.8 mm to (18.0, 42.9), turned to 270 degrees
- moved R19 22.1 mm to (16.6, 42.9), turned to 270 degrees
- moved C4 17.0 mm to (1.65, 38.9), turned to 90 degrees
- moved R8 14.9 mm to (4.95, 39.6), turned to 0 degrees
- moved R17 13.9 mm to (9.14, 24.3), turned to 270 degrees
- moved C6 13.6 mm to (7.75, 38.9), turned to 90 degrees
- moved C5 13.5 mm to (11.6, 27.4), turned to 90 degrees
- moved R6 13.2 mm to (4.95, 38.2), turned to 180 degrees
- moved U$10 13.0 mm to (14.6, 28.4), turned to 270 degrees
- moved R9 10.8 mm to (4.19, 27.4), turned to 90 degrees
- moved R16 10.5 mm to (9.02, 27.4), turned to 270 degrees
- moved C3 9.80 mm to (5.46, 27.4), turned to 90 degrees
- moved U$3 9.65 mm to (15.0, 16.5)
- moved U$5 9.65 mm to (5.33, 16.5)
- moved R15 9.62 mm to (7.75, 27.4), turned to 270 degrees
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Connections:
- removed net N$10: R4.1, U$16.1, U$16.2
- removed net N$3: R5.1, U$14.1, U$14.2
- net N$11: now also C9.2
- net N$12: now also R4.1; no longer U$16.3
- net N$13: now also C10.2
- net N$14: now also C7.1
- net N$17: now also C13.1
- net N$18: now also C13.2
- net N$2: now also C8.2, IC3.1; no longer IC1.7
- net N$20: now also R5.1; no longer U$14.3
- net N$24: now also C14.2, IC1.7; no longer IC3.1
- net N$25: now also C14.1, IC1.6; no longer IC3.2
- net N$5: now also C9.1
- net N$7: now also C7.2
- net N$8: now also C8.1, IC3.2; no longer IC1.6
- net N$9: now also C10.1

Commit message: Many small routing fixes & tracewidth improvements. Also split the tuesday over multiple pages.
Parts:
- moved C14 83.6 mm to (16.0, 47.9), turned to 90 degrees
- moved C7 71.1 mm to (6.73, 49.3), turned to 90 degrees
- moved C8 64.5 mm to (10.2, 39.4)
- moved C9 64.2 mm to (4.95, 37.7)
- moved C13 59.2 mm to (9.78, 26.7)
- moved C10 57.1 mm to (3.56, 28.3)
- moved R6 7.67 mm to (3.30, 45.7), turned to 270 degrees
- moved R10 5.97 mm to (1.91, 24.1)
- moved R18 5.73 mm to (9.91, 42.5), turned to 90 degrees
- moved R21 5.73 mm to (17.5, 42.5), turned to 90 degrees
- moved D3 5.71 mm to (6.35, 42.5)
- moved D4 5.71 mm to (14.0, 42.5)
- moved R19 4.99 mm to (17.3, 47.9)
- moved C1 4.35 mm to (17.0, 49.9)
- moved C2 4.33 mm to (5.59, 46.0)
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Routing:
- net -12V: track 0.00 -> 65.6 mm, vias 0 -> 6
- net N$14: track 0.00 -> 65.6 mm
- net 12V: track 0.00 -> 55.9 mm, vias 0 -> 5
- net N$7: track 0.00 -> 27.9 mm, vias 0 -> 2
- net N$2: track 0.00 -> 23.8 mm
- net N$9: track 0.00 -> 22.6 mm, vias 0 -> 2
- net N$19: track 0.00 -> 21.5 mm
- net N$8: track 0.00 -> 20.4 mm
- net N$24: track 0.00 -> 19.1 mm
- net GND: track 0.00 -> 18.2 mm, vias 0 -> 14
- net N$22: track 0.00 -> 16.1 mm
- net N$11: track 0.00 -> 16.1 mm, vias 0 -> 4
- net N$64: track 0.00 -> 10.2 mm, vias 0 -> 1
- net N$20: track 0.00 -> 9.87 mm
- net N$12: track 0.00 -> 9.87 mm
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
Commit message: FinalEffect & AddMixShift & EspDrum
Parts:
- added U$11: TINRS_ARTWORKROCKET, EurorackModularParts:TINRS_ROCKET
Changed lines of the file:
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@@
 <setting verticaltext="up"/>
 </settings>
-<grid distance="5" unitdist="mil" unit="mil" style="lines" multiple="1" display="yes" altdistance="0.025" altunitdist="inch" altunit="inch"/>
+<grid distance="5" unitdist="mil" unit="mm" style="lines" multiple="1" display="yes" altdistance="0.025" altunitdist="inch" altunit="inch"/>
 <layers>
 <layer number="1" name="Top" color="4" fill="1" visible="yes" active="yes"/>
@@
 <layer number="19" name="Unrouted" color="6" fill="1" visible="yes" active="yes"/>
 <layer number="20" name="Dimension" color="15" fill="1" visible="yes" active="yes"/>
-<layer number="21" name="tPlace" color="7" fill="1" visible="no" active="yes"/>
-<layer number="22" name="bPlace" color="7" fill="1" visible="no" active="yes"/>
-<layer number="23" name="tOrigins" color="15" fill="1" visible="no" active="yes"/>
-<layer number="24" name="bOrigins" color="15" fill="1" visible="no" active="yes"/>
+<layer number="21" name="tPlace" color="7" fill="1" visible="yes" active="yes"/>
+<layer number="22" name="bPlace" color="7" fill="1" visible="yes" active="yes"/>
+<layer number="23" name="tOrigins" color="15" fill="1" visible="yes" active="yes"/>
+<layer number="24" name="bOrigins" color="15" fill="1" visible="yes" active="yes"/>
 <layer number="25" name="tNames" color="57" fill="1" visible="no" active="yes"/>
 <layer number="26" name="bNames" color="7" fill="1" visible="no" active="yes"/>
@@
 <element name="C13" library="OPL" package="C0603" value="22pf" x="9.779" y="26.67"/>
 <element name="C14" library="OPL" package="C0603" value="22pf" x="16.002" y="47.879" rot="R90"/>
+<element name="U$11" library="EurorackModularParts" package="TINRS_ROCKET" value="TINRS_ARTWORKROCKET" x="10.287" y="72.644" rot="MR90"/>
 </elements>
 <signals>
