File: Eurorack Set 8 - Second Production Run/Edgecutter.sch (EAGLE design)
At the start: 147 parts, among them IC1 LD1117AS33TR, IC10 24LC16T-I/OT, IC2 TL072, IC3 MCP4822-E/SN, IC4 MCP6004, IC5 74HC595BQ, IC6 74HC595BQ, IC7 74HC595BQ, IC8 74HC595BQ, IC9 MKL02Z32VFK4, J1 PJ-341, J12 PJ-341, J13 PJ-341, J14 POWERSMT, J2 PJ-341, J3 PJ-341, J4 PJ-341, J5 PJ-341, J6 PJ-341, J7 PJ-341, J8 PJ-341, Q1 MMBT3904, Q2 MMBT3904, Q3 MMBT3904, Q5 MMBT3904, U1 LM4040DIM3-5.0

Commit message: Wobbler and Edgecutter progress
Parts:
- removed D10, D11, D12, D13, D14, D6, D7, D8, D9: yellow, EurorackModularParts:LED3MM
- removed IC10: 24LC16T-I/OT, EurorackModularParts:24LC00T-I/OT
- removed IC5, IC6, IC7, IC8: 74HC595BQ, FarnellThings:74HC595BQ
- removed IC9: MKL02Z32VFK4, FarnellThings:MKL02Z32VFK4
- removed Q5: MMBT3904, transistor:MMBT3904LT1-NPN-SOT23-BEC
- removed U$1: SWITCH_W_LED_PB6149L-X-102YELLOW, zephod-components:SWITCH_W_LED_PB6149L-X-102YELLOW
- added B1, B3: BUTTON-4P-3110040P1, zephod-components:BUTTON-4P-3110040P1
- added C23: 3.3nF, OPL:C-0603
- added D36, D37, D38, D39, D41, D43, D44: yellow, EurorackModularParts:LED3MM
- added FID1, FID2, FID3: FIDUCIAL, adafruit:FIDUCIAL
- added J10, J11: PJ-341, EurorackModularParts:AUDIO-JACKOUTPUT
- added J15, J9: PJ-341, EurorackModularParts:AUDIO-JACKINPUT
- added Q4, Q7, Q8: MMBT3904, transistor:MMBT3904LT1-NPN-SOT23-BEC
- added R4, R52, R53, R6, R76: 100k, OPL:R-0603
- added R74, R78: 56, OPL:R-0603
- added R75: 33k, OPL:R-0603
- added R77: 51k, OPL:R-0603
- added U$2: SWITCH_W_LED_PB6149L-X-102YELLOW, zephod-components:SWITCH_W_LED_PB6149L-X-102YELLOW
- added U2: LM4040DIM3-5.0, FarnellThings:LM4040DIM3-5.0
- added U3, U4, U5: 74HC595BQ, FarnellThings:74HC595BQ
- added U6: 24LC16T-I/OT, EurorackModularParts:24LC00T-I/OT
- added U7: MCP4822-E/SN, FarnellThings:MCP4822-E/SN
- C12, C13, C5: device EurorackModularParts:C-POLAR-A -> OPL:C-POLAR-A
- C20: value 100nF -> 3.3nF; MF MULTICOMP -> (none); MPN MC0603F104Z160CT -> (none); OC_FARNELL 1759017 -> unknown
- IC2: value TL072 -> MCP6004; device EurorackModularParts:TL072 -> EurorackModularParts:MCP6004; MF (none) -> MICROCHIP; MPN (none) -> MCP6004-I/SL.; OC_FARNELL (none) -> 1605572
- IC3: value MCP4822-E/SN -> TL074D; device FarnellThings:MCP4822-E/SN -> EurorackModularParts:TL074D; MF MICROCHIP -> TEXAS INSTRUMENTS; MPN (none) -> TL074CD; OC_FARNELL (none) -> 1103010
- J1, R17: DESC Frequency -> Decay
- J12: DESC Normal Out -> Linear
- J13: DESC Phased Out -> Curved
- J2, R68: DESC Shape -> Sustain
- J3, R69: DESC Mod -> Release
- J4: DESC Phase -> Curvature
- J5: DESC Reset -> Gate
- J6: device EurorackModularParts:AUDIO-JACKOUTPUT -> EurorackModularParts:AUDIO-JACKINPUT; DESC Loop -> Retrigger
- J7: DESC Mid -> ReleaseStartTrigger
- J8: device EurorackModularParts:AUDIO-JACKINPUT -> EurorackModularParts:AUDIO-JACKOUTPUT; DESC Sync -> ReleaseDoneTrigger
- R13: value 33k -> 100k
- R36: value 187k 0.1% -> 56
- R37: value 187k 0.1% -> 10k
- R38, R46, R65: value 56 -> 100k
- R39: value 10k -> 33k
- R40: value 100k -> 51k
- R41: value 51k -> 33k
- R42: value 10kB -> 10k; device EurorackModularParts:POTZEPHPOT -> OPL:R-0603; DESC Phase -> (none)
- R43: value 33k -> 10k
- R44: value 10kB -> 100k; device EurorackModularParts:POTZEPHPOT -> OPL:R-0603; DESC Normal Amp -> (none)
- R45: value 10kB -> 10k; device EurorackModularParts:POTZEPHPOT -> OPL:R-0603; DESC Phase Amp -> (none)
- R5, R8: value 187k 0.1% -> 30k
- R66: value 56 -> 33k
- R67: value 0 -> 56
- R7, R9: value 38.3k 0.1% -> 12k
- R70: value 56 -> 10kB; device OPL:R-0603 -> EurorackModularParts:POTZEPHPOT; DESC (none) -> Curvature
- R71: value 56 -> 51k
- R72: value 100k -> 33k
- R73: value 10k -> 10kB; device OPL:R-0603 -> EurorackModularParts:POTZEPHPOT; DESC (none) -> Attack
- U1: value LM4040DIM3-5.0 -> MKL02Z32VFK4; device FarnellThings:LM4040DIM3-5.0 -> FarnellThings:MKL02Z32VFK4; MF TEXAS INSTRUMENTS -> NXP; OC_FARNELL 9778330 -> (none)
Connections:
- net KNOB_FREQ renamed KNOB_DECAY
- net KNOB_MOD renamed KNOB_RELEASE
- net KNOB_SHAPE renamed KNOB_SUSTAIN
- removed net ADC_FREQ: C16.2, IC4N.OUT, IC9.PTA9/I2C1_SDA, R22.1
- removed net ADC_MOD: C1.2, IC4K.OUT, IC9.PTB13, R2.1
- removed net ADC_NORMAL: IC9.PTB10, R44.S
- removed net ADC_PHASE: C9.2, IC4L.OUT, IC9.PTB11, R13.1
- removed net ADC_PHASED: IC9.PTB2/IRQ_7/UART0_TX/UART0_RX, R45.S
- removed net ADC_SHAPE: C15.2, IC4M.OUT, IC9.PTA8/I2C1_SCL, R12.1
- removed net CLOCK_2: IC8.SHCP, IC9.PTA4/XTAL0/I2C0_SDA/I2C1_SCL
- removed net KNOB_PHASE: R42.S, R43.2
- removed net N$60: Q5.B, R40.2
- removed net N$62: IC8.Q2, R70.2
- removed net N$63: J12.RING, J13.RING, R67.2
- removed net N$65: D12.+, R66.1
- removed net N$66: IC8.Q3, R31.2
- removed net N$67: IC8.Q4, R34.2
- removed net NORMALOUT: C3.2, IC2VR1.OUT, R24.2, R8.1
- removed net OUT_LFOCYCLEMID: IC6.Q5, R10.2, R21.1
- removed net OUT_LFOCYCLESTART: IC6.Q4, R35.2, R40.1
- removed net PHASEDOUT: C2.2, IC2VR2.OUT, R25.2, R5.1
- removed net RESET_PATTERN: IC9.PTA12/IRQ_13/LPTMR0_ALT2, Q1.C, R20.1, U$1.1, U$1.2
- removed net SHIFTERS2TO3: IC6.Q7S, IC7.DS
- removed net SHIFTERS_2: IC8.DS, IC9.PTA3/EXTAL0/I2C0_SCL/I2C1_SDA
- removed net SYNC_LFO: IC9.PTB1/IRQ_6/UART0_RX/UART0_TX, Q2.C, R73.1
- removed net TRIGGERBUTTONLED: IC6.Q6, R38.2
- new net ADC_ATTACK: C9.2, IC4L.OUT, R66.1, U1.PTB13
- new net ADC_CURVE: C20.2, IC2K.OUT, R39.1, U1.PTB11
- new net ADC_DECAY: C16.2, IC4N.OUT, R22.1, U1.PTB2/IRQ_7/UART0_TX/UART0_RX
- new net ADC_RELEASE: C1.2, IC4K.OUT, R2.1, U1.PTA9/I2C1_SDA
- new net ADC_SUSTAIN: C15.2, IC4M.OUT, R12.1, U1.PTA8/I2C1_SCL
- new net ADC_VELOCITY: C23.2, IC2M.OUT, R75.1, U1.PTA12/IRQ_13/LPTMR0_ALT2
- new net BUTTON_LOOP: B3.A0, B3.A1, U1.PTA4/XTAL0/I2C0_SDA/I2C1_SCL
- new net BUTTON_TIMERANGE: B1.A0, B1.A1, U1.PTB10
- new net BUTTON_TRIGGER: U$2.1, U$2.2, U1.PTA3/EXTAL0/I2C0_SCL/I2C1_SDA
- new net D21: D43.-, R47.1
- new net EXTGATE: J14.GATE, J5.SWITCH
- new net KNOB_ATTACK: R72.2, R73.S
- new net KNOB_CURVE: R41.2, R70.S
- new net N$17: IC3C.-IN, R52.1, R53.2
- new net N$18: C3.2, IC3A.OUT, R4.1, R8.1
- new net N$2: IC3B.-IN, R4.2, R6.1
- new net N$24: C2.2, IC3D.OUT, R5.1, R53.1
- new net N$69: J10.TIP, Q7.C, R43.1
- new net N$71: Q8.B, R46.2
- new net N$72: J11.TIP, Q8.C, R45.1
- new net N$83: D36.+, R55.1
- new net N$84: D37.+, R54.1
- new net N$85: D38.+, R35.1
- new net N$86: D39.+, R36.1
- new net OUT_ATTACK: R44.1, R47.2, U3.Q0
- new net OUT_CUR_PRERES: IC2L.+IN, IC3C.OUT, R25.2, R52.2
- new net OUT_DECAY: R46.1, R48.2, U3.Q7
- new net OUT_LIN_PRERES: IC3B.OUT, R24.2, R6.2
- new net OUT_RELEASEDONE: R38.1, R49.2, U3.Q5
- new net OUT_RELEASESTART: R10.2, R21.1, U3.Q6
- new net RETRIGGER_ENVELOPE: Q2.C, R42.1, U1.PTA6/SPI0_MISO
- new net SHIFTER2TO3: U4.Q7S, U5.DS
- new net TRIGGER_ENVELOPE: Q1.C, R20.1, U1.PTB1/IRQ_6/UART0_RX/UART0_TX
- new net TRIGGER_LED: R78.2, U5.Q0
- net -12V: now also IC3P.V-; no longer IC2VR3.V-
- net 12V: now also IC3P.V+, J9.SWITCH, R37.2, R43.2, R45.2; no longer IC2VR3.V+, R39.2
- net 3.3V: now also C22.1, D41.+, D43.+, D44.+, IC2O.V+, R42.2, R70.A, R73.A, U1.VDD_VREFH, U3.!MR, U3.VCC, U4.!MR, U4.VCC, U5.!MR, U5.VCC, U6.VCC, U7.VDD; no longer C20.2, C22.2, D3.+, IC10.VCC, IC3.VDD, IC5.!MR, IC5.VCC, IC6.!MR, IC6.VCC, IC7.!MR, IC7.VCC, IC8.!MR, IC8.VCC, IC9.VDD_VREFH, R42.A, R44.A, R45.A, R73.2
- net CLOCK: now also U1.PTB6/IRQ_2/LPTMR0_ALT3, U3.SHCP, U4.SHCP, U5.SHCP; no longer IC5.SHCP, IC6.SHCP, IC7.SHCP, IC9.PTB6/IRQ_2/LPTMR0_ALT3
- net CPU_RESET: now also U1.PTA1/IRQ_1/LPTMR0_ALT1/RESET_B; no longer IC9.PTA1/IRQ_1/LPTMR0_ALT1/RESET_B
- net DACCS: now also U1.PTA5/SPI0_SS_B, U7./CS; no longer IC3./CS, IC9.PTA5/SPI0_SS_B
- net DACSCK: now also U1.PTB0/IRQ_5/SPI0_SCK, U7.SCK; no longer IC3.SCK, IC9.PTB0/IRQ_5/SPI0_SCK
- net DACSDI: now also U1.PTA7/IRQ_4/SPI0_MOSI/SPI0_MISO, U7.SDI; no longer IC3.SDI, IC9.PTA7/IRQ_4/SPI0_MOSI/SPI0_MISO
- net GND: now also B1.B0, B1.B1, B3.B0, B3.B1, C22.2, D3.-, D36.-, D37.-, D38.-, D39.-, IC2K.+IN, IC2M.+IN, IC2N.+IN, IC2O.V-, IC3A.+IN, IC3B.+IN, IC3C.+IN, IC3D.+IN, J10.RING, J11.RING, J12.RING, J13.RING, J15.RING, J15.SWITCH, J6.SWITCH, J9.RING, Q4.E, Q7.E, Q8.E, R70.E, R73.E, U$2.3, U$2.4, U$2.NEG, U1.E_PAD, U1.VREFL_VSS, U2.CATHODE, U3.!OE, U3.GND, U3.GND_2, U4.!OE, U4.GND, U4.GND_2, U5.!OE, U5.GND, U5.GND_2, U6.VSS, U6.WP, U7./LDAC, U7.VSS; no longer C20.1, C22.1, D10.-, D11.-, D12.-, D13.-, D14.-, D6.-, D7.-, D8.-, D9.-, IC10.VSS, IC10.WP, IC2VR1.+IN, IC2VR2.+IN, IC3./LDAC, IC3.VSS, IC5.!OE, IC5.GND, IC5.GND_2, IC6.!OE, IC6.GND, IC6.GND_2, IC7.!OE, IC7.GND, IC7.GND_2, IC8.!OE, IC8.GND, IC8.GND_2, IC9.E_PAD, IC9.VREFL_VSS, J5.SWITCH, J8.SWITCH, Q5.E, R42.E, R44.E, R45.E, R67.1, U$1.3, U$1.4, U$1.NEG, U1.CATHODE
- net LATCH: now also U1.PTB5/IRQ_12/NMI_B, U3.STCP, U4.STCP, U5.STCP; no longer IC5.STCP, IC6.STCP, IC7.STCP, IC8.STCP, IC9.PTB5/IRQ_12/NMI_B
- net N$1: now also R78.1, U$2.POS; no longer IC5.Q0, R33.2
- net N$10: now also IC3A.-IN; no longer IC2VR1.-IN, R36.1
- net N$11: now also J15.TIP, R65.2; no longer J4.TIP, R11.2
- net N$12: now also J4.TIP; no longer C9.1, IC4L.-IN, R11.1, R41.1, R43.1
- net N$14: now also R34.2, U4.Q7; no longer D7.+, R47.1
- net N$19: now also IC2L.-IN, IC2L.OUT, R74.2; no longer IC5.Q1, R64.2
- net N$22: now also C9.1, IC4L.-IN, R65.1, R66.2, R71.1, R72.1; no longer IC5.Q2, R63.2
- net N$26: now also IC2N.-IN, IC2N.OUT; no longer IC5.Q3, R61.2
- net N$27: now also R64.2, U4.Q0; no longer D3.-, R35.1
- net N$30: now also D4.+, R67.1; no longer IC5.Q4, R62.2
- net N$31: now also R60.2, U3.Q1; no longer IC5.Q5, R57.2
- net N$35: now also R33.2, U3.Q2; no longer IC5.Q6, R56.2
- net N$36: now also R55.2, U3.Q3; no longer IC5.Q7, R58.2
- net N$37: now also R35.2, U3.Q4; no longer IC6.Q3, R59.2
- net N$38: now also R56.2, U4.Q1; no longer IC7.Q7, R54.2
- net N$39: now also R54.2, U4.Q2; no longer IC7.Q6, R55.2
- net N$40: now also R67.2, U4.Q3; no longer IC7.Q5, R47.2
- net N$41: now also R32.2, U4.Q4; no longer R38.1, U$1.POS
- net N$42: now also R31.2, U4.Q5; no longer D13.+, R70.1
- net N$43: now also Q2.B, R11.2; no longer IC7.Q4, R46.2
- net N$44: now also D41.-, R49.1; no longer Q2.B, R72.2
- net N$45: now also D44.-, R48.1; no longer J8.TIP, R72.1
- net N$46: now also C20.1, IC2K.-IN, R13.1, R39.2, R40.1, R41.1; no longer D6.+, R46.1
- net N$47: now also J6.TIP, R11.1; no longer D5.+, R48.1
- net N$48: now also R36.2, U4.Q6; no longer D4.+, R49.1
- net N$49: now also R59.2, U5.Q1; no longer D8.+, R55.1
- net N$5: now also U7.VOUTA; no longer IC3.VOUTA
- net N$50: now also R58.2, U5.Q2; no longer D9.+, R54.1
- net N$51: now also D3.+; no longer D10.+
- net N$52: now also R57.2, U5.Q3; no longer D11.+, R65.1
- net N$53: now also R63.2, U5.Q4; no longer IC7.Q3, R48.2
- net N$54: now also R62.2, U5.Q5; no longer IC7.Q2, R49.2
- net N$55: now also R61.2, U5.Q6; no longer IC7.Q1, R32.2
- net N$56: now also C23.1, IC2M.-IN, R75.2, R76.1, R77.1; no longer IC7.Q0, R65.2
- net N$57: now also Q4.B, R38.2; no longer IC6.Q7, R60.2
- net N$58: now also J8.TIP, Q4.C, R37.1; no longer D14.+, R71.1
- net N$59: now also D5.+, R74.1; no longer IC8.Q1, R71.2
- net N$61: now also J9.TIP, R76.2; no longer J6.TIP, Q5.C, R39.1
- net N$68: now also Q7.B, R44.2; no longer IC8.Q5, R66.2
- net N$7: now also U7.VOUTB; no longer IC3.VOUTB
- net N$9: now also IC3D.-IN; no longer IC2VR2.-IN, R37.1
- net REF_-5V: now also R40.2, R71.2, R77.2, U2.ANODE; no longer R36.2, R37.2, R41.2, U1.ANODE
- net SCL: now also U1.PTB3/IRQ_10/I2C0_SCL/UART0_TX, U6.SCL; no longer IC10.SCL, IC9.PTB3/IRQ_10/I2C0_SCL/UART0_TX
- net SDA: now also U1.PTB4/IRQ_11/I2C0_SDA/UART0_RX, U6.SDA; no longer IC10.SDA, IC9.PTB4/IRQ_11/I2C0_SDA/UART0_RX
- net SHIFTER1TO2: now also U3.Q7S, U4.DS; no longer IC5.Q7S, IC6.DS
- net SHIFTERS: now also U1.PTB7/IRQ_3, U3.DS; no longer IC5.DS, IC9.PTB7/IRQ_3
- net SWD_CLK: now also U1.PTA0/IRQ_0/SWD_CLK; no longer IC9.PTA0/IRQ_0/SWD_CLK
- net SWD_DIO: now also U1.PTA2/SWD_DIO; no longer IC9.PTA2/SWD_DIO

Commit message: Many production tweaks for wobbler/edgecutter.
Parts:
- renumbered U1 to IC5, U3 to IC7, U4 to IC8, U5 to IC9, U6 to IC6, U7 to IC10

Commit message: Minor tweaks pre china
Parts:
- C12, C13, C5: device OPL:C-POLAR-A -> EurorackModularParts:C-POLAR-A
Changed lines of the file:
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@@
 <setting verticaltext="up"/>
 </settings>
-<grid distance="0.05" unitdist="inch" unit="inch" style="lines" multiple="1" display="no" altdistance="0.01" altunitdist="inch" altunit="inch"/>
+<grid distance="0.1" unitdist="inch" unit="inch" style="lines" multiple="1" display="no" altdistance="0.01" altunitdist="inch" altunit="inch"/>
 <layers>
 <layer number="1" name="Top" color="4" fill="1" visible="no" active="no"/>
@@
 <attribute name="OC_FARNELL" value="1759017"/>
 </part>
-<part name="C12" library="OPL" deviceset="C-POLAR*" device="-A" value="10uF">
+<part name="C12" library="EurorackModularParts" deviceset="C-POLAR*" device="-A" value="10uF">
 <attribute name="MF" value="AVX"/>
 <attribute name="MPN" value="TAJB106K020RNJ"/>
 <attribute name="OC_FARNELL" value="197427"/>
 </part>
-<part name="C13" library="OPL" deviceset="C-POLAR*" device="-A" value="10uF">
+<part name="C13" library="EurorackModularParts" deviceset="C-POLAR*" device="-A" value="10uF">
 <attribute name="MF" value="AVX"/>
 <attribute name="MPN" value="TAJB106K020RNJ"/>
@@
 <part name="GND2" library="SparkFun" deviceset="GND" device=""/>
 <part name="SUPPLY7" library="SparkFun-Aesthetics" deviceset="3.3V" device=""/>
-<part name="C5" library="OPL" deviceset="C-POLAR*" device="-A" value="10uF">
+<part name="C5" library="EurorackModularParts" deviceset="C-POLAR*" device="-A" value="10uF">
 <attribute name="MF" value="AVX"/>
 <attribute name="MPN" value="TAJB106K020RNJ"/>
