File: EuroForError/BigBus_Error.brd (EAGLE design)
At the start: 350 x 30 mm, 47 parts

Commit message: Perplexed, PowerBus, Wobbler/Edgecutter/Tuesday updates, FinalEffect
Parts:
- C1, C2, C3: value (none) -> 10uF
- C10, C13, C15, C18, C20, C27: value 10u -> 10uF; device EurorackModularParts:AVX-A -> EurorackModularParts:CASE-A_3216
- moved R1 37.6 mm to (28.6, 8.89), turned to 270 degrees
- moved D1 37.0 mm to (29.2, 6.10), turned to 0 degrees
- moved R2 27.6 mm to (28.6, 12.7)
- moved D2 27.2 mm to (29.2, 16.3), turned to 0 degrees
- moved R3 24.9 mm to (28.6, 21.6), turned to 270 degrees
- moved D3 23.1 mm to (29.2, 18.8), turned to 0 degrees
Routing:
- net +12: track 378.2 -> 380.6 mm, vias 2 -> 3
- net N$2: track 1.50 -> 2.85 mm
- net N$3: track 1.50 -> 2.57 mm
- net N$1: track 1.50 -> 2.08 mm
- net +5: track 378.8 -> 379.4 mm, vias 2 -> 3
- net -12: track 389.2 -> 389.5 mm, vias 2 -> 3
