File: Development/Eurorack Set 9/RectangularThing-SOICs.sch (EAGLE design)
At the start: 176 parts, among them IC1 CEM3310SOIC16, IC2 TL074D, IC3 CEM3320QFN24, IC4 CEM3310SOIC16, IC5 TL074D, IC7 CEM3340SOIC16, U1 LM4040DIM3-5.0

Commit message: RectangularThing Soics
Parts:
- added C37, C39, C42, C43, C48, C49: 100nF, OPL:C-0603
- added C40: 33p, OPL:C-0603
- added C41, C45: 0.01uF, OPL:C-0603
- added C44: 1000pF, OPL:C-0603
- added C46, C47: 0.001uF, OPL:C-0603
- added IC10, IC9: TL074D, EurorackModularParts:TL074D
- added IC6: 4013D, 40xx:4013D
- added IC8: CEM3340SOIC16, CEM:CEM3340SOIC16
- added R100: 820, OPL:R-0603
- added R101, R112, R113, R114, R116, R117, R118, R119, R120, R122, R123, R124, R125: 10k, OPL:R-0603
- added R102, R104, R105, R108, R75, R76: 100k, OPL:R-0603
- added R103, R74, R95: 1M, OPL:R-0603
- added R106: 140k, OPL:R-0603
- added R107: 560k, OPL:R-0603
- added R109: 1M 0.1%, OPL:R-0603
- added R110: 100k 0.1%, OPL:R-0603
- added R111, R72: (no value), OPL:R-0603
- added R115, R121, R126, R127, R128, R129, R130, R131: 20k, OPL:R-0603
- added R73, R97: 470, OPL:R-0603
- added R77: 360k, OPL:R-0603
- added R93: 1.8k, OPL:R-0603
- added R96: 1.5M, OPL:R-0603
- added R98: 24k, OPL:R-0603
- added R99: 5.6k, OPL:R-0603
- added TP1: TEST-POINT3X5, SparkFun-Passives:TEST-POINT3X5
- added U$44, U$45: (no value), EurorackModularParts:POTZEPHPOT_BIGKNOB
- added U$46, U$52, U$53, U$54, U$55: (no value), EurorackModularParts:POTZEPHPOT
- added U$47, U$48: (no value), adafruit:TRIMPOTTC33X
- added U$49: 100k, EurorackModularParts:POTZEPHPOT
- added U$50: PJ-341, EurorackModularParts:AUDIO-JACKINPUT
- added U$51: ONOFFON, EurorackModularParts:ONOFFON
- C18: value 0.001uF -> 33p
- R69: value 100k -> 100k 0.1%
- R70: value 1M -> 1M 0.1%
- U$3: DESC (none) -> Fine
- U$4: DESC (none) -> Coarse
Connections:
- net PULSE_OUT renamed PULSE_OUT_1
- net TRIANGLE_OUT renamed TRIANGLE_OUT_1
- removed net SAWTOOTH_OUT: IC7.8, R41.1
- removed net SOFTSYNC_IN: C18.1
- new net HARDSYNC_2_IN: C47.2, U$51.ON2
- new net N$100: IC8.7, U$48.E
- new net N$101: R105.2, U$49.S
- new net N$102: R106.1, U$49.A
- new net N$103: R107.1, R108.1, U$50.TIP
- new net N$104: R102.1, U$45.S
- new net N$105: R103.1, U$44.S
- new net N$106: C18.1, IC6B.CLK, R111.2
- new net N$107: IC6B.!Q, IC6B.D
- new net N$108: IC2D.-IN, R118.2, R119.2, R120.2, R124.2, R125.2, R47.2, R48.2, R49.2, R50.1, R71.2
- new net N$109: IC9A.OUT, R117.2, U$46.A
- new net N$110: IC9B.OUT, R116.2, U$52.A
- new net N$111: IC9B.-IN, R113.2, R116.1, R122.2
- new net N$112: IC9A.-IN, R112.2, R117.1, R123.2
- new net N$113: IC9C.-IN, R114.2, R115.1, R121.2
- new net N$114: IC9C.OUT, R115.2, U$53.A
- new net N$115: R120.1, U$53.S
- new net N$116: R119.1, U$52.S
- new net N$117: R118.1, U$46.S
- new net N$118: R125.1, U$55.S
- new net N$119: IC9D.OUT, R128.2, U$54.A
- new net N$120: IC9D.-IN, R126.2, R127.2, R128.1
- new net N$122: IC10D.OUT, R131.2, U$55.A
- new net N$123: IC10D.-IN, R129.2, R130.2, R131.1
- new net N$70: IC6A.!Q, IC6A.D
- new net N$71: C41.2, R73.2
- new net N$74: C40.1, IC6A.CLK, R72.2
- new net N$77: C45.2, R97.2
- new net N$87: IC8.13, R95.2, R96.2, R97.1
- new net N$88: C43.1, R95.1
- new net N$89: C44.1, IC8.11
- new net N$90: C46.2, IC8.9
- new net N$92: IC8.14, R93.2
- new net N$94: C47.1, IC8.6
- new net N$95: IC8.1, R98.1
- new net N$96: R98.2, U$47.E
- new net N$97: IC8.3, R100.1, R99.2, U$47.A, U$47.S
- new net N$98: IC8.2, R99.1
- new net N$99: R74.2, U$48.S
- new net PITCH_IN_2: IC8.15, R102.2, R103.2, R104.2, R109.2, R110.2, R73.1, R74.1, R75.2, R76.2, R77.2
- new net PULSE_OUT_2: IC8.4, R101.1, R113.1
- new net PWM_2_IN: IC8.5, R105.1, R107.2
- new net SAWTOOTH_OUT_1: IC7.8, R41.1, R72.1, U$51.CENTER
- new net SAWTOOTH_OUT_2: IC8.8, R111.1, R112.1
- new net SOFTSYNC_2_IN: C46.1, U$51.ON1
- new net SUBOSC_1_OUT: IC6A.Q, R127.1
- new net SUBOSC_2_OUT: IC6B.Q, R130.1
- new net TRIANGLE_OUT_2: IC8.10, R114.1
- net -12V: now also C39.1, C49.1, IC10P.V-, IC9P.V-, R100.2
- net -5V: now also R121.1, R122.1, R123.1, R126.1, R129.1, U$44.E, U$45.E
- net 10V: now also R106.2
- net 12V: now also C37.1, C42.1, C48.1, IC10P.V+, IC6P.VDD, IC8.16, IC9P.V+, R77.1, R96.1
- net 5V: now also U$44.A, U$45.A
- net EXP_FM_IN: now also R104.1
- net GND: now also C18.2, C37.2, C39.2, C40.2, C41.1, C42.2, C44.2, C45.1, C48.2, C49.2, IC10D.+IN, IC6A.R, IC6A.S, IC6B.R, IC6B.S, IC6P.VSS, IC8.12, IC9A.+IN, IC9B.+IN, IC9C.+IN, IC9D.+IN, R101.2, R108.2, R93.1, U$46.E, U$48.A, U$49.E, U$52.E, U$53.E, U$54.E, U$55.E
- net LINEAR_FM_IN: now also C43.2
- net MAIN_CV: now also R76.1
- net N$37: now also TP1.1; no longer C18.2
- net N$40: now also R124.1, U$54.S; no longer IC2D.-IN, R47.2, R48.2, R49.2, R50.1, R71.2
- net N$79: now also R110.1
- net N$80: now also R109.1
- net PITCH_ENV: now also R75.1
Other:
- note added: "Oscillator 1"
- note added: "Oscillator 2"
- note removed: "Oscillator"

Commit message: filter added..
Parts:
- removed R71: 10k, OPL:R-0603
- removed U$32: (no value), EurorackModularParts:POTZEPHPOT
- removed U$33: PJ-341, EurorackModularParts:AUDIO-JACKINPUT
- added C50, C51, C52, C53: 300pF, OPL:C-0603
- added C54: 1uF, adafruit:CPOL-US153CLV-0505
- added R132, R135: 1.8k, OPL:R-0603
- added R133, R136, R137, R138, R139, R140, R144, R145, R146, R147: 100k, OPL:R-0603
- added R134: BIAS, OPL:R-0603
- added R141, R142: 22k, OPL:R-0603
- added R143: 51k, OPL:R-0603
- added U$56: CEM3320_UNFOLDEDQFN, CEM:CEM3320_UNFOLDEDQFN
- added U$57: (no value), EurorackModularParts:POTZEPHPOT_BIGKNOB
- added U$58, U$59: (no value), EurorackModularParts:POTZEPHPOT
Connections:
- removed net N$75: R71.1, U$32.S
- removed net N$76: U$32.A, U$33.TIP
- new net CUTOFF_ENVELOPE_2: IC10B.OUT, R140.1, R142.2
- new net CUTOFF_KNOB_2: R139.1, U$57.S
- new net HPFILTER: C50.1, C9.-, R27.1
- new net HP_RESONANCE_IN: R133.2, U$58.S
- new net N$121: R132.1, U$56.NEGRAIL
- new net N$124: R133.1, U$56.RESONANCE_CV
- new net N$125: R134.1, R135.1, R136.2, R137.2, R138.2, R139.2, R140.2, U$56.FREQCV
- new net N$126: IC10B.-IN, R141.2, R142.1
- new net N$127: IC10B.+IN, U$59.S
- new net N$128: C50.2, U$56.STAGE1_CAP
- new net N$129: R147.1, U$56.STAGE1_IN
- new net N$130: C51.2, R147.2, U$56.STAGE1_OUT
- new net N$131: C51.1, U$56.STAGE2_CAP
- new net N$132: R146.1, U$56.STAGE2_IN
- new net N$133: C52.2, R146.2, U$56.STAGE2_OUT
- new net N$134: C52.1, U$56.STAGE3_CAP
- new net N$135: R145.1, U$56.STAGE3_IN
- new net N$136: C53.2, R145.2, U$56.STAGE3_OUT
- new net N$137: C53.1, U$56.STAGE4_CAP
- new net N$138: R144.1, U$56.STAGE4_IN
- new net N$139: C54.+, R144.2, U$56.STAGE4_OUT
- new net N$141: R143.2, U$56.FEEDBACK_IN
- net -12V: now also R132.2
- net -5V: now also R134.2, U$57.A
- net 12V: now also U$56.POSRAIL
- net 5V: now also U$57.E, U$58.A
- net CUTOFF_IN: now also R138.1
- net CUTOFF_KEYTRACK: now also R137.1
- net CUTOFF_KNOB: now also R136.1
- net FILTER_OUT: now also C54.-, R143.1; no longer C9.-, R27.1
- net GND: now also R135.2, U$56.GROUND, U$58.E, U$59.A; no longer U$32.E, U$33.RING, U$33.SWITCH
- net MODENVOUT: now also R141.1, U$59.E
- net N$108: no longer R71.2

Commit message: RectangularThing progress - new suboscs, separated opamps
Parts:
- removed IC5: TL074D, EurorackModularParts:TL074D
- added C55, C56, C57, C58, C59, C60: 100nF, OPL:C-0603
- added IC11: 4053D, 40xx:4053D
- added JP1: (no value), SparkFun-Connectors:M03X2NO_SILK
- added JP2: (no value), SparkFun-Connectors:M031X03_NO_SILK
- added JP3: JUMPER-31-2, SparkFun-Passives:JUMPER-31-2
- added R148, R71: 22k, OPL:R-0603
- added R149, R150, R151, R152, R153, R154: 100k, OPL:R-0603
- added TP2, TP3, TP5, TP6, TP7, TP8, TP9: TEST-POINT3X5, SparkFun-Passives:TEST-POINT3X5
- added U$32: 10k, EurorackModularParts:POTZEPHPOT
- added U$33, U$60, U$61, U$62, U$63: 100k, EurorackModularParts:TRIMPOT
- added U$64: TRIMPOT, EurorackModularParts:TRIMPOT
- added U$65, U$66: TL072, EurorackModularParts:TL072
- R118, R119, R120, R124, R125, R47, R48, R49, R50: value 10k -> 100k
- R127, R130: value 20k -> 10k
- R51: value 10k -> 100
- U$19: value (none) -> PJ-341; device adafruit:TRIMPOTTC33X -> EurorackModularParts:AUDIO-JACKINPUT
- U$20: value (none) -> 100k; device adafruit:TRIMPOTTC33X -> EurorackModularParts:TRIMPOT; DESC (none) -> Osc1: Scale
- U$21, U$22, U$23, U$46, U$52, U$53, U$54, U$55: value (none) -> 10kA
- U$44, U$45, U$59, U$6: value (none) -> 10k
- U$47: value (none) -> TL072; device adafruit:TRIMPOTTC33X -> EurorackModularParts:TL072
- U$48: value (none) -> TRIMPOT; device adafruit:TRIMPOTTC33X -> EurorackModularParts:TRIMPOT; DESC (none) -> Osc2: Scale
- U$5: value (none) -> 10k; DESC (none) -> Cutoff
- U$57: value (none) -> 10k; DESC (none) -> HP Cutoff
- U$58: value (none) -> 10k; DESC Resonance -> HP Resonance
Connections:
- net N$108 renamed MIXER_SUMLINE
- net N$125 renamed HP_FILTER_CUTOFF_IN
- removed net HPFILTER: C50.1, C9.-, R27.1
- new net CUTOFF1_MODENVINPUT: R65.1, U$30.E, U$62.P$2
- new net CUTOFF2_MODENVINPUT: R141.1, U$59.E, U$61.P$2
- new net FILTER_IN: R22.2, U$15.II2, U$19.TIP
- new net LP_TO_HP: C50.1, C9.-, R27.1, TP2.1
- new net N$75: IC10C.-IN, R148.2, R71.1
- new net N$76: IC10C.+IN, U$32.S
- new net PITCHENVMOD2: R148.1, U$32.A, U$33.P$2
- new net PITCHENVMODINP1: R68.1, U$31.A, U$60.P$2
- new net PITCH_ENV_2: IC10C.OUT, R71.2, R75.1
- new net RAMBLER2_SAW_IN: IC11A.Y0, IC11A.Z0, R153.1, R154.2
- new net RAMBLER_2_OPT: IC11A.Y1, JP3.2
- new net RAMBLER_IN_1B: IC11A.X1, R149.1, R150.2
- new net RAMBLER_OUT_1: IC11A.X, JP2.1, TP9.1
- new net RAMBLER_OUT_2: IC11A.Y, JP1.3, TP8.1
- new net SAWPULSE: IC11A.Z, JP1.5, TP7.1
- new net SAWPULSE_IN: IC11A.Z1, R151.2, R152.1
- new net SELECTEDSUB1: JP2.2, R127.1
- new net SELECTEDSUB2: JP1.2, JP1.4, JP1.6, R130.1
- net -12V: now also C58.1, C60.1, U$47VR3.V-, U$65VR3.V-, U$66VR3.V-; no longer IC5P.V-
- net -5V: now also C56.2, IC11P.VEE
- net 12V: now also C31.2, C57.2, C59.2, U$47VR3.V+, U$65VR3.V+, U$66VR3.V+; no longer C31.1, C42.1, IC5P.V+, IC6P.VDD
- net 5V: now also C42.1, C55.1, IC11P.VCC, IC6P.VDD
- net CUTOFF_ENVELOPE: now also U$47VR1.OUT; no longer IC5B.OUT
- net CUTOFF_ENVELOPE_2: now also U$47VR2.OUT; no longer IC10B.OUT
- net CUTOFF_KEYTRACK: now also U$66VR1.OUT; no longer IC5A.OUT
- net FILTER_OUT: now also TP3.1
- net GND: now also C31.1, C55.2, C56.1, C57.1, C58.2, C59.1, C60.2, IC11A.INH, IC11P.GND, JP3.1, R150.1, R151.1, R154.1, U$19.RING, U$32.E, U$33.P$1, U$60.P$1, U$61.P$1, U$62.P$1, U$63.P$3, U$64.P$3; no longer C31.2, U$20.A, U$48.A
- net MODENVOUT: now also U$33.P$3, U$60.P$3, U$61.P$3, U$62.P$3; no longer R141.1, R65.1, R68.1, U$30.E, U$31.A, U$59.E
- net N$100: now also U$64.P$1; no longer U$48.E
- net N$126: now also U$47VR2.-IN; no longer IC10B.-IN
- net N$127: now also U$47VR2.+IN; no longer IC10B.+IN
- net N$41: now also U$65VR1.OUT; no longer IC5D.OUT
- net N$44: now also U$20.P$3; no longer U$19.E
- net N$45: now also U$20.P$1, U$20.P$2; no longer U$19.A, U$19.S
- net N$46: now also U$63.P$2; no longer U$20.S
- net N$48: now also U$63.P$1; no longer U$20.E
- net N$66: now also U$65VR1.-IN; no longer IC5D.-IN
- net N$67: now also U$66VR1.-IN; no longer IC5A.-IN
- net N$68: now also U$66VR1.+IN; no longer IC5A.+IN
- net N$69: now also U$47VR1.-IN; no longer IC5B.-IN
- net N$72: now also U$66VR2.-IN; no longer IC5C.-IN
- net N$73: now also U$47VR1.+IN; no longer IC5B.+IN
- net N$78: now also U$66VR2.+IN; no longer IC5C.+IN
- net N$81: now also U$65VR1.+IN; no longer IC5D.+IN
- net N$96: now also U$48.P$3; no longer U$47.E
- net N$97: now also U$48.P$1, U$48.P$2; no longer U$47.A, U$47.S
- net N$99: now also U$64.P$2; no longer U$48.S
- net OSCSUM: now also U$19.SWITCH; no longer R22.2, U$15.II2
- net PITCH_ENV: now also U$66VR2.OUT; no longer IC5C.OUT, R75.1
- net PULSE_OUT_2: now also R152.2
- net SAWTOOTH_OUT_1: now also JP3.3, R149.2
- net SAWTOOTH_OUT_2: now also R153.2
- net SUBOSC_1_OUT: now also IC11A.A, JP2.3, TP6.1; no longer R127.1
- net SUBOSC_2_OUT: now also IC11A.B, IC11A.C, JP1.1, TP5.1; no longer R130.1
- net TRIANGLE_OUT_1: now also IC11A.X0
Other:
- moved on the sheet: C31, C32, IC10C, U$5, U$57, U$58, U$6

Commit message: Rectangular updates & library prefix namings
Parts:
- removed TP9: TEST-POINT3X5, SparkFun-Passives:TEST-POINT3X5
- removed U$21, U$22, U$23, U$46, U$52, U$53, U$54, U$55: 10kA, EurorackModularParts:POTZEPHPOT
- removed U$3, U$4: (no value), EurorackModularParts:POTZEPHPOT_BIGKNOB
- removed U$30, U$31, U$34: (no value), EurorackModularParts:POTZEPHPOT
- removed U$32, U$6: 10k, EurorackModularParts:POTZEPHPOT
- removed U$37, U$49: 100k, EurorackModularParts:POTZEPHPOT
- removed U$44, U$45, U$5: 10k, EurorackModularParts:POTZEPHPOT_BIGKNOB
- removed U$47, U$65: TL072, EurorackModularParts:TL072
- removed U$56: CEM3320_UNFOLDEDQFN, CEM:CEM3320_UNFOLDEDQFN
- added C61: 100nF, OPL:C-0603
- added H1, H2, H3, H4: MOUNT-HOLE, zephod-components:MOUNT-HOLE
- added IC16, IC17: CEM3310SOIC16, CEM:CEM3310SOIC16
- added IC5: TL074D, EurorackModularParts:TL074D
- added R155, R156, R157: 22k, OPL:R-0603
- added R159: 47k, OPL:R-0603
- added R162, R166, R168, R170, R171, R174, R175, R176: 470, OPL:R-0603
- added R163, R164, R167, R172, R177, R179: 10k, OPL:R-0603
- added R169, R173: 24k, OPL:R-0603
- added TP4: TEST-POINT3X5, SparkFun-Passives:TEST-POINT3X5
- C1, C2: value 0.02uF -> 100nF
- C10: value 300pF -> 1000pF
- C11, C13: value 300pF -> 10uF; device OPL:C-0603 -> EurorackModularParts:C-POLAR-A
- C12, C50, C51, C52: value 300pF -> 100nF
- C14, C41, C45: value 0.01uF -> 100nF
- C15, C23: value 100nF -> 0.001uF
- C16: value 1000pF -> 0.001uF
- C17: value 0.01uF -> 1000pF
- C18: value 33p -> 0.01uF
- C19, C47: value 0.001uF -> 100nF
- C20: value 10uF -> 100nF; device EurorackModularParts:C-POLAR-A -> OPL:C-0603
- C21: value 10uF -> 0.01uF; device EurorackModularParts:C-POLAR-A -> OPL:C-0603
- C26, C27: value 0.02uF -> 300pF
- C28: value 0.039uF -> 100nF
- C29, C33: value 100nF -> 1uF; device OPL:C-0603 -> adafruit:CPOL-US153CLV-0505
- C3: value 0.039uF -> 0.01uF
- C30, C31, C34, C35, C36, C37: value 100nF -> 300pF
- C38: MF AVX -> (none); MPN 06035C104KAT2A -> (none); OC_FARNELL 1301804 -> (none)
- C4: value 5nF -> 33p
- C40: value 33p -> 100nF
- C44: value 1000pF -> 100nF
- C46: value 0.001uF -> 5nF
- C49: MF (none) -> AVX; MPN (none) -> 06035C104KAT2A; OC_FARNELL (none) -> 1301804
- C53: value 300pF -> 0.039uF
- C54: value 1uF -> 0.039uF; device adafruit:CPOL-US153CLV-0505 -> OPL:C-0603
- C55, C56, C59, C60: value 100nF -> 0.02uF
- C6: value 100nF -> 0.01uF
- C8: value 100nF -> 33p
- C9: value 1uF -> 100nF; device adafruit:CPOL-US153CLV-0505 -> OPL:C-0603
- IC1: value CEM3310SOIC16 -> TL072; device CEM:CEM3310SOIC16 -> EurorackModularParts:TL072
- IC11: value 4053D -> TL072; device 40xx:4053D -> EurorackModularParts:TL072
- IC2: value TL074D -> 4013D; device EurorackModularParts:TL074D -> 40xx:4013D
- IC3: value CEM3320QFN24 -> CEM3340SOIC16; device CEM:CEM3320QFN24 -> CEM:CEM3340SOIC16
- IC4: value CEM3310SOIC16 -> CEM3340SOIC16; device CEM:CEM3310SOIC16 -> CEM:CEM3340SOIC16
- IC6: value 4013D -> 4053D; device 40xx:4013D -> 40xx:4053D
- IC7: value CEM3340SOIC16 -> TL072; device CEM:CEM3340SOIC16 -> EurorackModularParts:TL072
- IC8: value CEM3340SOIC16 -> CEM3320_UNFOLDEDQFN; device CEM:CEM3340SOIC16 -> CEM:CEM3320_UNFOLDEDQFN
- IC9: value TL074D -> CEM3320QFN24; device EurorackModularParts:TL074D -> CEM:CEM3320QFN24
- JP1: device SparkFun-Connectors:M03X2NO_SILK -> SparkFun-Connectors:M031X03_NO_SILK
- JP2: device SparkFun-Connectors:M031X03_NO_SILK -> SparkFun-Connectors:M03X2NO_SILK
- R1: value 10k -> (none); device OPL:R-0603 -> EurorackModularParts:POTZEPHPOT; DESC (none) -> FM
- R10: value 47k -> 100k
- R100: value 820 -> 10k
- R102, R133, R31, R81: value 100k -> 10k
- R103: value 1M -> 140k
- R106: value 140k -> 100k
- R107: value 560k -> 51k
- R109: value 1M 0.1% -> 100k
- R11: value 470 -> 10kA; device OPL:R-0603 -> EurorackModularParts:POTZEPHPOT; DESC (none) -> Saw 2
- R110: value 100k 0.1% -> 100k
- R111: value (none) -> 1.8k
- R112: value 10k -> BIAS
- R113, R122: value 10k -> 1.8k
- R114, R116, R117, R123, R41, R56, R57: value 10k -> 100k
- R115, R44: value 20k -> 100k
- R121: value 20k -> 1.8k
- R124, R91: value 100k -> 91k
- R126: value 20k -> 220k
- R127: value 10k -> 91k
- R128, R131, R83: value 20k -> 10k
- R13: value 1M -> 100
- R130, R86: value 10k -> 20k
- R132: value 1.8k -> 10k
- R134: value BIAS -> 10k; device OPL:R-0603 -> EurorackModularParts:POTZEPHPOT; DESC (none) -> Mod->Pitch 2
- R135: value 1.8k -> 22k
- R136: value 100k -> (none); device OPL:R-0603 -> EurorackModularParts:POTZEPHPOT; DESC (none) -> Mod->Cutoff
- R137: value 100k -> 10k; device OPL:R-0603 -> EurorackModularParts:POTZEPHPOT; DESC (none) -> Resonance
- R138: value 100k -> BIAS
- R139: value 100k -> 220k
- R14, R64, R65, R66, R67: value 22k -> 100k
- R141: value 22k -> 10k; device OPL:R-0603 -> EurorackModularParts:POTZEPHPOT_BIGKNOB; DESC (none) -> Cutoff
- R142: value 22k -> (none); device OPL:R-0603 -> EurorackModularParts:POTZEPHPOT; DESC (none) -> Mod->Pitch
- R143: value 51k -> 22k
- R144, R150, R152, R92: value 100k -> 22k
- R148: value 22k -> 10k; OC_FARNELL (none) -> unknown
- R15: value 91k -> 100k
- R151: value 100k -> 47k
- R153: value 100k -> 200k
- R16: value 100k -> 1M 0.1%
- R17: value 91k -> 100k 0.1%
- R18, R48, R52: value 100k -> 1M
- R187, R189: value TRIMPOT -> 100k
- R19: value 220k -> 360k
- R2: value 10k -> 1k
- R20: value 220k -> 1.8k
- R21: value 220k -> 470
- R22: value 91k -> 1M
- R23: value 100k -> 1.5M
- R24: value 91k -> 10kA; device OPL:R-0603 -> EurorackModularParts:POTZEPHPOT; DESC (none) -> Saw
- R26: value 100k -> (none); device OPL:R-0603 -> EurorackModularParts:POTZEPHPOT_BIGKNOB; DESC (none) -> Fine
- R27: value 51k -> 10k; device OPL:R-0603 -> EurorackModularParts:POTZEPHPOT_BIGKNOB; DESC (none) -> Coarse 2
- R29, R93: value 1.8k -> 100k
- R3: value 10k -> 22k
- R30: value 1.8k -> 560k
- R32: value 360k -> 820
- R33: value 1.8k -> 5.6k
- R34: value 1M -> 24k
- R35: value 1.5M -> 24k
- R36: value 470 -> 5.6k
- R37: value 24k -> 820
- R38: value 5.6k -> 10k
- R39: value 820 -> 100k
- R4: value 470 -> 22k
- R40: value 10k -> 560k
- R42: value 10k -> (none); device OPL:R-0603 -> EurorackModularParts:POTZEPHPOT_BIGKNOB; DESC (none) -> Coarse
- R43: value 10k -> 140k
- R45: value 10k -> 10kA; device OPL:R-0603 -> EurorackModularParts:POTZEPHPOT; DESC (none) -> Triangle 2
- R46: value 10k -> 1.5M
- R47, R54: value 100k -> 470
- R49: value 100k -> 1.8k
- R5: value 24k -> 10k
- R51: value 100 -> 360k
- R55: value 10k -> 1M
- R58: value 470 -> 1M 0.1%
- R59: value 470 -> 100k 0.1%
- R6: value 47k -> 470
- R60: value 470 -> 10kA; device OPL:R-0603 -> EurorackModularParts:POTZEPHPOT; DESC (none) -> Triangle
- R61, R7: value 470 -> 100k
- R62: value 24k -> 100k
- R63: value 22k -> 10kA; device OPL:R-0603 -> EurorackModularParts:POTZEPHPOT; DESC (none) -> Pulse 2
- R68: value 22k -> 10k
- R69: value 100k 0.1% -> 10k
- R70: value 1M 0.1% -> 10k
- R71: value 22k -> 20k
- R72: value (none) -> 20k
- R73, R8, R97: value 470 -> 10k
- R74: value 1M -> 10kA; device OPL:R-0603 -> EurorackModularParts:POTZEPHPOT; DESC (none) -> Pulse
- R76: device OPL:R-0603 -> EurorackModularParts:POTZEPHPOT; DESC (none) -> PWM
- R77: value 360k -> 100k
- R78: value 22k -> 10kA; device OPL:R-0603 -> EurorackModularParts:POTZEPHPOT; DESC (none) -> Sub 2
- R82: value 1k -> 10k
- R84: value 140k -> 20k
- R85: value 560k -> 10k
- R87: value 10k -> 10kA; device OPL:R-0603 -> EurorackModularParts:POTZEPHPOT; DESC (none) -> Sub 1
- R88: value BIAS -> 100k
- R89: value 200k -> 100k; device OPL:R-0603 -> EurorackModularParts:POTZEPHPOT; DESC (none) -> PWM
- R9: value 470 -> 10k; device OPL:R-0603 -> EurorackModularParts:POTZEPHPOT_BIGKNOB; DESC (none) -> Fine 2
- R90: value 100k -> 51k
- R94: value 10k -> 22k; OC_FARNELL unknown -> (none)
- R95: value 1M -> 220k
- R96: value 1.5M -> 91k
- R98: value 24k -> 20k
- R99: value 5.6k -> 20k
- TP1: DESC (none) -> SubOsc 2
- TP2: DESC LP -> HP -> SubOsc 1
- TP3: DESC Filter Out -> (none)
- TP5: DESC SubOsc 2 -> Rambler 1
- TP6: DESC SubOsc 1 -> SawPulse
- TP7: DESC SawPulse -> Filter Out
- TP8: DESC Rambler 2 -> LP -> HP
- renumbered U$1 to PCB1, U$10 to R183, U$11 to J10, U$12 to J12, U$13 to J13, U$14 to J2, U$15 to IC14, U$16 to J8, U$17 to J4, U$18 to J3, U$19 to J9, U$2 to J14, U$20 to R190, U$24 to R158, U$25 to R182, U$26 to R181, U$27 to R180, U$28 to R178, U$29 to J11, U$33 to R191, U$35 to S1, U$36 to J1, U$38 to J6, U$39 to S2, U$40 to J7, U$41 to IC12, U$42 to IC13, U$48 to R187, U$50 to J5, U$51 to S3, U$57 to R165, U$58 to R161, U$59 to R160, U$60 to R193, U$61 to R194, U$62 to R192, U$63 to R188, U$64 to R189, U$66 to IC15, U$7 to R186, U$8 to R185, U$9 to R184
Connections:
- net -12V: now also C1.1, C13.2, C14.1, C22.1, C24.1, C38.1, C40.1, C42.1, C43.1, C44.1, C47.1, C51.1, C58.2, D3.+, IC11VR3.V-, IC1VR3.V-, IC5P.V-, IC7VR3.V-, R113.2, R122.1, R126.2, R139.2, R148.1, R168.2, R174.2, R32.2, R37.2, R95.1; no longer C21.2, C24.2, C25.1, C30.1, C32.1, C34.1, C36.1, C39.1, C49.1, C58.1, C6.1, C60.1, C8.1, D2.+, IC2P.V-, IC9P.V-, R100.2, R132.2, R19.2, R20.2, R21.1, R30.1, R39.2, R4.2, R61.2, R94.1, U$47VR3.V-, U$65VR3.V-
- net -5V: now also C25.2, IC6P.VEE, R102.1, R112.2, R133.1, R138.1, R147.1, R154.1, R26.E, R27.E, R42.E, R68.1, R72.1, R82.1, R9.E, R98.1; no longer C56.2, IC11P.VEE, R121.1, R122.1, R123.1, R126.1, R134.2, R83.1, R87.1, R88.1, R91.1, R92.1, U$3.E, U$4.E, U$44.E, U$45.E
- net -5VIN: now also C49.2, R148.2; no longer C38.2, R94.2
- net 10V: now also R103.2, R141.E, R153.2, R43.2; no longer R106.2, R84.2, R89.2, U$5.E
- net 12V: now also C11.1, C12.1, C2.2, C28.2, C39.1, C41.2, C45.2, C48.2, C50.2, C52.2, C61.1, C9.2, D2.-, IC11VR3.V+, IC16.11, IC17.11, IC1VR3.V+, IC3.16, IC4.16, IC5P.V+, IC7VR3.V+, IC8.POSRAIL, IC9.14, R19.1, R23.1, R46.1, R51.1; no longer C22.1, C23.1, C29.2, C31.2, C33.2, C35.2, C37.1, C48.1, C5.2, C59.2, C7.2, D1.-, IC1.11, IC2P.V+, IC3.14, IC4.11, IC7.16, IC8.16, IC9P.V+, R32.1, R35.1, R77.1, R96.1, U$47VR3.V+, U$56.POSRAIL, U$65VR3.V+
- net 5V: now also C32.1, C5.1, IC2P.VDD, IC6P.VCC, R137.A, R149.2, R26.A, R27.A, R42.A, R9.A; no longer C42.1, C55.1, IC11P.VCC, IC6P.VDD, R90.2, U$3.A, U$4.A, U$44.A, U$45.A, U$6.A
- net A2_IN: now also R167.2; no longer R55.2
- net AMPENVELOPEOUT: now also IC16.2, R169.2; no longer IC1.2, R5.2
- net A_IN: now also R163.2; no longer R1.2
- net CUTOFF1_MODENVINPUT: now also R135.1, R136.E; no longer R65.1, U$30.E
- net CUTOFF2_MODENVINPUT: now also R152.1; no longer R141.1
- net CUTOFF_ENVELOPE: now also IC11VR1.OUT, R144.2, R145.1; no longer R54.1, R66.2, U$47VR1.OUT
- net CUTOFF_ENVELOPE_2: now also IC11VR2.OUT, R104.1, R143.2; no longer R140.1, R142.2, U$47VR2.OUT
- net CUTOFF_IN: now also R106.1, R120.1; no longer R138.1, R28.1
- net CUTOFF_INPUT: now also IC9.12, R120.2, R121.1, R138.2, R140.2, R145.2, R146.2; no longer IC3.12, R28.2, R29.1, R52.2, R53.2, R54.2, R88.2
- net CUTOFF_KEYTRACK: now also R109.1, R146.1, R150.2; no longer R137.1, R52.1, R63.2
- net CUTOFF_KNOB: now also R110.1, R140.1, R141.S; no longer R136.1, R53.1, U$5.S
- net CUTOFF_KNOB_2: now also R105.1; no longer R139.1
- net D2_IN: now also R177.2; no longer R56.2
- net D_IN: now also R172.2; no longer R2.2
- net EXP_FM_IN: now also R15.1, R53.1; no longer R104.1, R79.1
- net FILTER_IN: now also R96.2; no longer R22.2
- net FILTER_OUT: now also C33.-, R107.1, TP7.1; no longer C54.-, R143.1, TP3.1
- net GATE_IN: now also C56.1, C59.1, D1.-, IC16.4, IC17.4; no longer C2.1, C27.1, D3.-, IC1.4, IC4.4
- net GND: now also C1.2, C11.2, C12.2, C13.1, C14.2, C17.2, C18.1, C2.1, C24.2, C25.1, C30.1, C38.2, C43.2, C46.2, C47.2, C48.1, C49.1, C5.2, C50.1, C51.2, C52.1, C53.1, C54.1, C55.1, C58.1, C6.1, C60.1, C61.2, C9.1, IC10A.+IN, IC10B.+IN, IC10C.+IN, IC16.14, IC16.7, IC17.14, IC17.7, IC1VR2.+IN, IC2A.R, IC2A.S, IC2B.R, IC2B.S, IC2P.VSS, IC3.12, IC4.12, IC5A.+IN, IC5B.+IN, IC5C.+IN, IC5D.+IN, IC6A.INH, IC6P.GND, IC7VR2.+IN, IC7VR2.-IN, IC8.GROUND, IC9.3, R1.E, R11.E, R111.2, R121.2, R134.E, R136.A, R137.E, R141.A, R142.E, R151.2, R159.2, R162.2, R166.2, R170.2, R171.1, R175.2, R176.1, R2.2, R20.1, R24.E, R31.2, R38.2, R39.2, R45.E, R49.1, R60.E, R63.E, R64.1, R67.1, R74.E, R76.E, R78.E, R79.1, R87.E, R89.E; no longer C1.1, C11.1, C12.1, C13.2, C14.1, C16.2, C17.1, C18.2, C23.2, C24.1, C25.2, C26.1, C29.1, C30.2, C33.1, C34.2, C35.1, C38.1, C48.2, C49.2, C5.1, C55.2, C56.1, C58.2, C59.1, C6.2, C60.2, C7.1, IC1.14, IC1.7, IC11A.INH, IC11P.GND, IC2A.+IN, IC2B.+IN, IC2C.+IN, IC2D.+IN, IC3.3, IC4.14, IC4.7, IC6A.R, IC6A.S, IC6B.R, IC6B.S, IC6P.VSS, IC7.12, IC8.12, IC9A.+IN, IC9B.+IN, IC9C.+IN, IC9D.+IN, R10.2, R101.2, R108.2, R135.2, R150.1, R151.1, R154.1, R33.1, R40.2, R58.2, R59.2, R6.2, R60.1, R7.2, R8.2, R81.2, R82.2, R9.1, R93.1, U$21.E, U$22.E, U$23.E, U$30.A, U$31.E, U$32.E, U$34.E, U$37.E, U$46.E, U$49.E, U$5.A, U$52.E, U$53.E, U$54.E, U$55.E, U$56.GROUND, U$6.E
- net HARDSYNC_2_IN: now also C15.2; no longer C47.2
- net HARDSYNC_IN: now also C23.2; no longer C19.2
- net HP_FILTER_CUTOFF_IN: now also IC8.FREQCV, R104.2, R105.2, R106.2, R109.2, R110.2, R111.1, R112.1; no longer R134.1, R135.1, R136.2, R137.2, R138.2, R139.2, R140.2, U$56.FREQCV
- net HP_RESONANCE_IN: now also R108.2; no longer R133.2
- net LINEAR_FM_IN: now also C19.2, C7.2; no longer C15.2, C43.2
- net LP_TO_HP: now also C26.1, C29.-, R90.1, TP8.1; no longer C50.1, C9.-, R27.1, TP2.1
- net MAIN_CV: now also R14.1, R155.1, R57.1; no longer R31.1, R64.1, R76.1
- net MIXER_SUMLINE: now also IC1VR2.-IN, R10.2, R12.1, R25.2, R44.2, R61.2, R62.2, R75.2, R77.2, R88.2; no longer IC2D.-IN, R118.2, R119.2, R120.2, R124.2, R125.2, R47.2, R48.2, R49.2, R50.1
- net MODENVOUT: now also IC17.2, R173.2; no longer IC4.2, R62.2
- net N$1: now also IC16.15, R162.1, R163.1; no longer IC1.15, R1.1, R7.1
- net N$10: now also C55.2, IC16.8; no longer C1.2, IC1.8
- net N$100: now also IC4.7; no longer IC8.7
- net N$101: now also R28.2, R76.S; no longer R105.2, U$49.S
- net N$102: now also R43.1, R76.A; no longer R106.1, U$49.A
- net N$103: now also R29.1, R30.1; no longer R107.1, R108.1
- net N$104: now also R27.S, R50.1; no longer R102.1, U$45.S
- net N$105: now also R52.1, R9.S; no longer R103.1, U$44.S
- net N$106: now also C4.1, IC2B.CLK, R5.2; no longer C18.1, IC6B.CLK, R111.2
- net N$107: now also IC2B.!Q, IC2B.D; no longer IC6B.!Q, IC6B.D
- net N$109: now also IC5A.OUT, R11.A, R70.2; no longer IC9A.OUT, R117.2, U$46.A
- net N$11: now also IC16.10, R169.1; no longer IC1.10, R5.1
- net N$110: now also IC5B.OUT, R63.A, R83.2; no longer IC9B.OUT, R116.2, U$52.A
- net N$111: now also IC5B.-IN, R81.2, R82.2, R83.1; no longer IC9B.-IN, R113.2, R116.1, R122.2
- net N$112: now also IC5A.-IN, R68.2, R69.2, R70.1; no longer IC9A.-IN, R112.2, R117.1, R123.2
- net N$113: now also IC5C.-IN, R84.1, R85.2, R86.2; no longer IC9C.-IN, R114.2, R115.1, R121.2
- net N$114: now also IC5C.OUT, R45.A, R84.2; no longer IC9C.OUT, R115.2, U$53.A
- net N$115: now also R44.1, R45.S; no longer R120.1, U$53.S
- net N$116: now also R62.1, R63.S; no longer R119.1, U$52.S
- net N$117: now also R10.1, R11.S; no longer R118.1, U$46.S
- net N$118: now also R77.1, R78.S; no longer R125.1, U$55.S
- net N$119: now also IC10D.OUT, R130.2, R87.A; no longer IC9D.OUT, R128.2, U$54.A
- net N$120: now also IC10D.-IN, R128.2, R129.2, R130.1; no longer IC9D.-IN, R126.2, R127.2, R128.1
- net N$121: now also IC8.NEGRAIL, R113.1; no longer R132.1, U$56.NEGRAIL
- net N$122: now also IC5D.OUT, R71.2, R78.A; no longer IC10D.OUT, R131.2, U$55.A
- net N$123: now also IC5D.-IN, R71.1, R72.2, R73.2; no longer IC10D.-IN, R129.2, R130.2, R131.1
- net N$124: now also IC8.RESONANCE_CV, R108.1; no longer R133.1, U$56.RESONANCE_CV
- net N$126: now also IC11VR2.-IN, R143.1, R152.2; no longer R141.2, R142.1, U$47VR2.-IN
- net N$127: now also IC11VR2.+IN; no longer U$47VR2.+IN
- net N$128: now also C26.2, IC8.STAGE1_CAP; no longer C50.2, U$56.STAGE1_CAP
- net N$129: now also IC8.STAGE1_IN, R116.1; no longer R147.1, U$56.STAGE1_IN
- net N$13: now also R159.1; no longer R6.1
- net N$130: now also C27.2, IC8.STAGE1_OUT, R116.2; no longer C51.2, R147.2, U$56.STAGE1_OUT
- net N$131: now also C27.1, IC8.STAGE2_CAP; no longer C51.1, U$56.STAGE2_CAP
- net N$132: now also IC8.STAGE2_IN, R115.1; no longer R146.1, U$56.STAGE2_IN
- net N$133: now also C35.2, IC8.STAGE2_OUT, R115.2; no longer C52.2, R146.2, U$56.STAGE2_OUT
- net N$134: now also C35.1, IC8.STAGE3_CAP; no longer C52.1, U$56.STAGE3_CAP
- net N$135: now also IC8.STAGE3_IN, R114.1; no longer R145.1, U$56.STAGE3_IN
- net N$136: now also C34.2, IC8.STAGE3_OUT, R114.2; no longer C53.2, R145.2, U$56.STAGE3_OUT
- net N$137: now also C34.1, IC8.STAGE4_CAP; no longer C53.1, U$56.STAGE4_CAP
- net N$138: now also IC8.STAGE4_IN, R117.1; no longer R144.1, U$56.STAGE4_IN
- net N$139: now also C33.+, IC8.STAGE4_OUT, R117.2; no longer C54.+, R144.2, U$56.STAGE4_OUT
- net N$14: now also R151.1; no longer R10.1
- net N$141: now also IC8.FEEDBACK_IN, R107.2; no longer R143.2, U$56.FEEDBACK_IN
- net N$16: now also C3.2, R6.2; no longer C14.2, R11.2
- net N$17: now also C37.1, IC9.16; no longer C10.1, IC3.16
- net N$18: now also C31.2, IC9.4; no longer C11.2, IC3.4
- net N$19: now also C30.2, IC9.5; no longer C12.2, IC3.5
- net N$2: now also IC16.12, R171.2, R172.1; no longer IC1.12, R2.1, R9.2
- net N$20: now also C36.1, IC9.11; no longer C13.1, IC3.11
- net N$21: now also IC9.9, R118.1; no longer IC3.9, R26.1
- net N$22: now also R2.1; no longer R82.1
- net N$23: now also IC9.1, R125.1, R96.1; no longer IC3.1, R22.1, R23.1
- net N$24: now also IC9.7, R125.2, R91.2; no longer IC3.7, R23.2, R24.2
- net N$25: now also IC9.6, R124.1, R93.2; no longer IC3.6, R15.1, R25.2
- net N$26: now also IC9.18, R119.2, R126.1, R127.2; no longer IC3.18, R17.2, R18.2, R20.1
- net N$27: now also IC9.17, R123.2, R124.2, R139.1; no longer IC3.17, R12.2, R15.2, R19.1
- net N$28: now also IC9.15, R123.1, R127.1; no longer IC3.15, R12.1, R17.1
- net N$29: now also IC9.13, R122.2; no longer IC3.13, R30.2
- net N$3: now also IC16.13, R164.1, R170.1; no longer IC1.13, R3.1, R8.1
- net N$30: now also C29.+, IC9.10, R119.1; no longer C9.+, IC3.10, R18.1
- net N$31: now also C6.2, R21.2; no longer C17.2, R36.2
- net N$32: now also IC9.8, R90.2; no longer IC3.8, R27.2
- net N$33: now also IC9.2, R91.1, R93.1, R95.2; no longer IC3.2, R21.2, R24.1, R25.1
- net N$34: now also IC3.13, R21.1, R22.2, R23.2; no longer IC7.13, R34.2, R35.2, R36.1
- net N$35: now also C7.1, R22.1; no longer C15.1, R34.1
- net N$36: now also C10.1, IC3.11; no longer C16.1, IC7.11
- net N$37: now also IC3.9, TP3.1; no longer IC7.9, TP1.1
- net N$38: now also IC3.14, R20.2; no longer IC7.14, R33.2
- net N$39: now also IC1VR2.OUT, R12.2, R13.1; no longer IC2D.OUT, R50.2, R51.1
- net N$4: now also C53.2, IC16.1; no longer C3.2, IC1.1
- net N$40: now also R87.S, R88.1; no longer R124.1, U$54.S
- net N$41: now also IC1VR1.OUT, R4.2; no longer R14.2, U$65VR1.OUT
- net N$42: now also C23.1, IC3.6; no longer C19.1, IC7.6
- net N$43: now also IC3.1, R35.1; no longer IC7.1, R37.1
- net N$44: now also R35.2; no longer R37.2
- net N$45: now also IC3.3, R36.2, R37.1; no longer IC7.3, R38.2, R39.1
- net N$46: now also R18.2; no longer R13.2
- net N$47: now also IC3.2, R36.1; no longer IC7.2, R38.1
- net N$48: now also IC3.7; no longer IC7.7
- net N$49: now also R60.S, R61.1; no longer R49.1, U$23.S
- net N$5: now also C46.1; no longer C4.1
- net N$50: now also R74.S, R75.1; no longer R48.1, U$22.S
- net N$51: now also R24.S, R25.1; no longer R47.1, U$21.S
- net N$52: now also IC10A.OUT, R131.2, R24.A; no longer IC2A.OUT, R46.2, U$21.A
- net N$53: now also IC10B.OUT, R100.2, R74.A; no longer IC2B.OUT, R45.2, U$22.A
- net N$54: now also IC10B.-IN, R100.1, R101.2, R102.2; no longer IC2B.-IN, R42.2, R45.1, R86.2
- net N$55: now also IC10A.-IN, R131.1, R132.2, R133.2; no longer IC2A.-IN, R41.2, R46.1, R87.2
- net N$56: now also IC10C.-IN, R97.2, R98.2, R99.1; no longer IC2C.-IN, R43.2, R44.1, R83.2
- net N$57: now also IC10C.OUT, R60.A, R99.2; no longer IC2C.OUT, R44.2, U$23.A
- net N$58: now also IC17.15, R166.1, R167.1; no longer IC4.15, R55.1, R58.1
- net N$59: now also IC17.12, R176.2, R177.1; no longer IC4.12, R56.1, R60.2
- net N$6: now also C56.2, IC16.5; no longer C2.2, IC1.5
- net N$60: now also IC17.13, R175.1, R179.1; no longer IC4.13, R57.1, R59.1
- net N$61: now also C59.2, IC17.5; no longer C27.2, IC4.5
- net N$62: now also IC17.6, R174.1; no longer IC4.6, R61.1
- net N$63: now also C60.2, IC17.8; no longer C26.2, IC4.8
- net N$64: now also IC17.10, R173.1; no longer IC4.10, R62.1
- net N$65: now also C54.2, IC17.1; no longer C28.2, IC4.1
- net N$66: now also IC1VR1.-IN, R3.2, R4.1; no longer R14.1, R78.2, U$65VR1.-IN
- net N$67: now also R150.1, R155.2; no longer R63.1, R64.2
- net N$69: now also IC11VR1.-IN, R135.2, R144.1; no longer R65.2, R66.1, U$47VR1.-IN
- net N$7: now also D2.+; no longer D1.+
- net N$70: now also IC2A.!Q, IC2A.D; no longer IC6A.!Q, IC6A.D
- net N$71: now also C21.2, R54.2; no longer C41.2, R73.2
- net N$72: now also R156.1, R157.2; no longer R67.1, R68.2
- net N$73: now also IC11VR1.+IN, R136.S; no longer U$30.S, U$47VR1.+IN
- net N$74: now also C8.1, IC2A.CLK, R8.2; no longer C40.1, IC6A.CLK, R72.2
- net N$75: now also IC7VR1.-IN, R92.1, R94.2; no longer IC10C.-IN, R148.2, R71.1
- net N$76: now also IC7VR1.+IN, R134.S; no longer IC10C.+IN, U$32.S
- net N$77: now also C18.2, R47.2; no longer C45.2, R97.2
- net N$78: now also R142.S; no longer U$31.S
- net N$79: now also R17.1, R42.S, R59.1; no longer R110.1, R69.1, U$4.S
- net N$8: now also D3.-; no longer D2.-
- net N$80: now also R16.1, R26.S, R58.1; no longer R109.1, R70.1, U$3.S
- net N$81: now also IC1VR1.+IN, R1.S; no longer U$34.S, U$65VR1.+IN
- net N$82: now also R1.A, R3.1; no longer R78.1, U$34.A
- net N$83: now also R41.2, R89.S; no longer R80.2, U$37.S
- net N$84: now also R103.1, R89.A; no longer R84.1, U$37.A
- net N$85: now also R39.1, R40.1; no longer R81.1, R85.1
- net N$86: now also D1.+; no longer D3.+
- net N$87: now also IC4.13, R46.2, R47.1, R48.2; no longer IC8.13, R95.2, R96.2, R97.1
- net N$88: now also C19.1, R48.1; no longer C43.1, R95.1
- net N$89: now also C17.1, IC4.11; no longer C44.1, IC8.11
- net N$9: now also IC16.6, R168.1; no longer IC1.6, R4.1
- net N$90: now also C16.2, IC4.9; no longer C46.2, IC8.9
- net N$91: now also R153.1, R154.2; no longer R89.1, R92.2
- net N$92: now also IC4.14, R49.2; no longer IC8.14, R93.2
- net N$93: now also R147.2, R149.1; no longer R90.1, R91.2
- net N$94: now also C15.1, IC4.6; no longer C47.1, IC8.6
- net N$95: now also IC4.1, R34.1; no longer IC8.1, R98.1
- net N$96: now also R34.2; no longer R98.2
- net N$97: now also IC4.3, R32.1, R33.2; no longer IC8.3, R100.1, R99.2
- net N$98: now also IC4.2, R33.1; no longer IC8.2, R99.1
- net N$99: now also R55.2; no longer R74.2
- net OSCSUM: now also R13.2; no longer R51.2
- net PITCHENVMOD2: now also R134.A, R94.1; no longer R148.1, U$32.A
- net PITCHENVMODINP1: now also R142.A, R157.1; no longer R68.1, U$31.A
- net PITCH_ENV: now also R156.2, R7.1; no longer R16.1, R67.2
- net PITCH_ENV_2: now also IC7VR1.OUT, R56.1, R92.2; no longer IC10C.OUT, R71.2, R75.1
- net PITCH_IN: now also IC3.15, R14.2, R15.2, R17.2, R18.1, R19.2, R6.1, R7.2; no longer IC7.15, R11.1, R13.1, R31.2, R32.2, R69.2, R70.2, R79.2
- net PITCH_IN_2: now also IC4.15, R50.2, R51.2, R52.2, R53.2, R54.1, R55.1, R56.2, R57.2, R58.2, R59.2; no longer IC8.15, R102.2, R103.2, R104.2, R109.2, R110.2, R73.1, R74.1, R75.2, R76.2, R77.2
- net PULSE_OUT_1: now also IC3.4, R101.1, R38.1; no longer IC7.4, R40.1, R42.1
- net PULSE_OUT_2: now also IC4.4, R31.1, R65.2, R81.1; no longer IC8.4, R101.1, R113.1, R152.2
- net PWM_2_IN: now also IC4.5, R28.1, R30.2; no longer IC8.5, R105.1, R107.2
- net PWM_IN: now also IC3.5, R40.2, R41.1; no longer IC7.5, R80.1, R85.2
- net R2_IN: now also R179.2; no longer R57.2
- net RAMBLER2_SAW_IN: now also IC6A.Y0, IC6A.Z0, R66.1, R67.2; no longer IC11A.Y0, IC11A.Z0, R153.1, R154.2
- net RAMBLER_2_OPT: now also IC6A.Y1; no longer IC11A.Y1
- net RAMBLER_IN_1B: now also IC6A.X1, R79.2, R80.1; no longer IC11A.X1, R149.1, R150.2
- net RAMBLER_OUT_1: now also IC6A.X, JP1.1, TP5.1; no longer IC11A.X, JP2.1, TP9.1
- net RAMBLER_OUT_2: now also IC6A.Y, JP2.3, TP4.1; no longer IC11A.Y, JP1.3, TP8.1
- net RESONANCE_IN: now also R118.2, R137.S; no longer R26.2, U$6.S
- net R_IN: now also R164.2; no longer R3.2
- net S2_IN: now also IC17.9; no longer IC4.9
- net SAWPULSE: now also IC6A.Z, JP2.5, TP6.1; no longer IC11A.Z, JP1.5, TP7.1
- net SAWPULSE_IN: now also IC6A.Z1, R64.2, R65.1; no longer IC11A.Z1, R151.2, R152.1
- net SAWTOOTH_OUT_1: now also IC3.8, R132.1, R8.1, R80.2; no longer IC7.8, R149.2, R41.1, R72.1
- net SAWTOOTH_OUT_2: now also IC4.8, R5.1, R66.2, R69.1; no longer IC8.8, R111.1, R112.1, R153.2
- net SELECTEDSUB1: now also JP1.2, R128.1; no longer JP2.2, R127.1
- net SELECTEDSUB2: now also JP2.2, JP2.4, JP2.6, R73.1; no longer JP1.2, JP1.4, JP1.6, R130.1
- net SOFTSYNC_2_IN: now also C16.1; no longer C46.1
- net SUBOSC_1_OUT: now also IC2A.Q, IC6A.A, JP1.3, TP2.1; no longer IC11A.A, IC6A.Q, JP2.3, TP6.1
- net SUBOSC_2_OUT: now also IC2B.Q, IC6A.B, IC6A.C, JP2.1, TP1.1; no longer IC11A.B, IC11A.C, IC6B.Q, JP1.1, TP5.1
- net S_IN: now also IC16.9; no longer IC1.9
- net TRIANGLE_OUT_1: now also IC3.10, IC6A.X0, R97.1; no longer IC11A.X0, IC7.10, R43.1
- net TRIANGLE_OUT_2: now also IC4.10, R85.1; no longer IC8.10, R114.1
