File: Development/Eurorack Set 9/LineOut&Headphone.brd (EAGLE design)
At the start: 29.2 x 79.2 mm, 58 parts, among them IC1 NE5532D, IC2 NE5532D, U1 CJ1117-5.0-1310170P1

Commit message: Tweaks & Fixes...
Parts:
- moved U$2 12.7 mm to (8.89, 99.1)
- moved U$5 12.7 mm to (21.6, 99.1)
Routing:
- net N$14: track 104.0 -> 81.8 mm
- net N$22: track 84.6 -> 97.4 mm
Changed lines of the file:
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@@
 <setting verticaltext="up"/>
 </settings>
-<grid distance="1" unitdist="mm" unit="mm" style="dots" multiple="1" display="yes" altdistance="0.025" altunitdist="inch" altunit="inch"/>
+<grid distance="25" unitdist="mil" unit="mil" style="dots" multiple="1" display="yes" altdistance="0.025" altunitdist="inch" altunit="inch"/>
 <layers>
 <layer number="1" name="Top" color="4" fill="1" visible="yes" active="yes"/>
@@
 <element name="R9" library="OPL" package="R0603" value="27" x="8.5725" y="87.63" rot="R90"/>
 <element name="U$1" library="EurorackModularParts" package="POWER_10" value="POWER_SIMPLE10" x="15.24" y="41.91" rot="MR180"/>
-<element name="U$5" library="EurorackModularParts" package="3.5MM-JACK-SWITCH-13MM-INPUT" value="PJ-341" x="8.89" y="99.06">
-<attribute name="MPN" value="PJ-341" x="8.89" y="99.06" size="1.778" layer="27" display="off"/>
-<attribute name="DESC" value="Input" x="8.89" y="99.06" size="1.778" layer="27" display="off"/>
+<element name="U$5" library="EurorackModularParts" package="3.5MM-JACK-SWITCH-13MM-INPUT" value="PJ-341" x="21.59" y="99.06">
+<attribute name="MPN" value="PJ-341" x="21.59" y="99.06" size="1.778" layer="27" display="off"/>
+<attribute name="DESC" value="Input" x="21.59" y="99.06" size="1.778" layer="27" display="off"/>
 </element>
 <element name="C8" library="adafruit" package="153CLV-0505" value="220uF" x="26.67" y="88.5825" rot="R90"/>
@@
 <element name="C4" library="OPL" package="C0603" value="100nF" x="14.9225" y="46.355" rot="R270"/>
 <element name="IC2" library="EurorackModularParts" package="SO08" value="NE5532D" x="4.7625" y="65.7225"/>
-<element name="U$2" library="EurorackModularParts" package="3.5MM-JACK-SWITCH-13MM-INPUT" value="PJ-341" x="21.59" y="99.06">
-<attribute name="DESC" value="Input" x="-16.51" y="162.56" size="1.778" layer="27" display="off"/>
-<attribute name="MPN" value="PJ-341" x="-16.51" y="162.56" size="1.778" layer="27" display="off"/>
+<element name="U$2" library="EurorackModularParts" package="3.5MM-JACK-SWITCH-13MM-INPUT" value="PJ-341" x="8.89" y="99.06">
+<attribute name="DESC" value="Input" x="-29.21" y="162.56" size="1.778" layer="27" display="off"/>
+<attribute name="MPN" value="PJ-341" x="-29.21" y="162.56" size="1.778" layer="27" display="off"/>
 </element>
 <element name="C10" library="OPL" package="C0603" value="22p" x="4.7625" y="72.0725"/>
@@
 <contactref element="R2" pad="1"/>
 <contactref element="U$2" pad="SWITCH@3"/>
-<wire x1="8.89" y1="103.56" x2="17.5175" y2="103.56" width="0.2032" layer="1"/>
-<wire x1="17.5175" y1="103.56" x2="19.05" y2="105.0925" width="0.2032" layer="1"/>
-<wire x1="19.05" y1="105.0925" x2="23.495" y2="105.0925" width="0.2032" layer="1"/>
-<wire x1="23.495" y1="105.0925" x2="25.0825" y2="103.505" width="0.2032" layer="1"/>
-<wire x1="25.0825" y1="103.505" x2="25.0825" y2="99.2675" width="0.2032" layer="1"/>
-<wire x1="25.0825" y1="99.2675" x2="25.29" y2="99.06" width="0.2032" layer="1"/>
-<wire x1="25.29" y1="99.06" x2="20.955" y2="99.06" width="0.2032" layer="1"/>
-<wire x1="20.955" y1="99.06" x2="16.98625" y2="95.09125" width="0.2032" layer="1"/>
-<wire x1="16.98625" y1="95.09125" x2="11.43" y2="95.09125" width="0.2032" layer="1"/>
 <wire x1="5.87375" y1="94.13875" x2="1.5875" y2="89.8525" width="0.2032" layer="1"/>
 <wire x1="1.5875" y1="89.8525" x2="1.5875" y2="76.708" width="0.2032" layer="1"/>
 <wire x1="1.5875" y1="76.708" x2="2.7305" y2="75.565" width="0.2032" layer="1"/>
 <wire x1="5.87375" y1="94.13875" x2="10.4775" y2="94.13875" width="0.2032" layer="1"/>
-<wire x1="10.4775" y1="94.13875" x2="11.43" y2="95.09125" width="0.2032" layer="1"/>
 <wire x1="22.5425" y1="67.945" x2="22.225" y2="68.2625" width="0.2032" layer="1"/>
 <wire x1="22.225" y1="68.2625" x2="16.1925" y2="68.2625" width="0.2032" layer="1"/>
@@
 <wire x1="27.6225" y1="59.055" x2="26.24" y2="57.6725" width="0.2032" layer="1"/>
 <wire x1="26.24" y1="57.6725" x2="26.24" y2="57.61" width="0.2032" layer="1"/>
+<wire x1="10.4775" y1="94.13875" x2="12.59" y2="96.25125" width="0.2032" layer="1"/>
+<wire x1="12.59" y1="96.25125" x2="12.59" y2="99.06" width="0.2032" layer="1"/>
+<wire x1="12.59" y1="99.06" x2="17.09" y2="103.56" width="0.2032" layer="1"/>
+<wire x1="17.09" y1="103.56" x2="21.59" y2="103.56" width="0.2032" layer="1"/>
 </signal>
 <signal name="+12V" class="1">
@@
 <contactref element="R1" pad="1"/>
 <contactref element="U$5" pad="SWITCH@3"/>
-<wire x1="21.59" y1="103.56" x2="19.74" y2="103.56" width="0.2032" layer="1"/>
-<wire x1="19.74" y1="103.56" x2="18.415" y2="102.235" width="0.2032" layer="1"/>
-<wire x1="18.415" y1="102.235" x2="15.765" y2="102.235" width="0.2032" layer="1"/>
-<wire x1="15.765" y1="102.235" x2="12.59" y2="99.06" width="0.2032" layer="1"/>
-<wire x1="12.59" y1="99.06" x2="8.89" y2="99.06" width="0.2032" layer="1"/>
 <wire x1="8.89" y1="99.06" x2="0.9525" y2="91.1225" width="0.2032" layer="1"/>
 <wire x1="0.9525" y1="91.1225" x2="0.9525" y2="60.5155" width="0.2032" layer="1"/>
@@
 <wire x1="24.765" y1="57.785" x2="26.24" y2="59.26" width="0.2032" layer="1"/>
 <wire x1="26.24" y1="59.26" x2="26.24" y2="59.61" width="0.2032" layer="1"/>
+<wire x1="8.89" y1="103.56" x2="8.89" y2="99.06" width="0.2032" layer="1"/>
+<wire x1="25.29" y1="99.06" x2="25.4" y2="99.17" width="0.2032" layer="1"/>
+<wire x1="25.4" y1="99.17" x2="25.4" y2="103.505" width="0.2032" layer="1"/>
+<wire x1="25.4" y1="103.505" x2="23.495" y2="105.41" width="0.2032" layer="1"/>
+<wire x1="23.495" y1="105.41" x2="10.16" y2="105.41" width="0.2032" layer="1"/>
+<wire x1="10.16" y1="105.41" x2="8.89" y2="104.14" width="0.2032" layer="1"/>
+<wire x1="8.89" y1="104.14" x2="8.89" y2="103.56" width="0.2032" layer="1"/>
 </signal>
 <signal name="N$23">
