File: Development/Eurorack Set 9/DelayExperiments_Rev2.sch (EAGLE design)
At the start: 145 parts, among them IC1 TL074D, IC2 TL074D, IC3 TL074D, IC4 TL072, Q1 MMBT3904, Q2 MMBT3904, Q3 MMBT3904, Q5 MMBT3904, U1 CJ1117-5.0-1310170P1

Commit message: Tweaks, Powerboard, Caps in Echochamber fixed
Parts:
- C41, C42, C43, C44, C47, C48, C55: value 3.3n -> 33p
Changed lines of the file:
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@@
 <setting verticaltext="up"/>
 </settings>
-<grid distance="0.05" unitdist="inch" unit="inch" style="lines" multiple="1" display="no" altdistance="0.01" altunitdist="inch" altunit="inch"/>
+<grid distance="0.1" unitdist="inch" unit="inch" style="lines" multiple="1" display="no" altdistance="0.01" altunitdist="inch" altunit="inch"/>
 <layers>
 <layer number="1" name="Top" color="4" fill="1" visible="no" active="no"/>
@@
 <part name="SUPPLY4" library="SparkFun-Aesthetics" deviceset="5V" device=""/>
 <part name="SUPPLY5" library="SparkFun-Aesthetics" deviceset="5V" device=""/>
-<part name="C41" library="OPL" deviceset="C*" device="-0603" value="3.3n"/>
-<part name="C42" library="OPL" deviceset="C*" device="-0603" value="3.3n"/>
-<part name="C43" library="OPL" deviceset="C*" device="-0603" value="3.3n"/>
-<part name="C44" library="OPL" deviceset="C*" device="-0603" value="3.3n"/>
+<part name="C41" library="OPL" deviceset="C*" device="-0603" value="33p"/>
+<part name="C42" library="OPL" deviceset="C*" device="-0603" value="33p"/>
+<part name="C43" library="OPL" deviceset="C*" device="-0603" value="33p"/>
+<part name="C44" library="OPL" deviceset="C*" device="-0603" value="33p"/>
 <part name="IC2" library="EurorackModularParts" deviceset="TL074" device="D"/>
 <part name="C45" library="OPL" deviceset="C*" device="-0603" value="100n"/>
@@
 <part name="R34" library="OPL" deviceset="R*" device="-0603" value="51k"/>
 <part name="R35" library="OPL" deviceset="R*" device="-0603" value="100k"/>
-<part name="C47" library="OPL" deviceset="C*" device="-0603" value="3.3n"/>
-<part name="C48" library="OPL" deviceset="C*" device="-0603" value="3.3n"/>
+<part name="C47" library="OPL" deviceset="C*" device="-0603" value="33p"/>
+<part name="C48" library="OPL" deviceset="C*" device="-0603" value="33p"/>
 <part name="GND48" library="SparkFun-Aesthetics" deviceset="GND" device=""/>
 <part name="GND49" library="SparkFun-Aesthetics" deviceset="GND" device=""/>
@@
 <part name="R56" library="OPL" deviceset="R*" device="-0603" value="100k"/>
 <part name="R57" library="OPL" deviceset="R*" device="-0603" value="51k"/>
-<part name="C55" library="OPL" deviceset="C*" device="-0603" value="3.3n"/>
+<part name="C55" library="OPL" deviceset="C*" device="-0603" value="33p"/>
 <part name="GND66" library="SparkFun-Aesthetics" deviceset="GND" device=""/>
 <part name="R58" library="OPL" deviceset="R*" device="-0603" value="56"/>
