File: Development/Eurorack Set 10/TheRug-Andabil.brd (EAGLE design)
At the start: 59.6 x 106.5 mm, 157 parts, among them IC1 TL072, IC10 TL072, IC2 TL072, IC3 TL072, IC4 TL072, IC5 TL074D, IC6 TL074D, IC7 TL072, IC8 TL072, IC9 TL072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

Commit message: Edgecutter bodge, Ardabil, Labpower, RectangularThing & Calibrator
Parts:
- removed C23, C24: 1uF-BIDIR, adafruit:153CLV-0505
- removed IC4: TL072, EurorackModularParts:SO08
- removed U$21, U$22, U$23, U$24: 100K, adafruit:TC33X
- added C35, C36, C42, C49, C50: 100nF, OPL:C0603
- added IC12: TL072, EurorackModularParts:SO08
- added R147, R149: 100k, OPL:R0603
- added R148: 10k, OPL:R0603
- added R73, R74: 100K, OPL:R0603
- added R75, R76, R77, R78: 100k, EurorackModularParts:TRIMPOT
- added U2: LM4040DIM3-5.0, FarnellThings:SOT95P237X112-3N
- R2, R57: value 100K -> 49.9k
- R27, R28: value 220K -> 100K
- U$29, U$31, U$7, U$8: value 10K LINEAR -> 10KB
- moved R34 121.1 mm to (31.8, 90.8), turned to 180 degrees
- moved C18 117.5 mm to (34.9, 90.8), turned to 180 degrees
- moved R48 113.4 mm to (38.7, 90.8), turned to 0 degrees
- moved IC6 112.4 mm to (35.6, 85.7), turned to 0 degrees
- moved R24 111.5 mm to (31.1, 78.7), turned to 270 degrees
- moved R47 109.8 mm to (34.3, 78.7)
- moved C17 109.5 mm to (34.9, 81.3), turned to 0 degrees
- moved Q2 107.5 mm to (32.4, 74.6), turned to 90 degrees
- moved R29 100.8 mm to (38.7, 74.5)
- moved D8 100.4 mm to (39.6, 76.6), turned to 180 degrees
- moved R46 100.3 mm to (35.7, 74.5), turned to 180 degrees
- moved C28 89.6 mm to (27.3, 3.81)
- moved R43 88.9 mm to (28.6, 22.2), turned to 0 degrees
- moved R28 87.9 mm to (21.6, 12.7), turned to 0 degrees
- moved R32 85.0 mm to (28.6, 12.1)
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Connections:
- removed net N$40: C24.+, IC6.3, R27.2
- removed net N$42: IC6.1, IC6.2, R24.1
- removed net V+: IC10.8, IC4.8
- removed net V-: IC10.4, IC4.4
- new net -5V: IC12.1, IC12.2, R147.1, R75.P$1, R76.P$1, R77.P$1, R78.P$1, U$29.P$1, U$8.P$1
- new net -5VIN: C49.2, IC12.3, R148.2, U2.2
- new net -5V_TO_5V: IC12.6, R147.2, R149.1
- new net 5V: IC12.7, R149.2, R75.P$3, R76.P$3, R77.P$3, R78.P$3, U$29.P$3, U$8.P$3
- new net N$13: IC6.1, R24.1, R73.1
- new net N$49: IC6.2, R73.2, R74.1
- net -12V: now also C36.1, C42.1, IC10.4, IC12.4, R148.1; no longer U$21.1, U$22.1, U$23.1, U$24.1, U$29.P$1, U$8.P$1
- net 12V: now also C35.2, C50.2, IC10.8, IC12.8; no longer U$21.3, U$22.3, U$23.3, U$24.3, U$29.P$3, U$8.P$3
- net GND: now also C35.1, C36.2, C42.2, C49.1, C50.1, IC12.5, IC5.3, IC6.3, U2.1; no longer R27.1, R28.1
- net N$1: now also IC10.5; no longer IC4.3
- net N$10: now also IC10.6; no longer IC4.2
- net N$3: now also IC10.7; no longer IC4.1
- net N$33: now also R75.P$2; no longer U$23.2
- net N$34: now also R77.P$2; no longer U$21.2
- net N$35: now also R76.P$2; no longer U$24.2
- net N$36: now also R78.P$2; no longer U$22.2
- net N$37: now also R27.2; no longer C23.-
- net N$38: now also R74.2; no longer C24.-
- net N$39: now also IC5.2, R27.1; no longer C23.+, IC5.3
- net N$41: now also R28.1; no longer IC5.2
Routing:
- net -12V: track 0.00 -> 310.5 mm, vias 0 -> 27
- net 12V: track 0.00 -> 254.1 mm, vias 0 -> 29
- net 5V: track 0.00 -> 162.0 mm, vias 0 -> 18
- net -5V: track 0.00 -> 156.1 mm, vias 0 -> 8
- net OUTPUT2_SUM_TO_VCA2: track 0.00 -> 116.6 mm, vias 0 -> 8
- net N$70: track 0.00 -> 93.5 mm, vias 0 -> 12
- net GND: track 0.00 -> 91.7 mm, vias 0 -> 36
- net N$78: track 0.00 -> 87.3 mm, vias 0 -> 8
- net N$56: track 0.00 -> 81.2 mm, vias 0 -> 2
- net OUTPUT1_SUM_TO_VCA1: track 0.00 -> 76.9 mm, vias 0 -> 6
- net TRANS_OUT_B: track 0.00 -> 76.4 mm, vias 0 -> 8
- net N$53: track 0.00 -> 73.7 mm, vias 0 -> 8
- net N$24: track 0.00 -> 64.2 mm, vias 0 -> 10
- net N$67: track 0.00 -> 63.6 mm, vias 0 -> 8
- net N$44: track 0.00 -> 62.7 mm, vias 0 -> 10
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
Commit message: Value unification and value fixes
Parts:
- R147, R149: value 100k -> 100K
- R2, R57: value 49.9k -> 49.9K
- R4, R5, R52, R53: value 100k 0.1% -> 100K 0.1%
Changed lines of the file:
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@@
 <element name="R1" library="OPL" package="R0603" value="100K 0.1%" x="35.2425" y="99.695" rot="R270"/>
 <element name="R3" library="OPL" package="R0603" value="100K" x="24.4475" y="92.71"/>
-<element name="R4" library="OPL" package="R0603" value="100k 0.1%" x="24.13" y="105.0925"/>
-<element name="R5" library="OPL" package="R0603" value="100k 0.1%" x="24.13" y="103.8225"/>
+<element name="R4" library="OPL" package="R0603" value="100K 0.1%" x="24.13" y="105.0925"/>
+<element name="R5" library="OPL" package="R0603" value="100K 0.1%" x="24.13" y="103.8225"/>
 <element name="R10" library="OPL" package="R0603" value="56" x="6.35" y="60.0075"/>
 <element name="R11" library="OPL" package="R0603" value="100K 0.1%" x="13.97" y="80.9625" rot="R180"/>
@@
 </element>
 <element name="U$8" library="EurorackModularParts" package="ALPS_POT_SQUAREHOLES" value="10KB" x="22.86" y="69.85"/>
-<element name="R2" library="OPL" package="R0603" value="49.9k" x="24.4475" y="94.2975"/>
+<element name="R2" library="OPL" package="R0603" value="49.9K" x="24.4475" y="94.2975"/>
 <element name="R6" library="OPL" package="R0603" value="100K 0.1%" x="16.51" y="76.2" rot="R270"/>
 <element name="R7" library="OPL" package="R0603" value="100K 0.1%" x="18.0975" y="76.2" rot="R270"/>
@@
 <element name="R50" library="OPL" package="R0603" value="100K 0.1%" x="57.4675" y="29.21" rot="R270"/>
 <element name="R51" library="OPL" package="R0603" value="100K" x="31.4325" y="24.4475" rot="R270"/>
-<element name="R52" library="OPL" package="R0603" value="100k 0.1%" x="43.815" y="13.6525"/>
-<element name="R53" library="OPL" package="R0603" value="100k 0.1%" x="53.975" y="13.6525" rot="R180"/>
+<element name="R52" library="OPL" package="R0603" value="100K 0.1%" x="43.815" y="13.6525"/>
+<element name="R53" library="OPL" package="R0603" value="100K 0.1%" x="53.975" y="13.6525" rot="R180"/>
 <element name="R54" library="OPL" package="R0603" value="56" x="54.61" y="60.0075" rot="R180"/>
 <element name="R55" library="OPL" package="R0603" value="100K 0.1%" x="32.385" y="9.525" rot="R180"/>
@@
 </element>
 <element name="U$29" library="EurorackModularParts" package="ALPS_POT_SQUAREHOLES" value="10KB" x="38.1" y="36.83"/>
-<element name="R57" library="OPL" package="R0603" value="49.9k" x="57.4675" y="32.0675" rot="R270"/>
+<element name="R57" library="OPL" package="R0603" value="49.9K" x="57.4675" y="32.0675" rot="R270"/>
 <element name="R58" library="OPL" package="R0603" value="100K 0.1%" x="59.055" y="38.4175" rot="R270"/>
 <element name="R59" library="OPL" package="R0603" value="100K 0.1%" x="45.72" y="37.7825" rot="R90"/>
@@
 <element name="C50" library="OPL" package="C0603" value="100nF" x="44.1325" y="41.5925" rot="R180"/>
 <element name="C42" library="OPL" package="C0603" value="100nF" x="48.26" y="49.8475" rot="R90"/>
-<element name="R149" library="OPL" package="R0603" value="100k" x="39.37" y="45.4025" rot="R270"/>
-<element name="R147" library="OPL" package="R0603" value="100k" x="47.3075" y="41.5925" rot="R180"/>
+<element name="R149" library="OPL" package="R0603" value="100K" x="39.37" y="45.4025" rot="R270"/>
+<element name="R147" library="OPL" package="R0603" value="100K" x="47.3075" y="41.5925" rot="R180"/>
 <element name="U2" library="FarnellThings" package="SOT95P237X112-3N" value="LM4040DIM3-5.0" x="54.61" y="46.0375">
 <attribute name="MPN" value="LM4040DIM3-5.0" x="40.005" y="35.2425" size="1.778" layer="27" display="off"/>
