File: Development/Eurorack Set 10/TheRug-Andabil-R2.brd (EAGLE design)
At the start: 59.6 x 106.5 mm, 166 parts, among them IC1 TL072TSSOP8, IC10 TL072TSSOP8, IC12 TL072, IC2 TL072TSSOP8, IC3 TL072TSSOP8, IC5 TL074TSSOP14, IC6 TL074TSSOP14, IC7 TL072TSSOP8, IC8 TL072TSSOP8, IC9 TL072TSSOP8, J1 POWERSHROUDED, Q1 MMBT3906LT1SMD, Q2 MMBT3906LT1SMD, U1 LM13700M, U2 LM4040DIM3-5.0

Commit message: Ardabil progress
Parts:
- removed C21, C22, C25, C26, C27, C28, C35, C36, C5, C6: 100nF, OPL:C0603
- removed IC1, IC10, IC7, IC8, IC9: TL072TSSOP8, EurorackModularParts:TSSOP8
- added C23, C24, C37, C38: 100nF, OPL:C0603
- added IC11, IC4: TL074TSSOP14, EurorackModularParts:TSSOP14
- added S1, S2: ONOFFONNOHOLES, EurorackModularParts:MULTICOMP1MS-ONOFFON_NOHOLES
- IC12: value TL072 -> TL072TSSOP8; device EurorackModularParts:SO08 -> EurorackModularParts:TSSOP8
- IC2, IC3: value TL072TSSOP8 -> TL074TSSOP14; device EurorackModularParts:TSSOP8 -> EurorackModularParts:TSSOP14
- U$12, U$13, U$14, U$15, U$16, U$2, U$25, U$28, U$6, U$9: device EurorackModularParts:3.5MM-JACK-SWITCH-13MM-INPUT -> EurorackModularParts:3.5MM-JACK-SWITCH-13MM-NOHOLES
- U$17, U$18, U$19, U$20, U$26, U$27, U$3, U$30, U$4, U$5: device EurorackModularParts:3.5MM-JACK-SWITCH-13MM-OUTPUT -> EurorackModularParts:3.5MM-JACK-SWITCH-13MM-NOHOLES
- moved R57 190.8 mm to (-26.7, 30.5), turned to 0 degrees
- moved R58 189.9 mm to (-22.9, 15.9), turned to 180 degrees
- moved C31 189.8 mm to (-22.9, 14.6), turned to 0 degrees
- moved C42 189.4 mm to (-30.2, 9.53), turned to 180 degrees
- moved C4 189.3 mm to (-30.5, 25.4), turned to 180 degrees
- moved R60 188.6 mm to (-22.9, 13.3), turned to 0 degrees
- moved R50 187.2 mm to (-22.9, 21.6), turned to 0 degrees
- moved C29 186.0 mm to (-22.9, 20.3), turned to 0 degrees
- moved R61 183.2 mm to (-26.7, 13.3), turned to 180 degrees
- moved C32 181.7 mm to (-26.7, 14.6), turned to 180 degrees
- moved R59 180.4 mm to (-26.7, 15.9), turned to 0 degrees
- moved R69 179.8 mm to (-26.7, 17.1), turned to 0 degrees
- moved R68 175.9 mm to (-22.9, 29.2), turned to 180 degrees
- moved C34 174.6 mm to (-22.9, 30.5), turned to 0 degrees
- moved R71 172.7 mm to (-26.7, 29.2), turned to 180 degrees
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Connections:
- new net N$40: IC2.12, IC2.13, IC2.14
- new net N$42: IC3.12, IC3.13, IC3.14
- net -12V: now also C24.1, C38.1, IC11.11, IC2.11, IC3.11, IC4.11; no longer C22.1, C26.1, C28.1, C36.1, C6.1, IC1.4, IC10.4, IC2.4, IC3.4, IC7.4, IC8.4, IC9.4
- net 12V: now also C23.2, C37.2, IC11.4, IC2.4, IC3.4, IC4.4; no longer C21.2, C25.2, C27.2, C35.2, C5.2, IC1.8, IC10.8, IC2.8, IC3.8, IC7.8, IC8.8, IC9.8
- net GND: now also C23.1, C24.2, C37.1, C38.2, IC11.10, IC11.12, IC11.3, IC11.5, IC4.10, IC4.12, IC4.3, IC4.5, U$12.RING_B@1, U$12.RING_T@3, U$12.SWITCH_B@1, U$12.SWITCH_T@3, U$13.RING_B@1, U$13.RING_T@3, U$13.SWITCH_B@1, U$13.SWITCH_T@3, U$14.RING_B@1, U$14.RING_T@3, U$15.RING_B@1, U$15.RING_T@3, U$15.SWITCH_B@1, U$15.SWITCH_T@3, U$16.RING_B@1, U$16.RING_T@3, U$17.RING_B@1, U$17.RING_T@3, U$18.RING_B@1, U$18.RING_T@3, U$19.RING_B@1, U$19.RING_T@3, U$2.RING_B@1, U$2.RING_T@3, U$2.SWITCH_B@1, U$2.SWITCH_T@3, U$20.RING_B@1, U$20.RING_T@3, U$25.RING_B@1, U$25.RING_T@3, U$25.SWITCH_B@1, U$25.SWITCH_T@3, U$26.RING_B@1, U$26.RING_T@3, U$27.RING_B@1, U$27.RING_T@3, U$28.RING_B@1, U$28.RING_T@3, U$28.SWITCH_B@1, U$28.SWITCH_T@3, U$3.RING_B@1, U$3.RING_T@3, U$30.RING_B@1, U$30.RING_T@3, U$4.RING_B@1, U$4.RING_T@3, U$5.RING_B@1, U$5.RING_T@3, U$6.RING_B@1, U$6.RING_T@3, U$6.SWITCH_B@1, U$6.SWITCH_T@3, U$9.RING_B@1, U$9.RING_T@3, U$9.SWITCH_B@1, U$9.SWITCH_T@3; no longer C21.1, C22.2, C25.1, C26.2, C27.1, C28.2, C35.1, C36.2, C5.1, C6.2, IC1.3, IC1.5, IC7.3, IC7.5, IC8.3, IC8.5, IC9.3, IC9.5, U$12.RING@3, U$12.SWITCH@3, U$13.RING@3, U$13.SWITCH@3, U$14.RING@3, U$15.RING@3, U$15.SWITCH@3, U$16.RING@3, U$17.RING@3, U$18.RING@3, U$19.RING@3, U$2.RING@3, U$2.SWITCH@3, U$20.RING@3, U$25.RING@3, U$25.SWITCH@3, U$26.RING@3, U$27.RING@3, U$28.RING@3, U$28.SWITCH@3, U$3.RING@3, U$30.RING@3, U$4.RING@3, U$5.RING@3, U$6.RING@3, U$6.SWITCH@3, U$9.RING@3, U$9.SWITCH@3
- net N$1: now also IC2.10; no longer IC10.5
- net N$10: now also IC2.9; no longer IC10.6
- net N$11: now also IC4.7; no longer IC2.1
- net N$12: now also U$13.TIP_B@1, U$13.TIP_T@3; no longer U$13.TIP@3
- net N$14: now also IC2.2; no longer IC1.2
- net N$15: now also U$3.TIP_B@1, U$3.TIP_T@3; no longer U$3.TIP@3
- net N$16: now also U$5.TIP_B@1, U$5.TIP_T@3; no longer U$5.TIP@3
- net N$17: now also IC4.13; no longer IC3.6
- net N$18: now also IC4.14; no longer IC3.7
- net N$19: now also U$17.TIP_B@1, U$17.TIP_T@3; no longer U$17.TIP@3
- net N$2: now also IC4.1; no longer IC3.1
- net N$20: now also U$2.TIP_B@1, U$2.TIP_T@3; no longer U$2.TIP@3
- net N$22: now also U$4.TIP_B@1, U$4.TIP_T@3; no longer U$4.TIP@3
- net N$24: now also IC2.7; no longer IC1.7
- net N$25: now also IC2.6; no longer IC1.6
- net N$26: now also U$18.TIP_B@1, U$18.TIP_T@3; no longer U$18.TIP@3
- net N$3: now also IC2.8; no longer IC10.7
- net N$31: now also U$19.TIP_B@1, U$19.TIP_T@3; no longer U$19.TIP@3
- net N$37: now also U$12.TIP_B@1, U$12.TIP_T@3; no longer U$12.TIP@3
- net N$38: now also U$15.TIP_B@1, U$15.TIP_T@3; no longer U$15.TIP@3
- net N$4: now also U$6.TIP_B@1, U$6.TIP_T@3; no longer U$6.TIP@3
- net N$47: now also U$16.TIP_B@1, U$16.TIP_T@3; no longer U$16.TIP@3
- net N$48: now also U$14.TIP_B@1, U$14.TIP_T@3; no longer U$14.TIP@3
- net N$5: now also IC4.6; no longer IC2.2
- net N$53: now also IC11.1; no longer IC9.1
- net N$63: now also U$25.TIP_B@1, U$25.TIP_T@3; no longer U$25.TIP@3
- net N$65: now also IC3.2; no longer IC7.2
- net N$66: now also U$20.TIP_B@1, U$20.TIP_T@3; no longer U$20.TIP@3
- net N$67: now also IC3.1; no longer IC7.1
- net N$68: now also IC11.2; no longer IC9.2
- net N$69: now also U$9.TIP_B@1, U$9.TIP_T@3; no longer U$9.TIP@3
- net N$7: now also IC2.1; no longer IC1.1
- net N$70: now also U$28.TIP_B@1, U$28.TIP_T@3; no longer U$28.TIP@3
- net N$71: now also IC11.6; no longer IC8.2
- net N$72: now also IC11.9; no longer IC8.6
- net N$73: now also IC11.7; no longer IC8.1
- net N$75: now also U$26.TIP_B@1, U$26.TIP_T@3; no longer U$26.TIP@3
- net N$76: now also U$27.TIP_B@1, U$27.TIP_T@3; no longer U$27.TIP@3
- net N$77: now also IC11.13; no longer IC9.6
- net N$78: now also IC11.14; no longer IC9.7
- net N$79: now also U$30.TIP_B@1, U$30.TIP_T@3; no longer U$30.TIP@3
- net N$8: now also IC4.2; no longer IC3.2
- net N$81: now also IC3.7; no longer IC7.7
- net N$82: now also IC3.6; no longer IC7.6
- net N$84: now also IC3.10; no longer IC10.3
- net N$85: now also IC3.8; no longer IC10.1
- net N$86: now also IC3.9; no longer IC10.2
- net N$9: now also IC4.9; no longer IC2.6
- net OUTPUT1_SUM_TO_VCA1: now also IC4.8, U$14.SWITCH_B@1, U$14.SWITCH_T@3; no longer IC2.7, U$14.SWITCH@3
- net OUTPUT2_SUM_TO_VCA2: now also IC11.8, U$16.SWITCH_B@1, U$16.SWITCH_T@3; no longer IC8.7, U$16.SWITCH@3
Other:
- board size 59.6 x 106.5 mm -> 60.2 x 106.5 mm

Commit message: Nein & Ardabil
Parts:
- removed C14, C34: 22pf, OPL:C0603
- removed C19, C20, C42, C50: 100nF, OPL:C0603
- removed D3, D4: BAS16W, FenixBase:SOT-323
- removed IC12: TL072TSSOP8, EurorackModularParts:TSSOP8
- removed IC6: TL074TSSOP14, EurorackModularParts:TSSOP14
- removed Q1, Q2: MMBT3906LT1SMD, transistor-pnp:SOT23-BEC
- removed R18, R21, R67, R70: 1k, OPL:R0603
- removed R19, R20, R42, R49, R69, R73, R74: 100K, OPL:R0603
- removed R38: 249K, OPL:R0603
- removed R39, R41: 499, OPL:R0603
- removed R43, R44, R46, R48: 2K, OPL:R0603
- removed R45, R47: 200, OPL:R0603
- removed R75, R76, R77, R78: 100k, EurorackModularParts:TRIMPOT
- removed S1, S2: ONOFFONNOHOLES, EurorackModularParts:MULTICOMP1MS-ONOFFON_NOHOLES
- removed U1: LM13700M, FarnellThings:SOIC127P620X175-16N
- added C21, C22, C5, C6: 100n, OPL:C0603
- added C25, C26: 33p, OPL:C0603
- added C27, C28: 100p, OPL:C0603
- added C35, C36, C39, C40: 560p, OPL:C0603
- added IC1: TL074TSSOP14, EurorackModularParts:TSSOP14
- added R79, R81, R83, R84, R88, R95: 30k, OPL:R0603
- added R80, R82: 100, OPL:R0603
- added R85, R86, R91, R93: 100k, OPL:R0603
- added R87: 7.5k, OPL:R0603
- added R89, R92, R94, R96: 500, OPL:R0603
- added U$32: V2164, EurorackModularParts:SO16
- C15, C18: value 100nF -> 33p
- C16, C17: value 100nF -> 100n
- IC5: value TL074TSSOP14 -> TL072TSSOP8; device EurorackModularParts:TSSOP14 -> EurorackModularParts:TSSOP8
- R24, R26: value 49.9K -> 51k
- R25: value 499 -> 51k
- R27, R28: value 100K -> 51k
- R29, R30, R32, R33: value 220K -> 51k
- R31: value 249K -> 51k
- R34, R36: value 30.1K -> 100k
- R35, R37: value 100 -> 100k
- R40: value 499 -> 1.2K
- R68: value 100K -> 1.2K
- moved R30 149.1 mm to (-11.4, 93.5), turned to 90 degrees
- moved R40 141.2 mm to (-18.8, 33.0)
- moved R26 139.1 mm to (5.59, 83.1), turned to 0 degrees
- moved R36 137.1 mm to (20.6, 93.6), turned to 180 degrees
- moved R28 135.2 mm to (17.3, 86.9), turned to 180 degrees
- moved R32 131.1 mm to (1.52, 33.0), turned to 90 degrees
- moved R24 129.5 mm to (5.08, 86.9), turned to 180 degrees
- moved R27 128.7 mm to (17.3, 83.8), turned to 180 degrees
- moved C38 127.8 mm to (-5.08, 11.2), turned to 180 degrees
- moved C15 127.3 mm to (-5.08, 4.06), turned to 90 degrees
- moved IC5 122.1 mm to (0.51, 2.54), turned to 270 degrees
- moved R34 120.6 mm to (-19.1, 9.40)
- moved R2 120.2 mm to (-18.2, 84.6), turned to 90 degrees
- moved R22 117.6 mm to (-16.9, 84.6), turned to 270 degrees
- moved R33 115.8 mm to (4.83, 33.0), turned to 90 degrees
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Connections:
- removed net CV_IN_A: Q1.C, U1.16
- removed net CV_IN_B: Q2.C, U1.1
- removed net N$21: D_1POS.+, R21.1
- removed net N$23: D_1NEG.-, R18.1
- removed net N$24: C14.2, IC2.7, R18.2, R19.1, R21.2
- removed net N$25: C14.1, IC2.6, R19.2, R20.2
- removed net N$42: IC3.12, IC3.13, IC3.14
- removed net N$43: R25.2, R26.2, U1.13
- removed net N$46: R30.2, R41.2, U1.3
- removed net N$47: R49.1, U$16.TIP_B@1, U$16.TIP_T@3
- removed net N$48: R42.1, U$14.TIP_B@1, U$14.TIP_T@3
- removed net N$49: IC6.2, R73.2, R74.1
- removed net N$50: IC5.9, R42.2, R43.1
- removed net N$51: IC5.5, IC5.8, R43.2
- removed net N$52: D3.CATHODE, IC5.6, R32.2, R44.1
- removed net N$55: D3.ANODE, IC5.7, Q1.B
- removed net N$56: Q1.E, R44.2, R45.1
- removed net N$57: D4.CATHODE, IC6.6, R29.2, R46.1
- removed net N$58: D4.ANODE, IC6.7, Q2.B
- removed net N$59: Q2.E, R46.2, R47.1
- removed net N$60: IC6.5, IC6.8, R48.2
- removed net N$62: IC6.9, R48.1, R49.2
- removed net N$75: R62.2, U$26.TIP_B@1, U$26.TIP_T@3
- removed net N$79: R66.2, U$30.TIP_B@1, U$30.TIP_T@3
- removed net N$82: C34.1, IC3.6, R68.2, R69.2
- removed net N$83: D_2POS.+, R70.1
- removed net TRANS_OUT_A: IC5.13, R36.1, U1.12
- removed net TRANS_OUT_B: IC6.13, R34.1, U1.5
- new net N$100: C40.2, R95.2, U$32.10
- new net N$61: C25.2, IC1.8, R80.2
- new net N$74: C25.1, IC1.9, R79.2, U$32.12
- new net N$87: C26.2, IC1.14, R82.2
- new net N$88: C26.1, IC1.13, R81.2, U$32.4
- new net N$89: C27.2, IC1.1, U$32.3, U$32.6
- new net N$90: C28.1, IC1.6, R86.2, U$32.13
- new net N$91: C28.2, IC1.7, U$32.11, U$32.14
- new net N$92: R87.1, U$32.1
- new net N$93: C35.1, R89.2
- new net N$94: C35.2, R88.2, U$32.2
- new net N$95: C36.2, R91.1, U$32.7
- new net N$96: C36.1, R92.2
- new net N$97: C39.2, R93.1, U$32.15
- new net N$98: C39.1, R94.2
- new net N$99: C40.1, R96.2
- new net VCA1_CV: R85.1, U$14.TIP_B@1, U$14.TIP_T@3
- new net VCA1_FB: C27.1, IC1.2, R85.2, U$32.5
- new net VCA1_IN: R34.1, U$12.TIP_B@1, U$12.TIP_T@3
- new net VCA1_OUT: R81.1, R82.1, U$18.TIP_B@1, U$18.TIP_T@3
- new net VCA1_SUMIN: IC1.12, R84.1
- new net VCA2_CV: R86.1, U$16.TIP_B@1, U$16.TIP_T@3
- new net VCA2_IN: R36.1, U$15.TIP_B@1, U$15.TIP_T@3
- new net VCA2_OUT: R79.1, R80.1, U$19.TIP_B@1, U$19.TIP_T@3
- new net VCA2_SUMIN: IC1.10, R83.1
- net -12V: now also C16.2, C22.1, C6.1, IC1.11, IC5.4, U$32.9; no longer C16.1, C18.1, C20.2, C42.1, IC12.4, IC5.11, IC6.11, U1.6
- net -5V: now also IC2.13, IC2.14, R91.2, R93.2; no longer IC12.1, IC12.2, R75.P$1, R76.P$1, R77.P$1, R78.P$1
- net -5VIN: now also IC2.12; no longer IC12.3
- net -5V_TO_5V: now also IC3.13; no longer IC12.6
- net 12V: now also C17.1, C21.2, C5.2, IC1.4, IC5.8, R87.2, U$32.16; no longer C15.2, C17.2, C19.1, C50.2, IC12.8, IC5.4, IC6.4, R31.1, R38.1, U1.11
- net 5V: now also IC3.14; no longer IC12.7, R75.P$3, R76.P$3, R77.P$3, R78.P$3
- net GND: now also C16.1, C17.2, C21.1, C22.2, C5.1, C6.2, IC1.3, IC1.5, IC3.12, IC5.5, R24.2, R25.2, R26.1, R27.1, R28.1, R29.2, R30.2, R31.1, R32.1, R33.1, R40.2, R68.2, R83.2, R84.2, R89.1, R92.1, R94.1, R96.1, U$32.8; no longer C15.1, C16.2, C17.1, C18.2, C19.2, C20.1, C42.2, C50.1, D_1NEG.+, D_1POS.-, D_2NEG.+, D_2POS.-, IC11.10, IC11.12, IC11.3, IC11.5, IC12.5, IC2.3, IC2.5, IC3.3, IC3.5, IC4.10, IC4.12, IC4.3, IC4.5, IC5.10, IC5.12, IC6.10, IC6.12, IC6.3, R25.1, R39.1, R40.1, R41.1, R45.2, R47.2
- net N$11: no longer R8.2
- net N$13: now also R60.2, R62.2, U$26.TIP_B@1, U$26.TIP_T@3; no longer IC6.1, R24.1, R73.1
- net N$15: now also R8.2
- net N$16: now also R9.2
- net N$18: no longer R16.1
- net N$19: now also R16.1
- net N$2: no longer R12.2
- net N$22: now also R12.2
- net N$26: now also IC11.3, R24.1; no longer R37.2, U$18.TIP_B@1, U$18.TIP_T@3
- net N$27: now also IC3.3, R25.1; no longer IC5.14, R36.2, R37.1
- net N$29: now also IC11.5, R26.2; no longer R31.2, U1.2
- net N$30: now also IC11.10, R27.2; no longer R38.2, U1.15
- net N$31: now also R65.1, R66.2, U$30.TIP_B@1, U$30.TIP_T@3; no longer R35.2, U$19.TIP_B@1, U$19.TIP_T@3
- net N$32: now also IC11.12, R28.2; no longer IC6.14, R34.2, R35.1
- net N$33: now also IC4.3, R29.1; no longer R33.1, R75.P$2
- net N$34: now also IC2.3, R30.1; no longer R32.1, R77.P$2
- net N$35: now also IC4.5, R31.2; no longer R30.1, R76.P$2
- net N$36: now also IC4.10, R32.2; no longer R29.1, R78.P$2
- net N$37: now also IC4.12, R33.2; no longer R27.2, U$12.TIP_B@1, U$12.TIP_T@3
- net N$38: now also C15.1, IC5.2, R34.2, R35.1; no longer R74.2, U$15.TIP_B@1, U$15.TIP_T@3
- net N$39: now also C15.2, IC5.1, R35.2, R88.1; no longer IC5.2, R27.1, R28.2
- net N$40: now also C18.1, IC5.6, R36.2, R37.1; no longer IC2.12, IC2.13, IC2.14
- net N$41: now also C18.2, IC5.7, R37.2, R95.1; no longer IC5.1, R26.1, R28.1
- net N$44: now also D_1NEG.-, D_1POS.+, IC2.6, R40.1; no longer R24.2, R39.2, U1.4
- net N$45: now also D_1NEG.+, D_1POS.-, IC2.7; no longer R33.2, R40.2, U1.14
- net N$53: no longer R56.2
- net N$66: now also R56.2
- net N$67: now also IC3.5; no longer R69.1
- net N$7: now also IC2.5; no longer R20.1
- net N$73: no longer R60.2
- net N$76: now also R61.2
- net N$78: no longer R65.1
- net N$80: now also D_2POS.+, IC3.6, R68.1; no longer R67.1
- net N$81: now also D_2NEG.+, D_2POS.-; no longer C34.2, R67.2, R68.1, R70.2
- net OUTPUT1_SUM_TO_VCA1: no longer R9.2
- net OUTPUT2_SUM_TO_VCA2: no longer R61.2
Routing:
- net VCA2_CV: track 0.00 -> 84.4 mm, vias 0 -> 2
- net -12V: track 0.00 -> 82.3 mm
- net 12V: track 0.00 -> 50.9 mm
- net GND: track 0.00 -> 50.6 mm, vias 0 -> 39
- net 5V: track 0.00 -> 48.9 mm
- net N$39: track 0.00 -> 45.8 mm
- net N$67: track 0.00 -> 45.7 mm
- net -5VIN: track 0.00 -> 40.7 mm
- net N$6: track 0.00 -> 38.5 mm
- net N$76: track 0.00 -> 29.7 mm
- net N$65: track 0.00 -> 28.7 mm
- net N$16: track 0.00 -> 27.8 mm
- net VCA1_CV: track 0.00 -> 24.3 mm
- net OUTPUT2_SUM_TO_VCA2: track 0.00 -> 24.2 mm
- net N$38: track 0.00 -> 23.2 mm
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
Commit message: Ardabil update
Parts:
- moved R68 55.7 mm to (3.43, 76.1), turned to 180 degrees
- moved R91 14.4 mm to (-19.3, 22.4), turned to 90 degrees
- moved R36 7.38 mm to (27.9, 93.1), turned to 0 degrees
- moved R15 1.70 mm to (9.91, 39.1), turned to 90 degrees
- moved C17 0.89 mm to (5.08, 5.21)
- moved R14 0.76 mm to (-2.03, 34.3)
- moved R34 0.76 mm to (-19.1, 8.64)
- moved C24 0.76 mm to (3.05, 33.8)
- moved R32 0.76 mm to (1.52, 33.8)
- moved R33 0.76 mm to (4.83, 33.8)
- moved R85 0.72 mm to (-9.14, 13.2)
- moved C10 0.63 mm to (-1.02, 37.0)
- moved R9 0.63 mm to (-2.54, 37.0)
- moved R7 0.25 mm to (-5.21, 37.0)
Connections:
- net N$44: now also IC3.6; no longer IC2.6
- net N$45: now also IC3.7; no longer IC2.7
- net N$67: now also IC2.5; no longer IC3.5
- net N$7: now also IC3.5; no longer IC2.5
- net N$80: now also IC2.6; no longer IC3.6
- net N$81: now also IC2.7; no longer IC3.7
Routing:
- net 12V: track 50.9 -> 217.0 mm, vias 0 -> 16
- net VCA2_OUT: track 1.88 -> 161.2 mm, vias 0 -> 10
- net -5V: track 6.56 -> 162.0 mm, vias 0 -> 10
- net -12V: track 82.3 -> 207.2 mm, vias 0 -> 12
- net -5V_TO_5V: track 4.85 -> 103.5 mm, vias 0 -> 2
- net N$40: track 19.0 -> 115.5 mm, vias 0 -> 2
- net N$7: track 19.0 -> 103.5 mm, vias 0 -> 10
- net N$67: track 45.7 -> 109.9 mm, vias 0 -> 4
- net N$66: track 1.88 -> 63.6 mm, vias 0 -> 6
- net OUTPUT1_SUM_TO_VCA1: track 5.08 -> 66.0 mm, vias 0 -> 5
- net N$88: track 3.74 -> 50.7 mm
- net N$22: track 1.88 -> 47.7 mm, vias 0 -> 4
- net 5V: track 48.9 -> 93.5 mm, vias 0 -> 4
- net N$13: track 2.16 -> 43.7 mm, vias 0 -> 4
- net N$81: track 9.96 -> 47.8 mm
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
Commit message: some production files
Connections:
- net GND: now also U$31.P$1, U$7.P$1; no longer U$31.P$3, U$7.P$3
- net N$4: now also U$7.P$3; no longer U$7.P$1
- net N$70: now also U$31.P$3; no longer U$31.P$1
Routing:
- net N$4: track 30.7 -> 37.2 mm
- net N$70: track 50.6 -> 56.7 mm, vias 5 -> 6
- net N$45: track 50.0 -> 50.5 mm
Changed lines of the file:
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@@
 <layer number="19" name="Unrouted" color="6" fill="1" visible="yes" active="yes"/>
 <layer number="20" name="Dimension" color="15" fill="1" visible="yes" active="yes"/>
-<layer number="21" name="tPlace" color="7" fill="1" visible="no" active="yes"/>
+<layer number="21" name="tPlace" color="7" fill="1" visible="yes" active="yes"/>
 <layer number="22" name="bPlace" color="7" fill="1" visible="no" active="yes"/>
 <layer number="23" name="tOrigins" color="15" fill="1" visible="yes" active="yes"/>
@@
 <contactref element="J1" pad="6"/>
 <contactref element="J1" pad="4"/>
-<contactref element="U$7" pad="P$3"/>
 <contactref element="U$12" pad="SWITCH_B@1" route="any" routetag="G$1.SWITCH"/>
 <contactref element="U$14" pad="RING_B@1" route="any" routetag="G$1.RING"/>
@@
 <contactref element="U$28" pad="RING_B@1" route="any" routetag="G$1.RING"/>
 <contactref element="U$28" pad="SWITCH_B@1" route="any" routetag="G$1.SWITCH"/>
-<contactref element="U$31" pad="P$3"/>
 <contactref element="U$20" pad="RING_B@1" route="any" routetag="G$1.RING"/>
 <contactref element="U$26" pad="RING_B@1" route="any" routetag="G$1.RING"/>
@@
 <wire x1="4.572" y1="45.974" x2="3.81" y2="45.974" width="0.2032" layer="1"/>
 <wire x1="3.81" y1="45.974" x2="3.048" y2="45.974" width="0.2032" layer="1"/>
+<contactref element="U$7" pad="P$1"/>
+<contactref element="U$31" pad="P$1"/>
 </signal>
 <signal name="12V" class="1">
@@
 <wire x1="-11.303" y1="69.85" x2="-8.763" y2="72.39" width="0.2032" layer="1"/>
 <via x="-8.763" y="72.39" extent="1-16" drill="0.3048"/>
-<wire x1="-8.763" y1="72.39" x2="-6.35" y2="74.803" width="0.2032" layer="16"/>
-<via x="-6.35" y="74.803" extent="1-16" drill="0.3048"/>
-<wire x1="-6.35" y1="74.803" x2="-5.715" y2="74.803" width="0.2032" layer="1"/>
-<wire x1="-5.715" y1="74.803" x2="-4.318" y2="76.2" width="0.2032" layer="1"/>
+<wire x1="-8.763" y1="72.39" x2="-5.969" y2="75.184" width="0.2032" layer="16"/>
+<via x="-5.969" y="75.184" extent="1-16" drill="0.3048"/>
+<wire x1="-5.969" y1="75.184" x2="-5.334" y2="75.184" width="0.2032" layer="1"/>
+<wire x1="-5.334" y1="75.184" x2="-4.318" y2="76.2" width="0.2032" layer="1"/>
 <wire x1="-4.318" y1="76.2" x2="-4.318" y2="77.851" width="0.2032" layer="1"/>
 <wire x1="-4.318" y1="77.851" x2="-10.16" y2="83.693" width="0.2032" layer="1"/>
@@
 <contactref element="U$6" pad="TIP_B@1" route="any" routetag="G$1.TIP"/>
 <contactref element="R23" pad="1"/>
-<contactref element="U$7" pad="P$1"/>
 <contactref element="U$6" pad="TIP_T@3" route="any" routetag="G$1.TIP"/>
 <wire x1="-15.24" y1="79.502" x2="-16.637" y2="79.502" width="0.2032" layer="1"/>
@@
 <wire x1="-21.59" y1="88.9" x2="-24.975" y2="88.9" width="0.2032" layer="1"/>
 <wire x1="-24.975" y1="88.9" x2="-25" y2="88.875" width="0.2032" layer="1"/>
-<wire x1="-5.625" y1="76.875" x2="-7.707" y2="76.875" width="0.2032" layer="1"/>
-<wire x1="-7.707" y1="76.875" x2="-8.255" y2="76.327" width="0.2032" layer="1"/>
 <via x="-8.255" y="76.327" extent="1-16" drill="0.3048"/>
 <wire x1="-8.255" y1="76.327" x2="-10.287" y2="74.295" width="0.2032" layer="16"/>
@@
 <wire x1="-13.589" y1="75.184" x2="-15.24" y2="76.835" width="0.2032" layer="1"/>
 <wire x1="-15.24" y1="76.835" x2="-15.24" y2="79.502" width="0.2032" layer="1"/>
+<contactref element="U$7" pad="P$3"/>
+<wire x1="-8.255" y1="76.327" x2="-6.477" y2="74.549" width="0.2032" layer="1"/>
+<wire x1="-6.477" y1="74.549" x2="-2.871" y2="74.549" width="0.2032" layer="1"/>
+<wire x1="-2.871" y1="74.549" x2="-0.545" y2="76.875" width="0.2032" layer="1"/>
 </signal>
 <signal name="N$5">
@@
 <contactref element="U$28" pad="TIP_B@1" route="any" routetag="G$1.TIP"/>
 <contactref element="R72" pad="1"/>
-<contactref element="U$31" pad="P$1"/>
 <contactref element="U$28" pad="TIP_T@3" route="any" routetag="G$1.TIP"/>
 <wire x1="13.208" y1="12.446" x2="13.208" y2="12.192" width="0.2032" layer="1"/>
@@
 <wire x1="25.019" y1="17.356" x2="25" y2="17.375" width="0.2032" layer="1"/>
 <wire x1="14.351" y1="11.049" x2="20.828" y2="11.049" width="0.2032" layer="1"/>
-<wire x1="5.625" y1="29.375" x2="7.531" y2="29.375" width="0.2032" layer="16"/>
-<wire x1="7.531" y1="29.375" x2="8.89" y2="30.734" width="0.2032" layer="16"/>
-<via x="8.89" y="30.734" extent="1-16" drill="0.3048"/>
-<wire x1="8.89" y1="30.734" x2="10.414" y2="30.734" width="0.2032" layer="1"/>
+<via x="9.144" y="30.734" extent="1-16" drill="0.3048"/>
+<wire x1="9.144" y1="30.734" x2="10.414" y2="30.734" width="0.2032" layer="1"/>
 <wire x1="10.414" y1="30.734" x2="14.224" y2="34.544" width="0.2032" layer="1"/>
 <wire x1="14.224" y1="34.544" x2="14.224" y2="34.798" width="0.2032" layer="1"/>
@@
 <wire x1="17.145" y1="30.734" x2="19.304" y2="30.734" width="0.2032" layer="1"/>
 <wire x1="19.304" y1="30.734" x2="21.844" y2="28.194" width="0.2032" layer="1"/>
-<wire x1="21.844" y1="28.194" x2="21.844" y2="27.178" width="0.2032" layer="1"/>
-<wire x1="21.844" y1="27.178" x2="21.844" y2="24.511" width="0.2032" layer="1"/>
+<wire x1="21.844" y1="28.194" x2="21.844" y2="24.511" width="0.2032" layer="1"/>
 <wire x1="21.844" y1="24.511" x2="23.114" y2="23.241" width="0.2032" layer="1"/>
 <wire x1="23.114" y1="23.241" x2="23.114" y2="21.844" width="0.2032" layer="1"/>
@@
 <wire x1="25.019" y1="19.939" x2="25.019" y2="17.394" width="0.2032" layer="1"/>
 <wire x1="25.019" y1="17.394" x2="25" y2="17.375" width="0.2032" layer="1"/>
+<contactref element="U$31" pad="P$3"/>
+<wire x1="0.545" y1="29.375" x2="0.546" y2="29.375" width="0.2032" layer="1"/>
+<wire x1="0.546" y1="29.375" x2="1.778" y2="30.607" width="0.2032" layer="1"/>
+<wire x1="1.778" y1="30.607" x2="6.045" y2="30.607" width="0.2032" layer="1"/>
+<wire x1="6.045" y1="30.607" x2="7.277" y2="29.375" width="0.2032" layer="1"/>
+<via x="7.277" y="29.375" extent="1-16" drill="0.3048"/>
+<wire x1="7.277" y1="29.375" x2="8.5725" y2="30.6705" width="0.2032" layer="16"/>
+<wire x1="8.5725" y1="30.6705" x2="9.0805" y2="30.6705" width="0.2032" layer="16"/>
+<wire x1="9.0805" y1="30.6705" x2="9.144" y2="30.734" width="0.2032" layer="16"/>
 </signal>
 <signal name="N$71">
@@
 <wire x1="-10.541" y1="30.988" x2="-10.033" y2="30.48" width="0.2032" layer="1"/>
 <wire x1="-10.033" y1="30.48" x2="-2.921" y2="30.48" width="0.2032" layer="1"/>
-<wire x1="-2.921" y1="30.48" x2="-2.159" y2="31.242" width="0.2032" layer="1"/>
-<wire x1="-2.159" y1="31.242" x2="7.239" y2="31.242" width="0.2032" layer="1"/>
+<wire x1="-2.921" y1="30.48" x2="-1.905" y2="31.496" width="0.2032" layer="1"/>
+<wire x1="-1.905" y1="31.496" x2="7.366" y2="31.496" width="0.2032" layer="1"/>
 <via x="12.573" y="29.464" extent="1-16" drill="0.3048"/>
 <wire x1="12.573" y1="29.464" x2="13.432" y2="28.605" width="0.2032" layer="1"/>
 <wire x1="13.432" y1="28.605" x2="13.432" y2="22.2218" width="0.2032" layer="1"/>
-<wire x1="7.239" y1="31.242" x2="9.017" y2="29.464" width="0.2032" layer="1"/>
-<wire x1="9.017" y1="29.464" x2="9.398" y2="29.464" width="0.2032" layer="1"/>
+<wire x1="7.366" y1="31.496" x2="9.398" y2="29.464" width="0.2032" layer="1"/>
 <via x="9.398" y="29.464" extent="1-16" drill="0.3048"/>
 <wire x1="9.398" y1="29.464" x2="12.573" y2="29.464" width="0.2032" layer="16"/>
@@
 <wire x1="-11.2065" y1="29.6875" x2="-10.922" y2="29.972" width="0.2032" layer="1"/>
 <wire x1="-10.922" y1="29.972" x2="-2.667" y2="29.972" width="0.2032" layer="1"/>
-<wire x1="-2.667" y1="29.972" x2="-1.905" y2="30.734" width="0.2032" layer="1"/>
-<wire x1="-1.905" y1="30.734" x2="6.35" y2="30.734" width="0.2032" layer="1"/>
-<wire x1="6.35" y1="30.734" x2="9.017" y2="28.067" width="0.2032" layer="1"/>
-<via x="9.017" y="28.067" extent="1-16" drill="0.3048"/>
-<wire x1="9.017" y1="28.067" x2="9.398" y2="27.686" width="0.2032" layer="16"/>
+<wire x1="-2.667" y1="29.972" x2="-1.651" y2="30.988" width="0.2032" layer="1"/>
+<wire x1="-1.651" y1="30.988" x2="6.604" y2="30.988" width="0.2032" layer="1"/>
+<wire x1="6.604" y1="30.988" x2="8.763" y2="28.829" width="0.2032" layer="1"/>
+<wire x1="8.763" y1="28.829" x2="8.763" y2="28.321" width="0.2032" layer="1"/>
+<via x="8.763" y="28.321" extent="1-16" drill="0.3048"/>
+<wire x1="8.763" y1="28.321" x2="9.398" y2="27.686" width="0.2032" layer="16"/>
 <wire x1="9.398" y1="27.686" x2="12.192" y2="27.686" width="0.2032" layer="16"/>
 <via x="12.192" y="27.686" extent="1-16" drill="0.3048"/>
