File: Development/Eurorack Set 10/TheRug-Andabil-R2.sch (EAGLE design)
At the start: 166 parts, among them IC1 TL072TSSOP8, IC10 TL072TSSOP8, IC12 TL072, IC2 TL072TSSOP8, IC3 TL072TSSOP8, IC5 TL074TSSOP14, IC6 TL074TSSOP14, IC7 TL072TSSOP8, IC8 TL072TSSOP8, IC9 TL072TSSOP8, J1 POWERSHROUDED, Q1 MMBT3906LT1SMD, Q2 MMBT3906LT1SMD, U1 LM13700M, U2 LM4040DIM3-5.0

Commit message: Ardabil progress
Parts:
- removed C21, C22, C25, C26, C27, C28, C35, C36, C5, C6: 100nF, OPL:C-0603
- removed IC1, IC10, IC7, IC8, IC9: TL072TSSOP8, EurorackModularParts:TL072TSSOP8
- added C23, C24, C37, C38: 100nF, OPL:C-0603
- added IC11, IC4: TL074TSSOP14, EurorackModularParts:TL074TSSOP14
- added S1, S2: ONOFFONNOHOLES, EurorackModularParts:ONOFFONNOHOLES
- IC12: value TL072 -> TL072TSSOP8; device EurorackModularParts:TL072 -> EurorackModularParts:TL072TSSOP8
- IC2, IC3: value TL072TSSOP8 -> TL074TSSOP14; device EurorackModularParts:TL072TSSOP8 -> EurorackModularParts:TL074TSSOP14
- U$12: device EurorackModularParts:AUDIO-JACKINPUT -> EurorackModularParts:AUDIO-JACKNODRILL; DESC Input VCA1 -> (none)
- U$13: device EurorackModularParts:AUDIO-JACKINPUT -> EurorackModularParts:AUDIO-JACKNODRILL; DESC Input 1B -> 1: B
- U$14: device EurorackModularParts:AUDIO-JACKINPUT -> EurorackModularParts:AUDIO-JACKNODRILL; DESC Input VCA1 CV -> (none)
- U$15: device EurorackModularParts:AUDIO-JACKINPUT -> EurorackModularParts:AUDIO-JACKNODRILL; DESC Input VCA2 -> (none)
- U$16: device EurorackModularParts:AUDIO-JACKINPUT -> EurorackModularParts:AUDIO-JACKNODRILL; DESC Input VCA2 CV -> (none)
- U$17: device EurorackModularParts:AUDIO-JACKOUTPUT -> EurorackModularParts:AUDIO-JACKNODRILL; DESC Output 1inv -> 1: Inverted
- U$18: device EurorackModularParts:AUDIO-JACKOUTPUT -> EurorackModularParts:AUDIO-JACKNODRILL; DESC Output VCA1 -> (none)
- U$19: device EurorackModularParts:AUDIO-JACKOUTPUT -> EurorackModularParts:AUDIO-JACKNODRILL; DESC Output VCA2 -> (none)
- U$2: device EurorackModularParts:AUDIO-JACKINPUT -> EurorackModularParts:AUDIO-JACKNODRILL; DESC Input 1A -> 1: A
- U$20: device EurorackModularParts:AUDIO-JACKOUTPUT -> EurorackModularParts:AUDIO-JACKNODRILL; DESC Output 2a -> 2: Out 1
- U$25: device EurorackModularParts:AUDIO-JACKINPUT -> EurorackModularParts:AUDIO-JACKNODRILL; DESC Input 2B -> (none)
- U$26: device EurorackModularParts:AUDIO-JACKOUTPUT -> EurorackModularParts:AUDIO-JACKNODRILL; DESC Output 2b -> 2: Out 2
- U$27: device EurorackModularParts:AUDIO-JACKOUTPUT -> EurorackModularParts:AUDIO-JACKNODRILL; DESC Output 2c -> 2: Out 3
- U$28: device EurorackModularParts:AUDIO-JACKINPUT -> EurorackModularParts:AUDIO-JACKNODRILL; DESC Input 2C -> (none)
- U$3: device EurorackModularParts:AUDIO-JACKOUTPUT -> EurorackModularParts:AUDIO-JACKNODRILL; DESC Output 1b -> 1: Out 2
- U$30: device EurorackModularParts:AUDIO-JACKOUTPUT -> EurorackModularParts:AUDIO-JACKNODRILL; DESC Output 2inv -> 2: Inverted
- U$4: device EurorackModularParts:AUDIO-JACKOUTPUT -> EurorackModularParts:AUDIO-JACKNODRILL; DESC Output 1a -> 1: Out 1
- U$5: device EurorackModularParts:AUDIO-JACKOUTPUT -> EurorackModularParts:AUDIO-JACKNODRILL; DESC Output 1c -> 1: Out 3
- U$6: device EurorackModularParts:AUDIO-JACKINPUT -> EurorackModularParts:AUDIO-JACKNODRILL; DESC Input 1C -> 1: C
- U$7: DESC Amp 1 -> 1: C Amp
- U$8: DESC Offset 1 -> 1: Offset
- U$9: device EurorackModularParts:AUDIO-JACKINPUT -> EurorackModularParts:AUDIO-JACKNODRILL; DESC Input 2A -> (none)
Connections:
- new net N$40: IC2D.+IN, IC2D.-IN, IC2D.OUT
- new net N$42: IC3D.+IN, IC3D.-IN, IC3D.OUT
- net -12V: now also C24.1, C38.1, IC11P.V-, IC2P.V-, IC3P.V-, IC4P.V-; no longer C22.1, C26.1, C28.1, C36.1, C6.1, IC10VR3.V-, IC1VR3.V-, IC2VR3.V-, IC3VR3.V-, IC7VR3.V-, IC8VR3.V-, IC9VR3.V-
- net 12V: now also C23.2, C37.2, IC11P.V+, IC2P.V+, IC3P.V+, IC4P.V+; no longer C21.2, C25.2, C27.2, C35.2, C5.2, IC10VR3.V+, IC1VR3.V+, IC2VR3.V+, IC3VR3.V+, IC7VR3.V+, IC8VR3.V+, IC9VR3.V+
- net GND: now also C23.1, C24.2, C37.1, C38.2, IC11A.+IN, IC11B.+IN, IC11C.+IN, IC11D.+IN, IC2A.+IN, IC2B.+IN, IC3A.+IN, IC3B.+IN, IC4A.+IN, IC4B.+IN, IC4C.+IN, IC4D.+IN; no longer C21.1, C22.2, C25.1, C26.2, C27.1, C28.2, C35.1, C36.2, C5.1, C6.2, IC1VR1.+IN, IC1VR2.+IN, IC2VR1.+IN, IC2VR2.+IN, IC3VR1.+IN, IC3VR2.+IN, IC7VR1.+IN, IC7VR2.+IN, IC8VR1.+IN, IC8VR2.+IN, IC9VR1.+IN, IC9VR2.+IN
- net N$1: now also IC2C.+IN; no longer IC10VR2.+IN
- net N$10: now also IC2C.-IN; no longer IC10VR2.-IN
- net N$11: now also IC4B.OUT; no longer IC2VR1.OUT
- net N$14: now also IC2A.-IN; no longer IC1VR1.-IN
- net N$17: now also IC4D.-IN; no longer IC3VR2.-IN
- net N$18: now also IC4D.OUT; no longer IC3VR2.OUT
- net N$2: now also IC4A.OUT; no longer IC3VR1.OUT
- net N$24: now also IC2B.OUT; no longer IC1VR2.OUT
- net N$25: now also IC2B.-IN; no longer IC1VR2.-IN
- net N$3: now also IC2C.OUT; no longer IC10VR2.OUT
- net N$5: now also IC4B.-IN; no longer IC2VR1.-IN
- net N$53: now also IC11A.OUT; no longer IC9VR1.OUT
- net N$65: now also IC3A.-IN; no longer IC7VR1.-IN
- net N$67: now also IC3A.OUT; no longer IC7VR1.OUT
- net N$68: now also IC11A.-IN; no longer IC9VR1.-IN
- net N$7: now also IC2A.OUT; no longer IC1VR1.OUT
- net N$71: now also IC11B.-IN; no longer IC8VR1.-IN
- net N$72: now also IC11C.-IN; no longer IC8VR2.-IN
- net N$73: now also IC11B.OUT; no longer IC8VR1.OUT
- net N$77: now also IC11D.-IN; no longer IC9VR2.-IN
- net N$78: now also IC11D.OUT; no longer IC9VR2.OUT
- net N$8: now also IC4A.-IN; no longer IC3VR1.-IN
- net N$81: now also IC3B.OUT; no longer IC7VR2.OUT
- net N$82: now also IC3B.-IN; no longer IC7VR2.-IN
- net N$84: now also IC3C.+IN; no longer IC10VR1.+IN
- net N$85: now also IC3C.OUT; no longer IC10VR1.OUT
- net N$86: now also IC3C.-IN; no longer IC10VR1.-IN
- net N$9: now also IC4C.-IN; no longer IC2VR2.-IN
- net OUTPUT1_SUM_TO_VCA1: now also IC4C.OUT; no longer IC2VR2.OUT
- net OUTPUT2_SUM_TO_VCA2: now also IC11C.OUT; no longer IC8VR2.OUT
Other:
- moved on the sheet: C1, C2, C3, C4

Commit message: Nein & Ardabil
Parts:
- removed C14, C34: 22pf, OPL:C-0603
- removed C19, C20, C42, C50: 100nF, OPL:C-0603
- removed D3, D4: BAS16W, FenixBase:BAS16W
- removed IC12: TL072TSSOP8, EurorackModularParts:TL072TSSOP8
- removed IC6: TL074TSSOP14, EurorackModularParts:TL074TSSOP14
- removed Q1, Q2: MMBT3906LT1SMD, transistor-pnp:MMBT3906LT1SMD
- removed R18, R21, R67, R70: 1k, OPL:R-0603
- removed R19, R20, R42, R49, R69, R73, R74: 100K, OPL:R-0603
- removed R38: 249K, OPL:R-0603
- removed R39, R41: 499, OPL:R-0603
- removed R43, R44, R46, R48: 2K, OPL:R-0603
- removed R45, R47: 200, OPL:R-0603
- removed R75, R76, R77, R78: 100k, EurorackModularParts:TRIMPOT
- removed S1, S2: ONOFFONNOHOLES, EurorackModularParts:ONOFFONNOHOLES
- removed U1: LM13700M, FarnellThings:LM13700M
- added C21, C22, C5, C6: 100n, OPL:C-0603
- added C25, C26: 33p, OPL:C-0603
- added C27, C28: 100p, OPL:C-0603
- added C35, C36, C39, C40: 560p, OPL:C-0603
- added IC1: TL074TSSOP14, EurorackModularParts:TL074TSSOP14
- added R79, R81, R83, R84, R88, R95: 30k, OPL:R-0603
- added R80, R82: 100, OPL:R-0603
- added R85, R86, R91, R93: 100k, OPL:R-0603
- added R87: 7.5k, OPL:R-0603
- added R89, R92, R94, R96: 500, OPL:R-0603
- added U$32: V2164, EurorackModularParts:V2164
- C15, C18: value 100nF -> 33p
- C16, C17: value 100nF -> 100n
- IC5: value TL074TSSOP14 -> TL072TSSOP8; device EurorackModularParts:TL074TSSOP14 -> EurorackModularParts:TL072TSSOP8
- R24, R26: value 49.9K -> 51k
- R25: value 499 -> 51k
- R27, R28: value 100K -> 51k
- R29, R30, R32, R33: value 220K -> 51k
- R31: value 249K -> 51k
- R34, R36: value 30.1K -> 100k
- R35, R37: value 100 -> 100k
- R40: value 499 -> 1.2K
- R68: value 100K -> 1.2K
- U$12: device EurorackModularParts:AUDIO-JACKNODRILL -> EurorackModularParts:AUDIO-JACK_SMALLSYMBOLNODRILL; DESC (none) -> VCA1 In
- U$13, U$17, U$2, U$20, U$26, U$27, U$3, U$30, U$4, U$5, U$6: device EurorackModularParts:AUDIO-JACKNODRILL -> EurorackModularParts:AUDIO-JACK_SMALLSYMBOLNODRILL
- U$14: device EurorackModularParts:AUDIO-JACKNODRILL -> EurorackModularParts:AUDIO-JACK_SMALLSYMBOLNODRILL; DESC (none) -> VCA1 CV
- U$15: device EurorackModularParts:AUDIO-JACKNODRILL -> EurorackModularParts:AUDIO-JACK_SMALLSYMBOLNODRILL; DESC (none) -> VCA2 In
- U$16: device EurorackModularParts:AUDIO-JACKNODRILL -> EurorackModularParts:AUDIO-JACK_SMALLSYMBOLNODRILL; DESC (none) -> VCA2 CV
- U$18: device EurorackModularParts:AUDIO-JACKNODRILL -> EurorackModularParts:AUDIO-JACK_SMALLSYMBOLNODRILL; DESC (none) -> VCA1 Out
- U$19: device EurorackModularParts:AUDIO-JACKNODRILL -> EurorackModularParts:AUDIO-JACK_SMALLSYMBOLNODRILL; DESC (none) -> VCA2 Out
- U$25: device EurorackModularParts:AUDIO-JACKNODRILL -> EurorackModularParts:AUDIO-JACK_SMALLSYMBOLNODRILL; DESC (none) -> 2: B
- U$28: device EurorackModularParts:AUDIO-JACKNODRILL -> EurorackModularParts:AUDIO-JACK_SMALLSYMBOLNODRILL; DESC (none) -> 2: C
- U$9: device EurorackModularParts:AUDIO-JACKNODRILL -> EurorackModularParts:AUDIO-JACK_SMALLSYMBOLNODRILL; DESC (none) -> 2: A
Connections:
- removed net CV_IN_A: Q1.C, U1.AMP_BIAS_IN
- removed net CV_IN_B: Q2.C, U1.AMP_BIAS_IN_2
- removed net N$21: D_1POS.+, R21.1
- removed net N$23: D_1NEG.-, R18.1
- removed net N$24: C14.2, IC2B.OUT, R18.2, R19.1, R21.2
- removed net N$25: C14.1, IC2B.-IN, R19.2, R20.2
- removed net N$42: IC3D.+IN, IC3D.-IN, IC3D.OUT
- removed net N$43: R25.2, R26.2, U1.-IN
- removed net N$46: R30.2, R41.2, U1.+IN_2
- removed net N$47: R49.1, U$16.TIP
- removed net N$48: R42.1, U$14.TIP
- removed net N$49: IC6A.-IN, R73.2, R74.1
- removed net N$50: IC5C.-IN, R42.2, R43.1
- removed net N$51: IC5B.+IN, IC5C.OUT, R43.2
- removed net N$52: D3.CATHODE, IC5B.-IN, R32.2, R44.1
- removed net N$55: D3.ANODE, IC5B.OUT, Q1.B
- removed net N$56: Q1.E, R44.2, R45.1
- removed net N$57: D4.CATHODE, IC6B.-IN, R29.2, R46.1
- removed net N$58: D4.ANODE, IC6B.OUT, Q2.B
- removed net N$59: Q2.E, R46.2, R47.1
- removed net N$60: IC6B.+IN, IC6C.OUT, R48.2
- removed net N$62: IC6C.-IN, R48.1, R49.2
- removed net N$75: R62.2, U$26.TIP
- removed net N$79: R66.2, U$30.TIP
- removed net N$82: C34.1, IC3B.-IN, R68.2, R69.2
- removed net N$83: D_2POS.+, R70.1
- removed net TRANS_OUT_A: IC5D.-IN, R36.1, U1.OUT_2
- removed net TRANS_OUT_B: IC6D.-IN, R34.1, U1.OUT
- new net N$100: C40.2, R95.2, U$32C.IN
- new net N$61: C25.2, IC1C.OUT, R80.2
- new net N$74: C25.1, IC1C.-IN, R79.2, U$32C.OUT
- new net N$87: C26.2, IC1D.OUT, R82.2
- new net N$88: C26.1, IC1D.-IN, R81.2, U$32A.OUT
- new net N$89: C27.2, IC1A.OUT, U$32A.CV, U$32B.CV
- new net N$90: C28.1, IC1B.-IN, R86.2, U$32D.OUT
- new net N$91: C28.2, IC1B.OUT, U$32C.CV, U$32D.CV
- new net N$92: R87.1, U$32PWR.MODE
- new net N$93: C35.1, R89.2
- new net N$94: C35.2, R88.2, U$32A.IN
- new net N$95: C36.2, R91.1, U$32B.IN
- new net N$96: C36.1, R92.2
- new net N$97: C39.2, R93.1, U$32D.IN
- new net N$98: C39.1, R94.2
- new net N$99: C40.1, R96.2
- new net VCA1_CV: R85.1, U$14.TIP
- new net VCA1_FB: C27.1, IC1A.-IN, R85.2, U$32B.OUT
- new net VCA1_IN: R34.1, U$12.TIP
- new net VCA1_OUT: R81.1, R82.1, U$18.TIP
- new net VCA1_SUMIN: IC1D.+IN, R84.1
- new net VCA2_CV: R86.1, U$16.TIP
- new net VCA2_IN: R36.1, U$15.TIP
- new net VCA2_OUT: R79.1, R80.1, U$19.TIP
- new net VCA2_SUMIN: IC1C.+IN, R83.1
- net -12V: now also C16.2, C22.1, C6.1, IC1P.V-, IC5VR3.V-, U$32PWR.NEG; no longer C16.1, C18.1, C20.2, C42.1, IC12VR3.V-, IC5P.V-, IC6P.V-, U1.V-
- net -5V: now also IC2D.-IN, IC2D.OUT, R91.2, R93.2; no longer IC12VR1.-IN, IC12VR1.OUT, R75.P$1, R76.P$1, R77.P$1, R78.P$1
- net -5VIN: now also IC2D.+IN; no longer IC12VR1.+IN
- net -5V_TO_5V: now also IC3D.-IN; no longer IC12VR2.-IN
- net 12V: now also C17.1, C21.2, C5.2, IC1P.V+, IC5VR3.V+, R87.2, U$32PWR.POS; no longer C15.2, C17.2, C19.1, C50.2, IC12VR3.V+, IC5P.V+, IC6P.V+, R31.1, R38.1, U1.V+
- net 5V: now also IC3D.OUT; no longer IC12VR2.OUT, R75.P$3, R76.P$3, R77.P$3, R78.P$3
- net GND: now also C16.1, C17.2, C21.1, C22.2, C5.1, C6.2, IC1A.+IN, IC1B.+IN, IC3D.+IN, IC5VR1.+IN, IC5VR2.+IN, R24.2, R25.2, R26.1, R27.1, R28.1, R29.2, R30.2, R31.1, R32.1, R33.1, R40.2, R68.2, R83.2, R84.2, R89.1, R92.1, R94.1, R96.1, U$32PWR.GND; no longer C15.1, C16.2, C17.1, C18.2, C19.2, C20.1, C42.2, C50.1, D_1NEG.+, D_1POS.-, D_2NEG.+, D_2POS.-, IC11A.+IN, IC11B.+IN, IC11C.+IN, IC11D.+IN, IC12VR2.+IN, IC2A.+IN, IC2B.+IN, IC3A.+IN, IC3B.+IN, IC4A.+IN, IC4B.+IN, IC4C.+IN, IC4D.+IN, IC5A.+IN, IC5C.+IN, IC5D.+IN, IC6A.+IN, IC6C.+IN, IC6D.+IN, R25.1, R39.1, R40.1, R41.1, R45.2, R47.2
- net N$11: no longer R8.2
- net N$13: now also R60.2, R62.2, U$26.TIP; no longer IC6A.OUT, R24.1, R73.1
- net N$15: now also R8.2
- net N$16: now also R9.2
- net N$18: no longer R16.1
- net N$19: now also R16.1
- net N$2: no longer R12.2
- net N$22: now also R12.2
- net N$26: now also IC11A.+IN, R24.1; no longer R37.2, U$18.TIP
- net N$27: now also IC3A.+IN, R25.1; no longer IC5D.OUT, R36.2, R37.1
- net N$29: now also IC11B.+IN, R26.2; no longer R31.2, U1.DIODE_BIAS_2
- net N$30: now also IC11C.+IN, R27.2; no longer R38.2, U1.DIODE_BIAS
- net N$31: now also R65.1, R66.2, U$30.TIP; no longer R35.2, U$19.TIP
- net N$32: now also IC11D.+IN, R28.2; no longer IC6D.OUT, R34.2, R35.1
- net N$33: now also IC4A.+IN, R29.1; no longer R33.1, R75.P$2
- net N$34: now also IC2A.+IN, R30.1; no longer R32.1, R77.P$2
- net N$35: now also IC4B.+IN, R31.2; no longer R30.1, R76.P$2
- net N$36: now also IC4C.+IN, R32.2; no longer R29.1, R78.P$2
- net N$37: now also IC4D.+IN, R33.2; no longer R27.2, U$12.TIP
- net N$38: now also C15.1, IC5VR1.-IN, R34.2, R35.1; no longer R74.2, U$15.TIP
- net N$39: now also C15.2, IC5VR1.OUT, R35.2, R88.1; no longer IC5A.-IN, R27.1, R28.2
- net N$40: now also C18.1, IC5VR2.-IN, R36.2, R37.1; no longer IC2D.+IN, IC2D.-IN, IC2D.OUT
- net N$41: now also C18.2, IC5VR2.OUT, R37.2, R95.1; no longer IC5A.OUT, R26.1, R28.1
- net N$44: now also D_1NEG.-, D_1POS.+, IC2B.-IN, R40.1; no longer R24.2, R39.2, U1.-IN_2
- net N$45: now also D_1NEG.+, D_1POS.-, IC2B.OUT; no longer R33.2, R40.2, U1.+IN
- net N$53: no longer R56.2
- net N$66: now also R56.2
- net N$67: now also IC3B.+IN; no longer R69.1
- net N$7: now also IC2B.+IN; no longer R20.1
- net N$73: no longer R60.2
- net N$76: now also R61.2
- net N$78: no longer R65.1
- net N$80: now also D_2POS.+, IC3B.-IN, R68.1; no longer R67.1
- net N$81: now also D_2NEG.+, D_2POS.-; no longer C34.2, R67.2, R68.1, R70.2
- net OUTPUT1_SUM_TO_VCA1: no longer R9.2
- net OUTPUT2_SUM_TO_VCA2: no longer R61.2

Commit message: Ardabil update
Parts:
- U$29: DESC Offset 2 -> 2: Offset
- U$31: DESC Amp 2 -> 2: C Amp
Connections:
- net N$44: now also IC3B.-IN; no longer IC2B.-IN
- net N$45: now also IC3B.OUT; no longer IC2B.OUT
- net N$67: now also IC2B.+IN; no longer IC3B.+IN
- net N$7: now also IC3B.+IN; no longer IC2B.+IN
- net N$80: now also IC2B.-IN; no longer IC3B.-IN
- net N$81: now also IC2B.OUT; no longer IC3B.OUT
Other:
- moved on the sheet: IC2B, IC3B
Changed lines of the file:
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@@
 <setting verticaltext="up"/>
 </settings>
-<grid distance="0.05" unitdist="inch" unit="inch" style="lines" multiple="1" display="no" altdistance="0.01" altunitdist="inch" altunit="inch"/>
+<grid distance="0.1" unitdist="inch" unit="inch" style="lines" multiple="1" display="no" altdistance="0.01" altunitdist="inch" altunit="inch"/>
 <layers>
 <layer number="1" name="Top" color="4" fill="1" visible="no" active="no"/>
@@
 </part>
 <part name="U$29" library="EurorackModularParts" deviceset="POT" device="SQUAREHOLE_SMALLKNOB" value="10KB">
-<attribute name="DESC" value="Offset 2"/>
+<attribute name="DESC" value="2: Offset"/>
 </part>
 <part name="R57" library="OPL" deviceset="R*" device="-0603" value="49.9K"/>
@@
 <part name="R72" library="OPL" deviceset="R*" device="-0603" value="100K"/>
 <part name="U$31" library="EurorackModularParts" deviceset="POT" device="SQUAREHOLE_SMALLKNOB" value="10KB">
-<attribute name="DESC" value="Amp 2"/>
+<attribute name="DESC" value="2: C Amp"/>
 </part>
 <part name="GND50" library="SparkFun-Aesthetics" deviceset="GND" device=""/>
@@
 <instance part="IC3" gate="P" x="100.33" y="105.41"/>
 <instance part="IC2" gate="A" x="-59.69" y="205.74"/>
-<instance part="IC2" gate="B" x="8.89" y="63.5"/>
+<instance part="IC3" gate="B" x="8.89" y="63.5"/>
 <instance part="IC2" gate="C" x="-96.52" y="134.62" rot="MR180"/>
 <instance part="IC2" gate="D" x="152.4" y="-21.59"/>
 <instance part="IC3" gate="A" x="246.38" y="199.39"/>
-<instance part="IC3" gate="B" x="297.18" y="41.91"/>
+<instance part="IC2" gate="B" x="297.18" y="41.91"/>
 <instance part="IC3" gate="C" x="208.28" y="105.41" rot="MR180"/>
 <instance part="IC3" gate="D" x="207.01" y="-19.05"/>
@@
 <junction x="-52.07" y="205.74"/>
 <wire x1="-46.99" y1="66.04" x2="1.27" y2="66.04" width="0.1524" layer="91"/>
-<pinref part="IC2" gate="B" pin="+IN"/>
+<pinref part="IC3" gate="B" pin="+IN"/>
 </segment>
 </net>
@@
 <junction x="254" y="199.39"/>
 <wire x1="259.08" y1="44.45" x2="289.56" y2="44.45" width="0.1524" layer="91"/>
-<pinref part="IC3" gate="B" pin="+IN"/>
+<pinref part="IC2" gate="B" pin="+IN"/>
 </segment>
 </net>
@@
 <junction x="288.29" y="30.48"/>
 <wire x1="288.29" y1="33.02" x2="288.29" y2="39.37" width="0.1524" layer="91"/>
-<pinref part="IC3" gate="B" pin="-IN"/>
+<pinref part="IC2" gate="B" pin="-IN"/>
 <wire x1="288.29" y1="39.37" x2="289.56" y2="39.37" width="0.1524" layer="91"/>
 <junction x="288.29" y="33.02"/>
@@
 <segment>
 <wire x1="304.8" y1="41.91" x2="311.15" y2="41.91" width="0.1524" layer="91"/>
-<pinref part="IC3" gate="B" pin="OUT"/>
+<pinref part="IC2" gate="B" pin="OUT"/>
 <pinref part="D_2NEG" gate="LED" pin="+"/>
 <wire x1="302.26" y1="33.02" x2="311.15" y2="33.02" width="0.1524" layer="91"/>
@@
 <pinref part="D_1POS" gate="LED" pin="+"/>
 <wire x1="0" y1="44.45" x2="0" y2="60.96" width="0.1524" layer="91"/>
-<pinref part="IC2" gate="B" pin="-IN"/>
+<pinref part="IC3" gate="B" pin="-IN"/>
 <wire x1="0" y1="60.96" x2="1.27" y2="60.96" width="0.1524" layer="91"/>
 <junction x="0" y="44.45"/>
@@
 <pinref part="D_1NEG" gate="LED" pin="+"/>
 <pinref part="D_1POS" gate="LED" pin="-"/>
-<pinref part="IC2" gate="B" pin="OUT"/>
-</segment>
-</net>
+<pinref part="IC3" gate="B" pin="OUT"/>
+</segment>
+</net>

Commit message: some production files
Connections:
- net GND: now also U$31.E, U$7.E; no longer U$31.A, U$7.A
- net N$4: now also U$7.A; no longer U$7.E
- net N$70: now also U$31.A; no longer U$31.E
Changed lines of the file:
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@@
 <setting verticaltext="up"/>
 </settings>
-<grid distance="0.1" unitdist="inch" unit="inch" style="lines" multiple="1" display="no" altdistance="0.01" altunitdist="inch" altunit="inch"/>
+<grid distance="0.05" unitdist="inch" unit="inch" style="lines" multiple="1" display="no" altdistance="0.01" altunitdist="inch" altunit="inch"/>
 <layers>
 <layer number="1" name="Top" color="4" fill="1" visible="no" active="no"/>
@@
 <instance part="GND6" gate="1" x="-160.02" y="139.7"/>
 <instance part="GND7" gate="1" x="-129.54" y="137.16"/>
-<instance part="GND9" gate="1" x="-121.92" y="119.38"/>
+<instance part="GND9" gate="1" x="-118.11" y="139.7" rot="R90"/>
 <instance part="GND10" gate="1" x="-36.83" y="152.4"/>
 <instance part="GND12" gate="1" x="-34.29" y="114.3"/>
@@
 <instance part="GND62" gate="1" x="146.05" y="113.03"/>
 <instance part="GND63" gate="1" x="176.53" y="113.03"/>
-<instance part="GND64" gate="1" x="184.15" y="85.09"/>
+<instance part="GND64" gate="1" x="189.23" y="110.49" rot="R90"/>
 <instance part="GND65" gate="1" x="267.97" y="144.78"/>
 <instance part="GND66" gate="1" x="270.51" y="105.41"/>
@@
 </segment>
 <segment>
-<pinref part="GND9" gate="1" pin="GND"/>
-<wire x1="-121.92" y1="124.46" x2="-121.92" y2="121.92" width="0.1524" layer="91"/>
-<pinref part="U$7" gate="G$1" pin="A"/>
-</segment>
-<segment>
 <pinref part="U$4" gate="G$1" pin="RING"/>
 <pinref part="GND13" gate="1" pin="GND"/>
@@
 </segment>
 <segment>
-<pinref part="GND64" gate="1" pin="GND"/>
-<wire x1="184.15" y1="95.25" x2="184.15" y2="87.63" width="0.1524" layer="91"/>
-<pinref part="U$31" gate="G$1" pin="A"/>
-</segment>
-<segment>
 <pinref part="U$20" gate="G$1" pin="RING"/>
 <pinref part="GND67" gate="1" pin="GND"/>
@@
 <pinref part="R40" gate="R" pin="2"/>
 <pinref part="GND41" gate="1" pin="GND"/>
+</segment>
+<segment>
+<pinref part="U$7" gate="G$1" pin="E"/>
+<pinref part="GND9" gate="1" pin="GND"/>
+<wire x1="-120.65" y1="139.7" x2="-121.92" y2="139.7" width="0.1524" layer="91"/>
+</segment>
+<segment>
+<pinref part="U$31" gate="G$1" pin="E"/>
+<pinref part="GND64" gate="1" pin="GND"/>
+<wire x1="186.69" y1="110.49" x2="184.15" y2="110.49" width="0.1524" layer="91"/>
 </segment>
 </net>
@@
 <segment>
 <pinref part="U$6" gate="G$1" pin="TIP"/>
-<wire x1="-127" y1="146.05" x2="-121.92" y2="146.05" width="0.1524" layer="91"/>
-<wire x1="-121.92" y1="146.05" x2="-121.92" y2="139.7" width="0.1524" layer="91"/>
-<junction x="-121.92" y="146.05"/>
 <pinref part="R23" gate="R" pin="1"/>
-<wire x1="-121.92" y1="146.05" x2="-111.76" y2="146.05" width="0.1524" layer="91"/>
-<pinref part="U$7" gate="G$1" pin="E"/>
+<wire x1="-127" y1="146.05" x2="-125.73" y2="146.05" width="0.1524" layer="91"/>
+<wire x1="-125.73" y1="146.05" x2="-111.76" y2="146.05" width="0.1524" layer="91"/>
+<wire x1="-125.73" y1="146.05" x2="-125.73" y2="124.46" width="0.1524" layer="91"/>
+<pinref part="U$7" gate="G$1" pin="A"/>
+<wire x1="-125.73" y1="124.46" x2="-121.92" y2="124.46" width="0.1524" layer="91"/>
+<junction x="-125.73" y="146.05"/>
 </segment>
 </net>
@@
 <segment>
 <pinref part="U$28" gate="G$1" pin="TIP"/>
-<wire x1="179.07" y1="119.38" x2="184.15" y2="119.38" width="0.1524" layer="91"/>
-<wire x1="184.15" y1="119.38" x2="184.15" y2="110.49" width="0.1524" layer="91"/>
-<junction x="184.15" y="119.38"/>
 <pinref part="R72" gate="R" pin="1"/>
-<wire x1="184.15" y1="119.38" x2="193.04" y2="119.38" width="0.1524" layer="91"/>
-<pinref part="U$31" gate="G$1" pin="E"/>
-</segment>
-</net>
+<wire x1="179.07" y1="119.38" x2="180.34" y2="119.38" width="0.1524" layer="91"/>
+<wire x1="180.34" y1="119.38" x2="193.04" y2="119.38" width="0.1524" layer="91"/>
+<wire x1="180.34" y1="119.38" x2="180.34" y2="95.25" width="0.1524" layer="91"/>
+<pinref part="U$31" gate="G$1" pin="A"/>
+<wire x1="180.34" y1="95.25" x2="184.15" y2="95.25" width="0.1524" layer="91"/>
+<junction x="180.34" y="119.38"/>
+</segment>
+</net>
