File: Development/StageProjecten/AllOfTheAbove.sch (EAGLE design)
At the start: 19 parts, among them J1 JACK, J2 POWERSHROUDED, J3 JACK, J4 JACK, J5 JACK, J6 JACK, J7 JACK, J8 JACK, J9 JACK

Commit message: AllOfTheAbove
Parts:
- added J10, J11, J12, J13, J14, J15, J16: JACK, EurorackModularParts:AUDIO-JACK_SMALLSYMBOLNODRILL
- J4: DESC Input -> Input B
- J5: DESC Input -> Difference B
- J9: DESC Input -> Output B
Connections:
- new net INPUT_A: J6.TIP
- new net INPUT_B: J4.TIP
- new net INPUT_C: J11.TIP
- new net INPUT_D: J14.TIP
- new net MASTERINPUT: J1.TIP, J6.SWITCH
- new net OUTPUT_A: J4.SWITCH, J7.TIP
- new net OUTPUT_B: J11.SWITCH, J9.TIP
- new net OUTPUT_C: J13.TIP, J14.SWITCH
- new net OUTPUT_D: J16.TIP, J3.TIP
- net GND: now also J1.RING, J1.SWITCH, J10.RING, J11.RING, J12.RING, J13.RING, J14.RING, J15.RING, J16.RING, J3.RING, J4.RING, J5.RING, J6.RING, J7.RING, J8.RING, J9.RING

Commit message: 9pwr - opamp - testpad
Parts:
- added C10, C5, C6, C9: (no value), OPL:C-0603
- added C7, C8: (no value), EurorackModularParts:C-POLAR-A
- added IC1: 7809DT, adafruit:7805DT
- added IC2: TL074TSSOP14, EurorackModularParts:TL074TSSOP14
- added U$13: VOLTAGETESTPAD, FenixBase:VOLTAGETESTPAD
Connections:
- new net 9V: C5.2, C7.1, IC1.VO
- net -12V: now also C10.1, IC2P.V-
- net 12V: now also C6.2, C8.1, C9.2, IC1.VI, IC2P.V+
- net GND: now also C10.2, C5.1, C6.1, C7.2, C8.2, C9.1, IC1.GND
Changed lines of the file:
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@@
 <part name="GND20" library="FenixBase" deviceset="GND" device=""/>
 <part name="GND21" library="FenixBase" deviceset="GND" device=""/>
+<part name="IC1" library="adafruit" deviceset="78*" device="DT" technology="05" value="7809DT"/>
+<part name="GND22" library="FenixBase" deviceset="GND" device=""/>
+<part name="U$7" library="FenixBase" deviceset="12V" device=""/>
+<part name="U$9" library="FenixBase" deviceset="9V" device=""/>
+<part name="C5" library="OPL" deviceset="C*" device="-0603"/>
+<part name="C6" library="OPL" deviceset="C*" device="-0603"/>
+<part name="C7" library="EurorackModularParts" deviceset="C-POLAR*" device="-A"/>
+<part name="C8" library="EurorackModularParts" deviceset="C-POLAR*" device="-A"/>
+<part name="GND25" library="FenixBase" deviceset="GND" device=""/>
+<part name="GND26" library="FenixBase" deviceset="GND" device=""/>
+<part name="U$8" library="FenixBase" deviceset="9V" device=""/>
+<part name="U$10" library="FenixBase" deviceset="9V" device=""/>
+<part name="U$11" library="FenixBase" deviceset="12V" device=""/>
+<part name="U$12" library="FenixBase" deviceset="12V" device=""/>
+<part name="GND23" library="FenixBase" deviceset="GND" device=""/>
+<part name="GND24" library="FenixBase" deviceset="GND" device=""/>
+<part name="IC2" library="EurorackModularParts" deviceset="TL074" device="TSSOP14"/>
+<part name="C9" library="OPL" deviceset="C*" device="-0603"/>
+<part name="C10" library="OPL" deviceset="C*" device="-0603"/>
+<part name="GND29" library="FenixBase" deviceset="GND" device=""/>
+<part name="U$14" library="FenixBase" deviceset="12V" device=""/>
+<part name="U$16" library="FenixBase" deviceset="-12V" device=""/>
+<part name="U$17" library="FenixBase" deviceset="12V" device=""/>
+<part name="U$18" library="FenixBase" deviceset="-12V" device=""/>
+<part name="U$13" library="FenixBase" deviceset="VOLTAGETESTPAD" device="">
+<attribute name="DESC" value="MEET"/>
+</part>
 </parts>
 <sheets>
@@
 <instance part="GND20" gate="1" x="127" y="92.71"/>
 <instance part="GND21" gate="1" x="118.11" y="92.71"/>
+<instance part="IC2" gate="A" x="81.28" y="36.83"/>
+<instance part="IC2" gate="B" x="82.55" y="20.32"/>
+<instance part="IC2" gate="C" x="82.55" y="6.35"/>
+<instance part="IC2" gate="D" x="82.55" y="-8.89"/>
+<instance part="IC2" gate="P" x="114.3" y="16.51"/>
+<instance part="C9" gate="C" x="124.46" y="20.32" rot="R90"/>
+<instance part="C10" gate="C" x="124.46" y="12.7" rot="R90"/>
+<instance part="GND29" gate="1" x="128.27" y="16.51" rot="R90"/>
+<instance part="U$14" gate="G$1" x="124.46" y="24.13"/>
+<instance part="U$16" gate="G$1" x="124.46" y="8.89"/>
+<instance part="U$17" gate="G$1" x="114.3" y="24.13"/>
+<instance part="U$18" gate="G$1" x="114.3" y="8.89"/>
+<instance part="U$13" gate="G$1" x="29.21" y="5.08"/>
 </instances>
 <busses>
@@
 <pinref part="J14" gate="G$1" pin="RING"/>
 <pinref part="GND21" gate="1" pin="GND"/>
+</segment>
+<segment>
+<pinref part="C9" gate="C" pin="1"/>
+<pinref part="GND29" gate="1" pin="GND"/>
+<wire x1="125.73" y1="16.51" x2="124.46" y2="16.51" width="0.1524" layer="91"/>
+<pinref part="C10" gate="C" pin="2"/>
+<junction x="124.46" y="16.51"/>
 </segment>
 </net>
@@
 <wire x1="115.57" y1="128.27" x2="115.57" y2="157.48" width="0.1524" layer="91"/>
 <label x="118.11" y="146.05" size="1.778" layer="95" rot="R90"/>
+</segment>
+</net>
+<net name="12V" class="0">
+<segment>
+<pinref part="C9" gate="C" pin="2"/>
+<pinref part="U$14" gate="G$1" pin="12V"/>
+</segment>
+<segment>
+<pinref part="IC2" gate="P" pin="V+"/>
+<pinref part="U$17" gate="G$1" pin="12V"/>
+</segment>
+</net>
+<net name="-12V" class="0">
+<segment>
+<pinref part="C10" gate="C" pin="1"/>
+<pinref part="U$16" gate="G$1" pin="-12V"/>
+</segment>
+<segment>
+<pinref part="IC2" gate="P" pin="V-"/>
+<pinref part="U$18" gate="G$1" pin="-12V"/>
 </segment>
 </net>
@@
 <instance part="U$5" gate="G$1" x="80.01" y="39.37"/>
 <instance part="U$6" gate="G$1" x="82.55" y="40.64"/>
+<instance part="IC1" gate="A1" x="53.34" y="-1.27"/>
+<instance part="GND22" gate="1" x="53.34" y="-11.43"/>
+<instance part="U$7" gate="G$1" x="41.91" y="-1.27"/>
+<instance part="U$9" gate="G$1" x="64.77" y="-1.27"/>
+<instance part="C5" gate="C" x="20.32" y="-13.97" rot="R90"/>
+<instance part="C6" gate="C" x="31.75" y="-16.51" rot="R90"/>
+<instance part="C7" gate="C" x="16.51" y="-13.97" rot="R270"/>
+<instance part="C8" gate="C" x="29.21" y="-16.51" rot="R270"/>
+<instance part="GND25" gate="1" x="20.32" y="-20.32"/>
+<instance part="GND26" gate="1" x="16.51" y="-21.59"/>
+<instance part="U$8" gate="G$1" x="16.51" y="-7.62"/>
+<instance part="U$10" gate="G$1" x="20.32" y="-7.62"/>
+<instance part="U$11" gate="G$1" x="29.21" y="-11.43"/>
+<instance part="U$12" gate="G$1" x="31.75" y="-12.7"/>
+<instance part="GND23" gate="1" x="29.21" y="-24.13"/>
+<instance part="GND24" gate="1" x="31.75" y="-22.86"/>
 </instances>
 <busses>
@@
 <pinref part="GND5" gate="1" pin="GND"/>
 </segment>
+<segment>
+<pinref part="IC1" gate="A1" pin="GND"/>
+<pinref part="GND22" gate="1" pin="GND"/>
+</segment>
+<segment>
+<pinref part="C5" gate="C" pin="1"/>
+<pinref part="GND25" gate="1" pin="GND"/>
+</segment>
+<segment>
+<pinref part="C7" gate="C" pin="2"/>
+<pinref part="GND26" gate="1" pin="GND"/>
+</segment>
+<segment>
+<pinref part="C8" gate="C" pin="2"/>
+<pinref part="GND23" gate="1" pin="GND"/>
+</segment>
+<segment>
+<pinref part="C6" gate="C" pin="1"/>
+<pinref part="GND24" gate="1" pin="GND"/>
+</segment>
 </net>
 <net name="N$2" class="0">
@@
 <wire x1="71.12" y1="53.34" x2="71.12" y2="50.8" width="0.1524" layer="91"/>
 </segment>
+<segment>
+<pinref part="IC1" gate="A1" pin="VI"/>
+<pinref part="U$7" gate="G$1" pin="12V"/>
+<wire x1="41.91" y1="-1.27" x2="43.18" y2="-1.27" width="0.1524" layer="91"/>
+</segment>
+<segment>
+<pinref part="C8" gate="C" pin="1"/>
+<pinref part="U$11" gate="G$1" pin="12V"/>
+</segment>
+<segment>
+<pinref part="C6" gate="C" pin="2"/>
+<pinref part="U$12" gate="G$1" pin="12V"/>
+</segment>
 </net>
 <net name="N$3" class="0">
@@
 </segment>
 </net>
+<net name="9V" class="0">
+<segment>
+<pinref part="IC1" gate="A1" pin="VO"/>
+<pinref part="U$9" gate="G$1" pin="9V"/>
+<wire x1="64.77" y1="-1.27" x2="63.5" y2="-1.27" width="0.1524" layer="91"/>
+</segment>
+<segment>
+<pinref part="C7" gate="C" pin="1"/>
+<wire x1="16.51" y1="-7.62" x2="16.51" y2="-8.89" width="0.1524" layer="91"/>
+<pinref part="U$8" gate="G$1" pin="9V"/>
+</segment>
+<segment>
+<pinref part="C5" gate="C" pin="2"/>
+<wire x1="20.32" y1="-7.62" x2="20.32" y2="-10.16" width="0.1524" layer="91"/>
+<pinref part="U$10" gate="G$1" pin="9V"/>
+</segment>
+</net>

Commit message: differentiator and zerocrossing setup start
Parts:
- added C11, C12, C13, C14, C15, C16, C17, C18, C19, C20, C21: (no value), OPL:C-0603
- added D10, D3, D4, D5, D6, D7, D8, D9: BAS16W, FenixBase:BAS16W
- added IC3, IC4: TL074TSSOP14, EurorackModularParts:TL074TSSOP14
- added R10, R11, R12, R13, R14, R15, R16, R17, R18, R19, R20, R21, R4, R5, R6, R7, R8, R9: (no value), OPL:R-0603
Connections:
- new net N$1: IC3A.+IN, R4.2
- new net N$10: IC3C.OUT, R10.1
- new net N$11: IC4A.OUT, R16.1, R5.1, R8.1
- new net N$12: C13.2, IC4A.-IN, R16.2
- new net N$13: IC4C.OUT, R17.1
- new net N$14: IC4C.-IN, R17.2
- new net N$15: C14.2, D3.CATHODE, D4.ANODE, R6.2
- new net N$16: C13.1, R4.1, R9.1
- new net N$17: C15.2, D5.CATHODE, D6.ANODE, R7.2
- new net N$18: C16.2, D7.CATHODE, D8.ANODE, R10.2
- new net N$19: C17.2, D10.ANODE, D9.CATHODE, R11.2
- new net N$24: C19.2, D6.CATHODE, R14.2
- new net N$25: C20.2, D8.CATHODE, R13.2
- new net N$26: C21.2, D10.CATHODE, R12.2
- new net N$27: C18.2, D4.CATHODE, R15.2
- new net N$28: C18.1, R18.2
- new net N$29: C19.1, R19.2
- new net N$30: C20.1, R20.2
- new net N$31: C21.1, R21.2
- new net N$4: IC3B.+IN, R5.2
- new net N$5: IC3A.OUT, R6.1
- new net N$6: IC3B.OUT, R7.1
- new net N$7: IC3C.-IN, R9.2
- new net N$8: IC3D.-IN, R8.2
- new net N$9: IC3D.OUT, R11.1
- net -12V: now also C12.1, IC3P.V-
- net 12V: now also C11.2, IC3P.V+
- net GND: now also C11.1, C12.2, C14.1, C15.1, C16.1, C17.1, D3.ANODE, D5.ANODE, D7.ANODE, D9.ANODE, IC3A.-IN, IC3B.-IN, IC3C.+IN, IC3D.+IN, IC4A.+IN, R12.1, R13.1, R14.1, R15.1

Commit message: Dist+ added
Parts:
- added C22, C23, C24, C25, C26, C27, C28: (no value), OPL:C-0603
- added D11, D12: (no value), diode:DIODE-DO-214AC
- added IC5: UA741D, linear:UA741D
- added R23: 1M, EurorackModularParts:POTSQUAREHOLE_SMALLKNOB
- added R24: 10K, EurorackModularParts:POTSQUAREHOLE_SMALLKNOB
- added R25, R26, R27, R28: (no value), OPL:R-0603
Connections:
- new net N$20: C23.2, R25.2
- new net N$21: IC5.-IN, R25.1
- new net N$22: C26.2, IC5.+IN, R27.1
- new net N$23: C26.1, R26.1
- new net N$32: C27.1, IC5.OUT, R27.2
- new net N$33: R23.A, R26.2
- new net N$34: C28.2, D11.C, D12.A, R24.A, R28.1
- new net N$35: C27.2, R28.2
- net -12V: now also C25.1, IC5.V-
- net 12V: now also C24.2, IC5.V+
- net GND: now also C22.2, C24.1, C25.2, C28.1, D11.A, D12.C, R23.E, R23.S, R24.E
- net INPUT_A: now also C22.1, C23.1
- net OUTPUT_A: now also R24.S

Commit message: Rat added with powerjumpers
Parts:
- added C29, C30, C31, C32, C33, C34, C35, C36, C37, C38, C39: (no value), OPL:C-0603
- added D13, D14: (no value), OPL:D-D1206
- added IC6: UA741D, linear:UA741D
- added JP1, JP2, JP3: (no value), pinhead:PINHD-1X3
- added Q1: SST201, transistor-fet:SST201
- added R22, R29, R30, R31: (no value), EurorackModularParts:POTSQUAREHOLE_SMALLKNOB
- added R32, R33, R34, R35, R36, R37, R38, R39, R40: (no value), OPL:R-0603
- D11, D12: device diode:DIODE-DO-214AC -> OPL:D-D1206
Connections:
- new net +4.5V: R34.2
- new net N$36: R22.E, R22.S, R28.1
- new net N$37: C29.2, JP1.2, R33.1
- new net N$38: C30.2, IC6.+IN, R33.2
- new net N$39: IC6.V+, JP2.2
- new net N$40: IC6.V-, JP3.2
- new net N$41: JP1.1, R34.1
- new net N$42: C31.1, IC6.-IN, R31.E, R31.S, R35.2, R36.2
- new net N$43: C31.2, C34.2, IC6.OUT, R31.A
- new net N$44: C34.1, R37.1
- new net N$45: D13.-, D14.+, R30.E, R30.S, R37.2
- new net N$46: R30.A, R38.1
- new net N$47: C33.2, R36.1
- new net N$48: C32.2, R35.1
- new net N$49: C35.1, C36.1, R38.2
- new net N$50: C36.2, Q1.G, R39.2
- new net N$51: C37.1, Q1.S, R40.2
- new net N$52: C37.2, R29.A
- net -12V: now also C39.1, JP3.3
- net 12V: now also C38.2, JP2.3
- net 9V: now also JP2.1, Q1.D
- net GND: now also C30.1, C32.1, C33.1, C35.2, C38.1, C39.2, D11.+, D12.-, D13.+, D14.-, JP3.1, R29.E, R32.2, R39.1, R40.1; no longer D11.A, D12.C
- net INPUT_B: now also C29.1, R32.1
- net N$21: now also IC5.+IN; no longer IC5.-IN
- net N$22: now also IC5.-IN; no longer IC5.+IN
- net N$34: now also D11.-, D12.+, R22.A; no longer D11.C, D12.A, R28.1

Commit message: Added FF&Muff schematic (.brd not updated)
Parts:
- added C40, C41, C42, C43, C44, C45, C46, C47, C48, C49, C50, C51, C52, C53, C54, C55: (no value), OPL:C-0603
- added D15, D16, D17, D18: (no value), OPL:D-D1206
- added Q2, Q3: BCX71SMD, transistor-pnp:BCX71SMD
- added Q4, Q5, Q6, Q7: BC849SMD, transistor-npn:BC849SMD
- added R41, R44, R45, R46, R47, R48, R49, R50, R51, R52, R53, R54, R55, R56, R57, R58, R59, R60, R61, R62, R63, R64, R65, R66, R67, R68: (no value), OPL:R-0603
- added R42, R43, R69, R70, R71: (no value), EurorackModularParts:POTSQUAREHOLE_SMALLKNOB
Connections:
- new net N$53: Q3.E, R41.1, R43.A
- new net N$54: C40.2, Q2.B, R41.2
- new net N$55: Q2.C, Q3.B, R45.2
- new net N$56: C41.1, R43.S
- new net N$57: C42.2, R42.A
- new net N$58: C42.1, R44.1, R46.2
- new net N$59: Q3.C, R44.2
- new net N$60: C43.1, R47.2
- new net N$61: C43.2, C44.1, Q4.B, R48.2, R49.2
- new net N$62: Q4.E, R50.1
- new net N$63: C44.2, C45.1, Q4.C, R49.1, R51.2
- new net N$64: C45.2, R71.A
- new net N$65: C47.1, C48.1, Q5.B, R53.2, R54.2, R56.2
- new net N$66: C48.2, D15.+, D16.-
- new net N$67: Q5.E, R55.2
- new net N$68: C47.2, C49.1, D15.-, D16.+, Q5.C, R56.1, R57.2
- new net N$69: C49.2, R58.1
- new net N$70: C50.1, C51.1, Q6.B, R58.2, R59.2, R61.2
- new net N$71: Q6.E, R60.2
- new net N$72: C50.2, C52.1, D17.-, D18.+, Q6.C, R61.1, R62.2, R63.1
- new net N$73: C53.1, R70.S
- new net N$74: C55.2, R63.2, R70.E
- new net N$75: C52.2, R64.1, R70.A
- new net N$76: C51.2, D17.+, D18.-
- new net N$77: C53.2, Q7.B, R65.2, R66.1
- new net N$78: C54.1, Q7.C, R67.1
- new net N$79: Q7.E, R68.2
- new net N$80: C54.2, R69.A
- new net N$84: R52.1, R71.E
- new net N$85: C46.2, R53.1
- new net N$86: C46.1, R71.S
- net 9V: now also R45.1, R46.1, R51.1, R57.1, R62.1, R66.2, R67.2
- net GND: now also C41.2, C55.1, Q2.E, R42.E, R43.E, R48.1, R50.2, R52.2, R54.1, R55.1, R59.1, R60.1, R64.2, R65.1, R68.1, R69.E
- net INPUT_C: now also C40.1
- net INPUT_D: now also R47.1
- net OUTPUT_B: now also R29.S
- net OUTPUT_C: now also R42.S
- net OUTPUT_D: now also R69.S

Commit message: Added Modules/Guitar In
Parts:
- removed C28, C29, C30, C31, C32, C33, C34, C35, C36, C37, C38, C39, C40, C41, C42, C43, C44, C45, C46, C47, C48, C49, C50, C51, C52, C53, C54, C55: (no value), OPL:C-0603
- removed D11, D12, D13, D14, D15, D16, D17, D18: (no value), OPL:D-D1206
- removed IC6: UA741D, linear:UA741D
- removed JP1, JP2, JP3: (no value), pinhead:PINHD-1X3
- removed Q1: SST201, transistor-fet:SST201
- removed Q2, Q3: BCX71SMD, transistor-pnp:BCX71SMD
- removed Q4, Q5, Q6, Q7: BC849SMD, transistor-npn:BC849SMD
- removed R27, R28, R32, R33, R34, R35, R36, R37, R38, R39, R40, R41, R44, R45, R46, R47, R48, R49, R50, R51, R52, R53, R54, R55, R56, R57, R58, R59, R60, R61, R62, R63, R64, R65, R66, R67, R68: (no value), OPL:R-0603
- removed R29, R30, R31, R42, R43, R69, R70, R71: (no value), EurorackModularParts:POTSQUAREHOLE_SMALLKNOB
- C22: value (none) -> 10uF
- IC5: value UA741D -> TL071D; device linear:UA741D -> EurorackModularParts:TL071D
- R22: value (none) -> 1M; device EurorackModularParts:POTSQUAREHOLE_SMALLKNOB -> OPL:R-0603; DESC Tone -> (none)
- R23: value 1M -> 150K; device EurorackModularParts:POTSQUAREHOLE_SMALLKNOB -> OPL:R-0603; DESC Distortion -> (none)
- R24: value 10K -> (none); device EurorackModularParts:POTSQUAREHOLE_SMALLKNOB -> OPL:R-0603; DESC Volume -> (none)
Connections:
- removed net +4.5V: R34.2
- removed net N$37: C29.2, JP1.2, R33.1
- removed net N$39: IC6.V+, JP2.2
- removed net N$40: IC6.V-, JP3.2
- removed net N$41: JP1.1, R34.1
- removed net N$42: C31.1, IC6.-IN, R31.E, R31.S, R35.2, R36.2
- removed net N$43: C31.2, C34.2, IC6.OUT, R31.A
- removed net N$44: C34.1, R37.1
- removed net N$45: D13.-, D14.+, R30.E, R30.S, R37.2
- removed net N$46: R30.A, R38.1
- removed net N$47: C33.2, R36.1
- removed net N$48: C32.2, R35.1
- removed net N$49: C35.1, C36.1, R38.2
- removed net N$50: C36.2, Q1.G, R39.2
- removed net N$51: C37.1, Q1.S, R40.2
- removed net N$52: C37.2, R29.A
- removed net N$53: Q3.E, R41.1, R43.A
- removed net N$54: C40.2, Q2.B, R41.2
- removed net N$55: Q2.C, Q3.B, R45.2
- removed net N$56: C41.1, R43.S
- removed net N$57: C42.2, R42.A
- removed net N$58: C42.1, R44.1, R46.2
- removed net N$59: Q3.C, R44.2
- removed net N$60: C43.1, R47.2
- removed net N$61: C43.2, C44.1, Q4.B, R48.2, R49.2
- removed net N$62: Q4.E, R50.1
- removed net N$63: C44.2, C45.1, Q4.C, R49.1, R51.2
- removed net N$64: C45.2, R71.A
- removed net N$65: C47.1, C48.1, Q5.B, R53.2, R54.2, R56.2
- removed net N$66: C48.2, D15.+, D16.-
- removed net N$67: Q5.E, R55.2
- removed net N$68: C47.2, C49.1, D15.-, D16.+, Q5.C, R56.1, R57.2
- removed net N$69: C49.2, R58.1
- removed net N$70: C50.1, C51.1, Q6.B, R58.2, R59.2, R61.2
- removed net N$71: Q6.E, R60.2
- removed net N$72: C50.2, C52.1, D17.-, D18.+, Q6.C, R61.1, R62.2, R63.1
- removed net N$73: C53.1, R70.S
- removed net N$74: C55.2, R63.2, R70.E
- removed net N$75: C52.2, R64.1, R70.A
- removed net N$76: C51.2, D17.+, D18.-
- removed net N$77: C53.2, Q7.B, R65.2, R66.1
- removed net N$78: C54.1, Q7.C, R67.1
- removed net N$79: Q7.E, R68.2
- removed net N$80: C54.2, R69.A
- removed net N$84: R52.1, R71.E
- removed net N$85: C46.2, R53.1
- removed net N$86: C46.1, R71.S
- new net BIASMAINLINE: C7.1, D2.ANODE, D4.ANODE, D6.ANODE, D7.ANODE, D8.ANODE, IC1.OUT, R13.1
- new net GUITAR_IN: C22.1, R22.2
- new net GUITAR_OUT: R26.2
- new net INPUT_E: R14.2
- new net N$81: IC5.V+
- new net N$82: IC5.V-
- new net OUTPUT_E: R22.1, R23.1
- net -12V: now also C27.1, C4.1, C6.1, IC1.V-, IC3SUPPLY.V-, R12.1, R9.2, U$13.-12V; no longer C39.1, IC5.V-, JP3.3
- net 12V: now also C26.2, C3.2, C5.2, IC1.V+, IC3SUPPLY.V+, R2.A; no longer C38.2, IC5.V+, JP2.3
- net 9V: no longer JP2.1, Q1.D, R45.1, R46.1, R51.1, R57.1, R62.1, R66.2, R67.2
- net GND: now also C23.1, C25.1, C26.1, C27.2, C3.1, C4.2, C6.2, D1.CATHODE, D10.CATHODE, D3.CATHODE, D5.CATHODE, D9.CATHODE, IC1.+IN, IC3BUF1.B, IC3BUF2.B, IC3OTA2.IN_N, IC3OTA2.IN_P, R1.E, R2.E, R22.1, R23.1, R24.2, R25.1, R26.1, R4.2, R5.2, R7.1, R8.1; no longer C28.1, C30.1, C32.1, C33.1, C35.2, C38.1, C39.2, C41.2, C55.1, D11.+, D12.-, D13.+, D14.-, JP3.1, Q2.E, R29.E, R32.2, R39.1, R40.1, R42.E, R43.E, R48.1, R50.2, R52.2, R54.1, R55.1, R59.1, R60.1, R64.2, R65.1, R68.1, R69.E
- net INPUT_B: no longer C29.1, R32.1
- net INPUT_C: no longer C40.1
- net INPUT_D: no longer R47.1
- net N$1: now also R4.1
- net N$10: now also R6.1
- net N$11: now also C8.1, IC1.OUT, R15.1, R16.2, R17.2
- net N$12: now also C14.2, C8.2, IC1.-IN, R15.2
- net N$13: now also C14.1, IC3OTA1.OUT, R5.1
- net N$14: now also D3.ANODE, D4.CATHODE, IC2A.+IN, R16.1
- net N$15: now also C9.1, IC2A.OUT, R18.1
- net N$16: now also D5.ANODE, D6.CATHODE, IC2B.+IN
- net N$17: now also C9.2, IC2A.-IN, R17.1, R18.2
- net N$18: now also C11.2, IC2C.-IN, R20.1
- net N$19: now also C16.1, IC1.OUT
- net N$20: now also C22.2, D8.CATHODE, D9.ANODE, IC2D.+IN, IC5.+IN, R23.2
- net N$21: now also C10.2, IC2B.-IN, R19.2
- net N$22: now also C10.1, C24.1, IC2B.OUT, IC5.OUT, R19.1, R20.2, R24.2, R26.1; no longer R27.1
- net N$23: now also C24.2, D10.ANODE, D7.CATHODE, IC2C.+IN, IC5.-IN, R24.1, R25.2
- net N$24: now also C11.1, IC2C.OUT
- net N$25: now also C13.1, IC1.+IN, R25.2
- net N$26: now also C15.2, IC2D.-IN, R21.2
- net N$27: now also C15.1, IC2D.OUT, R21.1
- net N$28: now also D1.ANODE, D2.CATHODE, IC1.+IN
- net N$29: now also C12.1, IC1.OUT, R22.2
- net N$3: now also C7.2, IC1.-IN, R13.2, R14.1
- net N$30: now also C16.2, IC1.-IN
- net N$32: now also C12.2, C25.2, IC1.-IN, R23.2, R24.1, R25.1; no longer R27.2
- net N$33: now also R9.1
- net N$34: now also IC3OTA1.I_BIAS, R6.2; no longer C28.2, D11.-, D12.+
- net N$35: no longer R28.2
- net N$36: now also IC3OTA1.IN_P, R7.2; no longer R28.1
- net N$38: now also IC3OTA1.IN_N, R8.2; no longer C30.2, IC6.+IN, R33.2
- net N$5: now also R1.S, R10.2
- net N$6: now also R1.A
- net N$7: now also R10.1, R11.1, R12.2
- net N$8: now also R11.2, R2.S
- net N$9: now also C13.2, R26.2
- net OUTPUT_B: no longer R29.S
- net OUTPUT_C: no longer R42.S
- net OUTPUT_D: no longer R69.S

Commit message: VCA added
Parts:
- removed C23, C24, C25, C26, C27: (no value), OPL:C-0603
- added D17: (no value), OPL:D-D1206
- added IC6: TL072, EurorackModularParts:TL072
- added Q1: MMBT3906LT1SMD, transistor-pnp:MMBT3906LT1SMD
- added R27, R28, R30, R31, R32, R33: (no value), OPL:R-0603
- added R29, R34: TRIMPOT, EurorackModularParts:TRIMPOT
- added R69: (no value), EurorackModularParts:POTSQUAREHOLE_SMALLKNOB
- C22: value 10uF -> (none)
- IC5: value TL071D -> LM13700M; device EurorackModularParts:TL071D -> ota:LM13700M
- R22: value 1M -> (none)
- R23: value 150K -> (none)
Connections:
- new net +4.5V: R34.2
- new net N$37: D17.-, IC6VR2.-IN, R31.1, R32.2, R33.1, R33.2
- new net N$39: IC5OTA1.I_BIAS, IC6A.V+, Q1.C
- new net N$40: IC6A.V-, R33.1, R34.P$2
- new net N$41: R34.1
- new net N$42: IC6A.-IN, R31.E, R31.S, R32.1, R69.S
- new net N$43: IC6A.OUT, R31.A
- new net N$45: R30.E, R30.S
- new net N$46: R30.A
- new net N$50: Q1.G
- new net N$51: Q1.S
- new net N$52: R29.A
- new net N$72: D17.-
- new net N$76: D17.+
- new net N$80: R69.A
- new net VCA_CV_IN: R69.A
- new net VCA_OUTPUT: R28.2
- new net VCA_SIG_IN: R22.1
- net -12V: now also IC5A.V-, R29.P$1, R34.P$1; no longer C25.1, C27.1
- net 12V: now also IC5A.V+, R29.P$3, R34.P$3; no longer C24.2, C26.2
- net 9V: now also Q1.D
- net GND: now also IC6VR2.+IN, R26.2, R29.E, R30.1, R32.2, R69.E; no longer C23.1, C24.1, C25.1, C25.2, C26.1, C27.2
- net GUITAR_IN: no longer C22.1
- net INPUT_A: no longer C23.1
- net INPUT_B: now also R32.1
- net N$15: now also R31.2, R32.2
- net N$16: now also R31.1
- net N$19: now also R27.1, R28.2
- net N$20: now also IC5A.+IN, IC5OTA1.IN_N, R24.1, R25.1, R34.1; no longer C22.2, C23.2, IC5.+IN
- net N$21: now also IC5A.+IN, IC5OTA1.IN_P, R22.2, R23.2, R32.1; no longer IC5.+IN
- net N$22: now also IC5A.-IN, IC5A.OUT, IC5OTA1.OUT, IC6VR1.+IN, R27.1, R33.2; no longer C24.1, C26.2, IC5.-IN, IC5.OUT
- net N$23: now also C22.1, IC5A.-IN, IC6VR1.-IN, R27.1, R33.1; no longer C24.2, C26.1, IC5.-IN
- net N$24: now also R34.2
- net N$27: now also R29.1, R30.1
- net N$28: now also R29.2
- net N$30: now also R28.1, R30.2
- net N$32: now also IC5A.OUT, R25.2, R27.2, R29.P$2; no longer C25.2, C27.1, IC5.OUT, R25.1
- net N$33: now also C22.2, IC6VR1.OUT, R27.2, R28.1
- net N$35: now also R28.2; no longer C27.2
- net N$36: now also D17.+, IC6VR2.OUT, Q1.B, R28.1
- net N$38: now also IC6A.+IN, Q1.E, R30.2, R31.2, R33.2
- net N$81: now also IC5A.V+; no longer IC5.V+
- net N$82: now also IC5A.V-; no longer IC5.V-
- net N$9: now also R27.2
- net OUTPUT_B: now also R29.S
- net OUTPUT_D: now also R69.S
Other:
- moved on the sheet: C22, R22, R23, R24, R25, R26
