File: Development/StageProjecten/AllOfTheAbove7x_5nov3_v9fixed.sch (EAGLE design)
At the start: 231 parts, among them IC1 7809DT, IC10 LM13700M, IC2 TL074TSSOP14, IC3 TL074TSSOP14, IC4 TL074TSSOP14, IC5 LM13700M, IC6 TL074TSSOP14, IC8 TL074TSSOP14, IC9 TL074TSSOP14, J1 JACK, J10 JACK, J11 JACK, J12 JACK, J13 JACK, J14 JACK, J15 JACK, J16 JACK, J17 JACK, J18 JACK, J19 JACK, J2 POWERSHROUDED, J20 JACK, J21 JACK, J22 JACK, J23 JACK, J24 JACK, J25 JACK, J26 JACK, J3 JACK, J4 JACK, J5 JACK, J6 JACK, J7 JACK, J8 JACK, J9 JACK, Q1 MMBT3906LT1SMD, Q3 MMBT3906LT1SMD, Q4 MMBT3906LT1SMD, T1 3906

Commit message: Finished Board placements
Parts:
- added C42, C43: 100n, OPL:C-0603
- added IC7: TL074TSSOP14, EurorackModularParts:TL074TSSOP14
- added R116, R117, R92, R93, R94, R95, R96, R97: 100k, OPL:R-0603
Connections:
- new net N$13: IC7B.-IN, R94.2, R97.1
- new net N$31: IC7B.OUT, J9.TIP, R97.2
- new net N$6: IC7A.OUT, J7.TIP, R93.2
- net -12V: now also C43.1, IC7P.V-
- net 12V: now also C42.2, IC7P.V+
- net GND: now also C42.1, C43.2, IC7A.+IN, IC7B.+IN, IC7C.+IN, IC7D.+IN
- net N$1: now also IC7A.-IN, R92.2, R93.1
- net N$32: now also IC7C.-IN, R116.1, R95.2
- net N$36: now also IC7C.OUT, J13.TIP, R116.2
- net N$37: now also IC7D.-IN, R117.1, R96.2
- net N$42: now also IC7D.OUT, J16.TIP, R117.2
- net N$57: now also C42.2
- net N$58: now also C42.1
- net OUTPUT_A: now also R92.1; no longer J7.TIP
- net OUTPUT_B: now also R94.1; no longer J9.TIP
- net OUTPUT_C: now also R95.1; no longer J13.TIP
- net OUTPUT_D: now also R96.1; no longer J16.TIP
- net OUTPUT_E: no longer J19.TIP
Other:
- moved on the sheet: C10, C9, IC2P, J13, J16, J7, J9
