File: Development/StageProjecten/AllOfTheAbove7x14novTRIMS.brd (EAGLE design)
At the start: 180.7 x 105.1 mm, 357 parts, among them IC1 7809DT, IC10 LM13700M, IC2 TL074TSSOP14, IC3 TL074TSSOP14, IC4 TL074TSSOP14, IC5 LM13700M, IC6 TL074TSSOP14, IC7 TL074TSSOP14, IC8 TL074TSSOP14, IC9 TL074TSSOP14, J1 JACK, J10 JACK, J11 JACK, J12 JACK, J13 JACK, J14 JACK, J15 JACK, J16 JACK, J17 JACK, J18 JACK, J19 JACK, J2 POWERSHROUDED, J20 JACK, J21 JACK, J22 JACK, J23 JACK, J24 JACK, J25 JACK, J26 JACK, J3 JACK, J4 JACK, J5 JACK, J6 JACK, J7 JACK, J8 JACK, J9 JACK, Q1 MMBT3906LT1SMD, Q3 MMBT3906LT1SMD, Q4 MMBT3906LT1SMD, T1 3906

Commit message: Lijntjes trekken
Parts:
- ACID1:R24: value 10K -> 10KA
- R109: value 10kA -> 100KB
- R114: value 10k -> 10KB
- R49: value 100KB Lin -> 100KB
- R50: value 10KB Lin -> 10KB
- R69: value 100K Linear -> 100KB
- moved U$15 74.2 mm to (42.2, 49.5)
- moved U$71 13.5 mm to (63.5, 32.7)
- moved TR_IN_B 9.21 mm to (55.6, 31.4)
Routing:
- net 12V: track 105.0 -> 291.0 mm, vias 6 -> 33
- net OUTPUT_B: track 0.00 -> 163.1 mm, vias 0 -> 9
- net OUTPUT_A: track 0.00 -> 153.0 mm, vias 0 -> 20
- net INPUT_A: track 0.00 -> 151.8 mm, vias 0 -> 14
- net 4.5V: track 5.35 -> 151.2 mm, vias 0 -> 17
- net N$42: track 0.00 -> 141.7 mm, vias 0 -> 8
- net -12V: track 109.0 -> 242.8 mm, vias 8 -> 32
- net VCA_OUTPUT2: track 0.00 -> 129.6 mm, vias 0 -> 10
- net N$4: track 6.44 -> 130.9 mm, vias 1 -> 3
- net VCA_OUTPUT1: track 0.00 -> 122.8 mm, vias 0 -> 8
- net INPUT_B: track 0.00 -> 118.2 mm, vias 0 -> 12
- net N$13: track 7.25 -> 122.4 mm, vias 1 -> 6
- net OUTPUT_E: track 59.4 -> 173.0 mm, vias 0 -> 8
- net N$12: track 0.00 -> 99.8 mm, vias 0 -> 12
- net INPUT_C: track 0.00 -> 87.8 mm, vias 0 -> 4
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