File: Development/StageProjecten/StompBoard.brd (EAGLE design)
At the start: 162.6 x 27.9 mm, 16 parts

Commit message: STM32 KLAAR
Routing:
- net N$3: track 11.4 -> 12.1 mm
- net N$8: track 11.4 -> 12.1 mm
- net N$11: track 11.4 -> 12.1 mm
- net INP5_PCB: track 12.9 -> 12.1 mm
- net INP4_PCB: track 12.9 -> 12.1 mm
- net INP2_PCB: track 12.9 -> 12.1 mm
- net INP1_PCB: track 12.9 -> 12.1 mm
- net INP3_PCB: track 14.1 -> 13.4 mm
- net N$7: track 4.80 -> 5.30 mm
- net N$2: track 4.80 -> 5.30 mm
- net N$13: track 4.80 -> 5.30 mm
- net N$10: track 4.80 -> 5.30 mm
- net INP5_JACK: track 12.8 -> 12.3 mm
- net INP4_JACK: track 12.8 -> 12.3 mm
- net INP3_JACK: track 14.0 -> 13.5 mm
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