File: Development/StageProjecten/TiNRS&Navenant-Overstuurd versie 1.brd (EAGLE design)
At the start: 180.7 x 105.1 mm, 380 parts, among them IC1 7809DT, IC10 LM13700M, IC11 TL074TSSOP14, IC2 TL074TSSOP14, IC3 TL074TSSOP14, IC4 TL074TSSOP14, IC5 LM13700M, IC6 TL074TSSOP14, IC7 TL074TSSOP14, IC8 TL074TSSOP14, IC9 TL074TSSOP14, J1 JACK, J10 JACK, J11 JACK, J12 JACK, J13 JACK, J14 JACK, J15 JACK, J16 JACK, J17 JACK, J18 JACK, J19 JACK, J2 POWERSHROUDED, J20 JACK, J21 JACK, J22 JACK, J23 JACK, J24 JACK, J25 JACK, J26 JACK, J27 JACK, J3 JACK, J4 JACK, J5 JACK, J6 JACK, J7 JACK, J8 JACK, J9 JACK, Q1 MMBT3906LT1SMD, Q3 MMBT3906LT1SMD, Q4 MMBT3906LT1SMD, T1 3906, U1 LM358DR-1110010P1

Commit message: Some overstuur resistors
Parts:
- added R128, R129: 56, OPL:R0603
Connections:
- new net N$125: J26.TIP_B@1, J26.TIP_T@3, R128.1
- new net N$126: J10.TIP_B@1, J10.TIP_T@3, R129.1
- net CROSSFADER_OUT: now also R128.2; no longer J26.TIP_B@1, J26.TIP_T@3
- net N$38: now also R129.2; no longer J10.TIP_B@1, J10.TIP_T@3
Routing:
- net CROSSFADER_OUT: track 58.3 -> 35.8 mm
- net N$38: track 29.7 -> 28.4 mm
Changed lines of the file:
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@@
 <?xml version="1.0" encoding="utf-8"?>
 <!DOCTYPE eagle SYSTEM "eagle.dtd">
-<eagle version="9.5.2">
+<eagle version="9.5.1">
 <drawing>
 <settings>
@@
 <attribute name="VALUE" x="34.9725" y="43.053" size="0.508" layer="27" ratio="10" rot="R90"/>
 </element>
+<element name="R128" library="OPL" package="R0603" value="56" x="-0.3175" y="-11.7475" smashed="yes">
+<attribute name="NAME" x="-0.3175" y="-11.7475" size="0.508" layer="25" ratio="11" align="center"/>
+<attribute name="VALUE" x="-1.7145" y="-13.065" size="0.508" layer="27" ratio="10"/>
+</element>
+<element name="R129" library="OPL" package="R0603" value="56" x="-0.3175" y="-14.2875" smashed="yes">
+<attribute name="NAME" x="-0.3175" y="-14.2875" size="0.508" layer="25" ratio="11" align="center"/>
+<attribute name="VALUE" x="-1.7145" y="-15.605" size="0.508" layer="27" ratio="10"/>
+</element>
 </elements>
 <signals>
@@
 <contactref element="IC6" pad="7"/>
 <contactref element="R20" pad="1"/>
-<contactref element="J10" pad="TIP_T@3" route="any" routetag="G$1.TIP"/>
-<contactref element="J10" pad="TIP_B@1" route="any" routetag="G$1.TIP"/>
 <wire x1="151.5078" y1="71.4825" x2="150.7675" y2="71.4825" width="0.254" layer="1"/>
 <wire x1="149.733" y1="72.517" x2="149.733" y2="73.3425" width="0.254" layer="1"/>
@@
 <via x="170.815" y="73.9775" extent="1-16" drill="0.3048"/>
 <wire x1="170.815" y1="73.9775" x2="174.3625" y2="73.9775" width="0.254" layer="1"/>
-<wire x1="174.3625" y1="73.9775" x2="175.26" y2="73.08" width="0.254" layer="1"/>
+<contactref element="R129" pad="2"/>
+<wire x1="0.4445" y1="-14.2875" x2="149.733" y2="73.3425" width="0" layer="19" extent="1-1"/>
 </signal>
 <signal name="N$39">
@@
 <signal name="CROSSFADER_OUT">
 <contactref element="R110" pad="1"/>
-<contactref element="J26" pad="TIP_B@1" route="any" routetag="G$1.TIP"/>
-<contactref element="J26" pad="TIP_T@3" route="any" routetag="G$1.TIP"/>
 <contactref element="IC6" pad="14"/>
 <wire x1="146.8755" y1="65.7225" x2="146.8755" y2="64.643" width="0.254" layer="1"/>
@@
 <wire x1="167.9575" y1="53.34" x2="168.91" y2="53.34" width="0.254" layer="1"/>
 <wire x1="168.91" y1="53.34" x2="169.8625" y2="52.3875" width="0.254" layer="1"/>
-<wire x1="169.8625" y1="52.3875" x2="169.8625" y2="35.56" width="0.254" layer="1"/>
-<wire x1="169.8625" y1="35.56" x2="170.4975" y2="34.925" width="0.254" layer="1"/>
-<wire x1="170.4975" y1="34.925" x2="175.205" y2="34.925" width="0.254" layer="1"/>
-<wire x1="175.205" y1="34.925" x2="175.26" y2="34.98" width="0.254" layer="1"/>
 <wire x1="153.035" y1="62.23" x2="154.94" y2="62.23" width="0.254" layer="16"/>
 <wire x1="162.555009375" y1="56.519990625" x2="165.735" y2="53.34" width="0.254" layer="16"/>
+<contactref element="R128" pad="2"/>
+<wire x1="0.4445" y1="-11.7475" x2="145.6722" y2="67.5825" width="0" layer="19" extent="1-1"/>
 </signal>
 <signal name="CV_IN">
@@
 <wire x1="31.115" y1="30.48" x2="31.115" y2="31.5087" width="0.254" layer="1"/>
 </signal>
+<signal name="N$125">
+<contactref element="J26" pad="TIP_T@3" route="any" routetag="G$1.TIP"/>
+<contactref element="J26" pad="TIP_B@1" route="any" routetag="G$1.TIP"/>
+<contactref element="R128" pad="1"/>
+<wire x1="-1.0795" y1="-11.7475" x2="175.26" y2="34.98" width="0" layer="19" extent="1-1"/>
+</signal>
+<signal name="N$126">
+<contactref element="J10" pad="TIP_T@3" route="any" routetag="G$1.TIP"/>
+<contactref element="J10" pad="TIP_B@1" route="any" routetag="G$1.TIP"/>
+<contactref element="R129" pad="1"/>
+<wire x1="-1.0795" y1="-14.2875" x2="175.26" y2="73.08" width="0" layer="19" extent="1-1"/>
+</signal>
 </signals>

Commit message: tiny overstuur schematic fixes
Parts:
- added R130, R131, R132, R133, R134, R135: 56, OPL:R0603
Connections:
- new net N$127: J8.TIP_B@1, J8.TIP_T@3, R130.1
- new net N$128: J5.TIP_B@1, J5.TIP_T@3, R131.1
- new net N$129: IC2.14, R133.2, R16.1
- new net N$130: J12.TIP_B@1, J12.TIP_T@3, R132.1
- new net N$131: J27.TIP_B@1, J27.TIP_T@3, R134.1
- new net N$132: J3.TIP_B@1, J3.TIP_T@3, R135.1
- net N$18: now also R130.2; no longer J8.TIP_B@1, J8.TIP_T@3
- net N$23: now also R131.2; no longer J5.TIP_B@1, J5.TIP_T@3
- net N$28: now also R132.2; no longer J12.TIP_B@1, J12.TIP_T@3
- net N$33: now also R133.1; no longer IC2.14, R16.1
- net N$4: now also R134.2; no longer J27.TIP_B@1, J27.TIP_T@3
- net VCA_OUTPUT2: now also R135.2; no longer J3.TIP_B@1, J3.TIP_T@3
Routing:
- net N$33: track 103.9 -> 0.00 mm, vias 4 -> 0
- net N$28: track 95.3 -> 2.20 mm, vias 4 -> 0
- net N$4: track 32.1 -> 24.0 mm
- net N$18: track 62.1 -> 57.6 mm
- net VCA_OUTPUT2: track 183.6 -> 179.5 mm
- net N$23: track 49.1 -> 45.7 mm
