File: Development/Eurorack Set 12/SimpleKeyboardTeensy.sch (EAGLE design)
At the start: 151 parts, among them IC1 74AC04D, SW46 C_1, SW47 C#1, SW48 D_1, SW49 D#1, SW50 E_1, SW51 F_1, SW52 F#1, SW53 G_1, SW54 G#1, SW55 A_2, SW56 A#2, SW57 B_2, SW58 C_2, SW59 C#2, SW60 D_2, SW61 D#2, SW62 E_2, SW63 F_2, SW64 F#2, SW65 G_2, SW66 G#2, SW67 A_3, SW68 A#3, SW69 B_3, SW70 C_3, SW71 C#3, SW72 D_3, SW73 D#3, SW74 E_3, SW75 Right, SW76 Up, SW77 Down, SW78 Stop, SW79 Oct Down, SW80 Left, SW81 Play, SW82 Continue, SW83 Record, SW84 Empty, SW85 Oct Up, SW86 Delete, SW87 Insert, SW88 Sequence, SW89 Pattern, SW90 Machine

Commit message: TeensyKeyboard
Parts:
- added C13: 100n, OPL:C-0603
- added C14: 1u, OPL:C-0603
- added C15, C16: 22p, OPL:C-0603
- added ISP1: AVRISP-6, adafruit:AVRISP-6
- added JP1: USB-B, SparkFun-Connectors:USBPTH
- added LED13, LED14, LED15, LED16, LED17, LED18, LED19, LED20, LED21, LED22, LED23, LED24, LED25, LED26, LED27, LED28, LED29, LED30, LED31, LED32, LED33, LED34, LED35, LED36, LED37, LED38, LED39, LED40, LED41, LED42, LED43, LED44, LED45, LED46, LED47, LED48, LED49, LED50, LED51, LED52, LED53, LED54, LED55, LED56, LED57: WS2812B3535, EurorackModularParts:WS2812B3535
- added R10: 1M, OPL:R-0603
- added R11, R9: 10k, OPL:R-0603
- added R7, R8: 22, OPL:R-0603
- added U$60: RESONATOR, EurorackModularParts:RESONATOR
- added U$61: 2PSWITCH_SMT_SIDEMOUNT, zephod-components:2PSWITCH_SMT_SIDEMOUNT
- added U1: ATMEGA32U4-MU, IC:ATMEGA32U4-MU
Connections:
- new net MISO: ISP1.MISO, U1.PB3(PD0/PCINT3/MISO)
- new net MODE: R11.2, U$46.5, U$61.A, U1.PD4(ICP1/ADC8)
- new net MOSI: ISP1.MOSI, U1.PB2(PDI/PCINT2/MOSI)
- new net N$100: JP1.D+, R8.2
- new net N$101: LED32.DO, LED33.DI
- new net N$102: LED43.DO, LED44.DI
- new net N$103: LED44.DO, LED45.DI
- new net N$104: LED45.DO, LED46.DI
- new net N$105: LED46.DO, LED47.DI
- new net N$106: LED48.DO, LED49.DI
- new net N$107: LED49.DO, LED50.DI
- new net N$108: LED50.DO, LED51.DI
- new net N$109: LED51.DO, LED52.DI
- new net N$110: C13.1, U1.AREF
- new net N$111: R8.1, U1.D+
- new net N$112: LED42.DO, LED43.DI
- new net N$113: LED53.DO, LED54.DI
- new net N$114: LED54.DO, LED55.DI
- new net N$115: LED55.DO, LED56.DI
- new net N$116: LED56.DO, LED57.DI
- new net N$117: R7.1, U1.D-
- new net N$118: C14.1, U1.UCAP
- new net N$119: C15.1, R10.1, U$60.XTAL1, U1.XTAL1
- new net N$120: C16.1, R10.2, U$60.XTAL2, U1.XTAL2
- new net N$123: LED52.DO, LED53.DI
- new net N$48: LED13.DO, LED14.DI
- new net N$70: LED14.DO, LED15.DI
- new net N$71: LED15.DO, LED16.DI
- new net N$72: LED16.DO, LED17.DI
- new net N$73: LED18.DO, LED19.DI
- new net N$74: LED19.DO, LED20.DI
- new net N$75: LED20.DO, LED21.DI
- new net N$76: LED21.DO, LED22.DI
- new net N$77: LED17.DO, LED18.DI
- new net N$78: LED27.DO, LED28.DI
- new net N$79: LED12.DO, LED13.DI
- new net N$80: LED23.DO, LED24.DI
- new net N$81: LED24.DO, LED25.DI
- new net N$82: LED25.DO, LED26.DI
- new net N$83: LED26.DO, LED27.DI
- new net N$84: LED28.DO, LED29.DI
- new net N$85: LED29.DO, LED30.DI
- new net N$86: LED30.DO, LED31.DI
- new net N$87: LED31.DO, LED32.DI
- new net N$88: LED37.DO, LED38.DI
- new net N$89: LED47.DO, LED48.DI
- new net N$90: LED22.DO, LED23.DI
- new net N$91: LED33.DO, LED34.DI
- new net N$92: LED34.DO, LED35.DI
- new net N$93: LED35.DO, LED36.DI
- new net N$94: LED36.DO, LED37.DI
- new net N$95: LED38.DO, LED39.DI
- new net N$96: LED39.DO, LED40.DI
- new net N$97: LED40.DO, LED41.DI
- new net N$98: LED41.DO, LED42.DI
- new net N$99: JP1.D-, R7.2
- new net RESET: ISP1.RST, R9.1, U1.!RESET
- new net SCLK: ISP1.SCK, U1.PB1(PCINT1/SCLK)
- net 5V: now also ISP1.VCC, JP1.VBUS, LED13.VDD, LED14.VDD, LED15.VDD, LED16.VDD, LED17.VDD, LED18.VDD, LED19.VDD, LED20.VDD, LED21.VDD, LED22.VDD, LED23.VDD, LED24.VDD, LED25.VDD, LED26.VDD, LED27.VDD, LED28.VDD, LED29.VDD, LED30.VDD, LED31.VDD, LED32.VDD, LED33.VDD, LED34.VDD, LED35.VDD, LED36.VDD, LED37.VDD, LED38.VDD, LED39.VDD, LED40.VDD, LED41.VDD, LED42.VDD, LED43.VDD, LED44.VDD, LED45.VDD, LED46.VDD, LED47.VDD, LED48.VDD, LED49.VDD, LED50.VDD, LED51.VDD, LED52.VDD, LED53.VDD, LED54.VDD, LED55.VDD, LED56.VDD, LED57.VDD, R11.1, R9.2, U1.AVCC@1, U1.AVCC@2, U1.UVCC, U1.VBUS, U1.VCC@1, U1.VCC@2
- net COL1: now also U1.PF7(ADC7/TDI)
- net COL2: now also U1.PF6(ADC6/TDO)
- net COL3: now also U1.PF5(ADC5/TMS)
- net COL4: now also U1.PF4(ADC4/TCK)
- net COL5: now also U1.PF1(ADC1)
- net GND: now also C13.2, C14.2, C15.2, C16.2, ISP1.GND, JP1.GND, LED13.GND, LED14.GND, LED15.GND, LED16.GND, LED17.GND, LED18.GND, LED19.GND, LED20.GND, LED21.GND, LED22.GND, LED23.GND, LED24.GND, LED25.GND, LED26.GND, LED27.GND, LED28.GND, LED29.GND, LED30.GND, LED31.GND, LED32.GND, LED33.GND, LED34.GND, LED35.GND, LED36.GND, LED37.GND, LED38.GND, LED39.GND, LED40.GND, LED41.GND, LED42.GND, LED43.GND, LED44.GND, LED45.GND, LED46.GND, LED47.GND, LED48.GND, LED49.GND, LED50.GND, LED51.GND, LED52.GND, LED53.GND, LED54.GND, LED55.GND, LED56.GND, LED57.GND, U$60.GND, U$61.B, U$61.GND1, U$61.GND2, U1.GND@1, U1.GND@2, U1.GND@3, U1.GND@4, U1.UGND
- net LED: now also U1.PD7(T0/OC4D/ADC10)
- net MIDI1: now also U1.PD3(TXD1/INT3)
- net MIDI2: now also U1.PD2(RXD1/INT2)
- net ROW1: now also U1.PB0(SS/PCINT0)
- net ROW2: now also U1.PC7(ICP3/CLK0/OC4A)
- net ROW3: now also U1.PD6(T1/ADC9/!OC4D)
- net ROW4: now also U1.PB7(PCINT7/OC0A/OC1C/!RTS)
- net ROW5: now also U1.PB6(PCINT6/OC1B/OC4B/ADC13)
- net ROW6: now also U1.PB5(PCINT5/OC1A/ADC12/!OC4B)
- net ROW7: now also U1.PB4(PCINT4/ADC11)
- net ROW8: now also U1.PE6(INT.6/AIN0)
- net ROW9: now also U1.PC6(OC3A/!OC4A)

Commit message: Speaker order - Simplekeyboard TRS midi - Overstuur design
Parts:
- added J1: AUDIO-CONNECTOR-6P-SMD-3440030P1, OPL:AUDIO-CONNECTOR-6P-SMD-3440030P1
- added SW1: SWITCH-2CH-6P-3010010P1, OPL:SWITCH-2CH-6P-3010010P1
- added U$63: TINRS_ARTWORKTINYDATE, EurorackModularParts:TINRS_ARTWORKTINYDATE
- SW83: value Record -> Note Off
Connections:
- new net N$121: J1.R, J1.RS, SW1.COM1
- new net N$122: J1.L, J1.LS, SW1.COM2
- net GND: now also J1.COM1, J1.COM2
- net N$62: now also SW1.CH1A, SW1.CH2B
- net N$64: now also SW1.CH1B, SW1.CH2A
Other:
- moved on the sheet: R5
Changed lines of the file:
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@@
 <class number="0" name="default" width="0.254" drill="0">
+</class>
+<class number="1" name="power" width="0.381" drill="0">
 </class>
 </classes>
@@
 <part name="SW81" library="Cherry_MX_v7.0" deviceset="CHERRY_MX" device="_WITH_FIXING_PINS" value="Play"/>
 <part name="SW82" library="Cherry_MX_v7.0" deviceset="CHERRY_MX" device="_WITH_FIXING_PINS" value="Continue"/>
-<part name="SW83" library="Cherry_MX_v7.0" deviceset="CHERRY_MX" device="_WITH_FIXING_PINS" value="Record"/>
+<part name="SW83" library="Cherry_MX_v7.0" deviceset="CHERRY_MX" device="_WITH_FIXING_PINS" value="Note Off"/>
 <part name="SW84" library="Cherry_MX_v7.0" deviceset="CHERRY_MX" device="_WITH_FIXING_PINS" value="Empty"/>
 <part name="SW85" library="Cherry_MX_v7.0" deviceset="CHERRY_MX" device="_WITH_FIXING_PINS" value="Oct Up"/>
@@
 <part name="R11" library="OPL" deviceset="R*" device="-0603" value="10k"/>
 <part name="U$62" library="FenixBase" deviceset="5V" device=""/>
+<part name="SW1" library="OPL" deviceset="SWITCH-2CH-6P*" device="-3010010P1"/>
+<part name="J1" library="OPL" deviceset="AUDIO-CONNECTOR-6P-SMD" device="-3440030P1"/>
+<part name="GND37" library="FenixBase" deviceset="GND" device=""/>
+<part name="GND38" library="FenixBase" deviceset="GND" device=""/>
+<part name="U$63" library="EurorackModularParts" deviceset="TINRS_ARTWORK" device="TINYDATE"/>
 </parts>
 <sheets>
@@
 <instance part="R3" gate="R" x="-185.42" y="-30.48" rot="R180"/>
 <instance part="R4" gate="R" x="-187.96" y="-62.23" rot="R180"/>
-<instance part="R5" gate="R" x="-176.53" y="34.29" rot="R180"/>
+<instance part="R5" gate="R" x="-168.91" y="34.29" rot="R180"/>
 <instance part="R6" gate="R" x="-119.38" y="31.75" rot="R180"/>
-<instance part="U$13" gate="G$1" x="-172.72" y="34.29"/>
+<instance part="U$13" gate="G$1" x="-162.56" y="34.29"/>
 <instance part="U$14" gate="G$1" x="-115.57" y="31.75"/>
 <instance part="U$15" gate="G$1" x="-12.7" y="-147.32"/>
@@
 <instance part="R11" gate="R" x="156.21" y="-541.02" rot="R270"/>
 <instance part="U$62" gate="G$1" x="156.21" y="-537.21"/>
+<instance part="SW1" gate="SW" x="-264.16" y="20.32"/>
+<instance part="J1" gate="J" x="-228.6" y="48.26" rot="R90"/>
+<instance part="GND37" gate="1" x="-215.9" y="59.69" rot="R90"/>
+<instance part="GND38" gate="1" x="-241.3" y="57.15" rot="R270"/>
+<instance part="U$63" gate="G$1" x="-261.62" y="-11.43"/>
 </instances>
 <busses>
@@
 <pinref part="GND36" gate="1" pin="GND"/>
 </segment>
+<segment>
+<pinref part="J1" gate="J" pin="COM2"/>
+<pinref part="GND37" gate="1" pin="GND"/>
+</segment>
+<segment>
+<pinref part="J1" gate="J" pin="COM1"/>
+<pinref part="GND38" gate="1" pin="GND"/>
+</segment>
 </net>
 <net name="ROW9" class="0">
@@
 <pinref part="R5" gate="R" pin="1"/>
 <pinref part="U$13" gate="G$1" pin="5V"/>
+<wire x1="-162.56" y1="34.29" x2="-165.1" y2="34.29" width="0.1524" layer="91"/>
 </segment>
 <segment>
@@
 <pinref part="U$11" gate="G$1" pin="4"/>
 <pinref part="R5" gate="R" pin="2"/>
+<wire x1="-172.72" y1="34.29" x2="-175.26" y2="34.29" width="0.1524" layer="91"/>
+<wire x1="-175.26" y1="34.29" x2="-180.34" y2="34.29" width="0.1524" layer="91"/>
+<wire x1="-175.26" y1="34.29" x2="-175.26" y2="15.24" width="0.1524" layer="91"/>
+<pinref part="SW1" gate="SW" pin="CH2B"/>
+<wire x1="-175.26" y1="15.24" x2="-251.46" y2="15.24" width="0.1524" layer="91"/>
+<wire x1="-251.46" y1="15.24" x2="-257.81" y2="15.24" width="0.1524" layer="91"/>
+<wire x1="-257.81" y1="15.24" x2="-257.81" y2="17.78" width="0.1524" layer="91"/>
+<wire x1="-251.46" y1="15.24" x2="-251.46" y2="31.75" width="0.1524" layer="91"/>
+<pinref part="SW1" gate="SW" pin="CH1A"/>
+<wire x1="-251.46" y1="31.75" x2="-270.51" y2="31.75" width="0.1524" layer="91"/>
+<wire x1="-270.51" y1="31.75" x2="-270.51" y2="22.86" width="0.1524" layer="91"/>
+<junction x="-251.46" y="15.24"/>
+<junction x="-175.26" y="34.29"/>
 </segment>
 </net>
@@
 <pinref part="U$11" gate="G$1" pin="5"/>
 <wire x1="-205.74" y1="34.29" x2="-207.01" y2="34.29" width="0.1524" layer="91"/>
-<wire x1="-207.01" y1="34.29" x2="-207.01" y2="5.08" width="0.1524" layer="91"/>
+<wire x1="-207.01" y1="34.29" x2="-207.01" y2="22.86" width="0.1524" layer="91"/>
 <pinref part="R3" gate="R" pin="1"/>
+<wire x1="-207.01" y1="22.86" x2="-207.01" y2="5.08" width="0.1524" layer="91"/>
 <wire x1="-207.01" y1="5.08" x2="-181.61" y2="5.08" width="0.1524" layer="91"/>
 <wire x1="-181.61" y1="5.08" x2="-181.61" y2="-30.48" width="0.1524" layer="91"/>
+<pinref part="SW1" gate="SW" pin="CH2A"/>
+<wire x1="-257.81" y1="22.86" x2="-254" y2="22.86" width="0.1524" layer="91"/>
+<wire x1="-254" y1="22.86" x2="-207.01" y2="22.86" width="0.1524" layer="91"/>
+<wire x1="-254" y1="22.86" x2="-254" y2="11.43" width="0.1524" layer="91"/>
+<pinref part="SW1" gate="SW" pin="CH1B"/>
+<wire x1="-254" y1="11.43" x2="-270.51" y2="11.43" width="0.1524" layer="91"/>
+<wire x1="-270.51" y1="11.43" x2="-270.51" y2="17.78" width="0.1524" layer="91"/>
+<junction x="-207.01" y="22.86"/>
+<junction x="-254" y="22.86"/>
 </segment>
 </net>
@@
 </segment>
 </net>
+<net name="N$121" class="0">
+<segment>
+<pinref part="J1" gate="J" pin="R"/>
+<pinref part="J1" gate="J" pin="RS"/>
+<wire x1="-238.76" y1="52.07" x2="-238.76" y2="39.37" width="0.1524" layer="91"/>
+<wire x1="-238.76" y1="39.37" x2="-278.13" y2="39.37" width="0.1524" layer="91"/>
+<wire x1="-278.13" y1="39.37" x2="-278.13" y2="20.32" width="0.1524" layer="91"/>
+<pinref part="SW1" gate="SW" pin="COM1"/>
+<wire x1="-278.13" y1="20.32" x2="-270.51" y2="20.32" width="0.1524" layer="91"/>
+<junction x="-238.76" y="39.37"/>
+</segment>
+</net>
+<net name="N$122" class="0">
+<segment>
+<pinref part="J1" gate="J" pin="L"/>
+<pinref part="J1" gate="J" pin="LS"/>
+<wire x1="-218.44" y1="41.91" x2="-218.44" y2="36.83" width="0.1524" layer="91"/>
+<wire x1="-218.44" y1="36.83" x2="-219.71" y2="36.83" width="0.1524" layer="91"/>
+<wire x1="-219.71" y1="36.83" x2="-219.71" y2="29.21" width="0.1524" layer="91"/>
+<wire x1="-219.71" y1="29.21" x2="-248.92" y2="29.21" width="0.1524" layer="91"/>
+<wire x1="-248.92" y1="29.21" x2="-248.92" y2="20.32" width="0.1524" layer="91"/>
+<pinref part="SW1" gate="SW" pin="COM2"/>
+<wire x1="-248.92" y1="20.32" x2="-257.81" y2="20.32" width="0.1524" layer="91"/>
+<junction x="-219.71" y="36.83"/>
+</segment>
+</net>
