File: Development/Eurorack Set 12/MiniKeyb.sch (EAGLE design)
At the start: 63 parts, among them J1 MINI-USB-5P-3400030P1, SW46 1, SW47 2, SW48 3, SW49 4, SW51 5, SW52 6, SW53 7, SW54 8, SW55 9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

Commit message: Minikeyb, STM32
Parts:
- removed J1: MINI-USB-5P-3400030P1, OPL:MINI-USB-5P-3400030P1
- removed R11: 10k, OPL:R-0603
- removed U$61: 2PSWITCH_SMT_SIDEMOUNT, zephod-components:2PSWITCH_SMT_SIDEMOUNT
- added C1, C2, C3, C4: 100n, OPL:C-0603
- added D15, D16: CGRM4001-G, diode:CGRM4001-G
- added JP2, JP3: (no value), SparkFun-Connectors:M03X2
- added LED1, LED2: WS2812B3535, EurorackModularParts:WS2812B3535
- added SW1: A, Cherry_MX_v7.0:CHERRY_MX_WITH_FIXING_PINS
- added SW2: B, Cherry_MX_v7.0:CHERRY_MX_WITH_FIXING_PINS
Connections:
- removed net COL5: U1.PF1(ADC1)
- removed net MIDI1: U1.PD3(TXD1/INT3)
- removed net MIDI2: U1.PD2(RXD1/INT2)
- removed net MODE: R11.2, U$61.A, U1.PD4(ICP1/ADC8)
- removed net N$30: D13.A, D2.A, D6.A, D9.A
- removed net ROW6: U1.PB5(PCINT5/OC1A/ADC12/!OC4B)
- removed net ROW7: U1.PB4(PCINT4/ADC11)
- removed net ROW8: U1.PE6(INT.6/AIN0)
- removed net ROW9: U1.PC6(OC3A/!OC4A)
- new net A1: JP3.1, U1.PF1(ADC1)
- new net A2: JP3.2, U1.PF0(ADC0)
- new net A3: JP3.3, U1.PF5(ADC5/TMS)
- new net A4: JP3.4, U1.PF4(ADC4/TCK)
- new net B1: JP2.1, U1.PF7(ADC7/TDI)
- new net B2: JP2.2, U1.PF6(ADC6/TDO)
- new net B3: JP2.3, U1.PD4(ICP1/ADC8)
- new net B4: JP2.4, U1.PC6(OC3A/!OC4A)
- new net N$15: D15.C, SW1.1
- new net N$16: D16.C, SW2.1
- new net N$17: LED1.DO, LED2.DI
- new net N$18: LED1.DI, LED28.DO
- net 5V: now also C1.2, C2.2, C3.2, C4.2, JP2.5, JP3.5, LED1.VDD, LED2.VDD; no longer R11.1
- net COL1: now also D15.A, U1.PD3(TXD1/INT3); no longer U1.PF7(ADC7/TDI)
- net COL2: now also D13.A, D16.A, D2.A, D6.A, D9.A, U1.PD2(RXD1/INT2); no longer U1.PF6(ADC6/TDO)
- net COL3: now also U1.PD1(SDA/INT1); no longer U1.PF5(ADC5/TMS)
- net COL4: now also U1.PD0(OC0B/SCL/INT0); no longer U1.PF4(ADC4/TCK)
- net GND: now also C1.1, C2.1, C3.1, C4.1, JP2.6, JP3.6, LED1.GND, LED2.GND; no longer U$61.B, U$61.GND1, U$61.GND2
- net ROW5: now also SW1.2, SW2.2
