File: Development/StageProjecten/STM32test/stm32_02.brd (EAGLE design)
At the start: 60.2 x 106.5 mm, 172 parts, among them IC1 LD1117AS33TR, IC2 STM32F10XCXT6, IC3 MCP6004, IC4 TL074TSSOP14, IC5 TL074TSSOP14, IC6 MCP4822-E/SN, IC7 MCP4822-E/SN, IC8 74HC595D, IC9 74HC595D, J1 POWERSHROUDED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

Commit message: new boardfile
Parts:
- moved C31 82.2 mm to (99.2, 71.6)
- moved IC9 82.2 mm to (93.5, 66.8)
- moved C34 59.6 mm to (91.3, 89.4)
- moved IC7 59.6 mm to (87.8, 87.6)
- moved C20 57.6 mm to (79.2, 103.2)
- moved C21 57.6 mm to (71.3, 103.2)
- moved C24 57.6 mm to (75.2, 107.2)
- moved C25 57.6 mm to (75.2, 97.0)
- moved IC5 57.6 mm to (75.2, 102.1)
- moved R43 57.6 mm to (79.2, 104.8)
- moved R45 57.6 mm to (79.2, 101.0)
- moved R49 57.6 mm to (71.3, 104.8)
- moved R50 57.6 mm to (72.1, 107.2)
- moved R51 57.6 mm to (71.3, 101.0)
- moved R44 57.6 mm to (78.4, 107.2)
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Connections:
- net N$79 renamed RESET
Routing:
- net BTN_IN3: track 66.6 -> 6.00 mm, vias 2 -> 0
- net BTN_IN2: track 34.4 -> 6.00 mm, vias 2 -> 0
- net BTN_IN4: track 31.8 -> 6.00 mm, vias 2 -> 0
- net GND: track 48.0 -> 26.0 mm, vias 34 -> 20
- net LED_BTN4: track 16.8 -> 0.00 mm, vias 2 -> 0
- net LED_BTN3: track 12.2 -> 0.00 mm
- net CS1: track 11.5 -> 0.00 mm
- net CS2: track 10.7 -> 0.00 mm
- net SWDIO: track 9.21 -> 0.00 mm, vias 2 -> 0
- net N$52: track 9.18 -> 0.00 mm
- net N$47: track 8.23 -> 0.00 mm, vias 2 -> 0
- net SWCLK: track 7.29 -> 0.00 mm
- net RESET: track 18.1 -> 10.9 mm, vias 5 -> 2
- net SCK1: track 7.01 -> 0.00 mm, vias 2 -> 0
- net N$48: track 9.18 -> 2.71 mm
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
Commit message: more edits to board
Parts:
- moved R70 124.8 mm to (31.1, 105.1), turned to 180 degrees
- moved R71 122.9 mm to (27.3, 105.1), turned to 180 degrees
- moved IC7 70.1 mm to (17.8, 83.3), turned to 0 degrees
- moved C20 58.7 mm to (27.6, 75.2)
- moved C21 58.7 mm to (19.7, 75.2)
- moved C24 58.7 mm to (23.7, 79.2)
- moved C25 58.7 mm to (23.7, 69.1)
- moved IC5 58.7 mm to (23.7, 74.1)
- moved R43 58.7 mm to (27.6, 76.8)
- moved R44 58.7 mm to (26.8, 79.2)
- moved R45 58.7 mm to (27.6, 73.0)
- moved R46 58.7 mm to (27.6, 71.4)
- moved R48 58.7 mm to (22.1, 79.2)
- moved R49 58.7 mm to (19.7, 76.8)
- moved R50 58.7 mm to (20.5, 79.2)
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Connections:
- net BTN_IN2: now also IC2.31; no longer IC2.29
- net BTN_IN4: now also IC2.29; no longer IC2.31
Routing:
- net BTN_IN2: track 6.00 -> 36.9 mm, vias 0 -> 2
- net BTN_IN4: track 6.00 -> 33.5 mm, vias 0 -> 2
- net MOSI2: track 0.00 -> 21.8 mm
- net SCK2: track 0.00 -> 19.0 mm
- net CS2: track 0.00 -> 17.5 mm
- net BTN_IN3: track 6.00 -> 23.2 mm, vias 0 -> 2
- net 3.3V: track 42.9 -> 58.5 mm, vias 7 -> 6
- net GND: track 26.0 -> 40.5 mm, vias 20 -> 35
- net CS1: track 0.00 -> 14.0 mm
- net SCK1: track 0.00 -> 13.1 mm
- net MOSI1: track 0.00 -> 12.3 mm
- net N$39: track 0.00 -> 9.70 mm
- net N$33: track 0.00 -> 8.85 mm
- net SCK595: track 0.00 -> 5.52 mm
- net SER595: track 0.00 -> 5.46 mm
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
Commit message: nieuwste board!
Parts:
- moved IC6 7.60 mm to (36.2, 79.7), turned to 270 degrees
- moved IC7 6.52 mm to (23.2, 79.7), turned to 270 degrees
- moved U1 6.35 mm to (30.3, 35.4)
- moved IC1 6.35 mm to (31.8, 41.9)
- moved C18 4.61 mm to (40.8, 70.6)
- moved C19 4.61 mm to (32.9, 70.6)
- moved C20 4.61 mm to (27.8, 70.6)
- moved C21 4.61 mm to (19.8, 70.6)
- moved C22 4.61 mm to (36.8, 74.6)
- moved C23 4.61 mm to (36.8, 64.5)
- moved C24 4.61 mm to (23.8, 74.6)
- moved C25 4.61 mm to (23.8, 64.5)
- moved IC4 4.61 mm to (36.8, 69.5)
- moved IC5 4.61 mm to (23.8, 69.5)
- moved R30 4.61 mm to (38.4, 74.6)
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Routing:
- net MOSI2: track 21.8 -> 0.00 mm
- net SCK2: track 19.0 -> 0.00 mm
- net BTN_IN2: track 36.9 -> 18.0 mm, vias 2 -> 0
- net CS2: track 17.5 -> 0.00 mm
- net BTN_IN3: track 23.2 -> 6.00 mm, vias 2 -> 0
- net CS1: track 14.0 -> 0.00 mm
- net SCK1: track 13.1 -> 0.00 mm
- net BTN_IN4: track 33.5 -> 20.6 mm, vias 2 -> 0
- net MOSI1: track 12.3 -> 0.00 mm
- net N$39: track 9.70 -> 2.09 mm
- net N$33: track 8.85 -> 2.14 mm
- net GATE_IN4: track 4.08 -> 0.00 mm
- net 3.3V: track 58.5 -> 55.7 mm
- net GND: track 40.5 -> 37.8 mm, vias 35 -> 29
- net N$45: track 4.56 -> 2.09 mm
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
Commit message: power beter
Parts:
- X2: value USB-B-FEMALE -> USB_B_FEMALE_VERT; device ld-components:FCI61729 -> ld-components:USB_B_VERT
- moved R1 44.9 mm to (27.0, 32.1)
- moved C6 44.6 mm to (27.0, 33.5)
- moved C5 43.2 mm to (29.4, 29.1), turned to 90 degrees
- moved U$7 42.5 mm to (24.8, 47.0), turned to 0 degrees
- moved U$38 40.2 mm to (24.8, 41.9), turned to 180 degrees
- moved C2 39.9 mm to (32.4, 36.7)
- moved U$37 39.3 mm to (27.3, 47.0), turned to 0 degrees
- moved C1 39.0 mm to (32.4, 34.9)
- moved U$8 37.5 mm to (27.3, 41.9), turned to 180 degrees
- moved X2 34.5 mm to (13.0, 47.0), flipped to the bottom, turned to 0 degrees
- moved C4 32.2 mm to (37.9, 44.8)
- moved C3 31.8 mm to (36.5, 41.8), turned to 90 degrees
- moved U1 3.16 mm to (27.3, 36.4), turned to 270 degrees
- moved IC1 0.65 mm to (32.4, 41.8)
- moved C9 0.64 mm to (32.9, 80.2)
Connections:
- net GND: now also X2.G1, X2.G2; no longer X2.P$1, X2.P$2
Routing:
- net 12V: track 2.80 -> 32.4 mm
- net -12V: track 2.80 -> 21.3 mm
- net 3.3V: track 55.7 -> 72.1 mm
- net MOSI1: track 0.00 -> 14.9 mm
- net BTN_IN4: track 20.6 -> 6.00 mm
- net -5V: track 0.00 -> 10.6 mm
- net CS1: track 0.00 -> 9.48 mm
- net SCK1: track 0.00 -> 5.54 mm
- net BTN_IN2: track 18.0 -> 13.9 mm
- net USB-: track 3.77 -> 0.00 mm, vias 1 -> 0
- net USB+: track 2.49 -> 0.00 mm, vias 1 -> 0
- net SWCLK: track 0.00 -> 2.44 mm

Commit message: Chips neergezet
Parts:
- moved R55 145.7 mm to (51.8, 44.0), turned to 180 degrees
- moved T6 144.9 mm to (55.2, 52.7), turned to 270 degrees
- moved T5 141.1 mm to (55.2, 43.2), turned to 270 degrees
- moved R65 110.7 mm to (51.8, 45.6), turned to 180 degrees
- moved R64 106.5 mm to (51.8, 47.1), turned to 180 degrees
- moved R62 98.9 mm to (51.8, 48.7), turned to 180 degrees
- moved R61 94.8 mm to (51.8, 50.3), turned to 180 degrees
- moved R59 87.3 mm to (51.8, 51.9), turned to 180 degrees
- moved IC9 87.1 mm to (6.51, 71.0), turned to 0 degrees
- moved R58 83.1 mm to (51.8, 53.5), turned to 180 degrees
- moved C14 82.4 mm to (2.70, 42.5), turned to 0 degrees
- moved T8 81.2 mm to (55.2, 46.4), turned to 270 degrees
- moved R11 80.5 mm to (2.70, 44.1), turned to 0 degrees
- moved R7 78.5 mm to (2.70, 45.7), turned to 0 degrees
- moved R8 76.6 mm to (2.70, 47.3), turned to 0 degrees
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Routing:
- net N$16: track 0.00 -> 53.3 mm
- net N$62: track 0.00 -> 50.0 mm
- net N$46: track 0.00 -> 44.3 mm
- net N$58: track 0.00 -> 42.4 mm
- net USB+: track 0.00 -> 40.6 mm
- net USB-: track 0.00 -> 37.9 mm
- net N$12: track 0.00 -> 35.9 mm
- net N$54: track 0.00 -> 34.9 mm
- net N$40: track 0.00 -> 33.3 mm
- net N$8: track 0.00 -> 26.3 mm
- net N$34: track 0.00 -> 22.6 mm
- net 3.3V: track 72.1 -> 93.6 mm
- net -5V: track 10.6 -> 31.3 mm, vias 0 -> 2
- net GATE_OUT2: track 0.00 -> 17.9 mm
- net N$4: track 0.00 -> 17.4 mm
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
Commit message: Added final components?
Parts:
- removed R14, R19: 33k, OPL:R0603
- added C35, C36, C37, C38: 100nF, OPL:C0603
- added R4: 20r, OPL:R0603
- R9: value 33k -> 20r
- moved R9 108.0 mm to (-12.9, -24.0)
- moved R54 1.59 mm to (47.6, 17.1)
- moved R63 1.59 mm to (47.6, 6.99)
- moved R57 1.59 mm to (47.6, 27.3)
- moved R60 1.59 mm to (47.6, 37.5)
- moved C4 1.11 mm to (36.7, 46.4)
- moved C1 0.63 mm to (31.8, 34.9)
- turned D3 to 180 degrees
- turned D4 to 180 degrees
- turned D5 to 180 degrees
- turned D6 to 180 degrees
- flipped J1 to the top
Connections:
- new net N$56: IC2.32, R4.2
- new net N$60: IC2.33, R9.2
- net LED_IN1: now also IC9.6, R76.2; no longer IC9.4, R74.2
- net LED_IN2: now also IC9.7, R77.2; no longer IC9.5, R75.2
- net LED_IN3: now also IC9.5, R75.2; no longer IC9.6, R76.2
- net LED_IN4: now also IC9.4, R74.2; no longer IC9.7, R77.2
- net N$11: now also C37.1; no longer R14.1
- net N$13: no longer R14.2
- net N$15: now also C38.1; no longer R19.1
- net N$17: no longer R19.2
- net N$3: now also C35.1
- net N$7: now also C36.1; no longer R9.1
- net N$9: no longer R9.2
- net POT1: now also C35.2
- net POT2: now also C36.2
- net POT3: now also C37.2
- net POT4: now also C38.2
- net USB+: now also R9.1; no longer IC2.33
- net USB-: now also R4.1; no longer IC2.32
Routing:
- net LED_OUT4: track 0.00 -> 32.5 mm
- net USB+: track 40.6 -> 8.59 mm
- net USB-: track 37.9 -> 5.84 mm
- net LED_OUT3: track 0.00 -> 22.0 mm
- net LED_OUT2: track 0.00 -> 11.8 mm
- net N$25: track 0.00 -> 7.04 mm
- net 12V: track 23.4 -> 24.2 mm

Commit message: powertesters onderin
Parts:
- moved C38 103.3 mm to (53.2, 60.2)
- moved C37 92.4 mm to (37.5, 60.6)
- moved R4 84.1 mm to (26.8, 52.7)
- moved C36 82.6 mm to (22.7, 60.2)
- moved R9 80.5 mm to (26.8, 46.0)
- moved C35 75.5 mm to (7.14, 60.8)
- moved U$37 43.8 mm to (34.1, 1.43), turned to 180 degrees
- moved U$8 43.8 mm to (29.1, 1.43), turned to 180 degrees
- moved R72 42.9 mm to (23.8, 46.0), turned to 180 degrees
- moved U$38 41.0 mm to (26.5, 1.43), turned to 180 degrees
- moved U$7 41.0 mm to (31.6, 1.43), turned to 180 degrees
- moved SJ1 36.1 mm to (13.0, 88.9), turned to 180 degrees
- moved C4 10.4 mm to (40.5, 36.7)
- moved C3 10.1 mm to (38.7, 36.2), turned to 270 degrees
- moved C18 0.16 mm to (41.0, 70.6)
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Connections:
- net LED_IN1: now also IC9.4, R74.2; no longer IC9.6, R76.2
- net LED_IN2: now also IC9.5, R75.2; no longer IC9.7, R77.2
- net LED_IN3: now also IC9.6, R76.2; no longer IC9.5, R75.2
- net LED_IN4: now also IC9.7, R77.2; no longer IC9.4, R74.2
Routing:
- net 12V: track 24.2 -> 69.5 mm
- net 3.3V: track 93.8 -> 138.5 mm
- net N$60: track 0.00 -> 39.2 mm
- net N$56: track 0.00 -> 32.3 mm
- net -5V: track 31.3 -> 61.1 mm
- net -12V: track 26.0 -> 54.7 mm
- net USB+: track 8.59 -> 4.13 mm
- net USB-: track 5.84 -> 2.63 mm
