File: Development/JacThing/PowerBoard.brd (EAGLE design)
At the start: 7.1 x 7.3 mm, 27 parts, among them J1 POWER_JACKSLT, J2 POWERSHROUDED, J3 POWERSHROUDED, J4 POWERSHROUDED, J5 POWERSHROUDED, J6 POWERSHROUDED

Commit message: RectangularThing LEDboard v1
Parts:
- removed JP1, JP3: (no value), EurorackModularParts:AUDIO-JACK-.25-INCH-HORIZ-PTH
- removed R7: 10k, OPL:R0603
- removed R8: 20k, OPL:R0603
- added C1, C2, C3: 100uF 50V, rcl:153CLV-1010
- added J7: POWERSHROUDED, EurorackModularParts:POWER_16_SHROUDED
- moved C15 99.4 mm to (118.0, 71.4), flipped to the top
- moved U$22 98.3 mm to (113.5, 57.1)
- moved U$28 97.6 mm to (120.7, 139.7)
- moved U$17 96.6 mm to (116.8, 65.8), flipped to the top
- moved C12 92.5 mm to (114.3, 71.4), flipped to the top
- moved J5 71.2 mm to (113.0, 118.1), turned to 90 degrees
- moved C19 53.9 mm to (86.4, 144.8), flipped to the top
- moved L6 53.9 mm to (95.2, 141.0), flipped to the top
- moved C18 53.9 mm to (86.4, 137.2), flipped to the top, turned to 90 degrees
- moved J6 43.2 mm to (47.0, 118.1), turned to 270 degrees
- moved U$19 40.7 mm to (108.0, 139.7)
- moved C16 32.5 mm to (69.8, 144.8), flipped to the top
- moved J2 30.9 mm to (113.0, 88.9), turned to 90 degrees
- moved L3 30.7 mm to (77.5, 141.0), flipped to the top
- moved D7 26.3 mm to (40.3, 136.8), flipped to the top, turned to 90 degrees
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Connections:
- removed net 3.3V: R7.1, R8.2
- removed net AUDIO_OUT_LEFT_RING: JP1.P$4
- removed net AUDIO_OUT_LEFT_TIP: JP1.P$6
- removed net AUDIO_OUT_RIGHT_RING: JP3.P$4
- removed net AUDIO_OUT_RIGHT_TIP: JP3.P$6
- removed net N$1: J2.10, J2.9, J3.10, J3.9, J4.10, J4.9, J5.10, J5.9, J6.10, J6.9
- removed net N$2: J2.3, J2.4, J2.5, J2.6, J2.7, J2.8, J3.3, J3.4, J3.5, J3.6, J3.7, J3.8, J4.3, J4.4, J4.5, J4.6, J4.7, J4.8, J5.3, J5.4, J5.5, J5.6, J5.7, J5.8, J6.3, J6.4, J6.5, J6.6, J6.7, J6.8
- removed net N$3: J2.1, J2.2, J3.1, J3.2, J4.1, J4.2, J5.1, J5.2, J6.1, J6.2
- removed net N$4: J2.11, J2.12, J3.11, J3.12, J4.11, J4.12, J5.11, J5.12, J6.11, J6.12
- net -12V: now also C2.-, J2.1, J2.2, J3.1, J3.2, J4.1, J4.2, J5.1, J5.2, J6.1, J6.2, J7.1, J7.2
- net 12V: now also C3.+, J2.10, J2.9, J3.10, J3.9, J4.10, J4.9, J5.10, J5.9, J6.10, J6.9, J7.10, J7.9
- net 5V_1: now also C1.+, J2.11, J2.12, J3.11, J3.12, J4.11, J4.12, J5.11, J5.12, J6.11, J6.12, J7.11, J7.12; no longer R7.2
- net GND: now also C1.-, C2.+, C3.-, J2.3, J2.4, J2.5, J2.6, J2.7, J2.8, J3.3, J3.4, J3.5, J3.6, J3.7, J3.8, J4.3, J4.4, J4.5, J4.6, J4.7, J4.8, J5.3, J5.4, J5.5, J5.6, J5.7, J5.8, J6.3, J6.4, J6.5, J6.6, J6.7, J6.8, J7.3, J7.4, J7.5, J7.6, J7.7, J7.8; no longer JP1.P$2, JP1.P$3, JP3.P$2, JP3.P$3, R8.1
- net N$6: now also J7.13, J7.14
- net N$7: now also J7.15, J7.16
Routing:
- added copper zone on layer 16, net GND
- removed copper zone on layer 1, net GND
Other:
- board size 7.1 x 7.3 mm -> 90 x 100 mm

Commit message: Jac Powerboard
Parts:
- moved L3 17.8 mm to (95.2, 141.0)
- moved L6 17.8 mm to (77.5, 141.0)
- moved C15 1.36 mm to (119.4, 71.1)
- moved C11 0.77 mm to (62.2, 141.0)
- moved C12 0.26 mm to (114.3, 71.1)
- turned C16 to 270 degrees
Routing:
- net -12V: track 0.00 -> 297.4 mm, vias 0 -> 2
- net 5V_1: track 0.00 -> 249.8 mm, vias 0 -> 8
- net 12V: track 0.00 -> 238.8 mm, vias 0 -> 4
- net N$6: track 0.00 -> 236.9 mm, vias 0 -> 15
- net N$7: track 0.00 -> 236.5 mm, vias 0 -> 16
- net N$12: track 0.00 -> 107.8 mm
- net 9TO18V: track 0.00 -> 71.9 mm
- net GND: track 0.00 -> 51.8 mm, vias 0 -> 14
- net N$10: track 0.00 -> 16.2 mm
- net N$5: track 0.00 -> 8.76 mm
