File: Development/Eurorack Set 13/TINRS - Faust On ESP32.brd (EAGLE design)
At the start: 60.2 x 106.5 mm, 77 parts, among them J1 JACK, J10 JACK, J11 JACK, J12 JACK, J13 JACK, J14 JACK, J15 POWERSHROUDED, J2 JACK, J3 JACK, J4 JACK, J5 MICRO-SDCARD-CONNECTOR-330006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, J8 JACK, J9 JACK, U1 ESP-WROOM-32, U2 LD1117S, U3 LD1117S, X1 12.288MHZ

Commit message: bunch of experiments + pjb things added
Parts:
- removed C12: (no value), adafruit:153CLV-0605
- removed J5: MICRO-SDCARD-CONNECTOR-3300060P1, OPL:9P-SMD-W-RING
- added C1, C2, C3, C32, C35, C36, C37, C39: 3.3nF, OPL:C0603
- added C33: 10uF, EurorackModularParts:CASE-A_3216
- added C34, C38, C5: 100nF, OPL:C0603
- added C40, C41: 100n, OPL:C0603
- added C42: 33n, OPL:C0603
- added IC1, IC4: MCP6004, EurorackModularParts:SO14
- added IC2: TL072, EurorackModularParts:SO08
- added Q1, Q2: MMBT3904, transistor:SOT23-BEC
- added R10, R11, R50, R53: 56, OPL:R0603
- added R12, R13, R26, R31, R73: 10k, OPL:R0603
- added R14, R19, R22, R23, R25, R27, R30, R33, R36, R38, R39, R42, R43, R45, R47, R49, R52, R55: 33k, OPL:R0603
- added R16, R18, R21, R24, R29, R32, R35, R40, R46, R51, R54, R72: 100k, OPL:R0603
- added R17, R20, R28, R34, R37, R41, R44, R48: 51k, OPL:R0603
- added U4: LM4040DIM3-5.0, FarnellThings:SOT95P237X112-3N
- C11: value (none) -> 33n; device adafruit:153CLV-0605 -> OPL:C0603
- moved C8 57.8 mm to (15.4, 22.0)
- moved C4 57.3 mm to (13.5, 21.5)
- moved D1 52.8 mm to (17.4, 21.0), turned to 90 degrees
- moved C26 51.7 mm to (21.1, 60.2)
- moved C6 50.8 mm to (13.0, 10.7), turned to 90 degrees
- moved C7 49.6 mm to (15.0, 11.2), turned to 90 degrees
- moved C10 48.4 mm to (39.1, 21.3), turned to 90 degrees
- moved C9 47.9 mm to (46.2, 24.4)
- moved C25 47.0 mm to (21.3, 58.4), turned to 0 degrees
- moved C11 44.3 mm to (46.0, 15.1), turned to 0 degrees
- moved D2 43.4 mm to (17.3, 9.65), turned to 270 degrees
- moved L1 39.5 mm to (17.3, 15.4), turned to 270 degrees
- moved U2 38.1 mm to (8.76, 67.8), turned to 270 degrees
- moved C21 36.5 mm to (12.2, 63.5), turned to 90 degrees
- moved L2 31.7 mm to (17.3, 3.94), turned to 270 degrees
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Connections:
- removed net N$3: C9.-, J8.TIP_B@1, J8.TIP_T@3
- removed net N$4: C10.-, J4.TIP_B@1, J4.TIP_T@3
- removed net SD_CMD: J5.3
- removed net SD_CS: J5.2
- removed net SD_DAT0: J5.7
- removed net SD_DAT1: J5.8
- removed net SD_DAT2: J5.1
- removed net SD_SCLK: J5.5
- new net ANALOG0: C3.2, IC4.14, R22.1, U1.4
- new net ANALOG1: C1.2, IC4.8, R14.1, U1.5
- new net ANALOG2: C2.2, IC4.1, R19.1, U1.6
- new net ANALOG3: C32.2, IC4.7, R25.1, U1.7
- new net ANALOG4: C37.2, IC1.14, R42.1, U1.8
- new net ANALOG5: C35.2, IC1.8, R33.1, U1.23
- new net ANALOG6: C36.2, IC1.1, R36.1, U1.24
- new net ANALOG7: C39.2, IC1.7, R47.1, U1.26
- new net GATEJACK: Q1.C, R31.1, U1.32
- new net KNOB_DECAY: R2.P$2, R43.2
- new net KNOB_DELAYBEFORETAIL: R45.2, R5.P$2
- new net KNOB_MOD: R39.2
- new net KNOB_PITCH: R1.P$2, R49.2
- new net KNOB_SPACE: R23.2, R6.P$2
- new net KNOB_TONE: R3.P$2, R38.2
- new net KNOB_TRIGGERSPACE: R30.2, R7.P$2
- new net KNOB_TRIGGERTYPE: R27.2, R4.P$2
- new net N$22: R10.2, U$1.LEDPOS
- new net N$23: R11.2, U$2.LEDPOS
- new net N$24: J10.TIP_B@1, J10.TIP_T@3, R16.2
- new net N$25: C1.1, IC4.9, R14.2, R16.1, R17.1, R23.1
- new net N$26: J12.TIP_B@1, J12.TIP_T@3, R18.2
- new net N$27: C2.1, IC4.2, R18.1, R19.2, R20.1, R27.1
- new net N$29: J9.TIP_B@1, J9.TIP_T@3, R24.2
- new net N$30: C32.1, IC4.6, R24.1, R25.2, R41.1, R43.1
- new net N$31: Q1.B, R29.2
- new net N$32: J2.TIP_B@1, J2.TIP_T@3, R29.1
- new net N$33: J13.TIP_B@1, J13.TIP_T@3, R21.2
- new net N$34: C3.1, IC4.13, R21.1, R22.2, R28.1, R30.1
- new net N$35: J11.TIP_B@1, J11.TIP_T@3, R32.2
- new net N$36: C35.1, IC1.9, R32.1, R33.2, R34.1, R38.1
- new net N$37: R35.2
- new net N$38: C36.1, IC1.2, R35.1, R36.2, R37.1, R39.1
- new net N$39: J14.TIP_B@1, J14.TIP_T@3, R40.2
- new net N$40: C37.1, IC1.13, R40.1, R42.2, R44.1, R45.1
- new net N$41: J1.TIP_B@1, J1.TIP_T@3, R46.2
- new net N$42: C39.1, IC1.6, R46.1, R47.2, R48.1, R49.1
- new net N$43: C42.1, IC2.1, R50.2
- new net N$44: Q2.B, R72.2
- new net N$45: J3.TIP_B@1, J3.TIP_T@3, R72.1
- new net N$47: C42.2, IC2.2, R51.2, R52.1
- new net N$48: J4.TIP_B@1, J4.TIP_T@3, R50.1, R51.1
- new net N$49: C10.+, U$9.P$12
- new net N$50: C9.+, U$9.P$13
- new net N$51: C10.-, R52.2
- new net N$52: C11.1, IC2.7, R53.2
- new net N$53: C11.2, IC2.6, R54.2, R55.1
- new net N$55: J8.TIP_B@1, J8.TIP_T@3, R53.1, R54.1
- new net N$56: C9.-, R55.2
- new net REF_-5V: C34.2, R17.2, R20.2, R26.2, R28.2, R34.2, R37.2, R41.2, R44.2, R48.2, U4.2
- new net TRIGGER1: R13.1, U$1.1, U$1.2, U1.30
- new net TRIGGER2: R12.1, U$2.1, U$2.2, U1.28
- new net TRIGGERJACK: Q2.C, R73.1, U1.31
- new net TRIGGERLED1: R10.1, U1.29
- new net TRIGGERLED2: R11.1, U1.27
- net -12V: now also C33.-, C40.2, IC2.4, R26.1
- net 12V: now also C41.1, IC2.8
- net 3.3V: now also C38.1, C5.1, IC1.4, IC4.4, R1.P$3, R12.2, R13.2, R2.P$3, R3.P$3, R31.2, R4.P$3, R5.P$3, R6.P$3, R7.P$3, R73.2; no longer J5.4
- net GND: now also C33.+, C34.1, C38.2, C40.1, C41.2, C5.2, IC1.10, IC1.11, IC1.12, IC1.3, IC1.5, IC2.3, IC2.5, IC4.10, IC4.11, IC4.12, IC4.3, IC4.5, Q1.E, Q2.E, U$1.3, U$1.4, U$1.LEDNEG, U$2.3, U$2.4, U$2.LEDNEG, U4.1; no longer J5.6, J5.G1, J5.G2, J5.G3, J5.G4
- net WM_CS: now also U1.33; no longer U1.26
Routing:
- net N$30: track 0.00 -> 9.04 mm
- net N$27: track 0.00 -> 8.86 mm
- net N$34: track 0.00 -> 8.73 mm
- net N$25: track 0.00 -> 8.37 mm
- net GND: track 0.00 -> 6.55 mm
- net ANALOG2: track 0.00 -> 4.27 mm
- net ANALOG3: track 0.00 -> 4.14 mm
- net ANALOG0: track 0.00 -> 3.89 mm
- net 3.3V: track 0.00 -> 2.35 mm
