File: Development/USB_MiniPower.brd (EAGLE design)
At the start: 118 x 32 mm, 32 parts, among them J1 POWERSHROUDED, J2 POWERSHROUDED, U1 CJ1117-3.3-1310190P1, X1 USB-B-FEMALE

Commit message: Bunch of stuff again..
Parts:
- added L2: FERRITE_1812, EurorackModularParts:FERRITE_1812
- added R1, R2: 75k, OPL:R0603
- added R3, R4: 49.9k, OPL:R0603
- added U$17: TINRS_ARTWORKTINYDATE, EurorackModularParts:JUSTATINYROCKET_DATECODE
- added X2: USB-B-FEMALE, ld-components:FCI61729
- J1: value POWERSHROUDED -> POWER_SHROUDED_NOTEXT; device EurorackModularParts:POWER_16_SHROUDED -> EurorackModularParts:POWER_16_SHROUDED_NOTEXT
- moved R91 4.20 mm to (57.0, 19.0)
- moved C27 2.51 mm to (54.5, 26.8), turned to 0 degrees
- moved C26 1.25 mm to (50.0, 27.8)
Connections:
- new net N$3: L2.P$2, X2.P$1, X2.P$2
- new net N$7: R2.1, R3.2, X2.2
- new net N$8: R1.1, R4.2, X2.3
- net 5V: now also R1.2, R2.2, X2.1
- net GND: now also L2.P$1, R3.1, R4.1, X2.4
Routing:
- net 5V: track 0.00 -> 202.0 mm, vias 0 -> 1
- net -12V: track 0.00 -> 121.3 mm, vias 0 -> 2
- net N$2: track 0.00 -> 103.9 mm, vias 0 -> 2
- net N$1: track 0.00 -> 103.4 mm, vias 0 -> 1
- net 12V: track 0.00 -> 101.2 mm, vias 0 -> 4
- net 3.3V: track 0.00 -> 34.4 mm
- net GND: track 0.00 -> 22.9 mm, vias 0 -> 17
- net N$3: track 0.00 -> 17.3 mm
- net N$4: track 0.00 -> 17.0 mm, vias 0 -> 1
- net N$8: track 0.00 -> 11.8 mm
- net N$6: track 0.00 -> 9.67 mm, vias 0 -> 2
- net N$7: track 0.00 -> 8.91 mm
- net N$5: track 0.00 -> 6.84 mm, vias 0 -> 2
- net N$13: track 0.00 -> 3.28 mm
- net N$19: track 0.00 -> 3.22 mm
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