File: Development/PJB-Box/MainBoard.brd (EAGLE design)
At the start: 240 x 240 mm, 65 parts, among them IC2 NE5532D, J1 POWER_JACKSLT, X1 USB-A-FEMALERECEPTACLE, X2 USB-B-FEMALE

Commit message: PJB Mainboard, OPL fixes, teensyparts, powerbackpack
Parts:
- removed U$33: VOLTAGETESTPAD, FenixBase:POWERTESTPAD
- added C10, C15, C16, C3, C4, C5: 3.3nF, OPL:C0603
- added C13: 100n, OPL:C0603
- added C14: 2.2u 35v, OPL:C0603
- added C17: 10u 50v, OPL:C0603
- added C18, C19, C6, C7, C9: 100nF, OPL:C0603
- added C28: 10u X7R, OPL:C3216
- added C35: 100u, resistor:PANASONIC_D
- added C8: 10uF, EurorackModularParts:CASE-A_3216
- added IC3: TL074D, EurorackModularParts:SO14
- added IC4: MCP6004, EurorackModularParts:SO14
- added J2, J3, J4, J5, J6, J7, J8, J9: POWERSHROUDED, EurorackModularParts:POWER_16_SHROUDED
- added JP2, JP3, JP4, JP5: (no value), pinhead:1X03
- added JP7, JP8: (no value), pinhead:1X14
- added L5: 68uH, EurorackModularParts:SWRB120XS
- added MAINTEENSY, SECONDTEENSY: TEENSY_LC_ALL_PINS, Teensy_3_and_LC_Series_Boards_v1.4:TEENSY_3.0-3.2&LC_ALL_PINS
- added Q1, Q2, Q3, Q4, Q5, Q6, Q7: MMBT3904, transistor:SOT23-BEC
- added R14, R16, R18, R2, R22, R39, R4, R54: 10k, OPL:R0603
- added R15, R17, R21, R23, R3, R36, R37, R38, R40, R43, R48, R52, R53, R55, R6: 100k, OPL:R0603
- added R24, R26: 30k, OPL:R0603
- added R25, R27: 12k, OPL:R0603
- added R28, R35: 100, OPL:R0603
- added R41, R44, R46, R47, R49, R51, R56, R58: 33k, OPL:R0603
- added R42, R45, R50, R57: 51k, OPL:R0603
- added U$21: RECOM_REGULATOR, EurorackModularParts:R-78E5.0-1.0
- added U$24, U$3, U$5: VOLTAGETESTPAD, FenixBase:POWERTESTPAD
- added U2: LM4040DIM3-5.0, FarnellThings:SOT95P237X112-3N
- added U7: MCP4822-E/SN, FarnellThings:SOIC8-N_MC
- added X3: USB-A-FEMALERECEPTACLE, ld-components:FCI87520
- added X4: USB-B-FEMALE, ld-components:FCI61729
- moved U$35 239.0 mm to (29.8, 2.54), turned to 90 degrees
- moved U$34 158.5 mm to (29.8, 2.54), turned to 270 degrees
- moved L1 154.7 mm to (171.1, 17.1), turned to 0 degrees
- moved D1 149.5 mm to (180.4, 13.7)
- moved U$20 148.9 mm to (180.6, 21.4), turned to 270 degrees
- moved C22 147.9 mm to (137.3, 21.7), turned to 0 degrees
- moved R11 146.9 mm to (131.7, 19.7)
- moved R13 146.9 mm to (131.7, 21.7)
- moved R19 146.9 mm to (131.7, 23.7)
- moved R20 146.9 mm to (131.7, 25.7)
- moved R10 146.9 mm to (131.7, 17.3), turned to 0 degrees
- moved R5 146.0 mm to (171.7, 23.3), turned to 90 degrees
- moved R9 145.9 mm to (173.5, 23.3), turned to 270 degrees
- moved C1 142.5 mm to (169.7, 25.8), turned to 270 degrees
- moved C2 141.5 mm to (171.7, 26.5), turned to 270 degrees
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Connections:
- removed net 5V_1: C2.2, R5.2, U$20.8
- removed net LEFTOUT: R7.2, U$32.P$1, U$32.P$2, U$32.P$3
- removed net RIGHTOUT: U$33.P$1, U$33.P$2, U$33.P$3
- new net 26/A12/DAC: MAINTEENSY.RESET/DAC, SECONDTEENSY.RESET/DAC
- new net 3.3V: SECONDTEENSY.3.3V, SECONDTEENSY.3.3V1, U7.1
- new net 3V3: C2.2, JP2.3, JP3.3, JP4.3, JP5.3, MAINTEENSY.3.3V, MAINTEENSY.3.3V1, R5.2, U$20.8
- new net 5V: C13.1, C28.P$2, C35.+, J2.11, J2.12, J3.11, J3.12, J4.11, J4.12, J5.11, J5.12, J6.11, J6.12, J7.11, J7.12, J8.11, J8.12, J9.11, J9.12, MAINTEENSY.VIN, SECONDTEENSY.VIN, U$21.P$3, U$24.P$1, U$24.P$2, U$24.P$3
- new net AREF: MAINTEENSY.AREF, SECONDTEENSY.AREF
- new net DACCS: MAINTEENSY.15/A1, U7.2
- new net DACSCK: MAINTEENSY.13, U7.3
- new net DACSDI: MAINTEENSY.11, U7.4
- new net KNOB_L1: JP3.2, R46.2
- new net KNOB_L2: JP5.2, R47.2
- new net KNOB_X1: JP2.2, R51.2
- new net KNOB_X2: JP4.2, R58.2
- new net L1_ADC: C15.2, IC4.8, JP8.4, MAINTEENSY.16/A2, R41.1, SECONDTEENSY.16/A2
- new net L2_ADC: C5.2, IC4.1, JP8.5, MAINTEENSY.17/A3, R44.1, SECONDTEENSY.17/A3
- new net MAIN_TO_SECOND: JP7.9, MAINTEENSY.8, SECONDTEENSY.7
- new net N$10: MAINTEENSY.VBAT, U$3.P$1, U$3.P$2, U$3.P$3
- new net N$11: C14.2, L5.P$2, U$21.P$1
- new net N$12: SECONDTEENSY.VBAT, U$5.P$1, U$5.P$2, U$5.P$3
- new net N$17: Q1.B, R3.2
- new net N$18: Q2.B, R6.2
- new net N$19: Q3.B, R15.2
- new net N$20: Q4.B, R17.2
- new net N$21: Q6.B, R21.2
- new net N$22: Q7.B, R23.2
- new net N$23: C4.2, IC3.1, R26.1, R36.1
- new net N$24: C3.2, IC3.14, R24.1, R53.1
- new net N$25: C3.1, IC3.13, R24.2, R27.1
- new net N$26: C4.1, IC3.2, R25.1, R26.2
- new net N$27: C10.1, IC4.6, R55.1, R56.2, R57.1, R58.1
- new net N$30: JP7.2, SECONDTEENSY.0
- new net N$31: IC3.6, R36.2, R37.1
- new net N$35: IC3.7, R28.2, R37.2
- new net N$36: IC3.9, R52.1, R53.2
- new net N$37: R27.2, U7.8
- new net N$38: R25.2, U7.6
- new net N$39: JP7.3, SECONDTEENSY.1
- new net N$44: C15.1, IC4.9, R38.1, R41.2, R42.1, R46.1
- new net N$45: JP7.4, SECONDTEENSY.2
- new net N$46: C5.1, IC4.2, R43.1, R44.2, R45.1, R47.1
- new net N$47: JP7.5, SECONDTEENSY.3
- new net N$48: C16.1, IC4.13, R48.1, R49.2, R50.1, R51.1
- new net N$49: JP7.6, SECONDTEENSY.4
- new net N$50: JP7.7, SECONDTEENSY.5
- new net N$51: JP7.8, SECONDTEENSY.6
- new net N$52: JP7.11, SECONDTEENSY.9
- new net N$53: JP7.12, SECONDTEENSY.10
- new net N$54: JP7.13, SECONDTEENSY.11
- new net N$55: JP7.14, SECONDTEENSY.12
- new net N$56: JP8.1, SECONDTEENSY.13
- new net N$57: JP8.2, SECONDTEENSY.14/A0
- new net N$58: JP8.3, SECONDTEENSY.15/A1
- new net N$59: JP8.8, SECONDTEENSY.20/A6
- new net N$60: Q5.B, R40.2
- new net N$61: JP8.9, SECONDTEENSY.21/A7
- new net N$62: JP8.10, SECONDTEENSY.22/A8
- new net N$63: JP8.11, SECONDTEENSY.23/A9
- new net N$8: X3.P1, X4.1
- new net N$9: X3.P4, X4.4
- new net N$94: IC3.8, R35.2, R52.2
- new net OUT_CLOCK1: MAINTEENSY.5, R15.1
- new net OUT_CLOCK2: MAINTEENSY.6, R17.1
- new net OUT_CLOCK3: MAINTEENSY.10, R21.1
- new net OUT_G1: MAINTEENSY.2, R40.1
- new net OUT_G2: MAINTEENSY.3, R3.1
- new net OUT_G3: MAINTEENSY.4, R6.1
- new net OUT_RESET: MAINTEENSY.14/A0, R23.1
- new net REF_-5V: C9.2, R42.2, R45.2, R50.2, R54.2, R57.2, U2.2
- new net SECOND_TO_MAIN: JP7.10, MAINTEENSY.7, SECONDTEENSY.8
- new net USB_N2: X3.P2, X4.2
- new net USB_P2: X3.P3, X4.3
- new net VUSB: MAINTEENSY.VUSB, SECONDTEENSY.VUSB
- new net X1: R48.2
- new net X1_ADC: C16.2, IC4.14, JP8.6, MAINTEENSY.18/A4, R49.1, SECONDTEENSY.18/A4
- new net X2: R55.2
- new net X2_ADC: C10.2, IC4.7, JP8.7, MAINTEENSY.19/A5, R56.1, SECONDTEENSY.19/A5
- net -12V: now also C19.2, C7.2, C8.-, IC3.11, IC4.11, J2.1, J2.2, J3.1, J3.2, J4.1, J4.2, J5.1, J5.2, J6.1, J6.2, J7.1, J7.2, J8.1, J8.2, J9.1, J9.2, R54.1
- net 12V: now also C18.2, C6.2, IC3.4, IC4.4, J2.10, J2.9, J3.10, J3.9, J4.10, J4.9, J5.10, J5.9, J6.10, J6.9, J7.10, J7.9, J8.10, J8.9, J9.10, J9.9, R14.2, R16.2, R18.2, R2.2, R22.2, R39.2, R4.2
- net 9TO18V: now also C17.2, L5.P$1
- net CLOCK1: now also Q3.C, R14.1
- net CLOCK2: now also Q4.C, R16.1
- net CLOCK3: now also Q6.C, R18.1
- net CV1: now also J2.13, J2.14, J3.13, J3.14, J4.13, J4.14, J5.13, J5.14, J6.13, J6.14, J7.13, J7.14, J8.13, J8.14, J9.13, J9.14, R28.1
- net CV2: now also R35.1
- net G1: now also J2.15, J2.16, J3.15, J3.16, J4.15, J4.16, J5.15, J5.16, J6.15, J6.16, J7.15, J7.16, J8.15, J8.16, J9.15, J9.16, Q5.C, R39.1
- net G2: now also Q1.C, R2.1
- net G3: now also Q2.C, R4.1
- net GND: now also C13.2, C14.1, C17.1, C18.1, C19.1, C28.P$1, C35.-, C6.1, C7.1, C8.+, C9.1, IC3.10, IC3.12, IC3.3, IC3.5, IC4.10, IC4.12, IC4.3, IC4.5, J2.3, J2.4, J2.5, J2.6, J2.7, J2.8, J3.3, J3.4, J3.5, J3.6, J3.7, J3.8, J4.3, J4.4, J4.5, J4.6, J4.7, J4.8, J5.3, J5.4, J5.5, J5.6, J5.7, J5.8, J6.3, J6.4, J6.5, J6.6, J6.7, J6.8, J7.3, J7.4, J7.5, J7.6, J7.7, J7.8, J8.3, J8.4, J8.5, J8.6, J8.7, J8.8, J9.3, J9.4, J9.5, J9.6, J9.7, J9.8, JP2.1, JP3.1, JP4.1, JP5.1, MAINTEENSY.AGND, MAINTEENSY.GND, MAINTEENSY.GND1, Q1.E, Q2.E, Q3.E, Q4.E, Q5.E, Q6.E, Q7.E, SECONDTEENSY.AGND, SECONDTEENSY.GND, SECONDTEENSY.GND1, U$21.P$2, U2.1, U7.5, U7.7, X3.P$1, X3.P$2, X4.P$1, X4.P$2
- net L1: now also R38.2
- net L2: now also R43.2
- net MIDI: now also MAINTEENSY.9
- net OUTPUT: now also R7.2, U$32.P$1, U$32.P$2, U$32.P$3
- net RESET: now also Q7.C, R22.1
Routing:
- net MIDI: track 157.6 -> 5.78 mm, vias 6 -> 0
- net 12V: track 177.0 -> 50.4 mm, vias 6 -> 2
- net -12V: track 56.1 -> 9.03 mm, vias 4 -> 0
- net 5V_1: track 41.0 -> 0.00 mm, vias 4 -> 0
- net N$14: track 40.1 -> 4.45 mm, vias 2 -> 0
- net OUTTIPLEFT: track 32.5 -> 6.02 mm
- net N$4: track 14.1 -> 0.00 mm
- net LEFTOUT: track 13.4 -> 0.00 mm
- net USB_N: track 8.49 -> 0.00 mm
- net USB_P: track 8.04 -> 0.00 mm
- net RIGHTOUT: track 7.23 -> 0.00 mm
- net N$40: track 7.04 -> 0.05 mm
- net VIN: track 6.72 -> 0.00 mm
- net 3V3: track 0.00 -> 6.47 mm
- net GND: track 62.3 -> 56.1 mm, vias 214 -> 211
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- removed copper zone on layer 16, net N$5
- removed copper zone on layer 16, net VIN
Other:
- board size 240 x 240 mm -> 240 x 60 mm

Commit message: bunch of pjb boards - tentative mixer design..
Parts:
- removed C13: 100n, OPL:C0603
- removed C14: 2.2u 35v, OPL:C0603
- removed C17: 10u 50v, OPL:C0603
- removed C28: 10u X7R, OPL:C3216
- removed C35, C47: 100u, resistor:PANASONIC_D
- removed C42, C43: 100p 50V, OPL:C0603
- removed C44, C45, C56, C57, C58, C59, C65: 10u, OPL:C0805
- removed C49: 56u, resistor:PANASONIC_D
- removed C52, C53, C54, C55: 47u, OPL:C0805
- removed C63, C64: 100uF 50V, rcl:153CLV-1010
- removed C9: 100nF, OPL:C0603
- removed D5: SS34, dp_devices:DO-214AC
- removed D7: 1N4004 SMD SMA, diode:DO214AC
- removed J3, J6, J7, J8, J9: POWERSHROUDED, EurorackModularParts:POWER_16_SHROUDED
- removed JP6: M02PTH4, SparkFun-Connectors:1X02_XTRA_BIG
- removed L5: 68uH, EurorackModularParts:SWRB120XS
- removed R29, R32: 47k 1%, OPL:R0603
- removed R30, R33: 10k 1%, OPL:R0603
- removed R31, R34: 110k 1%, OPL:R0603
- removed R54: 10k, OPL:R0603
- removed U$21: RECOM_REGULATOR, EurorackModularParts:R-78E5.0-1.0
- removed U$24: VOLTAGETESTPAD, FenixBase:POWERTESTPAD
- removed U$39, U$40: LMZM33606, EurorackModularParts:LMZM33606
- removed U2: LM4040DIM3-5.0, FarnellThings:SOT95P237X112-3N
- added LEDPOWER, LEDPOWER1, POWERSWITCH: M02PTH4, SparkFun-Connectors:1X02_XTRA_BIG
- added U$17: HEARTOFGOLD, FenixBase:HEARTOFGOLD
- added U$23: FENIXPOWERBACKPACK_MODULE, EurorackModularParts:FENIXPOWERBACKPACK
- added U$25: FENIXPOWERBACKPACKART_MODULE, EurorackModularParts:FENIXPOWERBACKPACK_MODULE
- C8: value 10uF -> 100nF; device EurorackModularParts:CASE-A_3216 -> OPL:C0603
- J2: value POWERSHROUDED -> POWER_SHROUDED_NOTEXT; device EurorackModularParts:POWER_16_SHROUDED -> EurorackModularParts:POWER_16_SHROUDED_NOTEXT
- moved U$29 168.5 mm to (237.5, 17.9), turned to 0 degrees
- moved J2 111.0 mm to (234.0, 36.0), flipped to the bottom, turned to 90 degrees
- moved U$19 107.1 mm to (70.1, 31.5), flipped to the bottom, turned to 0 degrees
- moved C21 63.6 mm to (99.9, 34.7)
- moved C26 63.6 mm to (98.8, 32.2)
- moved C27 63.6 mm to (91.9, 38.7)
- moved IC2 63.6 mm to (92.9, 34.7)
- moved R12 63.6 mm to (94.9, 38.7)
- moved R7 63.6 mm to (99.2, 37.9)
- moved R8 63.6 mm to (97.9, 34.7)
- moved U$32 63.5 mm to (103.2, 38.3)
- moved C20 62.3 mm to (84.5, 34.9), turned to 270 degrees
- moved C22 61.3 mm to (77.5, 34.9), turned to 270 degrees
- moved J1 60.0 mm to (138.1, -3.00)
- moved R9 59.0 mm to (114.5, 24.3)
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Connections:
- removed net 12V_AGND: R29.1, R30.1, U$39.16A, U$39.16B, U$39.16C, U$39.16PAD, U$39.19, U$39.21
- removed net 26/A12/DAC: MAINTEENSY.RESET/DAC, SECONDTEENSY.RESET/DAC
- removed net 3V3: C2.2, JP2.3, JP3.3, JP4.3, JP5.3, MAINTEENSY.3.3V, MAINTEENSY.3.3V1, R5.2, U$20.8
- removed net AREF: MAINTEENSY.AREF, SECONDTEENSY.AREF
- removed net N$1: X1.P1, X2.1
- removed net N$11: C14.2, L5.P$2, U$21.P$1
- removed net N$28: R29.2, U$39.12
- removed net N$29: C42.1, R30.2, R31.1, U$39.15
- removed net N$32: R32.2, U$40.12
- removed net N$33: R32.1, R33.1, U$40.16A, U$40.16B, U$40.16C, U$40.16PAD, U$40.19, U$40.21
- removed net N$34: C43.1, R33.2, R34.1, U$40.15
- removed net N$4: X1.P4, X2.4
- removed net N$8: X3.P1, X4.1
- removed net N$9: X3.P4, X4.4
- removed net SW-12: U$40.1, U$40.2A, U$40.2B, U$40.2PAD, U$40.31A, U$40.31B, U$40.31C, U$40.31PAD, U$40.32, U$40.33, U$40.3A, U$40.3B, U$40.3PAD, U$40.4A, U$40.4B, U$40.4PAD, U$40.5A, U$40.5B, U$40.5PAD, U$40.6A, U$40.6B, U$40.6PAD
- removed net SW12: U$39.1, U$39.2A, U$39.2B, U$39.2PAD, U$39.31A, U$39.31B, U$39.31C, U$39.31PAD, U$39.32, U$39.33, U$39.3A, U$39.3B, U$39.3PAD, U$39.4A, U$39.4B, U$39.4PAD, U$39.5A, U$39.5B, U$39.5PAD, U$39.6A, U$39.6B, U$39.6PAD
- new net VUSB2: SECONDTEENSY.VUSB, X3.P1, X4.1
- net -12V: now also U$23.-12V@1, U$23.-12V@2, U$23.-12V@3; no longer C44.1, C49.-, C55.2, C8.-, D5.2, J3.1, J3.2, J6.1, J6.2, J7.1, J7.2, J8.1, J8.2, J9.1, J9.2, R54.1, U$40.10A, U$40.10B, U$40.10PAD, U$40.11, U$40.23A, U$40.23B, U$40.23C, U$40.23PAD, U$40.30A, U$40.30B, U$40.30C, U$40.30PAD, U$40.34, U$40.35, U$40.38, U$40.40, U$40.41, U$40.8
- net 12V: now also U$23.12V@1, U$23.12V@2, U$23.12V@4; no longer C42.2, C47.+, C52.2, C53.2, C54.2, J3.10, J3.9, J6.10, J6.9, J7.10, J7.9, J8.10, J8.9, J9.10, J9.9, R31.2, U$39.24A, U$39.24B, U$39.24PAD, U$39.25A, U$39.25B, U$39.25PAD, U$39.26A, U$39.26B, U$39.26PAD, U$39.27A, U$39.27B, U$39.27PAD, U$39.28, U$39.29A, U$39.29B, U$39.29C, U$39.29PAD, U$39.36, U$39.37
- net 3.3V: now also C2.2, C8.2, JP2.3, JP3.3, JP4.3, JP5.3, MAINTEENSY.3.3V, MAINTEENSY.3.3V1, R5.2, U$20.8; no longer SECONDTEENSY.3.3V, SECONDTEENSY.3.3V1
- net 5V: now also LEDPOWER.2, LEDPOWER1.2, U$23.5V@1, U$23.5V@2, U$23.5V@3, U$23.5V@4; no longer C13.1, C28.P$2, C35.+, J3.11, J3.12, J6.11, J6.12, J7.11, J7.12, J8.11, J8.12, J9.11, J9.12, U$21.P$3, U$24.P$1, U$24.P$2, U$24.P$3
- net 9TO18V: now also POWERSWITCH.2, U$23.VIN@1, U$23.VIN@2, U$23.VIN@3, U$23.VIN@4; no longer C17.2, C44.2, C45.2, C56.1, C57.1, C58.1, C59.1, C63.+, C64.+, C65.2, D7.C, JP6.2, L5.P$1, U$39.20, U$39.22A, U$39.22B, U$39.22PAD, U$39.39, U$40.20, U$40.22A, U$40.22B, U$40.22PAD, U$40.39
- net CV1: no longer J2.13, J2.14, J3.13, J3.14, J4.13, J4.14, J6.13, J6.14, J7.13, J7.14, J8.13, J8.14, J9.13, J9.14
- net CV2: now also J2.13, J2.14, J4.13, J4.14
- net G1: no longer J2.15, J2.16, J3.15, J3.16, J4.15, J4.16, J6.15, J6.16, J7.15, J7.16, J8.15, J8.16, J9.15, J9.16
- net G2: now also J2.15, J2.16, J4.15, J4.16
- net GND: now also C8.1, LEDPOWER.1, LEDPOWER1.1, U$23.GND@1, U$23.GND@10, U$23.GND@11, U$23.GND@12, U$23.GND@13, U$23.GND@14, U$23.GND@2, U$23.GND@3, U$23.GND@4, U$23.GND@5, U$23.GND@6, U$23.GND@7, U$23.GND@8, U$23.GND@9, X1.P4, X2.4, X3.P4, X4.4; no longer C13.2, C14.1, C17.1, C28.P$1, C35.-, C43.2, C45.1, C47.-, C49.+, C52.1, C53.1, C54.1, C55.1, C56.2, C57.2, C58.2, C59.2, C63.-, C64.-, C65.1, C8.+, C9.1, D5.1, D7.A, J3.3, J3.4, J3.5, J3.6, J3.7, J3.8, J6.3, J6.4, J6.5, J6.6, J6.7, J6.8, J7.3, J7.4, J7.5, J7.6, J7.7, J7.8, J8.3, J8.4, J8.5, J8.6, J8.7, J8.8, J9.3, J9.4, J9.5, J9.6, J9.7, J9.8, R34.2, U$21.P$2, U$39.10A, U$39.10B, U$39.10PAD, U$39.11, U$39.23A, U$39.23B, U$39.23C, U$39.23PAD, U$39.30A, U$39.30B, U$39.30C, U$39.30PAD, U$39.34, U$39.35, U$39.38, U$39.40, U$39.41, U$39.8, U$40.24A, U$40.24B, U$40.24PAD, U$40.25A, U$40.25B, U$40.25PAD, U$40.26A, U$40.26B, U$40.26PAD, U$40.27A, U$40.27B, U$40.27PAD, U$40.28, U$40.29A, U$40.29B, U$40.29C, U$40.29PAD, U$40.36, U$40.37, U2.1
- net REF_-5V: now also U$23.-5V, U$23.-5V@2; no longer C9.2, R54.2, U2.2
- net VIN: now also POWERSWITCH.1; no longer JP6.1
- net VUSB: now also X1.P1, X2.1; no longer SECONDTEENSY.VUSB
Routing:
- net CV2: track 0.00 -> 364.8 mm, vias 0 -> 9
- net 12V: track 50.4 -> 323.3 mm, vias 2 -> 10
- net G2: track 0.00 -> 267.0 mm, vias 0 -> 11
- net -12V: track 9.03 -> 247.3 mm, vias 0 -> 10
- net CV1: track 0.00 -> 219.7 mm, vias 0 -> 2
- net 5V: track 0.00 -> 214.0 mm, vias 0 -> 8
- net REF_-5V: track 0.00 -> 186.8 mm, vias 0 -> 2
- net G1: track 0.00 -> 145.1 mm, vias 0 -> 9
- net OUTPUT: track 0.00 -> 140.6 mm, vias 0 -> 4
- net 3.3V: track 0.00 -> 116.0 mm, vias 0 -> 4
- net L2: track 0.00 -> 108.0 mm, vias 0 -> 12
- net VIN: track 0.00 -> 107.9 mm
- net L2_ADC: track 0.00 -> 76.4 mm, vias 0 -> 8
- net X2_ADC: track 0.00 -> 75.0 mm, vias 0 -> 6
- net MIDI: track 5.78 -> 76.6 mm, vias 0 -> 2
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- removed copper zone on layer 16, net -12V
- removed copper zone on layer 16, net 12V
- removed copper zone on layer 16, net 12V_AGND
- removed copper zone on layer 16, net 9TO18V
- removed copper zone on layer 16, net GND
- removed copper zone on layer 16, net N$33
- removed copper zone on layer 1, net SW-12
- removed copper zone on layer 16, net SW-12
- removed copper zone on layer 1, net SW12
- removed copper zone on layer 16, net SW12
Other:
- outline, holes or cut-outs redrawn

Commit message: SWD isolator -pjb board progress
Parts:
- removed C7: 100nF, OPL:C0603
Connections:
- net -12V: no longer C7.2, IC4.11
- net 12V: no longer C6.2, IC4.4
- net 3.3V: now also C6.2, IC4.4
- net GND: now also IC4.11; no longer C7.1
- net N$6: no longer U$4.3
Routing:
- net 12V: track 323.3 -> 285.0 mm, vias 10 -> 6
- net 3.3V: track 116.0 -> 127.3 mm, vias 4 -> 6
- net -12V: track 247.3 -> 243.9 mm
- net N$6: track 8.51 -> 6.44 mm
- net GND: track 41.0 -> 41.8 mm
Changed lines of the file:
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@@
 <attribute name="OC_FARNELL" value="1759017" x="85.598" y="48.133" size="1.778" layer="28" rot="MR0" display="off"/>
-</element>
-<element name="C7" library="OPL" package="C0603" value="100nF" x="74.295" y="48.26" rot="MR180">
-<attribute name="MPN" value="MC0603F104Z160CT" x="74.295" y="48.26" size="1.778" layer="28" rot="MR180" display="off"/>
-<attribute name="MF" value="MULTICOMP" x="74.295" y="48.26" size="1.778" layer="28" rot="MR180" display="off"/>
-<attribute name="OC_FARNELL" value="1759017" x="74.295" y="48.26" size="1.778" layer="28" rot="MR180" display="off"/>
 </element>
 <element name="R55" library="OPL" package="R0603" value="100k" x="89.027" y="46.101" rot="MR180">
@@
 <contactref element="IC4" pad="3"/>
 <contactref element="IC4" pad="12"/>
-<contactref element="C7" pad="1"/>
 <contactref element="C6" pad="1"/>
 <contactref element="IC4" pad="5"/>
@@
 <via x="113.919" y="20.193" extent="1-16" drill="0.3048"/>
 <wire x1="113.919" y1="20.193" x2="113.919" y2="20.574" width="0.254" layer="1"/>
-<wire x1="73.533" y1="48.26" x2="72.779" y2="48.252" width="0.254" layer="16"/>
-<wire x1="72.779" y1="48.252" x2="72.771" y2="48.133" width="0.254" layer="16"/>
-<via x="72.771" y="48.133" extent="1-16" drill="0.3048"/>
-<wire x1="72.771" y1="48.133" x2="72.517" y2="48.133" width="0.254" layer="1"/>
 <wire x1="26.67" y1="35.052" x2="27.432" y2="35.052" width="0.254" layer="16"/>
 <wire x1="27.432" y1="35.052" x2="27.686" y2="35.306" width="0.254" layer="16"/>
 <via x="27.686" y="35.306" extent="1-16" drill="0.3048"/>
 <wire x1="27.686" y1="35.306" x2="27.686" y2="35.433" width="0.254" layer="1"/>
+<contactref element="IC4" pad="11"/>
+<wire x1="77.41" y1="48.133" x2="79.121" y2="48.133" width="0.254" layer="16"/>
+<via x="79.121" y="48.133" extent="1-16" drill="0.3048"/>
+<wire x1="79.121" y1="48.133" x2="79.375" y2="48.133" width="0.254" layer="1"/>
 </signal>
 <signal name="12V" class="1">
@@
 <contactref element="C18" pad="2"/>
 <contactref element="IC3" pad="4"/>
-<contactref element="C6" pad="2"/>
-<contactref element="IC4" pad="4"/>
 <contactref element="J4" pad="9"/>
 <contactref element="J4" pad="10"/>
@@
 <wire x1="21.59" y1="39.878" x2="22.733" y2="39.878" width="1" layer="16"/>
 <wire x1="11.43" y1="51.562" x2="9.017" y2="51.562" width="1" layer="16"/>
-<wire x1="82.61" y1="48.133" x2="84.836" y2="48.133" width="1" layer="16"/>
 <wire x1="97.993" y1="32.235" x2="97.993" y2="31.166" width="1" layer="16"/>
 <wire x1="97.993" y1="31.166" x2="98.933" y2="30.226" width="1" layer="16"/>
@@
 <wire x1="26.035" y1="52.07" x2="25.146" y2="51.181" width="1" layer="16"/>
 <wire x1="25.146" y1="51.181" x2="24.282" y2="51.181" width="1" layer="16"/>
-<wire x1="84.836" y1="48.133" x2="81.28" y2="48.133" width="1" layer="16"/>
-<wire x1="81.28" y1="48.133" x2="80.772" y2="47.625" width="1" layer="16"/>
-<wire x1="80.772" y1="47.625" x2="80.772" y2="42.926" width="1" layer="16"/>
-<wire x1="80.772" y1="42.926" x2="81.407" y2="42.291" width="1" layer="16"/>
-<wire x1="81.407" y1="42.291" x2="86.487" y2="42.291" width="1" layer="16"/>
-<via x="86.487" y="42.291" extent="1-16" drill="0.3048"/>
-<wire x1="86.487" y1="42.291" x2="86.487" y2="39.116" width="1" layer="1"/>
-<wire x1="86.487" y1="39.116" x2="86.614" y2="38.989" width="1" layer="1"/>
-<via x="86.614" y="38.989" extent="1-16" drill="0.3048"/>
-<wire x1="86.614" y1="38.989" x2="86.614" y2="33.655" width="1" layer="16"/>
-<wire x1="86.614" y1="33.655" x2="87.884" y2="32.385" width="1" layer="16"/>
-<via x="87.884" y="32.385" extent="1-16" drill="0.3048"/>
-<wire x1="87.884" y1="32.385" x2="93.726" y2="32.385" width="1" layer="1"/>
-<wire x1="93.726" y1="32.385" x2="94.742" y2="31.369" width="1" layer="1"/>
-<via x="94.742" y="31.369" extent="1-16" drill="0.3048"/>
-<wire x1="94.742" y1="31.369" x2="97.79" y2="31.369" width="1" layer="16"/>
-<wire x1="97.79" y1="31.369" x2="97.993" y2="31.166" width="1" layer="16"/>
 <wire x1="99.949" y1="58.42" x2="100.711" y2="57.658" width="1" layer="16"/>
 <wire x1="100.711" y1="57.658" x2="101.854" y2="57.658" width="1" layer="16"/>
@@
 <contactref element="C19" pad="2"/>
 <contactref element="IC3" pad="11"/>
-<contactref element="C7" pad="2"/>
-<contactref element="IC4" pad="11"/>
 <contactref element="J4" pad="1"/>
 <contactref element="J4" pad="2"/>
@@
 <wire x1="227.33" y1="21.71" x2="232.73" y2="27.11" width="1" layer="16"/>
 <wire x1="6.975" y1="33.775" x2="6.975" y2="36.128" width="1" layer="16"/>
-<wire x1="77.41" y1="48.133" x2="75.184" y2="48.133" width="1" layer="16"/>
-<wire x1="75.184" y1="48.133" x2="75.057" y2="48.26" width="1" layer="16"/>
-<wire x1="77.41" y1="48.133" x2="78.74" y2="48.133" width="1" layer="16"/>
-<wire x1="78.74" y1="48.133" x2="79.375" y2="47.498" width="1" layer="16"/>
-<wire x1="79.375" y1="47.498" x2="79.375" y2="41.91" width="1" layer="16"/>
-<wire x1="79.375" y1="41.91" x2="80.645" y2="40.64" width="1" layer="16"/>
-<wire x1="80.645" y1="40.64" x2="89.188" y2="40.64" width="1" layer="16"/>
-<wire x1="89.188" y1="40.64" x2="91.143" y2="38.685" width="1" layer="16"/>
 <wire x1="6.975" y1="36.128" x2="7.553" y2="36.128" width="1" layer="16"/>
 <wire x1="7.553" y1="36.128" x2="8.128" y2="36.703" width="1" layer="16"/>
@@
 <wire x1="9.017" y1="44.323" x2="8.89" y2="44.45" width="1" layer="16"/>
 <wire x1="113.03" y1="48.26" x2="113.03" y2="50.8" width="1" layer="16"/>
-<wire x1="75.057" y1="48.26" x2="75.057" y2="47.625" width="1" layer="16"/>
-<wire x1="75.057" y1="47.625" x2="74.676" y2="47.244" width="1" layer="16"/>
-<via x="74.676" y="47.244" extent="1-16" drill="0.3048"/>
-<wire x1="74.676" y1="47.244" x2="74.676" y2="50.419" width="1" layer="1"/>
 <wire x1="74.676" y1="50.419" x2="76.454" y2="52.197" width="1" layer="1"/>
 <wire x1="76.454" y1="52.197" x2="76.454" y2="56.769" width="1" layer="1"/>
@@
 <wire x1="25.4" y1="40.386" x2="25.4" y2="40.767" width="1" layer="16"/>
 <wire x1="25.4" y1="40.767" x2="25.654" y2="41.021" width="1" layer="16"/>
+<wire x1="90.305" y1="37.981" x2="89.654" y2="37.981" width="1" layer="16"/>
+<wire x1="89.654" y1="37.981" x2="86.614" y2="41.021" width="1" layer="16"/>
+<wire x1="86.614" y1="41.021" x2="81.788" y2="41.021" width="1" layer="16"/>
+<wire x1="81.788" y1="41.021" x2="81.026" y2="41.783" width="1" layer="16"/>
+<wire x1="81.026" y1="41.783" x2="78.232" y2="41.783" width="1" layer="16"/>
+<via x="78.232" y="41.783" extent="1-16" drill="0.3048"/>
+<wire x1="78.232" y1="41.783" x2="77.47" y2="41.783" width="1" layer="1"/>
+<wire x1="77.47" y1="41.783" x2="74.676" y2="44.577" width="1" layer="1"/>
+<wire x1="74.676" y1="44.577" x2="74.676" y2="50.419" width="1" layer="1"/>
 </signal>
 <signal name="USB_P" class="3">
@@
 <contactref element="U$4" pad="5"/>
 <contactref element="L1" pad="2"/>
-<contactref element="U$4" pad="3"/>
-<wire x1="122.08" y1="15.02" x2="124.52" y2="12.58" width="0.508" layer="16"/>
-<wire x1="124.52" y1="12.58" x2="124.52" y2="12.6705" width="0.254" layer="16"/>
-<wire x1="124.52" y1="12.6705" x2="128.037" y2="16.1875" width="0.254" layer="16"/>
+<wire x1="122.08" y1="15.02" x2="126.8695" y2="15.02" width="0.254" layer="16"/>
+<wire x1="126.8695" y1="15.02" x2="128.037" y2="16.1875" width="0.254" layer="16"/>
 </signal>
 <signal name="N$7">
@@
 <wire x1="65.056" y1="44.99" x2="63.5" y2="44.99" width="1" layer="16"/>
 <wire x1="108.674" y1="26.708" x2="112.707" y2="26.708" width="1" layer="16"/>
+<contactref element="C6" pad="2"/>
+<contactref element="IC4" pad="4"/>
+<wire x1="82.61" y1="48.133" x2="84.836" y2="48.133" width="1" layer="16"/>
+<wire x1="84.836" y1="48.133" x2="84.836" y2="47.879" width="0.254" layer="16"/>
+<wire x1="84.836" y1="47.879" x2="85.598" y2="47.117" width="0.254" layer="16"/>
+<wire x1="85.598" y1="47.117" x2="88.138" y2="47.117" width="0.254" layer="16"/>
+<wire x1="88.138" y1="47.117" x2="88.392" y2="47.371" width="0.254" layer="16"/>
+<via x="88.392" y="47.371" extent="1-16" drill="0.3048"/>
+<wire x1="88.392" y1="47.371" x2="89.789" y2="47.371" width="0.254" layer="1"/>
+<via x="89.789" y="47.371" extent="1-16" drill="0.3048"/>
+<wire x1="89.789" y1="47.371" x2="91.44" y2="47.371" width="0.254" layer="16"/>
+<wire x1="91.44" y1="47.371" x2="92.71" y2="46.101" width="0.254" layer="16"/>
 </signal>
 <signal name="VUSB">
@@
 <wire x1="82.61" y1="44.323" x2="82.169" y2="44.323" width="0.254" layer="16"/>
 <wire x1="82.169" y1="44.323" x2="81.915" y2="44.069" width="0.254" layer="16"/>
-<wire x1="81.915" y1="44.069" x2="81.915" y2="43.561" width="0.254" layer="16"/>
-<via x="81.915" y="43.561" extent="1-16" drill="0.3048"/>
-<wire x1="81.915" y1="43.561" x2="81.788" y2="43.561" width="0.254" layer="1"/>
-<wire x1="81.788" y1="43.561" x2="78.994" y2="40.767" width="0.254" layer="1"/>
-<via x="78.994" y="40.767" extent="1-16" drill="0.3048"/>
-<wire x1="78.994" y1="40.767" x2="76.581" y2="40.767" width="0.254" layer="16"/>
+<wire x1="81.915" y1="44.069" x2="81.915" y2="43.307" width="0.254" layer="16"/>
+<via x="81.915" y="43.307" extent="1-16" drill="0.3048"/>
+<wire x1="81.915" y1="43.307" x2="79.375" y2="40.767" width="0.254" layer="1"/>
+<via x="79.375" y="40.767" extent="1-16" drill="0.3048"/>
+<wire x1="79.375" y1="40.767" x2="76.581" y2="40.767" width="0.254" layer="16"/>
 <wire x1="76.581" y1="40.767" x2="72.898" y2="37.084" width="0.254" layer="16"/>
 <via x="72.898" y="37.084" extent="1-16" drill="0.3048"/>
