File: Development/Eurorack Set 2021/TINRS - PicoLooper.sch (EAGLE design)
At the start: 182 parts, among them IC10 4052D, IC2 TL072, IC3 MCP4822-E/SN, IC4 MCP6004, IC5 74HC595BQ, IC6 74HC595BQ, IC7 74HC595BQ, IC8 74HC595BQ, IC9 74HC595BQ, J1 MICRO-USB-5P, J14 POWERSHROUDED, K1 BUTTON-4P-3100010P1, Q1 MMBT3904, Q2 MMBT3904, Q3 MMBT3904, Q4 12mhz, Q5 MMBT3904, U1 LM4040DIM3-5.0

Commit message: Wobbler ordered.. picolooper?
Parts:
- removed C38: 100nF, resistor:C-EUC0402
- removed D10, D11, D12, D13, D14, D16, D17, D20, D21, D22, D24, D25, D26, D27, D28, D29, D30, D31, D32, D33, D34, D35, D4, D40, D5: yellow, EurorackModularParts:LED3MM
- removed IC2: TL072, EurorackModularParts:TL072
- removed IC3: MCP4822-E/SN, FarnellThings:MCP4822-E/SN
- removed IC8, IC9: 74HC595BQ, FarnellThings:74HC595BQ
- removed Q3: MMBT3904, transistor:MMBT3904LT1-NPN-SOT23-BEC
- removed R69: 10kB, EurorackModularParts:POTSQUAREHOLE_SMALLKNOB
- removed RN3, RN9: 56, resistor-dil:4R-N0402ARV341
- added C12, C13: 100n, resistor:C-EUC0402
- added IC1: PCM3060, FenixBase:PCM3060
- added JACK11: (no value), EurorackModularParts:AUDIO-JACK_SMALLSYMBOL
- added Q6, Q7: MMBT3904, transistor:MMBT3904LT1-NPN-SOT23-BEC
- added R35, R38, R46, R49, R50, R54, R55, R58, R59: 56, OPL:R-0603
- added R43, R47, R48, R51, R53, R56, R57, R60, R61: 10k, OPL:R-0603
- added U$11, U$12, U$13, U$23, U$24, U$31, U$32, U$33, U$34, U$35, U$36, U$37, U$38, U$39, U$40, U$41, U$42, U$43, U$44: SWITCH_W_LED_PB6149L-X-102YELLOW, zephod-components:SWITCH_W_LED_PB6149L-X-102YELLOW
- added U2: CJ1117-5.0, OPL:CJ1117-3.3-1310190P1
- C1: value 3.3nF -> 100n; OC_FARNELL unknown -> (none)
- C10, C18, C40: value 100nF -> 10u; device resistor:C-EUC0402 -> EurorackModularParts:C-POLAR-A; MF MULTICOMP -> (none); MPN MC0603F104Z160CT -> (none); OC_FARNELL 1759017 -> (none)
- C19: value 100nF -> 100n; MF MULTICOMP -> (none); MPN MC0603F104Z160CT -> (none); OC_FARNELL 1759017 -> (none)
- C2: value 3.3nF C0G -> 100n; OC_FARNELL unknown -> (none)
- C21, C22: value 100nF -> 2.2n; device resistor:C-EUC0402 -> OPL:C-0603; MF MULTICOMP -> (none); MPN MC0603F104Z160CT -> (none); OC_FARNELL 1759017 -> (none)
- C3: value 3.3nF COG -> 10u; device OPL:C-0603 -> EurorackModularParts:C-POLAR-A; OC_FARNELL unknown -> (none)
- C9: value 3.3nF -> 10u; device OPL:C-0603 -> EurorackModularParts:C-POLAR-A; OC_FARNELL unknown -> (none)
- JACK1: DESC Frequency -> Balance 1
- JACK10: DESC Phased Cycle -> Out 1
- JACK2: DESC Shape -> Balance 2
- JACK3: DESC Mod -> START1
- JACK6: DESC Phase -> START2
- JACK7: DESC Normal Out -> In 1
- JACK8: DESC Phased Out -> In 2
- JACK9: DESC Normal Cycle -> Clock
- R11: value 100k -> 10k
- R13, R2: value 33k -> 10k
- R17: DESC (none) -> Balance 1
- R21: value 100k -> 56
- R24: value 100 -> 56
- R25: value 100 -> 10k
- R27: value 56 -> 10k
- R3: value 51k -> 100k
- R36, R37: value 187k 0.1% -> 10k
- R41: value 51k -> 56
- R42: value 10kB -> 10k; device EurorackModularParts:POTSQUAREHOLE_SMALLKNOB -> OPL:R-0603
- R44: DESC (none) -> Tempo
- R45: value 10kB -> 56; device EurorackModularParts:POTSQUAREHOLE_SMALLKNOB -> OPL:R-0603
- R5, R8: value 187k 0.1% -> 56
- R68: DESC (none) -> Balance 2
- R7, R9: value 38.3k 0.1% -> 56
Connections:
- net ADC_FREQ renamed ADC_BALANCE_1
- net ADC_NORMAL renamed KNOB_TEMPO
- net ADC_SHAPE renamed ADC_BALANCE_2
- net FASTMODE_BUT renamed ARM_1_BUT
- net KNOB_FREQ renamed KNOB_BALANCE_1
- net KNOB_SHAPE renamed KNOB_BALANCE_2
- net N$51 renamed SHIFT_LED
- net OUT_LFOCYCLESTART renamed OUT_CLOCK
- net RESET_PATTERN_BUT renamed SHIFT_BUT
- net SYNC_LFO renamed CLOCK_IN
- removed net FASTMODE_LED: IC9.Q6, R30.2
- removed net N$67: D35.+, RN3B.2
- removed net N$68: IC9.Q5, RN9A.1
- removed net N$72: D20.+, RN9C.2
- removed net N$73: D30.+, RN2C.2
- removed net N$75: D32.+, RN2A.2
- removed net N$77: D27.+, RN1B.2
- removed net N$78: D26.+, RN1C.2
- removed net N$79: D25.+, RN1D.2
- removed net N$83: D16.+, R29.1
- removed net N$84: D21.+, RN9D.2
- removed net N$85: D17.+, RN9B.2
- removed net N$88: D22.+, RN9A.2
- removed net N$89: IC9.Q4, RN9B.1
- removed net N$90: IC9.Q3, RN9C.1
- removed net N$91: IC9.Q2, RN9D.1
- removed net N$92: IC9.Q1, R29.2
- removed net N$94: IC8.Q7S, IC9.DS
- removed net NORMALOUT: C3.2, IC2VR1.OUT, R24.2, R8.1
- removed net PHASEDOUT: C2.2, IC2VR2.OUT, R25.2, R5.1
- new net 1_1_BUT: R13.2, U$23.1, U$23.2
- new net 1_1_LED: R9.2
- new net 1_2_BUT: R25.2, U$31.1, U$31.2
- new net 1_2_LED: R21.2
- new net 1_3_BUT: R36.2, U$33.1, U$33.2
- new net 1_3_LED: R29.2
- new net 1_4_BUT: R42.2, U$35.1, U$35.2
- new net 1_4_LED: R38.2
- new net 1_5_BUT: R47.2, U$37.1, U$37.2
- new net 1_5_LED: R45.2
- new net 1_6_BUT: R51.2, U$39.1, U$39.2
- new net 1_6_LED: R49.2
- new net 1_7_BUT: R56.2, U$41.1, U$41.2
- new net 1_7_LED: R54.2
- new net 1_8_BUT: R60.2, U$43.1, U$43.2
- new net 1_8_LED: R58.2
- new net 2_1_BUT: R19.2, U$24.1, U$24.2
- new net 2_1_LED: R10.2
- new net 2_2_BUT: R27.2, U$32.1, U$32.2
- new net 2_2_LED: R24.2
- new net 2_3_BUT: R37.2, U$34.1, U$34.2
- new net 2_3_LED: R35.2
- new net 2_4_BUT: R43.2, U$36.1, U$36.2
- new net 2_4_LED: R41.2
- new net 2_5_BUT: R48.2, U$38.1, U$38.2
- new net 2_5_LED: R46.2
- new net 2_6_BUT: R53.2, U$40.1, U$40.2
- new net 2_6_LED: R50.2
- new net 2_7_BUT: R57.2, U$42.1, U$42.2
- new net 2_7_LED: R55.2
- new net 2_8_BUT: R61.2, U$44.1, U$44.2
- new net 2_8_LED: R59.2
- new net 5V: C13.2, C18.1, C2.1, C3.1, IC1.VCC, U2.OUT
- new net ARM_1_LED: R30.2
- new net ARM_2_BUT: U$13.1, U$13.2
- new net ARM_2_LED: R8.2
- new net BIAS_AUDIO: C10.1, C12.1, IC1.VCOM
- new net CODEC_SCL: IC1.MC/SCL/FMT
- new net CODEC_SDA: IC1.MD/SDA/DEMP
- new net I2S_BCK1: IC1.BCK1
- new net I2S_DIN: IC1.DIN
- new net I2S_DOUT: IC1.DOUT
- new net I2S_LRCK1: IC1.LRCK1
- new net I2S_SCKI1: IC1.SCKI1
- new net INL: C22.1, IC1.VINL
- new net INR: C21.1, IC1.VINR
- new net N$51: R49.1, U$39.POS
- new net START_1: Q6.C, R2.1
- new net START_1_BUT: U$11.1, U$11.2
- new net START_1_LED: R5.2
- new net START_2: Q7.C, R11.1
- new net START_2_BUT: U$12.1, U$12.2
- new net START_2_LED: R7.2
- net -12V: no longer C19.2, IC2VR3.V-
- net 12V: now also C1.1, C9.1, U2.IN; no longer C18.2, IC2VR3.V+, R19.2
- net 3.3V: now also C19.1, C40.1, IC1.VDD, R11.2, R13.1, R19.1, R2.2, R25.1, R27.1, R36.1, R37.1, R42.1, R43.1, R47.1, R48.1, R51.1, R53.1, R56.1, R57.1, R60.1, R61.1; no longer C22.2, C38.2, D40.+, IC3.VDD, IC8.!MR, IC8.VCC, IC9.!MR, IC9.VCC, R42.A, R45.A, R69.A
- net ADC_MOD: no longer C1.2, IC4N.OUT, R2.1
- net ADC_PHASE: no longer C9.2, IC4K.OUT, R13.1
- net ADC_PHASED: no longer C40.1, R45.S
- net CLOCK_2: no longer IC8.SHCP, IC9.SHCP
- net DACCS: no longer IC3./CS
- net DACSCK: no longer IC3.SCK
- net DACSDI: no longer IC3.SDI
- net GND: now also C1.2, C12.2, C13.1, C18.2, C19.2, C2.2, C22.2, C3.2, C9.2, IC1.!MS!/ADR/IFMD, IC1.AGND1, IC1.AGND2, IC1.BCK2, IC1.DGND, IC1.LRCK2, IC1.MODE, IC1.SCKI2, IC1.SGND, JACK11.RING, JACK7.SWITCH, JACK8.SWITCH, Q6.E, Q7.E, U$11.3, U$11.4, U$11.NEG, U$12.3, U$12.4, U$12.NEG, U$13.3, U$13.4, U$13.NEG, U$23.3, U$23.4, U$23.NEG, U$24.3, U$24.4, U$24.NEG, U$31.3, U$31.4, U$31.NEG, U$32.3, U$32.4, U$32.NEG, U$33.3, U$33.4, U$33.NEG, U$34.3, U$34.4, U$34.NEG, U$35.3, U$35.4, U$35.NEG, U$36.3, U$36.4, U$36.NEG, U$37.3, U$37.4, U$37.NEG, U$38.3, U$38.4, U$38.NEG, U$39.3, U$39.4, U$39.NEG, U$40.3, U$40.4, U$40.NEG, U$41.3, U$41.4, U$41.NEG, U$42.3, U$42.4, U$42.NEG, U$43.3, U$43.4, U$43.NEG, U$44.3, U$44.4, U$44.NEG, U2.GND; no longer C18.1, C19.1, C22.1, C38.1, D10.-, D11.-, D12.-, D13.-, D14.-, D16.-, D17.-, D20.-, D21.-, D22.-, D24.-, D25.-, D26.-, D27.-, D28.-, D29.-, D30.-, D31.-, D32.-, D33.-, D34.-, D35.-, D4.-, D5.-, IC2VR1.+IN, IC2VR2.+IN, IC3./LDAC, IC3.VSS, IC4K.+IN, IC4N.+IN, IC8.!OE, IC8.GND, IC8.GND_2, IC9.!OE, IC9.GND, IC9.GND_2, Q3.E, R42.E, R45.E, R69.E
- net KNOB_MOD: no longer C10.1, R69.S
- net KNOB_PHASE: no longer C21.1, R42.S
- net LATCH_2: no longer IC8.STCP, IC9.STCP
- net N$10: now also R9.1, U$23.POS; no longer C3.1, IC2VR1.-IN, R36.1, R7.1, R8.2
- net N$11: now also Q7.B, R3.2; no longer JACK6.TIP, R11.2
- net N$12: now also JACK6.TIP, R3.1; no longer C9.1, IC4K.-IN, R11.1, R13.2, R41.1
- net N$20: now also R10.1, U$24.POS; no longer JACK8.TIP, R25.1
- net N$21: now also R21.1, U$31.POS; no longer JACK7.TIP, R24.1
- net N$23: now also R24.1, U$32.POS; no longer D40.-, R10.1
- net N$25: now also R29.1, U$33.POS; no longer Q3.B, R21.2
- net N$28: now also R35.1, U$34.POS; no longer D29.+, RN2D.2
- net N$29: now also R38.1, U$35.POS; no longer JACK10.TIP, Q3.C, R19.1
- net N$32: now also R41.1, U$36.POS; no longer D28.+, RN1A.2
- net N$37: now also R45.1, U$37.POS; no longer IC8.Q2, RN3D.1
- net N$41: no longer D10.+
- net N$42: now also R46.1, U$38.POS; no longer D13.+, RN3C.2
- net N$47: no longer D5.+
- net N$48: no longer D4.+
- net N$5: now also R5.1, U$11.POS; no longer IC3.VOUTA, R9.2
- net N$52: no longer D11.+
- net N$57: now also R50.1, U$40.POS; no longer IC8.Q3, RN3C.1
- net N$58: now also R54.1, U$41.POS; no longer D14.+, RN3D.2
- net N$59: now also R55.1, U$42.POS; no longer IC8.Q4, RN3B.1
- net N$6: now also Q6.B; no longer JACK3.TIP
- net N$62: now also R58.1, U$43.POS; no longer IC8.Q5, RN3A.1
- net N$63: now also R59.1, U$44.POS; no longer IC8.Q1, R27.2
- net N$65: now also IC1.VOUTL+; no longer D12.+, R27.1
- net N$66: now also IC1.VOUTR+; no longer D34.+, RN3A.2
- net N$7: now also R7.1, U$12.POS; no longer IC3.VOUTB, R7.2
- net N$74: now also IC1.!RST!; no longer D31.+, RN2B.2
- net N$76: no longer D24.+
- net N$8: now also JACK3.TIP; no longer C1.1, IC4N.-IN, R2.2, R3.1
- net N$80: no longer D33.+
- net N$9: now also R8.1, U$13.POS; no longer C2.1, IC2VR2.-IN, R37.1, R5.2, R9.1
- net OUT_LFOCYCLEMID: no longer R10.2, R21.1
- net REF_-5V: no longer R3.2, R36.2, R37.2, R41.2
- net SHIFTERS_2: no longer IC8.DS
Other:
- moved on the sheet: JACK10, JACK3, JACK6, R1, R10, R11, R19, R2, R21, R27, R29, R3

Commit message: looper and stuff
Parts:
- removed C10, C18, C3, C40, C9: 10u, EurorackModularParts:C-POLAR-A
- removed C100: 1u, resistor:C-EUC0402
- removed C12, C13, C19, C74, C99: 100n, resistor:C-EUC0402
- removed C21, C22: 2.2n, OPL:C-0603
- removed C25, C26, C27, C28, C29, C30, C31, C35, C36, C37: 100n, Discrete:C-0402
- removed C32, C33: 27p, Discrete:C-0402
- removed C34: 1u, Discrete:C-0402
- removed C39: 4.7n 100v, OPL:C-1206
- removed IC10: 4052D, 40xx:4052D
- removed J1: MICRO-USB-5P, OPL:MICRO-USB-5P
- removed K1: BUTTON-4P-3100010P1, OPL:BUTTON-4P-3100010P1
- removed Q4: 12mhz, adafruit:XTAL-4-3225
- removed R103, R33: 1k, Discrete:R-0402
- removed R34: 10k DNP, Discrete:R-0402
- removed R52: 10k, Discrete:R-0402
- removed R74: 1M, OPL:R-0603
- removed SWD2: CORTEX_SWD, carrilib with jtags:CORTEX_SWD
- removed TP1, TP2, TP3, TP4: PTR1B1,27, testpad:PTR1B1,27
- removed U$2: RP2040, RP2040:RP2040
- removed U$25: W25Q256JVEIQTR, RP2040:W25Q128JVSIQ
- removed U2: CJ1117-5.0, OPL:CJ1117-3.3-1310190P1
- added C38, C47: 100p, OPL:C-0603
- added C49, C54, C55, C58, C59: 100n, OPL:C-0603
- added C50, C52: 470p, OPL:C-0603
- added C51, C53, C56, C57: 47p, OPL:C-0603
- added IC2: TL074TSSOP14, EurorackModularParts:TL074TSSOP14
- added IC3: NE5532D, EurorackModularParts:NE5532D
- added IC8: 74HC165D, 74xx-eu:74HC165D
- added JACK12: (no value), EurorackModularParts:AUDIO-JACK_SMALLSYMBOL
- added Q3: MMBT3904, transistor:MMBT3904LT1-NPN-SOT23-BEC
- added R62, R63, R70, R71, R84, R85, R86, R87, R88, R89: 100k, OPL:R-0603
- added R64, R65, R75, R76: 12.1k, OPL:R-0603
- added R66, R80: 4.42k, OPL:R-0603
- added R67, R69: 100, OPL:R-0603
- added R77, R81: 4.02k, OPL:R-0603
- added R78, R82: 35.7k, OPL:R-0603
- added R79, R83: 56, OPL:R-0603
- added U$50: MCP6022I/ST, EurorackModularParts:MCP6022I/ST
- added U$55: MCUPLUGIN2, FenixBase:MCUPLUGIN2
- C1, C2: value 100n -> 100nF; device OPL:C-0603 -> resistor:C-EUC0402; MF (none) -> MULTICOMP; MPN (none) -> MC0603F104Z160CT; OC_FARNELL (none) -> 1759017
- IC1: value PCM3060 -> 74HC165D; device FenixBase:PCM3060 -> 74xx-eu:74HC165D
- J14: value POWERSHROUDED -> POWER_SIMPLE10; device EurorackModularParts:POWERSHROUDED -> EurorackModularParts:POWER_SIMPLE10
- JACK3: DESC START1 -> Start 1
- JACK6: DESC START2 -> Start 2
- R4: value 27 -> 100k; device Discrete:R-0402 -> OPL:R-0603; OC_FARNELL (none) -> unknown
- R6: value 27 -> 10k; device Discrete:R-0402 -> OPL:R-0603; OC_FARNELL (none) -> unknown
Connections:
- removed net 1.1V: C29.1, C34.1, C99.1, U$2.DVDD, U$2.VREG_VOUT
- removed net 5V: C13.2, C18.1, C2.1, C3.1, IC1.VCC, U2.OUT
- removed net ADC0: IC10A.X, U$2.GPIO26/ADC0
- removed net ADC1: IC10A.Y, U$2.GPIO27/ADC1
- removed net ADC_MOD: IC10A.Y1
- removed net ADC_PHASE: IC10A.Y0
- removed net ADC_PHASED: IC10A.Y2
- removed net BOOTSEL_BUT: K1.A0, K1.A1, R33.2
- removed net CLOCK_2: U$2.GPIO10
- removed net CODEC_SCL: IC1.MC/SCL/FMT
- removed net CODEC_SDA: IC1.MD/SDA/DEMP
- removed net DACCS: U$2.GPIO1
- removed net DACSCK: U$2.GPIO0
- removed net DACSDI: U$2.GPIO2
- removed net I2S_BCK1: IC1.BCK1
- removed net I2S_DIN: IC1.DIN
- removed net I2S_DOUT: IC1.DOUT
- removed net I2S_LRCK1: IC1.LRCK1
- removed net I2S_SCKI1: IC1.SCKI1
- removed net INL: C22.1, IC1.VINL
- removed net INR: C21.1, IC1.VINR
- removed net KNOB_MOD: IC10A.X0
- removed net KNOB_PHASE: IC10A.X3
- removed net LATCH_2: U$2.GPIO11
- removed net MEM_CLK: U$2.QSPI_SCLK, U$25.CLK
- removed net MEM_CS: R33.1, R34.1, U$2.QSPI_CSN, U$25./CS
- removed net MEM_IO0: U$2.QSPI_SD0, U$25.DI
- removed net MEM_IO1: U$2.QSPI_SD1, U$25.DO
- removed net MEM_IO2: U$2.QSPI_SD2, U$25.IO2
- removed net MEM_IO3: U$2.QSPI_SD3, U$25.IO3
- removed net MUX_A: IC10A.A, U$2.GPIO24
- removed net MUX_B: IC10A.B, U$2.GPIO25
- removed net N$100: TP3.TP, U$2.GPIO8
- removed net N$18: R4.2, U$2.USB_DP
- removed net N$24: R6.2, U$2.USB_DM
- removed net N$65: IC1.VOUTL+
- removed net N$66: IC1.VOUTR+
- removed net N$69: C39.2, J1.GND@2, J1.GND@3, R74.2
- removed net N$74: IC1.!RST!
- removed net N$81: J1.VCC, TP1.TP
- removed net N$82: TP2.TP, U$2.GPIO15
- removed net N$86: TP4.TP, U$2.GPIO7
- removed net N$87: R103.2, U$2.XOUT
- removed net RUN: R52.2, SWD2.RESET, U$2.RUN
- removed net SHIFTERS_2: U$2.GPIO9
- removed net SWCLK: SWD2.SWCLK, U$2.SWCLK
- removed net SWDIO: SWD2.SWDIO, U$2.SWDIO
- removed net USB_N: J1.DM, R6.1
- removed net USB_P: J1.DP, R4.1
- new net 3V3_AUDIO: C49.2, U$50G$3.V+, U$55.AUDIO3.3V
- new net ARM_1: Q3.C, R6.1
- new net BIAS_BUFFERED: IC2B.-IN, IC2B.OUT, R70.1
- new net BIAS_INVERTED: IC2A.OUT, R71.2, R75.1, R76.1, R85.1, R87.1
- new net N$101: C56.2, IC2C.-IN, R84.2, R85.2, R89.1
- new net N$102: C57.2, IC2D.-IN, R86.2, R87.2, R88.1
- new net N$103: C56.1, IC2C.OUT, R80.1, R89.2
- new net N$104: R86.1, U$55.AUDIOOUT2
- new net N$105: R84.1, U$55.AUDIOOUT1
- new net N$106: C57.1, IC2D.OUT, R66.1, R88.2
- new net N$107: JACK7.TIP, R63.1
- new net N$108: JACK8.TIP, R62.1
- new net N$75: C38.2, R62.2, R65.1, R76.2, U$50G$2.-IN
- new net N$77: C47.2, R63.2, R64.1, R75.2, U$50G$1.-IN
- new net N$78: C38.1, R65.2, R69.1, U$50G$2.OUT
- new net N$79: C47.1, R64.2, R67.1, U$50G$1.OUT
- new net N$83: IC2A.-IN, R70.2, R71.1
- new net N$84: C51.2, IC3A.-IN, R77.2
- new net N$85: C50.2, R66.2, R77.1, R78.1
- new net N$88: C51.1, IC3A.OUT, R78.2, R79.1
- new net N$89: JACK11.TIP, R79.2
- new net N$90: C53.2, IC3B.-IN, R81.2
- new net N$91: C52.2, R80.2, R81.1, R82.1
- new net N$92: C53.1, IC3B.OUT, R82.2, R83.1
- new net N$94: JACK10.TIP, R83.2
- new net TO_AUDIOIN_1: R67.2, U$55.AUDIOIN1
- new net TO_AUDIOIN_2: R69.2, U$55.AUDIOIN2
- net -12V: now also C55.1, C59.1, IC2P.V-, IC3P.V-
- net 12V: now also C54.2, C58.2, IC2P.V+, IC3P.V+, U$55.12V; no longer C1.1, C9.1, U2.IN
- net 1_1_BUT: now also IC1A.A
- net 1_2_BUT: now also IC1A.B
- net 1_3_BUT: now also IC1A.C
- net 1_4_BUT: now also IC1A.D
- net 1_5_BUT: now also IC1A.E
- net 1_6_BUT: now also IC1A.F
- net 1_7_BUT: now also IC1A.G
- net 1_8_BUT: now also IC1A.H
- net 2_1_BUT: now also IC8A.A
- net 2_2_BUT: now also IC8A.B
- net 2_3_BUT: now also IC8A.C
- net 2_4_BUT: now also IC8A.D
- net 2_5_BUT: now also IC8A.E
- net 2_6_BUT: now also IC8A.F
- net 2_7_BUT: now also IC8A.G
- net 2_8_BUT: now also IC8A.H
- net 3.3V: now also C1.2, C2.2, IC1P.VCC, IC8P.VCC, R6.2, U$55.3.3V; no longer C100.1, C19.1, C25.2, C26.2, C27.2, C28.2, C30.2, C31.2, C35.2, C36.2, C37.2, C40.1, C74.2, IC1.VDD, IC10P.VCC, R34.2, R52.1, SWD2.VCC, U$2.ADC_IOVDD, U$2.IOVDD, U$2.USB_IOVDD, U$2.VREG_IOVDD, U$25.VCC
- net ADC_BALANCE_1: now also U$55.ADC3; no longer U$2.GPIO28/ADC2
- net ADC_BALANCE_2: now also U$55.ADC4; no longer U$2.GPIO29/ADC3
- net ARM_1_BUT: no longer U$2.GPIO5
- net BIAS_AUDIO: now also IC2B.+IN, U$55.VCOM; no longer C10.1, C12.1, IC1.VCOM
- net CLOCK: no longer U$2.GPIO13
- net CLOCK_IN: no longer U$2.GPIO22
- net GND: now also C1.1, C2.1, C49.1, C50.1, C52.1, C54.1, C55.2, C58.1, C59.2, IC1P.GND, IC2A.+IN, IC2C.+IN, IC2D.+IN, IC3A.+IN, IC3B.+IN, IC8P.GND, JACK12.RING, JACK12.SWITCH, Q3.E, U$50G$1.+IN, U$50G$2.+IN, U$50G$3.V-, U$55.GND1, U$55.GND2, U$55.GND3, U$55.GND4, U$55.GND5, U$55.GND6, U$55.GND7, U$55.GND8, U$55.GND9; no longer C1.2, C10.2, C100.2, C12.2, C13.1, C18.2, C19.2, C2.2, C21.2, C22.2, C25.1, C26.1, C27.1, C28.1, C29.2, C3.2, C30.1, C31.1, C32.2, C33.2, C34.2, C35.1, C36.1, C37.1, C39.1, C40.2, C74.1, C9.2, C99.2, IC1.!MS!/ADR/IFMD, IC1.AGND1, IC1.AGND2, IC1.BCK2, IC1.DGND, IC1.LRCK2, IC1.MODE, IC1.SCKI2, IC1.SGND, IC10A.INH, IC10P.GND, IC10P.VEE, J1.GND@1, K1.B0, K1.B1, Q4.G1, Q4.G2, R74.1, SWD2.GND1, SWD2.GND2, U$2.GND, U$2.TESTEN, U$25.GND, U2.GND
- net KNOB_BALANCE_1: now also U$55.ADC0; no longer IC10A.X1
- net KNOB_BALANCE_2: now also U$55.ADC1; no longer IC10A.X2
- net KNOB_TEMPO: now also U$55.ADC2; no longer IC10A.Y3
- net LATCH: no longer U$2.GPIO14
- net N$17: now also JACK12.TIP, R4.1; no longer C32.1, Q4.X1, R103.1
- net N$2: now also Q3.B, R4.2; no longer C33.1, Q4.X2, U$2.XIN
- net RESET_PATTERN: no longer U$2.GPIO21
- net SHIFTERS: no longer U$2.GPIO12
- net SHIFT_BUT: no longer U$2.GPIO20
Other:
- note added: "TODO: CALCULATE r29 and r30 for correct bias!!"
