File: Development/Eurorack Set 2021/FenixCaseMixer.sch (EAGLE design)
At the start: 27 parts, among them IC2 TL072TSSOP8

Commit message: Minor Updates..
Parts:
- added C3, C6: 10u, EurorackModularParts:C-POLAR-A
- added D1, D2: (no value), OPL:D-SMA
- added R7: 22K, OPL:R-0603
- added U$10, U$11, U$12, U$13: VOLTAGETESTPAD, FenixBase:VOLTAGETESTPAD
- added U$7: POWER_SIMPLE10, EurorackModularParts:POWER_SIMPLE10
- R1: DESC A -> C
- R2: DESC A -> B
- R3: DESC B -> A
- R5: DESC A -> D
- U$5: value FENIXGRID -> VOLTAGETESTPAD_BIG; device FenixBase:FENIXGRID -> FenixBase:VOLTAGETESTPAD_BIG; DESC Mixer -> IN
- U$6: value MODULEEND -> VOLTAGETESTPAD_BIG; device FenixBase:MODULEEND -> FenixBase:VOLTAGETESTPAD_BIG; DESC (none) -> OUT
Connections:
- new net N$17: D1.+, U$7.+12V
- new net N$18: D2.-, U$7.-12V
- new net N$5: R7.1, U$5.VOLTAGE
- net -12V: now also C6.2, D2.+
- net 12V: now also C3.1, D1.-
- net GND: now also C3.2, C6.1, U$10.VOLTAGE, U$11.VOLTAGE, U$12.VOLTAGE, U$13.VOLTAGE, U$7.GND; no longer JACK1.RING, JACK2.RING, JACK4.RING, JACK5.RING
- net MIXO: now also U$6.VOLTAGE
- net N$8: now also R7.2
