File: Development/Eurorack Set 2021/Wobbler2_kicad/_autosave-TINRS - Wobbler (pico)sch.kicad_sch (KiCad schematic)
At the start: 2 parts

Commit message: Wobbler2 Kicad Version
Parts:
- A1, A2: renamed from A?; value (none) -> Wobbler2_PCBArt; footprint (none) -> TINRS - Wobbler (pico)sch:Wobbler2_art
Changed lines of the file:
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@@
   (symbol (lib_id "Wobbler2_art:Wobbler2_PCBArt") (at 237.49 -3.048 0) (unit 1)
     (in_bom no) (on_board yes) (fields_autoplaced)
-    (property "Reference" "A?" (id 0) (at 237.49 -3.048 0)
+    (property "Reference" "A2" (id 0) (at 237.49 -3.048 0)
       (effects (font (size 1.27 1.27)) hide)
     )
-    (property "Value" "" (id 1) (at 237.49 -4.318 0)
+    (property "Value" "Wobbler2_PCBArt" (id 1) (at 237.49 -4.318 0)
       (effects (font (size 1.27 1.27)) hide)
     )
-    (property "Footprint" "" (id 2) (at 237.49 -3.048 0)
+    (property "Footprint" "TINRS - Wobbler (pico)sch:Wobbler2_art" (id 2) (at 237.49 -3.048 0)
       (effects (font (size 1.27 1.27)) hide)
     )
@@
   (symbol (lib_id "Wobbler2_art:Wobbler2_PCBArt") (at 111.506 77.978 0) (unit 1)
     (in_bom no) (on_board yes) (fields_autoplaced)
-    (property "Reference" "A?" (id 0) (at 111.506 77.978 0)
+    (property "Reference" "A1" (id 0) (at 111.506 77.978 0)
       (effects (font (size 1.27 1.27)) hide)
     )
-    (property "Value" "" (id 1) (at 111.506 76.708 0)
+    (property "Value" "Wobbler2_PCBArt" (id 1) (at 111.506 76.708 0)
       (effects (font (size 1.27 1.27)) hide)
     )
-    (property "Footprint" "" (id 2) (at 111.506 77.978 0)
+    (property "Footprint" "TINRS - Wobbler (pico)sch:Wobbler2_art" (id 2) (at 111.506 77.978 0)
       (effects (font (size 1.27 1.27)) hide)
     )
@@
       (reference "#PWR0155") (unit 1) (value "+3.3V") (footprint "")
     )
+    (path "/9327f1aa-dbea-4fcc-bdc3-4fd2e32fe928"
+      (reference "A1") (unit 1) (value "Wobbler2_PCBArt") (footprint "TINRS - Wobbler (pico)sch:Wobbler2_art")
+    )
     (path "/7d2f4232-978c-4971-8416-a0c02d0f59ac"
-      (reference "A?") (unit 1) (value "Wobbler2_PCBArt") (footprint "TINRS - Wobbler (pico)sch:Wobbler2_art")
-    )
-    (path "/9327f1aa-dbea-4fcc-bdc3-4fd2e32fe928"
-      (reference "A?") (unit 1) (value "Wobbler2_PCBArt") (footprint "TINRS - Wobbler (pico)sch:Wobbler2_art")
+      (reference "A2") (unit 1) (value "Wobbler2_PCBArt") (footprint "TINRS - Wobbler (pico)sch:Wobbler2_art")
     )
     (path "/c13cb299-c112-4746-b939-055f3bcd5f66/bb16a516-4131-4a51-bbea-b711bad6e2cf"
