File: Development/Eurorack Set 2021/Space/Space/Space.kicad_pcb (KiCad board)
At the start: 2 copper layers, 119.4 x 109.2 mm, 174 parts, among them IC1 PCM3060, J1 Conn_02x08_Odd_Even, J10 AudioJack3_SwitchTR, J11 AudioJack3_SwitchTR, J12 AudioJack3_SwitchTR, J13 AudioJack3_SwitchTR, J2 AudioJack3_SwitchTR, J3 AudioJack3_SwitchTR, J4 AudioJack3_SwitchTR, J5 AudioJack3_SwitchTR, J6 AudioJack3_SwitchTR, J7 AudioJack3_SwitchTR, J8 AudioJack3_SwitchTR, J9 AudioJack3_SwitchTR, SW1 SW_Push_LED_PB614, SW2 SW_Push_LED_PB614, SW3 SW_Push_LED_PB614, SW4 SW_Push_LED_PB614, U1 Teensy4.0, U10 MCP6004, U2 R-78E5.0-0.5, U3 4052, U4 TL074, U5 4052, U6 74HC595, U7 74HC595, U8 4052, U9 MCP6004

Commit message: Space..
Parts:
- moved J13 168.3 mm to (174.2, 113.0)
- moved D7 165.1 mm to (168.0, 46.8)
- moved D19 162.4 mm to (169.5, 52.3)
- moved D11 160.1 mm to (174.5, 63.0)
- moved D13 157.5 mm to (177.5, 130.0)
- moved D8 155.4 mm to (171.5, 57.8)
- moved D10 152.5 mm to (172.5, 130.0)
- moved J7 152.0 mm to (174.0, 94.5)
- moved J12 146.3 mm to (155.5, 44.5)
- moved D9 142.0 mm to (167.5, 130.0)
- moved D15 104.6 mm to (123.0, 127.8)
- moved D20 103.0 mm to (123.0, 119.3)
- moved J6 102.1 mm to (99.0, 137.0)
- moved SW2 94.0 mm to (124.0, 139.5)
- moved D18 91.5 mm to (117.0, 114.0)
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
Commit message: a lot of module progress.. ducktape, space etc
Parts:
- removed C17, C18: 1500p, Capacitor_SMD:C_0402_1005Metric
- removed C19: 10u, Capacitor_SMD:CP_Elec_5x5.9
- removed C20, C21, C22, C23, C30: 470p, Capacitor_SMD:C_0402_1005Metric
- removed C4, C5: 10u, Capacitor_SMD:C_0805_2012Metric
- removed C6: 100n, Capacitor_SMD:C_0402_1005Metric
- removed D2: D, Diode_SMD:D_SMA
- removed D5, D6: BAT54S, Package_TO_SOT_SMD:SOT-23
- removed J10, J11, J12, J13, J2, J3, J4, J5, J6, J7, J8, J9: AudioJack3_SwitchTR, AudioJacks:Jack_3.5mm_QingPu_WQP-PJ3410_Vertical
- removed R10, R16, R17, R9: 7.5k, Resistor_SMD:R_0402_1005Metric
- removed R11, R12, R13, R14: 820, Resistor_SMD:R_0402_1005Metric
- removed R15, R22: 20k, Resistor_SMD:R_0402_1005Metric
- removed R18, R23, R5, R6, R7, R8: 10k, Resistor_SMD:R_0402_1005Metric
- removed R19, R20: 100, Resistor_SMD:R_0402_1005Metric
- removed R21, R24: 1k, Resistor_SMD:R_0402_1005Metric
- removed R3: 47, Resistor_SMD:R_0402_1005Metric
- removed RV12, RV7: R_Potentiometer, Potentiometer_THT:Potentiometer_Alps_RK09K_Single_Vertical
- removed SW2, SW3, SW4: SW_Push_LED_PB614, footprints:PB614_LED_SW_6pin
- added C46: 100n, Capacitor_SMD:C_0402_1005Metric, F.Cu at (74.5, 118.2)
- added C47: 100n, Capacitor_SMD:C_0402_1005Metric, F.Cu at (145.9, 114.0)
- added C48: 1759017, Capacitor_SMD:C_0402_1005Metric, F.Cu at (143.6, 43.2)
- added C49: 10uF, Capacitor_SMD:C_0805_2012Metric, F.Cu at (140.7, 50.1)
- added C50: 197427, TiNRS_Eagle_Footprints:CASE-A_3216, F.Cu at (140.4, 59.4)
- added C51: 1759017, Capacitor_SMD:C_0402_1005Metric, F.Cu at (139.8, 55.6)
- added C52: 1759017, Capacitor_SMD:C_0402_1005Metric, F.Cu at (139.7, 51.9)
- added C53: 1759017, Capacitor_SMD:C_0402_1005Metric, F.Cu at (143.6, 49.6)
- added C54: 22u, Capacitor_SMD:C_0805_2012Metric, F.Cu at (150.0, 39.7)
- added C55: 197427, TiNRS_Eagle_Footprints:CASE-A_3216, F.Cu at (151.7, 37.4)
- added C56: 1759017, Capacitor_SMD:C_0402_1005Metric, F.Cu at (142.1, 38.2)
- added C57: 1301804, Capacitor_SMD:C_0402_1005Metric, F.Cu at (119.8, 58.7)
- added C58: 197427, TiNRS_Eagle_Footprints:CASE-A_3216, F.Cu at (120.2, 52.4)
- added C59: 4.7n 100v, TiNRS_Eagle_Footprints:C3216, F.Cu at (112.2, 142.0)
- added C60: 1u, Capacitor_SMD:C_0402_1005Metric, F.Cu at (102.9, 119.8)
- added C61: 22u, Capacitor_SMD:C_0805_2012Metric, F.Cu at (102.4, 116.4)
- added C62: 100n, Capacitor_SMD:C_0402_1005Metric, F.Cu at (104.0, 116.8)
- added C63: 100n, Capacitor_SMD:C_0402_1005Metric, F.Cu at (81.4, 87.0)
- added C64: 100n, Capacitor_SMD:C_0402_1005Metric, F.Cu at (151.6, 96.3)
- added C65: 100p, Capacitor_SMD:C_0402_1005Metric, F.Cu at (139.3, 115.7)
- added C66: 100p, Capacitor_SMD:C_0402_1005Metric, F.Cu at (148.1, 116.4)
- added C67: 47p, Capacitor_SMD:C_0402_1005Metric, F.Cu at (152.1, 128.8)
- added C68: 47p, Capacitor_SMD:C_0402_1005Metric, F.Cu at (168.2, 119.5)
- added C69: 47p, Capacitor_SMD:C_0402_1005Metric, F.Cu at (166.8, 128.1)
- added C70: 47p, Capacitor_SMD:C_0402_1005Metric, F.Cu at (152.1, 125.4)
- added D21: D-SMA, TiNRS_Eagle_Footprints:DO-214AC, F.Cu at (133.0, 60.3)
- added D22: D-SMA, TiNRS_Eagle_Footprints:DO-214AC, F.Cu at (125.2, 60.5)
- added D23: LED, LED_THT:LED_D3.0mm_FlatTop, F.Cu at (95.8, 136.8)
- added D24: LED, LED_THT:LED_D3.0mm_FlatTop, F.Cu at (95.8, 140.5)
- added D25: LED, LED_THT:LED_D3.0mm_FlatTop, F.Cu at (95.7, 144.2)
- added D26: LED, LED_THT:LED_D3.0mm_FlatTop, F.Cu at (79.9, 46.3)
- added D27: LED, LED_THT:LED_D3.0mm_FlatTop, F.Cu at (79.9, 50.0)
- added D28: LED, LED_THT:LED_D3.0mm_FlatTop, F.Cu at (79.9, 53.7)
- added D29: LED, LED_THT:LED_D3.0mm_FlatTop, F.Cu at (131.0, 46.3)
- added D30: LED, LED_THT:LED_D3.0mm_FlatTop, F.Cu at (131.0, 50.1)
- added D31: LED, LED_THT:LED_D3.0mm_FlatTop, F.Cu at (131.0, 53.9)
- added D32: LED, LED_THT:LED_D3.0mm_FlatTop, F.Cu at (76.0, 108.5)
- added D33: LED, LED_THT:LED_D3.0mm_FlatTop, F.Cu at (76.0, 112.7)
- added J14: MICRO-USB-5P, TiNRS_Eagle_Footprints:C132563, F.Cu at (105.1, 146.5)
- added JACK1: AUDIO-JACK_SMALLSYMBOLNODRILL, TiNRS_Eagle_Footprints:3.5MM-JACK-SWITCH-13MM-NOHOLES-TESTPAD, F.Cu at (68.8, 65.7)
- added JACK10: AUDIO-JACK_SMALLSYMBOLNODRILL, TiNRS_Eagle_Footprints:3.5MM-JACK-SWITCH-13MM-NOHOLES-TESTPAD, F.Cu at (68.7, 51.0)
- added JACK11: AUDIO-JACK_SMALLSYMBOLNODRILL, TiNRS_Eagle_Footprints:3.5MM-JACK-SWITCH-13MM-NOHOLES-TESTPAD, F.Cu at (176.8, 98.3)
- added JACK12: AUDIO-JACK_SMALLSYMBOLNODRILL, TiNRS_Eagle_Footprints:3.5MM-JACK-SWITCH-13MM-NOHOLES-TESTPAD, F.Cu at (177.0, 110.3)
- added JACK13: AUDIO-JACK_SMALLSYMBOLNODRILL, TiNRS_Eagle_Footprints:3.5MM-JACK-SWITCH-13MM-NOHOLES-TESTPAD, F.Cu at (68.7, 98.3)
- added JACK14: AUDIO-JACK_SMALLSYMBOLNODRILL, TiNRS_Eagle_Footprints:3.5MM-JACK-SWITCH-13MM-NOHOLES-TESTPAD, F.Cu at (68.8, 110.2)
- added JACK2: AUDIO-JACK_SMALLSYMBOLNODRILL, TiNRS_Eagle_Footprints:3.5MM-JACK-SWITCH-13MM-NOHOLES-TESTPAD, F.Cu at (68.7, 79.6)
- added JACK3: AUDIO-JACK_SMALLSYMBOLNODRILL, TiNRS_Eagle_Footprints:3.5MM-JACK-SWITCH-13MM-NOHOLES-TESTPAD, F.Cu at (68.7, 140.7)
- added JACK4: AUDIO-JACK_SMALLSYMBOLNODRILL, TiNRS_Eagle_Footprints:3.5MM-JACK-SWITCH-13MM-NOHOLES-TESTPAD, F.Cu at (148.2, 140.6)
- added JACK5: AUDIO-JACK_SMALLSYMBOLNODRILL, TiNRS_Eagle_Footprints:3.5MM-JACK-SWITCH-13MM-NOHOLES-TESTPAD, F.Cu at (176.8, 79.4)
- added JACK6: AUDIO-JACK_SMALLSYMBOLNODRILL, TiNRS_Eagle_Footprints:3.5MM-JACK-SWITCH-13MM-NOHOLES-TESTPAD, F.Cu at (176.7, 65.3)
- added JACK7: AUDIO-JACK_SMALLSYMBOLNODRILL, TiNRS_Eagle_Footprints:3.5MM-JACK-SWITCH-13MM-NOHOLES-TESTPAD, F.Cu at (176.7, 124.2)
- added JACK8: AUDIO-JACK_SMALLSYMBOLNODRILL, TiNRS_Eagle_Footprints:3.5MM-JACK-SWITCH-13MM-NOHOLES-TESTPAD, F.Cu at (176.9, 140.7)
- added JACK9: AUDIO-JACK_SMALLSYMBOLNODRILL, TiNRS_Eagle_Footprints:3.5MM-JACK-SWITCH-13MM-NOHOLES-TESTPAD, F.Cu at (176.7, 51.2)
- added L5: 0.1uH C76737, Inductor_SMD:L_0805_2012Metric, F.Cu at (141.7, 56.5)
- added L6: 0.1uH C76737, Inductor_SMD:L_0805_2012Metric, F.Cu at (141.7, 53.0)
- added L7: 4.7uH, TiNRS_Eagle_Footprints:L0420, F.Cu at (147.0, 43.4)
- added L8: 0.1uH C76737, Inductor_SMD:L_0805_2012Metric, F.Cu at (147.0, 38.9)
- added Q3: MMBT3904, Package_TO_SOT_SMD:SOT-23, F.Cu at (167.9, 50.1)
- added Q4: MMBT3904, Package_TO_SOT_SMD:SOT-23, F.Cu at (75.7, 57.0)
- added R100: 12.1k, Resistor_SMD:R_0603_1608Metric, F.Cu at (144.3, 119.0)
- added R101: 12.1k, Resistor_SMD:R_0603_1608Metric, F.Cu at (149.4, 116.3)
- added R102: 100k, Resistor_SMD:R_0402_1005Metric, F.Cu at (142.1, 126.0)
- added R103: 100k, Resistor_SMD:R_0402_1005Metric, F.Cu at (143.2, 125.0)
- added R104: 100k, Resistor_SMD:R_0402_1005Metric, F.Cu at (153.1, 128.8)
- added R105: 100k, Resistor_SMD:R_0402_1005Metric, F.Cu at (154.1, 128.8)
- added R106: 100k, Resistor_SMD:R_0402_1005Metric, F.Cu at (148.7, 130.5)
- added R107: 4.42k, Resistor_SMD:R_0603_1608Metric, F.Cu at (164.9, 119.1)
- added R108: 4.02k, Resistor_SMD:R_0603_1608Metric, F.Cu at (167.3, 117.0)
- added R109: 37.5k, Resistor_SMD:R_0603_1608Metric, F.Cu at (168.8, 117.0)
- added R110: 56, Resistor_SMD:R_0402_1005Metric, F.Cu at (170.2, 117.3)
- added R111: 37.5k, Resistor_SMD:R_0603_1608Metric, F.Cu at (167.7, 130.1)
- added R112: 4.42k, Resistor_SMD:R_0603_1608Metric, F.Cu at (162.7, 130.6)
- added R113: 4.02k, Resistor_SMD:R_0603_1608Metric, F.Cu at (166.2, 130.1)
- added R114: 100k, Resistor_SMD:R_0402_1005Metric, F.Cu at (154.1, 125.4)
- added R115: 56, Resistor_SMD:R_0402_1005Metric, F.Cu at (169.5, 129.1)
- added R116: 100k, Resistor_SMD:R_0402_1005Metric, F.Cu at (153.1, 125.4)
- added R117: 100k, Resistor_SMD:R_0402_1005Metric, F.Cu at (148.7, 123.7)
- added R66: 12.1k, Resistor_SMD:R_0603_1608Metric, F.Cu at (138.0, 115.7)
- added R67: 100k, Resistor_SMD:R_0402_1005Metric, F.Cu at (136.2, 116.5)
- added R68: 12.1k, Resistor_SMD:R_0603_1608Metric, F.Cu at (138.0, 118.7)
- added R69: unknown, Resistor_SMD:R_0402_1005Metric, F.Cu at (140.4, 46.9)
- added R70: unknown, Resistor_SMD:R_0402_1005Metric, F.Cu at (142.2, 39.8)
- added R71: unknown, Resistor_SMD:R_0402_1005Metric, F.Cu at (138.6, 42.7)
- added R72: unknown, Resistor_SMD:R_0402_1005Metric, F.Cu at (123.5, 56.8)
- added R73: 0, Resistor_SMD:R_0402_1005Metric, F.Cu at (103.1, 133.5)
- added R74: 0, Resistor_SMD:R_0402_1005Metric, F.Cu at (103.1, 132.2)
- added R75: 1M, Resistor_SMD:R_0402_1005Metric, F.Cu at (110.2, 142.7)
- added R76: 2k, Resistor_SMD:R_0402_1005Metric, F.Cu at (125.3, 106.9)
- added R77: 2k, Resistor_SMD:R_0402_1005Metric, F.Cu at (120.8, 106.8)
- added R78: 10k, Resistor_SMD:R_0402_1005Metric, F.Cu at (104.0, 118.8)
- added R79: 56, Resistor_SMD:R_0402_1005Metric, F.Cu at (73.4, 37.4)
- added R80: 56, Resistor_SMD:R_0402_1005Metric, F.Cu at (93.8, 145.0)
- added R81: 56, Resistor_SMD:R_0402_1005Metric, F.Cu at (156.8, 89.1)
- added R82: 56, Resistor_SMD:R_0402_1005Metric, F.Cu at (78.1, 46.9)
- added R83: 56, Resistor_SMD:R_0402_1005Metric, F.Cu at (78.1, 49.6)
- added R84: 56, Resistor_SMD:R_0402_1005Metric, F.Cu at (78.1, 53.4)
- added R85: 56, Resistor_SMD:R_0402_1005Metric, F.Cu at (76.5, 41.2)
- added R86: 56, Resistor_SMD:R_0402_1005Metric, F.Cu at (98.9, 128.4)
- added R87: 56, Resistor_SMD:R_0402_1005Metric, F.Cu at (129.2, 45.8)
- added R88: 56, Resistor_SMD:R_0402_1005Metric, F.Cu at (129.1, 49.6)
- added R89: 56, Resistor_SMD:R_0402_1005Metric, F.Cu at (129.2, 53.5)
- added R90: 56, Resistor_SMD:R_0402_1005Metric, F.Cu at (127.4, 40.7)
- added R91: 56, Resistor_SMD:R_0402_1005Metric, F.Cu at (74.2, 107.1)
- added R92: 56, Resistor_SMD:R_0402_1005Metric, F.Cu at (74.2, 113.5)
- added R93: unknown, Resistor_SMD:R_0402_1005Metric, F.Cu at (75.7, 60.0)
- added R94: unknown, Resistor_SMD:R_0402_1005Metric, F.Cu at (76.7, 53.9)
- added R95: unknown, Resistor_SMD:R_0402_1005Metric, F.Cu at (168.0, 53.1)
- added R96: unknown, Resistor_SMD:R_0402_1005Metric, F.Cu at (168.9, 46.9)
- added R97: 100, Resistor_SMD:R_0402_1005Metric, F.Cu at (139.3, 113.7)
- added R98: 100, Resistor_SMD:R_0402_1005Metric, F.Cu at (148.1, 114.5)
- added R99: 100k, Resistor_SMD:R_0402_1005Metric, F.Cu at (148.1, 118.3)
- added U$2: BL9342, Package_TO_SOT_SMD:SOT-23-6, F.Cu at (141.4, 43.5)
- added U$3: SWITCH_W_LED_PB6149L-X-102YELLOW, TINRS - Wobbler (pico)sch:PB6149L, F.Cu at (68.7, 40.5)
- added U$4: SWITCH_W_LED_PB6149L-X-102YELLOW, TINRS - Wobbler (pico)sch:PB6149L, F.Cu at (176.8, 40.8)
- added U$5: SWITCH_W_LED_PB6149L-X-102YELLOW, TINRS - Wobbler (pico)sch:PB6149L, F.Cu at (118.2, 142.1)
- added U$6: SWITCH_W_LED_PB6149L-X-102YELLOW, TINRS - Wobbler (pico)sch:PB6149L, F.Cu at (157.0, 94.1)
- added U$7: SWITCH_W_LED_PB6149L-X-102YELLOW, TINRS - Wobbler (pico)sch:PB6149L, F.Cu at (81.2, 40.7)
- added U$8: SWITCH_W_LED_PB6149L-X-102YELLOW, TINRS - Wobbler (pico)sch:PB6149L, F.Cu at (97.1, 131.2)
- added U$9: SWITCH_W_LED_PB6149L-X-102YELLOW, TINRS - Wobbler (pico)sch:PB6149L, F.Cu at (132.3, 40.8)
- added U11: 74HC595, Package_SO:TSSOP-16_4.4x5mm_P0.65mm, F.Cu at (78.0, 120.5)
- added U12: ESP32-S3-WROOM-1, Espressif:ESP32-S3-WROOM-1, F.Cu at (114.9, 125.4)
- added U13: 74HC595, Package_SO:TSSOP-16_4.4x5mm_P0.65mm, F.Cu at (84.9, 88.5)
- added U14: 74HC595, Package_SO:TSSOP-16_4.4x5mm_P0.65mm, F.Cu at (148.1, 94.7)
- added U15: HT7550-1, Package_TO_SOT_SMD:SOT-89-3, F.Cu at (149.9, 62.0)
- added U16: MCP6022, Package_SO:TSSOP-8_4.4x3mm_P0.65mm, F.Cu at (143.7, 116.3)
- added U17: NE5532, Package_SO:SOIC-8_3.9x4.9mm_P1.27mm, F.Cu at (166.8, 123.8)
- C1, C2: value 100n -> 1759017
- C24: value 100n -> 470p
- C28: value 10u -> 100n; footprint Capacitor_SMD:CP_Elec_5x5.9 -> Capacitor_SMD:C_0402_1005Metric
- C3, C8: value 10u -> 197427; footprint Capacitor_SMD:C_0805_2012Metric -> TiNRS_Eagle_Footprints:CASE-A_3216
- C7: value 100n -> 22u; footprint Capacitor_SMD:C_0402_1005Metric -> Capacitor_SMD:C_0805_2012Metric
- D3: value D -> D-SOD-123; footprint Diode_SMD:D_SMA -> TiNRS_Eagle_Footprints:SOD123
- J1: value Conn_02x08_Odd_Even -> unknown; footprint Connector_IDC:IDC-Header_2x08_P2.54mm_Vertical -> TiNRS_Eagle_Footprints:POWER_16_SHROUDED
- SW1: value SW_Push_LED_PB614 -> SW_Push; footprint footprints:PB614_LED_SW_6pin -> Button_Switch_SMD:SW_Push_1P1T_NO_6x6mm_H9.5mm; moved to B.Cu
- U1: value Teensy4.0 -> 9778330; footprint teensy:Teensy40 -> TINRS - Wobbler (pico)sch:SOT95P237X112-3N
- U2: value R-78E5.0-0.5 -> AT24CS01-STUM; footprint Converter_DCDC:Converter_DCDC_RECOM_R-78E-0.5_THT -> Package_TO_SOT_SMD:SOT-23-5
- moved D3 166.0 mm to (145.0, 47.2), turned to 180 degrees
- moved C2 160.2 mm to (153.1, 62.9), turned to -90 degrees
- moved C1 154.7 mm to (153.1, 60.8), turned to -90 degrees
- moved C8 154.2 mm to (156.6, 61.9), turned to -90 degrees
- moved C3 153.6 mm to (150.9, 65.7), turned to 0 degrees
- moved J1 143.3 mm to (132.4, 64.8), turned to 0 degrees
- moved R65 138.2 mm to (93.9, 142.7), turned to -90 degrees
- moved R64 137.2 mm to (93.9, 138.8), turned to -90 degrees
- moved U1 131.8 mm to (119.8, 55.8)
- moved R29 131.3 mm to (165.4, 106.9)
- moved R27 131.1 mm to (165.3, 104.7), turned to -90 degrees
- moved R25 130.5 mm to (165.2, 100.6), turned to -90 degrees
- moved R31 130.5 mm to (165.0, 113.0), turned to -90 degrees
- moved R4 118.9 mm to (154.1, 122.2), turned to 180 degrees
- moved R2 115.8 mm to (165.2, 96.0), turned to -90 degrees
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Connections:
- net /LEDs/LED2 renamed /LED_PP_DRY
- net Net-(D2-Pad1) renamed /Power/min12in
- C1 pad 1: -12V -> +5V
- C12 pad 1: /CodecBuffer/VCOM -> /PCM3060/VCOM
- C13 pad 1: /CodecBuffer/VCOM -> /PCM3060/VCOM
- C24 pad 2: /CodecBuffer/VCOM -> Net-(C24-Pad2)
- C25 pad 1: Net-(C25-Pad1) -> GND
- C28 pad 1: /CodecBuffer/In_Jack_Right -> +12V
- C28 pad 2: Net-(C28-Pad2) -> GND
- C29 pad 1: GND -> -12V
- C29 pad 2: /CodecBuffer/VCOM -> GND
- C7 pad 1: +5V -> GND
- C7 pad 2: GND -> +5V
- D1 pad 2: /LEDs/LED0 -> /LED_ENVTRACKER_OUT
- D10 pad 2: /LEDs/LED5 -> /LED_VU_OUT_3
- D11 pad 2: /LEDs/LED6 -> /LED_PP_DIFFUSE
- D12 pad 2: /LEDs/LED7 -> /LED_VU_OUT_4
- D13 pad 2: /LEDs/LED8 -> /LED_PP_DELAY_FEEDBACK
- D14 pad 2: /LEDs/LED9 -> /LED_VU_OUT_5
- D15 pad 2: /LEDs/LED10 -> /LED_PP_DELAY
- D16 pad 2: /LEDs/LED11 -> /LED_VU_IN_1
- D17 pad 2: /LEDs/LED12 -> /LED_PP_MAINPOST
- D18 pad 2: /LEDs/LED13 -> /LED_VU_IN_2
- D19 pad 2: /LEDs/LED14 -> /LED_PP_TAIL
- D20 pad 2: /LEDs/LED15 -> /LED_VU_IN_3
- D4 pad 2: /LEDs/LED1 -> /LED_VU_OUT_1
- D8 pad 2: /LEDs/LED3 -> /LED_VU_OUT_2
- D9 pad 2: /LEDs/LED4 -> /LED_PP_MAINPRE
- IC1 pad 21: /CodecBuffer/VCOM -> /PCM3060/VCOM
- IC1 pad 6: Net-(IC1-Pad6) -> /MCLK
- J1 pad 10: Net-(D3-Pad2) -> /Power/plus12in
- J1 pad 11: unconnected-(J1-Pad11) -> unconnected-(J1-+5V-Pad11)
- J1 pad 12: unconnected-(J1-Pad12) -> unconnected-(J1-+5V-Pad11)
- J1 pad 13: unconnected-(J1-Pad13) -> unconnected-(J1-CV-Pad13)
- J1 pad 14: unconnected-(J1-Pad14) -> unconnected-(J1-CV-Pad13)
- J1 pad 15: unconnected-(J1-Pad15) -> unconnected-(J1-GATE-Pad15)
- J1 pad 16: unconnected-(J1-Pad16) -> unconnected-(J1-GATE-Pad15)
- J1 pad 9: Net-(D3-Pad2) -> /Power/plus12in
- R39 pad 1: /CVJacks/CV4 -> /CVJacks/CV_DELAY_LENGTH
- R41 pad 1: /CVJacks/CV0 -> /CVJacks/CV_DELAY_FEEDBACK
- R45 pad 1: /CVJacks/CV5 -> /CVJacks/CV_PITCH_TRANSPOSE
- R47 pad 1: /CVJacks/CV1 -> /CVJacks/CV_PITCH_CONTROL
- R51 pad 1: /CVJacks/CV6 -> /CVJacks/CV_TAIL_TEMPERATURE
- R53 pad 1: /CVJacks/CV2 -> /CVJacks/CV_TAIL_LENGTH
- R57 pad 1: /CVJacks/CV7 -> /CVJacks/CV_MIX
- R59 pad 1: /CVJacks/CV3 -> unconnected-(R59-Pad1)
- R62 pad 1: /LED_TARGET -> /LED_FREEZE
- R62 pad 2: Net-(SW1-Pad2) -> Net-(U$4-POS)
- R63 pad 1: /LED_STYLE -> /LED_PITCHPOINT
- R64 pad 1: /LED_FREEZE -> Net-(D23-K)
- R64 pad 2: Net-(SW3-Pad2) -> GND
- R65 pad 1: /LED_SENDONLY -> Net-(D24-K)
- R65 pad 2: Net-(SW4-Pad2) -> GND
- RV1 pad 2: /Knobs/KNOB0 -> /Knobs/KNOB_TAIL_LENGTH
- RV10 pad 2: /Knobs/KNOB6 -> /Knobs/KNOB_TAIL_TEMPERATURE
- RV11 pad 2: /Knobs/KNOB14 -> /Knobs/KNOB_DIFFUSE
- RV13 pad 2: /Knobs/KNOB3 -> /Knobs/KNOB_DELAY_LENGTH
- RV14 pad 2: /Knobs/KNOB15 -> /Knobs/KNOB_DELAY
- RV15 pad 2: /Knobs/KNOB11 -> /Knobs/KNOB_MAIN
- RV16 pad 2: /Knobs/KNOB7 -> /Knobs/KNOB_PITCH_CONTROL
- RV2 pad 2: /Knobs/KNOB12 -> /Knobs/KNOB_DELAY_FEEDBACK
- RV3 pad 2: /Knobs/KNOB4 -> /Knobs/KNOB_TAIL_CHORALITY
- RV4 pad 2: /Knobs/KNOB8 -> /Knobs/KNOB_DIFFUSE_STYLE
- RV5 pad 2: /Knobs/KNOB1 -> /Knobs/KNOB_DELAY_PATTERN
- RV6 pad 2: /Knobs/KNOB5 -> /Knobs/KNOB_TAIL
- RV8 pad 2: /Knobs/KNOB9 -> /Knobs/KNOB_PITCH_TRANSPOSE
- RV9 pad 2: /Knobs/KNOB2 -> /Knobs/KNOB_ENVTRACK
- SW1 pad 2: Net-(SW1-Pad2) -> /BOOTSEL_BUT
- U1 pad 2: /BUT_STYLE -> -5V
- U1 pad 3: /BUT_FREEZE -> unconnected-(U1-NC-Pad3)
- U2 pad 1: +12V -> /EEPROM_SCL
- U2 pad 3: +5V -> /EEPROM_SDA
- U3 pad 1: /Knobs/KNOB4 -> /Knobs/KNOB_DELAY
- U3 pad 10: /KNOBMUX0 -> /CVMUX0
- U3 pad 11: /Knobs/KNOB3 -> /Knobs/KNOB_DIFFUSE
- U3 pad 12: /Knobs/KNOB0 -> /Knobs/KNOB_DELAY_LENGTH
- U3 pad 14: /Knobs/KNOB1 -> /Knobs/KNOB_DELAY_FEEDBACK
- U3 pad 15: /Knobs/KNOB2 -> /Knobs/KNOB_DELAY_PATTERN
- U3 pad 2: /Knobs/KNOB6 -> /Knobs/KNOB_PITCH_TRANSPOSE
- U3 pad 4: /Knobs/KNOB7 -> GND
- U3 pad 5: /Knobs/KNOB5 -> /Knobs/KNOB_DIFFUSE_STYLE
- U3 pad 9: /KNOBMUX1 -> /CVMUX1
- U4 pad 1: Net-(C22-Pad2) -> /CodecBuffer/BIAS_INVERTED
- U4 pad 10: Net-(C21-Pad2) -> GND
- U4 pad 12: /CodecBuffer/VCOM -> GND
- U4 pad 13: Net-(C25-Pad1) -> Net-(U4D--)
- U4 pad 14: Net-(C25-Pad2) -> Net-(C70-Pad1)
- U4 pad 3: Net-(C20-Pad2) -> GND
- U4 pad 5: /CodecBuffer/VCOM -> /PCM3060/VCOM
- U4 pad 6: Net-(C30-Pad1) -> /CodecBuffer/BIAS_BUFFERED
- U4 pad 7: Net-(C30-Pad2) -> /CodecBuffer/BIAS_BUFFERED
- U5 pad 1: /Knobs/KNOB12 -> /Knobs/KNOB_MAIN
- U5 pad 10: /KNOBMUX0 -> /CVMUX0
- U5 pad 11: /Knobs/KNOB11 -> /Knobs/KNOB_TAIL
- U5 pad 12: /Knobs/KNOB8 -> /Knobs/KNOB_TAIL_LENGTH
- U5 pad 14: /Knobs/KNOB9 -> /Knobs/KNOB_TAIL_TEMPERATURE
- U5 pad 15: /Knobs/KNOB10 -> /Knobs/KNOB_TAIL_CHORALITY
- U5 pad 2: /Knobs/KNOB14 -> /Knobs/KNOB_PITCH_CONTROL
- U5 pad 4: /Knobs/KNOB15 -> GND
- U5 pad 5: /Knobs/KNOB13 -> /Knobs/KNOB_ENVTRACK
- U5 pad 9: /KNOBMUX1 -> /CVMUX1
- U6 pad 1: /LEDs/LED9 -> /LED_DELAYMODE_2
- U6 pad 14: Net-(U6-Pad14) -> /LEDDAT
- U6 pad 15: /LEDs/LED8 -> /LED_DELAYMODE_1
- U6 pad 2: /LEDs/LED10 -> /LED_DELAYMODE_3
- U6 pad 3: /LEDs/LED11 -> /LED_DELAY
- U6 pad 4: /LEDs/LED12 -> /LED_TAILMODE_1
- U6 pad 5: /LEDs/LED13 -> /LED_TAILMODE_2
- U6 pad 6: /LEDs/LED14 -> /LED_TAILMODE_3
- U6 pad 7: /LEDs/LED15 -> /LED_TAIL
- U6 pad 9: unconnected-(U6-Pad9) -> Net-(U6-QH')
- U7 pad 1: /LEDs/LED1 -> /LED_TAP
- U7 pad 14: /LEDDAT -> Net-(U6-QH')
- U7 pad 15: /LEDs/LED0 -> /LED_FREEZE
- U7 pad 3: /LEDs/LED3 -> /LED_PP_MAINPRE
- U7 pad 4: /LEDs/LED4 -> /LED_PP_DIFFUSE
- U7 pad 5: /LEDs/LED5 -> /LED_PP_DELAY_FEEDBACK
- U7 pad 6: /LEDs/LED6 -> /LED_PP_DELAY
- U7 pad 7: /LEDs/LED7 -> /LED_PP_MAINPOST
- U7 pad 9: Net-(U6-Pad14) -> Net-(U11-SER)
Other:
- board size 119.4 x 109.2 mm -> 119.4 x 110.4 mm
- board text added: "TiNRS Void"
